File: Light.kicad_sch (KiCad schematic)
At the start: 87 parts, among them J8 PGMR, SW1 SW_Push, U1 CD74HC4067SM, U2 STM32F103CBTx, U3 CD74HC4067SM, Y1 Crystal

Commit message: switches to stm32f0
Parts:
- removed C10, C11, C2, C3, C5, C6, C7, C8, C9: 1u, Capacitor_SMD:C_0603_1608Metric_Pad1.08x0.95mm_HandSolder, symbol Device:C
- removed D1: LED, LED_SMD:LED_0201_0603Metric_Pad0.64x0.40mm_HandSolder, symbol Device:LED
- removed R23: 10K, Resistor_SMD:R_0603_1608Metric_Pad0.98x0.95mm_HandSolder, symbol Device:R
- removed SW1: SW_Push, symbol Switch:SW_Push
- removed U2: STM32F103CBTx, Package_QFP:LQFP-48_7x7mm_P0.5mm, symbol MCU_ST_STM32F1:STM32F103CBTx
- removed Y1: Crystal, symbol Device:Crystal
- added C? (x4): C_Small, symbol Device:C_Small
- added D?: LED, symbol Device:LED
- added U?: STM32F042F4Px, Package_SO:TSSOP-20_4.4x6.5mm_P0.65mm, symbol MCU_ST_STM32F0:STM32F042F4Px
- added Y?: 8Mhz, symbol Device:Crystal
- renumbered U3 to U2
Connections:
- net M2_0 is gone; now on net M_S0: U2.10 (S0)
- net M2_1 is gone; now on net M_S1: U2.11 (S1)
- net M2_2 is gone; now on net M_S2: U2.14 (S2)
- net +3V3: now also C?.1, C?.1
- net GND: now also C?.1, C?.2, D?.1 (K), U?.15 (VSS)
- net M1: now also U?.6 (PA0)
- net M2: now also U?.7 (PA1)
- net PTX: now also U?.17 (PA9/PA11)
- net TX: now also U?.8 (PA2)
- net CLK renamed SWCLK
- net SWCLK: now also U?.20 (PA14)
- net DIO renamed SWDIO
- net SWDIO: now also U?.19 (PA13)
- net M1_0 renamed M_S0
- net M_S0: now also U?.10 (PA4)
- net M1_1 renamed M_S1
- net M_S1: now also U?.11 (PA5)
- net M1_2 renamed M_S2
- net M_S2: now also U?.12 (PA6)
- net M1_3 renamed MS_3
- net M2_3 renamed M_S3
- net M_S3: now also U?.13 (PA7)
- new net: C?.2, U?.2 (PF0), Y?.2
- new net: D?.2 (A), U?.14 (PB1)
- new net: C?.2, U?.16 (VDD)
- new net: C?.1, U?.3 (PF1), Y?.1
- new net: C?.2, U?.5 (VDDA)
- no-connect marks 18 -> 1
Other:
- note added: "PRX"
- note added: "RX"
- note added: "STM32F042F4P6"
- note removed: "STMF103CBT6"
- moved on the sheet: D10, D11, D12, D13, D14, D15, D16, D17, D18, D19, D2, D20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
