File: 2024l1.kicad_pcb (KiCad board)
At the start: 2 copper layers, 176 x 167.7 mm, 88 parts, among them IC1 SN74LVC2G04DBVTG4, IC2 SN74LVC2G04DBVTG4, IC3 LM2587S-ADJ_NOPB, J1 LG LED, J10 XT30, J2 LG RES, J3 ESC, J4 XT60, J5 FL, J6 FR, J7 52610-1233, J8 BL, J9 BR, Q1 STP75NF75, Q2 AO3400A, SW1 SW_SPDT, SW2 5V SW, SW3 M SW, U1 Seeed Studio XIAO ESP32C3, U2 CD74HC4067SM, U3 TPS5430DDA, U4 VNH5050A-E, U5 VNH5050A-E, U6 VNH5050A-E, U7 VNH5050A-E

Commit message: group driver
Parts:
- moved D19 15.2 mm to (114.3, 147.6), turned to 180 degrees
- moved D18 10.2 mm to (111.2, 152.7), turned to 180 degrees
- moved J10 5.20 mm to (103.6, 119.0), turned to 180 degrees
Routing:
- removed copper zone on F.Cu, net +48V
- removed copper zone on F.Cu, net Net-(D18-K)
- removed copper zone on F.Cu, net Net-(D19-A)
Changed lines of the file:
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@@
   (net 94 "unconnected-(U1-A2-Pad2)")
   (footprint "Diode_THT:D_DO-201AD_P15.24mm_Horizontal" (layer "F.Cu")
-    (at 99.04557 147.591132)
+    (at 114.28557 147.591132 180)
     (descr "Diode, DO-201AD series, Axial, Horizontal, pin pitch=15.24mm, , length*diameter=9.5*5.2mm^2, , http://www.diodes.com/_files/packages/DO-201AD.pdf")
     (tags "Diode DO-201AD series Axial Horizontal pin pitch 15.24mm  length 9.5mm diameter 5.2mm")
@@
     (fp_line (start 15.24 0) (end 12.37 0)
       (stroke (width 0.1) (type solid)) (layer "F.Fab"))
-    (pad "1" thru_hole rect (at 0 0) (size 3.2 3.2) (drill 1.6) (layers "*.Cu" "*.Mask")
+    (pad "1" thru_hole rect (at 0 0 180) (size 3.2 3.2) (drill 1.6) (layers "*.Cu" "*.Mask")
       (net 85 "Net-(D18-K)") (pinfunction "K") (pintype "passive"))
-    (pad "2" thru_hole oval (at 15.24 0) (size 3.2 3.2) (drill 1.6) (layers "*.Cu" "*.Mask")
+    (pad "2" thru_hole oval (at 15.24 0 180) (size 3.2 3.2) (drill 1.6) (layers "*.Cu" "*.Mask")
       (net 86 "Net-(D19-A)") (pinfunction "A") (pintype "passive"))
     (model "${KICAD6_3DMODEL_DIR}/Diode_THT.3dshapes/D_DO-201AD_P15.24mm_Horizontal.wrl"
@@
   )
   (footprint "footprints:AMASS_XT30-F" (layer "F.Cu")
-    (at 108.77757 119.031132)
+    (at 103.57757 119.031132 180)
     (descr "Connector XT30 Vertical Cable Male, https://www.tme.eu/en/Document/3cbfa5cfa544d79584972dd5234a409e/XT30U%20SPEC.pdf")
     (tags "RC Connector XT30")
@@
     (property "Sheetname" "")
     (attr through_hole)
-    (fp_text reference "J10" (at -2.54 -3.81 180) (layer "F.SilkS") hide
+    (fp_text reference "J10" (at -2.54 -3.81) (layer "F.SilkS") hide
         (effects (font (size 1 1) (thickness 0.15)))
     )
-    (fp_text value "XT30" (at -2.54 3.81 180) (layer "F.Fab") hide
+    (fp_text value "XT30" (at -2.54 3.81) (layer "F.Fab") hide
         (effects (font (size 1 1) (thickness 0.15)))
     )
-    (fp_text user "+" (at -9.08 0 180) (layer "F.SilkS") hide
+    (fp_text user "+" (at -9.08 0) (layer "F.SilkS") hide
         (effects (font (size 1.5 1.5) (thickness 0.15)))
     )
-    (fp_text user "-" (at 3.92 0 180) (layer "F.SilkS") hide
+    (fp_text user "-" (at 3.92 0) (layer "F.SilkS") hide
         (effects (font (size 1.5 1.5) (thickness 0.15)))
     )
-    (fp_text user "${REFERENCE}" (at -2.58 0 180) (layer "F.Fab") hide
+    (fp_text user "${REFERENCE}" (at -2.58 0) (layer "F.Fab") hide
         (effects (font (size 1 1) (thickness 0.15)))
     )
@@
     (fp_line (start 2.52 1.3) (end 2.52 -1.3)
       (stroke (width 0.1) (type solid)) (layer "F.Fab"))
-    (pad "1" thru_hole circle (at -0.08 0 180) (size 3.8 3.8) (drill 2.5) (layers "*.Cu" "*.Mask")
+    (pad "1" thru_hole circle (at -0.08 0) (size 3.8 3.8) (drill 2.5) (layers "*.Cu" "*.Mask")
       (net 86 "Net-(D19-A)") (pinfunction "NEG") (pintype "passive"))
-    (pad "2" thru_hole rect (at -5.08 0 180) (size 3.8 3.8) (drill 2.5) (layers "*.Cu" "*.Mask")
+    (pad "2" thru_hole rect (at -5.08 0) (size 3.8 3.8) (drill 2.5) (layers "*.Cu" "*.Mask")
       (net 84 "+48V") (pinfunction "POS") (pintype "passive"))
     (model "C:/Users/vince/OneDrive/Documents/KiCad/7.0/3dmodels/XT30UPB-F.step"
@@
   )
   (footprint "Diode_THT:D_DO-41_SOD81_P10.16mm_Horizontal" (layer "F.Cu")
-    (at 101.07757 152.671132)
+    (at 111.23757 152.671132 180)
     (descr "Diode, DO-41_SOD81 series, Axial, Horizontal, pin pitch=10.16mm, , length*diameter=5.2*2.7mm^2, , http://www.diodes.com/_files/packages/DO-41%20(Plastic).pdf")
     (tags "Diode DO-41_SOD81 series Axial Horizontal pin pitch 10.16mm  length 5.2mm diameter 2.7mm")
@@
     (fp_line (start 10.16 0) (end 7.68 0)
       (stroke (width 0.1) (type solid)) (layer "F.Fab"))
-    (pad "1" thru_hole rect (at 0 0) (size 2.2 2.2) (drill 1.1) (layers "*.Cu" "*.Mask")
+    (pad "1" thru_hole rect (at 0 0 180) (size 2.2 2.2) (drill 1.1) (layers "*.Cu" "*.Mask")
       (net 85 "Net-(D18-K)") (pinfunction "K") (pintype "passive"))
-    (pad "2" thru_hole oval (at 10.16 0) (size 2.2 2.2) (drill 1.1) (layers "*.Cu" "*.Mask")
+    (pad "2" thru_hole oval (at 10.16 0 180) (size 2.2 2.2) (drill 1.1) (layers "*.Cu" "*.Mask")
       (net 84 "+48V") (pinfunction "A") (pintype "passive"))
     (model "${KICAD6_3DMODEL_DIR}/Diode_THT.3dshapes/D_DO-41_SOD81_P10.16mm_Horizontal.wrl"
@@
   (segment (start 118.45307 169.435132) (end 117.32357 169.435132) (width 1) (layer "F.Cu") (net 90))
   (segment (start 114.90707 161.815132) (end 113.12607 161.815132) (width 1) (layer "F.Cu") (net 92))
-  (zone (net 86) (net_name "Net-(D19-A)") (layer "F.Cu") (hatch edge 0.5)
-    (priority 1)
-    (connect_pads (clearance 0.5))
-    (min_thickness 0.25) (filled_areas_thickness no)
-    (fill (thermal_gap 0.5) (thermal_bridge_width 0.5) (island_removal_mode 1) (island_area_min 10))
-    (polygon
-      (pts
-        (xy 106.15757 116.079132)
-        (xy 106.15757 121.175132)
-        (xy 114.79357 121.175132)
-        (xy 114.79357 144.543132)
-        (xy 111.23757 144.543132)
-        (xy 111.23757 150.639132)
-        (xy 121.39757 150.639132)
-        (xy 121.39757 116.079132)
-      )
-    )
-  )
-  (zone (net 85) (net_name "Net-(D18-K)") (layer "F.Cu") (hatch edge 0.5)
-    (priority 2)
-    (connect_pads (clearance 0.5))
-    (min_thickness 0.25) (filled_areas_thickness no)
-    (fill yes (thermal_gap 0.5) (thermal_bridge_width 0.5) (island_removal_mode 1) (island_area_min 10))
-    (polygon
-      (pts
-        (xy 97.01357 144.543132)
-        (xy 97.01357 154.703132)
-        (xy 104.63357 154.703132)
-        (xy 104.63357 144.543132)
-      )
-    )
-  )
-  (zone (net 84) (net_name "+48V") (layer "F.Cu") (hatch edge 0.5)
-    (connect_pads (clearance 0.5))
-    (min_thickness 0.25) (filled_areas_thickness no)
-    (fill (thermal_gap 0.5) (thermal_bridge_width 0.5))
-    (polygon
-      (pts
-        (xy 97.52157 116.079132)
-        (xy 97.52157 133.875132)
-        (xy 114.79357 133.875132)
-        (xy 114.79357 121.175132)
-        (xy 106.15757 121.175132)
-        (xy 106.15757 116.079132)
-      )
+  (group "" (id 08725436-c702-4056-9982-256f1cdd291e)
+    (members
+      61842971-29b9-460e-a328-8e93e849ccc4
+      a896f5c4-5ff5-4641-bf3c-2f9c28e6a841
+      c29a8908-faea-44e7-8466-aa417cf79d45
+    )
+  )
+  (group "" (id 482d8e49-3e24-49ac-a01b-61ed317a959c)
+    (members
+      31bb66a4-bb57-4838-a43a-9f9d320c7999
+      aec90297-a06e-480c-8212-55d6ec92aab4
+      bab992f5-07c9-46fa-a4d1-7a8bda61c431
+    )
+  )
+  (group "" (id 8be6000e-feea-4568-843c-ff048ca2cf74)
+    (members
+      4d4aae5d-3e68-4d75-97f4-2f02974cedb2
+      6f7163d4-decd-4d2f-a7cd-be1ef648cf37
+      aa090134-e64c-4dbb-8aff-b22d69198016
+    )
+  )
+  (group "" (id f0d9db46-b6c8-4dd2-a601-a0806c834e05)
+    (members
+      21c121bf-4540-4258-9700-bd6b3a6ea1af
+      a519b7ea-c577-441e-a73c-070f4800cbe4
+      e7dd98fa-974a-4119-a2a4-900ec4bedc72
     )
   )

Commit message: moved esp32 to the left
Parts:
- moved U1 105.1 mm to (31.2, 112.0), turned to 90 degrees
- moved C7 102.7 mm to (102.1, 190.5)
- moved D16 102.7 mm to (106.2, 174.3)
- moved U3 102.7 mm to (112.8, 185.4)
- moved C2 102.7 mm to (107.9, 187.5)
- moved L1 102.7 mm to (104.6, 180.9)
- moved R18 102.7 mm to (110.2, 190.8)
- moved R19 102.7 mm to (113.8, 190.8)
- moved C8 102.7 mm to (112.3, 177.8)
- moved SW2 102.7 mm to (109.2, 193.3)
Routing:
- net /M1: track 96.7 -> 90.4 mm
- net /S2: track 84.3 -> 78.0 mm
- net /S0: track 81.9 -> 76.8 mm
- net /S1: track 76.1 -> 71.9 mm
- net /S3: track 77.5 -> 73.6 mm

Commit message: starting to wire mdrivers
Parts:
- removed the SW1 at (51.6, 140.0)
- C3, C4, C5, C6, C9: value 100u -> 220u
- moved IC1 108.1 mm to (154.2, 112.0)
- moved D12 31.4 mm to (129.7, 146.7)
- moved D8 31.4 mm to (129.7, 129.3)
- moved D13 31.4 mm to (136.7, 152.2)
- moved D14 31.4 mm to (136.7, 156.6)
- moved D2 31.4 mm to (136.8, 129.3)
- moved D6 31.4 mm to (136.8, 146.7)
- moved D10 31.4 mm to (129.7, 138.0)
- moved D7 31.4 mm to (129.7, 125.0)
- moved D9 31.4 mm to (129.7, 133.7)
- moved D1 31.4 mm to (136.8, 125.0)
- moved D15 31.4 mm to (136.7, 160.9)
- moved D3 31.4 mm to (136.8, 133.7)
- moved D4 31.4 mm to (136.8, 138.0)
- moved D11 31.4 mm to (129.7, 142.4)
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- renumbered SW2 to SW1, SW3 to SW2
Connections:
- D1 pad 2: Net-(D1-A) -> +5V
- D10 pad 2: Net-(D1-A) -> +5V
- D11 pad 2: Net-(D1-A) -> +5V
- D12 pad 2: Net-(D1-A) -> +5V
- D13 pad 2: Net-(D1-A) -> +5V
- D14 pad 2: Net-(D1-A) -> +5V
- D15 pad 2: Net-(D1-A) -> +5V
- D2 pad 2: Net-(D1-A) -> +5V
- D3 pad 2: Net-(D1-A) -> +5V
- D4 pad 2: Net-(D1-A) -> +5V
- D5 pad 2: Net-(D1-A) -> +5V
- D6 pad 2: Net-(D1-A) -> +5V
- D7 pad 2: Net-(D1-A) -> +5V
- D8 pad 2: Net-(D1-A) -> +5V
- D9 pad 2: Net-(D1-A) -> +5V
- IC1 pad 1: /FL DIR -> /BR DIR
- IC1 pad 5: +5V -> +3V3
- IC1 pad 6: /!FL DIR -> /!BR DIR
- IC2 pad 1: /BL DIR -> /FL DIR
- IC2 pad 3: /BR DIR -> /BL DIR
- IC2 pad 4: /!BR DIR -> /!BL DIR
- IC2 pad 5: +5V -> +3V3
- IC2 pad 6: /!BL DIR -> /!FL DIR
- J7 pad 3: /TX -> /RX
- J7 pad 5: /RX -> /TX
- U1 pad 11: unconnected-(U1-3V3-Pad11) -> +3V3
- U4 pad 15: /FL DIR -> /!FL DIR
- U4 pad 22: /!FL DIR -> /FL DIR
- U7 pad 15: /BR DIR -> /!BR DIR
- U7 pad 22: /!BR DIR -> /BR DIR
Routing:
- net +3V3: track 0.00 -> 94.1 mm, vias 0 -> 2
- net /M1: track 90.4 -> 5.80 mm
- net /M SW: track 0.00 -> 83.7 mm, vias 0 -> 2
- net /BL PWM: track 0.00 -> 36.4 mm, vias 0 -> 2
- net /TX: track 0.00 -> 26.9 mm, vias 0 -> 1
- net /RX: track 0.00 -> 22.0 mm, vias 0 -> 1
- net /!BL DIR: track 0.00 -> 12.4 mm
- net /!FR DIR: track 0.00 -> 12.4 mm
- net /!BR DIR: track 0.00 -> 12.4 mm
- net /!FL DIR: track 0.00 -> 12.4 mm
- net /BL DIR: track 0.00 -> 9.00 mm
- net /FL DIR: track 0.00 -> 8.59 mm
- net /FL PWM: track 0.00 -> 5.46 mm, vias 0 -> 1
- net /FR PWM: track 0.00 -> 5.43 mm, vias 0 -> 1
- net /FR DIR: track 0.00 -> 5.43 mm, vias 0 -> 1
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- added copper zone on F.Cu, net /BL A
- added copper zone on F.Cu, net /BL B
- added copper zone on F.Cu, net /BR B
- added copper zone on F.Cu, net /FL A
- added copper zone on F.Cu, net /FL B
- added copper zone on F.Cu, net /FR A
- added copper zone on F.Cu, net /FR B

Commit message: left with power
Parts:
- moved D1 19.7 mm to (151.6, 138.0)
- moved D7 19.7 mm to (144.5, 138.0)
- moved D2 19.7 mm to (151.6, 142.3)
- moved D3 19.7 mm to (151.6, 146.7)
- moved D8 19.7 mm to (144.5, 142.3)
- moved D9 19.7 mm to (144.5, 146.7)
Routing:
- net /BR DIR: track 5.41 -> 138.0 mm, vias 1 -> 2
- net /FR DIR: track 5.43 -> 137.6 mm, vias 1 -> 2
- net /BR PWM: track 5.36 -> 112.7 mm, vias 1 -> 2
- net /FR PWM: track 5.43 -> 104.5 mm, vias 1 -> 2
- net /S2: track 78.0 -> 13.6 mm
- net /S0: track 76.8 -> 14.5 mm
- net /S3: track 73.6 -> 11.4 mm
- net /S1: track 71.9 -> 13.1 mm
- net +3V3: track 94.1 -> 138.9 mm, vias 2 -> 4
- net /M SW: track 83.7 -> 125.0 mm, vias 2 -> 4
- net /FL DIR: track 8.59 -> 39.0 mm
- net /BL DIR: track 9.00 -> 37.8 mm
- net +5V: track 19.2 -> 46.3 mm
- net /FL PWM: track 5.46 -> 28.3 mm, vias 1 -> 2
- net /LG: track 78.0 -> 65.6 mm
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- added copper zone on F.Cu, net /BR A

Commit message: i hate elec
Parts:
- moved R10 24.7 mm to (106.6, 99.9)
- moved R11 24.7 mm to (106.6, 102.5)
- moved R3 24.7 mm to (110.8, 97.3)
- moved R4 24.7 mm to (110.8, 99.9)
- moved R5 24.7 mm to (110.8, 102.5)
- moved R9 24.7 mm to (106.6, 97.3)
- moved R6 8.73 mm to (102.5, 102.1)
- moved R12 5.74 mm to (97.0, 104.9)
- moved R1 4.33 mm to (104.6, 91.7), turned to -90 degrees
Changed lines of the file:
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@@
   )
   (footprint "footprints:ALS-PT19" (layer "B.Cu")
-    (at 86.33557 101.031132 180)
+    (at 110.77 97.282 180)
     (property "Sheetfile" "2024l1.kicad_sch")
     (property "Sheetname" "")
@@
   )
   (footprint "footprints:ALS-PT19" (layer "B.Cu")
-    (at 97.33557 109.144496 180)
+    (at 102.504 102.108 180)
     (property "Sheetfile" "2024l1.kicad_sch")
     (property "Sheetname" "")
@@
   )
   (footprint "footprints:ALS-PT19" (layer "B.Cu")
-    (at 82.15757 106.279132 180)
+    (at 106.592 102.53 180)
     (property "Sheetfile" "2024l1.kicad_sch")
     (property "Sheetname" "")
@@
   )
   (footprint "footprints:ALS-PT19" (layer "B.Cu")
-    (at 104.64707 96.024496 180)
+    (at 104.64707 91.694 -90)
     (property "Sheetfile" "2024l1.kicad_sch")
     (property "Sheetname" "")
@@
     (property "ki_keywords" "resistor variable light sensitive opto LDR")
     (attr smd)
-    (fp_text reference "R1" (at 0.254 1.524 unlocked) (layer "B.SilkS")
-        (effects (font (size 1 1) (thickness 0.1)) (justify mirror))
-    )
-    (fp_text value "R_Photo" (at 0 0.278 unlocked) (layer "B.Fab")
-        (effects (font (size 1 1) (thickness 0.15)) (justify mirror))
-    )
-    (fp_text user "${REFERENCE}" (at 0 -1.222 unlocked) (layer "B.Fab")
+    (fp_text reference "R1" (at 0.254 1.524 -270 unlocked) (layer "B.SilkS") hide
+        (effects (font (size 1 1) (thickness 0.1)) (justify mirror))
+    )
+    (fp_text value "R_Photo" (at 0 0.278 -270 unlocked) (layer "B.Fab") hide
+        (effects (font (size 1 1) (thickness 0.15)) (justify mirror))
+    )
+    (fp_text user "${REFERENCE}" (at 0 -1.222 -270 unlocked) (layer "B.Fab") hide
         (effects (font (size 1 1) (thickness 0.15)) (justify mirror))
     )
     (fp_line (start -1.778 0.762) (end -1.778 -0.762)
       (stroke (width 0.1) (type default)) (layer "B.SilkS"))
-    (pad "1" smd roundrect (at -0.85 0 180) (size 1 1) (layers "B.Cu" "B.Paste" "B.Mask") (roundrect_rratio 0.1)
+    (pad "1" smd roundrect (at -0.85 0 270) (size 1 1) (layers "B.Cu" "B.Paste" "B.Mask") (roundrect_rratio 0.1)
       (net 1 "+5V") (pintype "passive") (thermal_bridge_angle 45))
-    (pad "2" smd roundrect (at 0.85 0 180) (size 1 1) (layers "B.Cu" "B.Paste" "B.Mask") (roundrect_rratio 0.1)
+    (pad "2" smd roundrect (at 0.85 0 270) (size 1 1) (layers "B.Cu" "B.Paste" "B.Mask") (roundrect_rratio 0.1)
       (net 41 "Net-(U2-I0)") (pintype "passive") (thermal_bridge_angle 45))
     (model "C:/Users/vince/OneDrive/Documents/KiCad/7.0/3dmodels/ALS-PT19.step"
@@
   )
   (footprint "footprints:ALS-PT19" (layer "B.Cu")
-    (at 82.15757 101.031132 180)
+    (at 106.592 97.282 180)
     (property "Sheetfile" "2024l1.kicad_sch")
     (property "Sheetname" "")
@@
   )
   (footprint "footprints:ALS-PT19" (layer "B.Cu")
-    (at 93.15757 109.144496 180)
+    (at 97.028 104.902 180)
     (property "Sheetfile" "2024l1.kicad_sch")
     (property "Sheetname" "")
@@
   )
   (footprint "footprints:ALS-PT19" (layer "B.Cu")
-    (at 82.15757 103.655132 180)
+    (at 106.592 99.906 180)
     (property "Sheetfile" "2024l1.kicad_sch")
     (property "Sheetname" "")
@@
   )
   (footprint "footprints:ALS-PT19" (layer "B.Cu")
-    (at 86.33557 106.279132 180)
+    (at 110.77 102.53 180)
     (property "Sheetfile" "2024l1.kicad_sch")
     (property "Sheetname" "")
@@
   )
   (footprint "footprints:ALS-PT19" (layer "B.Cu")
-    (at 86.33557 103.655132 180)
+    (at 110.77 99.906 180)
     (property "Sheetfile" "2024l1.kicad_sch")
     (property "Sheetname" "")
@@
         (xy 149.84557 114.315132)
         (xy 157.33857 114.315132)
-        (xy 157.33857 114.315132)
         (xy 157.33857 120.032132)
         (xy 157.33857 120.031132)
@@
         (xy 145.15757 107.586132)
         (xy 149.84557 107.586132)
-        (xy 149.84557 107.586132)
         (xy 149.84557 109.618132)
-        (xy 157.33857 109.618132)
         (xy 157.33857 109.618132)
         (xy 157.33857 104.030132)
@@
         (xy 149.84557 125.747132)
         (xy 157.33857 125.747132)
-        (xy 157.33857 125.747132)
         (xy 157.33857 120.032132)

Commit message: shit is screwed
Routing:
- net +5V: track 46.3 -> 41.7 mm
- net GND: vias 1 -> 9
- added copper zone on B.Cu, net GND
- added copper zone on F.Cu, net GND
Changed lines of the file:
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@@
   (gr_arc (start 33.325708 135.365415) (mid 34.739921 134.779628) (end 36.154135 135.365415)
     (stroke (width 0.2) (type solid)) (layer "Edge.Cuts"))
-  (segment (start 48.54657 106.531132) (end 47.552438 105.537) (width 0.3) (layer "F.Cu") (net 1))
-  (segment (start 157.18957 174.271132) (end 156.35457 173.436132) (width 0.3) (layer "F.Cu") (net 1))
-  (segment (start 41.021 106.553) (end 25.019 106.553) (width 0.3) (layer "F.Cu") (net 1))
+  (segment (start 27.686 109.22) (end 23.53757 105.07157) (width 0.3) (layer "F.Cu") (net 1))
+  (segment (start 47.552438 105.537) (end 42.037 105.537) (width 0.3) (layer "F.Cu") (net 1))
+  (segment (start 38.354 109.22) (end 27.686 109.22) (width 0.3) (layer "F.Cu") (net 1))
   (segment (start 103.82057 189.044132) (end 102.09357 187.317132) (width 0.3) (layer "F.Cu") (net 1))
-  (segment (start 47.552438 105.537) (end 42.037 105.537) (width 0.3) (layer "F.Cu") (net 1))
-  (segment (start 25.019 106.553) (end 23.53757 105.07157) (width 0.3) (layer "F.Cu") (net 1))
   (segment (start 104.83657 190.060132) (end 103.82057 189.044132) (width 0.3) (layer "F.Cu") (net 1))
   (segment (start 105.54757 190.771132) (end 103.82057 189.044132) (width 0.3) (layer "F.Cu") (net 1))
-  (segment (start 42.037 105.537) (end 41.021 106.553) (width 0.3) (layer "F.Cu") (net 1))
-  (segment (start 156.35457 173.436132) (end 156.35457 167.819132) (width 0.3) (layer "F.Cu") (net 1))
+  (segment (start 48.54657 106.531132) (end 47.552438 105.537) (width 0.3) (layer "F.Cu") (net 1))
+  (segment (start 42.037 105.537) (end 38.354 109.22) (width 0.3) (layer "F.Cu") (net 1))
   (segment (start 109.30907 190.771132) (end 105.54757 190.771132) (width 0.3) (layer "F.Cu") (net 1))
   (segment (start 23.53757 105.07157) (end 23.53757 104.411132) (width 0.3) (layer "F.Cu") (net 1))
@@
   (segment (start 127.49357 112.031132) (end 136.15757 112.031132) (width 5) (layer "F.Cu") (net 4))
   (via (at 55.48457 112.158132) (size 0.8) (drill 0.4) (layers "F.Cu" "B.Cu") (net 5))
+  (via (at 61.214 113.919) (size 0.8) (drill 0.4) (layers "F.Cu" "B.Cu") (free) (net 5))
+  (via (at 57.912 126.238) (size 0.8) (drill 0.4) (layers "F.Cu" "B.Cu") (free) (net 5))
+  (via (at 60.325 113.919) (size 0.8) (drill 0.4) (layers "F.Cu" "B.Cu") (free) (net 5))
+  (via (at 60.96 126.238) (size 0.8) (drill 0.4) (layers "F.Cu" "B.Cu") (free) (net 5))
+  (via (at 58.928 126.238) (size 0.8) (drill 0.4) (layers "F.Cu" "B.Cu") (free) (net 5))
+  (via (at 62.103 113.919) (size 0.8) (drill 0.4) (layers "F.Cu" "B.Cu") (free) (net 5))
+  (via (at 59.944 126.238) (size 0.8) (drill 0.4) (layers "F.Cu" "B.Cu") (free) (net 5))
+  (via (at 59.436 113.919) (size 0.8) (drill 0.4) (layers "F.Cu" "B.Cu") (free) (net 5))
   (segment (start 69.469 96.647) (end 56.134 96.647) (width 0.3) (layer "F.Cu") (net 6))
   (segment (start 56.35757 110.531132) (end 54.737 110.531132) (width 0.3) (layer "F.Cu") (net 6))
@@
   (segment (start 69.90757 110.689132) (end 69.51557 111.081132) (width 0.25) (layer "F.Cu") (net 9))
   (segment (start 69.90757 108.989132) (end 69.90757 110.689132) (width 0.25) (layer "F.Cu") (net 9))
-  (segment (start 56.261 127.127) (end 54.737 125.603) (width 0.3) (layer "F.Cu") (net 10))
-  (segment (start 69.90757 126.68843) (end 69.469 127.127) (width 0.3) (layer "F.Cu") (net 10))
-  (segment (start 69.469 127.127) (end 56.261 127.127) (width 0.3) (layer "F.Cu") (net 10))
-  (segment (start 54.737 125.603) (end 54.737 114.531132) (width 0.3) (layer "F.Cu") (net 10))
+  (segment (start 56.769 127.635) (end 54.737 125.603) (width 0.3) (layer "F.Cu") (net 10))
   (segment (start 56.90757 112.981132) (end 55.35757 114.531132) (width 0.3) (layer "F.Cu") (net 10))
   (segment (start 69.90757 124.989132) (end 69.90757 126.68843) (width 0.25) (layer "F.Cu") (net 10))
+  (segment (start 68.961 127.635) (end 56.769 127.635) (width 0.3) (layer "F.Cu") (net 10))
+  (segment (start 69.90757 126.68843) (end 68.961 127.635) (width 0.3) (layer "F.Cu") (net 10))
   (segment (start 54.737 114.531132) (end 48.54657 114.531132) (width 0.3) (layer "F.Cu") (net 10))
   (segment (start 55.35757 114.531132) (end 54.737 114.531132) (width 0.3) (layer "F.Cu") (net 10))
+  (segment (start 54.737 125.603) (end 54.737 114.531132) (width 0.3) (layer "F.Cu") (net 10))
   (segment (start 53.870573 116.531132) (end 53.87107 116.530635) (width 0.3) (layer "F.Cu") (net 11))
   (segment (start 143.129 128.143) (end 142.40757 127.42157) (width 0.25) (layer "F.Cu") (net 11))
@@
   )
   (zone (net 17) (net_name "/FR B") (layer "F.Cu") (hatch edge 0.5)
-    (priority 1)
     (connect_pads (clearance 0.5))
     (min_thickness 0.25) (filled_areas_thickness no)
@@
       )
     )
+  )
+  (zone (net 5) (net_name "GND") (layers "F&B.Cu") (hatch edge 0.5)
+    (connect_pads (clearance 0.5))
+    (min_thickness 0.25) (filled_areas_thickness no)
+    (fill yes (thermal_gap 0.5) (thermal_bridge_width 0.5) (smoothing fillet))
+    (polygon
+      (pts
+        (xy 12.7 25.4)
+        (xy 12.7 203.2)
+        (xy 195.58 203.2)
+        (xy 195.58 25.4)
+      )
+    )

Commit message: i hate pcbs
Parts:
- moved J3 6.61 mm to (175.2, 109.1)
- moved J4 5.32 mm to (182.9, 112.0)
Routing:
- net +12V: track 280.6 -> 26.2 mm
- net +3V3: track 138.9 -> 0.00 mm, vias 4 -> 0
- net /BR DIR: track 138.0 -> 0.00 mm, vias 2 -> 0
- net /FR DIR: track 137.6 -> 0.00 mm, vias 2 -> 0
- net /M SW: track 125.0 -> 0.00 mm, vias 4 -> 0
- net /BR PWM: track 112.7 -> 0.00 mm, vias 2 -> 0
- net /FR PWM: track 104.5 -> 0.00 mm, vias 2 -> 0
- net /LG: track 65.6 -> 0.00 mm
- net +5V: track 41.7 -> 0.00 mm
- net /FL DIR: track 39.0 -> 0.00 mm
- net /BL DIR: track 38.2 -> 0.00 mm
- net /BL PWM: track 38.1 -> 0.00 mm, vias 2 -> 0
- net /FL PWM: track 28.3 -> 0.00 mm, vias 2 -> 0
- net /TX: track 23.9 -> 0.00 mm, vias 1 -> 0
- net /RX: track 19.2 -> 0.00 mm, vias 1 -> 0
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- removed copper zone on F.Cu, net /BL A
- removed copper zone on F.Cu, net /BL B
- removed copper zone on F.Cu, net /BR A
- removed copper zone on F.Cu, net /BR B
- removed copper zone on F.Cu, net /FL A
- removed copper zone on F.Cu, net /FL B
- removed copper zone on F.Cu, net /FR A
- removed copper zone on F.Cu, net /FR B
