File: 2024l1.kicad_pcb (KiCad board)
At the start: 2 copper layers, 176 x 167.7 mm, 87 parts, among them IC1 SN74LVC2G04DBVTG4, IC2 SN74LVC2G04DBVTG4, IC3 LM2587S-ADJ_NOPB, J1 LG LED, J10 XT30, J2 LG RES, J3 ESC, J4 XT60, J5 FL, J6 FR, J7 52610-1233, J8 BL, J9 BR, Q1 STP75NF75, Q2 AO3400A, SW1 5V SW, SW2 M SW, U1 Seeed Studio XIAO ESP32C3, U2 CD74HC4067SM, U3 TPS5430DDA, U4 VNH5050A-E, U5 VNH5050A-E, U6 VNH5050A-E, U7 VNH5050A-E

Commit message: find btr place for buck
Parts:
- SW1: footprint Connector_PinHeader_2.54mm:PinHeader_1x03_P2.54mm_Vertical -> footprints:SS12D00G3
- moved SW1 117.5 mm to (24.4, 112.0)
- moved C7 94.9 mm to (101.7, 95.6), turned to 180 degrees
- moved R18 87.5 mm to (101.4, 103.7), turned to -90 degrees
- moved C2 86.1 mm to (104.7, 101.4), turned to 0 degrees
- moved R19 84.4 mm to (101.4, 107.3), turned to -90 degrees
- moved L1 83.0 mm to (111.3, 98.1), turned to 90 degrees
- moved U3 79.4 mm to (106.8, 106.3), turned to 0 degrees
- moved D16 75.5 mm to (117.9, 99.7), turned to 90 degrees
- moved C8 72.2 mm to (114.4, 105.7), turned to 0 degrees
- moved R24 28.6 mm to (106.8, 177.2), turned to -90 degrees
- moved C12 26.6 mm to (105.2, 177.2), turned to 90 degrees
- moved R26 25.8 mm to (108.5, 177.2), turned to -90 degrees
- moved C9 24.4 mm to (114.8, 158.5)
- moved RV1 23.9 mm to (108.2, 181.6)
- moved IC3 21.3 mm to (102.6, 169.5), turned to 180 degrees
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Connections:
- U3 pad 5: /EN 5V -> unconnected-(U3-EN-Pad5)
Routing:
- net +12V: track 26.2 -> 199.1 mm
- net /Sol: track 0.00 -> 92.3 mm, vias 0 -> 1
- net +48V: track 0.00 -> 68.0 mm
- net Net-(D19-A): track 0.00 -> 54.7 mm
- net Net-(D17-A): track 0.00 -> 24.9 mm
- net Net-(IC3-FDBK): track 0.00 -> 21.0 mm
- net Net-(D16-K): track 0.00 -> 16.1 mm
- net Net-(Q2-D): track 0.00 -> 15.9 mm
- net +5V: track 0.00 -> 15.4 mm
- net Net-(R21-Pad2): track 0.00 -> 11.8 mm
- net /FL B: track 0.00 -> 7.44 mm
- net /BL A: track 0.00 -> 7.44 mm
- net /FR A: track 0.00 -> 7.44 mm
- net /FL A: track 0.00 -> 7.38 mm
- net /BL B: track 0.00 -> 7.38 mm
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