File: Step Down.kicad_sch (KiCad schematic)
At the start: 16 parts, among them U1 3V3 Buck, U2 5V Buck

Commit message: added switches for the tps5430
Parts:
- added SW? (x2): SW_SPDT, symbol Switch:SW_SPDT
Connections:
- net 3V3_ENA: now also SW?.2 (B)
- net 5V_ENA: now also SW?.2 (B)
- net GND: now also SW?.1 (A), SW?.1 (A)
- no-connect marks 0 -> 2
Other:
- note added: "ENA. Below 0.5 V, the device stops switching. Float the pin to enable."
Changed lines of the file:
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@@
   (junction (at 105.41 118.11) (diameter 0) (color 0 0 0 0)
   )
+  (no_connect (at 240.03 105.41))
+  (no_connect (at 240.03 88.9))
   (wire (pts (xy 114.3 128.27) (xy 124.46 128.27))
     (stroke (width 0) (type default))
@@
     (stroke (width 0) (type default))
   )
+  (wire (pts (xy 240.03 83.82) (xy 243.84 83.82))
+    (stroke (width 0) (type default))
+  )
+  (wire (pts (xy 219.71 86.36) (xy 229.87 86.36))
+    (stroke (width 0) (type default))
+  )
   (wire (pts (xy 187.96 89.535) (xy 187.96 88.9))
     (stroke (width 0) (type default))
@@
     (stroke (width 0) (type default))
   )
+  (wire (pts (xy 240.03 100.33) (xy 243.84 100.33))
+    (stroke (width 0) (type default))
+  )
   (wire (pts (xy 149.86 88.9) (xy 162.56 88.9))
     (stroke (width 0) (type default))
@@
     (stroke (width 0) (type default))
   )
+  (wire (pts (xy 219.71 102.87) (xy 229.87 102.87))
+    (stroke (width 0) (type default))
+  )
   (wire (pts (xy 162.56 78.74) (xy 162.56 83.82))
     (stroke (width 0) (type default))
+  )
+  (text "ENA. Below 0.5 V, the device stops switching. Float the pin to enable."
+    (at 104.14 151.13 0)
+    (effects (font (size 1.27 1.27)) (justify left bottom))
+  )
+  (label "3V3_ENA" (at 220.98 86.36 0) (fields_autoplaced)
+    (effects (font (size 1.27 1.27)) (justify left bottom))
   )
   (label "5V_ENA" (at 115.57 128.27 0) (fields_autoplaced)
     (effects (font (size 1.27 1.27)) (justify left bottom))
   )
+  (label "5V_ENA" (at 220.98 102.87 0) (fields_autoplaced)
+    (effects (font (size 1.27 1.27)) (justify left bottom))
+  )
   (label "3V3_ENA" (at 115.57 88.9 0) (fields_autoplaced)
     (effects (font (size 1.27 1.27)) (justify left bottom))
+  )
+  (symbol (lib_id "Switch:SW_SPDT") (at 234.95 86.36 0) (unit 1)
+    (in_bom yes) (on_board yes) (dnp no) (fields_autoplaced)
+    (property "Reference" "SW?" (at 234.95 78.74 0)
+      (effects (font (size 1.27 1.27)))
+    )
+    (property "Value" "SW_SPDT" (at 234.95 81.28 0)
+      (effects (font (size 1.27 1.27)))
+    )
+    (property "Footprint" "" (at 234.95 86.36 0)
+      (effects (font (size 1.27 1.27)) hide)
+    )
+    (property "Datasheet" "~" (at 234.95 86.36 0)
+      (effects (font (size 1.27 1.27)) hide)
+    )
+    (pin "1")
+    (pin "2")
+    (pin "3")
+    (instances
+      (project "2024l1"
+        (path "/5be543b5-1bdc-438f-a916-f916127c0a2b/557de726-edfd-4324-bc0e-6d5b81e56087"
+          (reference "SW?") (unit 1)
+        )
+      )
+    )
   )
   (symbol (lib_id "power:GND") (at 187.96 140.97 0) (unit 1)
@@
         (path "/df3073b9-8d60-44a4-89ea-71f9aa763c80"
           (reference "#PWR01") (unit 1)
+        )
+      )
+    )
+  )
+  (symbol (lib_id "power:GND") (at 243.84 100.33 90) (unit 1)
+    (in_bom yes) (on_board yes) (dnp no) (fields_autoplaced)
+    (property "Reference" "#PWR078" (at 250.19 100.33 0)
+      (effects (font (size 1.27 1.27)) hide)
+    )
+    (property "Value" "GND" (at 247.65 100.3299 90)
+      (effects (font (size 1.27 1.27)) (justify right))
+    )
+    (property "Footprint" "" (at 243.84 100.33 0)
+      (effects (font (size 1.27 1.27)) hide)
+    )
+    (property "Datasheet" "" (at 243.84 100.33 0)
+      (effects (font (size 1.27 1.27)) hide)
+    )
+    (pin "1")
+    (instances
+      (project "2024l1"
+        (path "/5be543b5-1bdc-438f-a916-f916127c0a2b/557de726-edfd-4324-bc0e-6d5b81e56087"
+          (reference "#PWR078") (unit 1)
         )
       )
@@
     )
   )
+  (symbol (lib_id "Switch:SW_SPDT") (at 234.95 102.87 0) (unit 1)
+    (in_bom yes) (on_board yes) (dnp no) (fields_autoplaced)
+    (property "Reference" "SW?" (at 234.95 95.25 0)
+      (effects (font (size 1.27 1.27)))
+    )
+    (property "Value" "SW_SPDT" (at 234.95 97.79 0)
+      (effects (font (size 1.27 1.27)))
+    )
+    (property "Footprint" "" (at 234.95 102.87 0)
+      (effects (font (size 1.27 1.27)) hide)
+    )
+    (property "Datasheet" "~" (at 234.95 102.87 0)
+      (effects (font (size 1.27 1.27)) hide)
+    )
+    (pin "1")
+    (pin "2")
+    (pin "3")
+    (instances
+      (project "2024l1"
+        (path "/5be543b5-1bdc-438f-a916-f916127c0a2b/557de726-edfd-4324-bc0e-6d5b81e56087"
+          (reference "SW?") (unit 1)
+        )
+      )
+    )
+  )
   (symbol (lib_id "power:GND") (at 137.16 100.33 0) (unit 1)
     (in_bom yes) (on_board yes) (dnp no) (fields_autoplaced)
@@
         )
       )
+    )
+  )
+  (symbol (lib_id "power:GND") (at 243.84 83.82 90) (unit 1)
+    (in_bom yes) (on_board yes) (dnp no) (fields_autoplaced)
+    (property "Reference" "#PWR077" (at 250.19 83.82 0)
+      (effects (font (size 1.27 1.27)) hide)
+    )
+    (property "Value" "GND" (at 247.65 83.8199 90)
+      (effects (font (size 1.27 1.27)) (justify right))
+    )
+    (property "Footprint" "" (at 243.84 83.82 0)
+      (effects (font (size 1.27 1.27)) hide)
+    )
+    (property "Datasheet" "" (at 243.84 83.82 0)
+      (effects (font (size 1.27 1.27)) hide)
+    )
+    (pin "1")
+    (instances
+      (project "2024l1"
+        (path "/5be543b5-1bdc-438f-a916-f916127c0a2b/557de726-edfd-4324-bc0e-6d5b81e56087"
+          (reference "#PWR077") (unit 1)
+        )
+      )
