File: Drive.kicad_sch (KiCad schematic)
At the start: 55 parts, among them IC1 SN74LVC2G04DBVTG4, IC2 SN74LVC2G04DBVTG4, M1 VNH5050A-E, M1C1 680u, M1C2 33n, M1R1 3K3, M1R2 3K3, M1R3 1K, M1R4 1K, M1R5 1K, M1R6 1K, M1R7 1K, M1R8 10K, M1R9 1K5, M1_CONN XT30, M2 VNH5050A-E, M2C2 33n, M2C2 680u, M2R1 3K3, M2R2 3K3, M2R3 1K, M2R4 1K, M2R5 1K, M2R6 1K, M2R7 1K, M2R8 10K, M2R9 1K5, M2_CONN XT30, M3 VNH5050A-E, M3C1 680u, M3C2 33n, M3R1 3K3, M3R2 3K3, M3R3 1K, M3R4 1K, M3R5 1K, M3R6 1K, M3R7 1K, M3R8 10K, M3R9 1K5, M3_CONN XT30, M4 VNH5050A-E, M4C1 680u, M4C2 33n, M4R1 3K3, M4R2 3K3, M4R3 1K, M4R4 1K, M4R5 1K, M4R6 1K, M4R7 1K, M4R8 10K, M4R9 1K5, M4_CONN XT30

Commit message: 5050 - ❌ Enc - ❌ CS
Other:
- moved on the sheet: M2, M2C2, M2R1, M2R2, M2R3, M2R4, M2R5, M2R6, M2R7, M2R8, M2R9, M2_CONN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
