File: Processing.kicad_sch (KiCad schematic)
At the start: 48 parts

Commit message: stm32
Parts:
- added C? (x4): 0.1u, symbol vincent:C
- added C? (x2): 22p, symbol vincent:C
- added D?: LED, symbol Device:LED
- added J?: PGMR, symbol Connector_Generic:Conn_01x04
- added R? (x2): 10K, symbol vincent:R
- added R?: 1K, symbol vincent:R
- added SW?: SW_Push, symbol Switch:SW_Push
- added SW?: SW_SPDT, symbol Switch:SW_SPDT
- added U?: STM32F103CBTx, Package_QFP:LQFP-48_7x7mm_P0.5mm, symbol vincent:STM32F103CBTx
- added Y?: 8Mhz, symbol vincent:Crystal
Connections:
- net +3V3: now also C?.2, C?.2, C?.2, C?.2, R?.2, SW?.1 (A), U?.24 (VDD), U?.36 (VDD), U?.48 (VDD), U?.9 (VDDA)
- net GND: now also C?.1, C?.1, C?.1, C?.1, C?.1, C?.1, D?.1 (K), J?.4 (Pin_4), R?.1, R?.1, U?.23 (VSS), U?.35 (VSS), U?.47 (VSS), U?.8 (VSSA)
- net M1: now reaches R?.2, U?.1 (COM)
- net M3: now reaches R?.2, U?.1 (COM)
- net M3: now also U?.39 (PB3)
- net M3_S0: now reaches U?.10 (S0)
- net M3_S0: now also U?.26 (PB13)
- net M3_S1: now reaches U?.11 (S1)
- net M3_S1: now also U?.27 (PB14)
- net M3_S3: now reaches U?.13 (S3)
- net M3_S3: now also U?.22 (PB11)
- net M3_S2: now reaches U?.14 (S2)
- net M3_S2: now also U?.25 (PB12)
- net M2: now reaches R?.2, U?.1 (COM)
- net M2: now also U?.19 (PB1)
- net M2_S0: now reaches U?.10 (S0)
- net M2_S0: now also U?.20 (PB2)
- net M2_S1: now reaches U?.11 (S1)
- net M2_S1: now also U?.21 (PB10)
- net M2_S3: now reaches U?.13 (S3)
- net M2_S3: now also U?.16 (PA6), U?.17 (PA7)
- net M2_S2: now reaches U?.14 (S2)
- net M2_S2: now also U?.18 (PB0)
- net M1_S0: now reaches U?.10 (S0)
- net M1_S0: now also U?.42 (PB6)
- net M1_S1: now reaches U?.11 (S1)
- net M1_S1: now also U?.43 (PB7)
- net M1_S3: now reaches U?.13 (S3)
- net M1_S3: now also U?.40 (PB4)
- net M1_S2: now reaches U?.14 (S2)
- net M1_S2: now also U?.41 (PB5)
- new net: C?.2, U?.5 (PD0), Y?.2
- new net: C?.2, U?.6 (PD1), Y?.1
- new net: R?.2, SW?.1
- new net BOOT: R?.2, U?.44 (BOOT0)
- new net LED: D?.2 (A), U?.2 (PC13)
- new net PGMR_3V3: J?.1 (Pin_1), SW?.2 (B)
- new net RST: R?.1, SW?.2, U?.7 (NRST)
- new net RX: U?.13 (PA3)
- new net SWCLK: J?.3 (Pin_3), U?.37 (PA14)
- new net SWDIO: J?.2 (Pin_2), U?.34 (PA13)
- new net Sol: U?.29 (PA8)
- new net TX: U?.12 (PA2)
- no-connect marks 4 -> 17

Commit message: Removed Encoders since we are using motors with built in encoders
Parts:
- removed C?: 100n, symbol vincent:C
- removed R? (x4): R_Photo, symbol Device:R_Photo
- removed R?: 10K, symbol vincent:R
- removed R?: 3K24, symbol vincent:R
- removed U?: CD74HC4067SM, Package_SO:SSOP-24_5.3x8.2mm_P0.65mm, symbol 74xx:CD74HC4067SM
Connections:
- net M3: no longer names the net of U?.39 (PB3)
- net M3_S0: no longer names the net of U?.26 (PB13)
- net M3_S1: no longer names the net of U?.27 (PB14)
- net M3_S2: no longer names the net of U?.25 (PB12)
- net M3_S3: no longer names the net of U?.22 (PB11)
- no-connect marks 17 -> 21

Commit message: 5050 - ❌ Enc - ❌ CS
Parts:
- removed R? (x2): R_Photo, symbol Device:R_Photo
Connections:
- no-connect marks 21 -> 23
Changed lines of the file:
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@@
   (junction (at 60.96 24.13) (diameter 0) (color 0 0 0 0)
   )
-  (junction (at 170.18 24.13) (diameter 0) (color 0 0 0 0)
-  )
   (junction (at 95.25 173.99) (diameter 0) (color 0 0 0 0)
   )
@@
   (junction (at 31.75 52.07) (diameter 0) (color 0 0 0 0)
   )
-  (junction (at 81.28 24.13) (diameter 0) (color 0 0 0 0)
-  )
   (junction (at 85.09 186.69) (diameter 0) (color 0 0 0 0)
   )
@@
   )
   (no_connect (at 111.76 165.1))
+  (no_connect (at 83.82 39.37))
   (no_connect (at 144.78 132.08))
   (no_connect (at 111.76 160.02))
+  (no_connect (at 172.72 39.37))
   (no_connect (at 111.76 152.4))
   (no_connect (at 144.78 124.46))
@@
     (stroke (width 0) (type default))
   )
-  (wire (pts (xy 172.72 24.13) (xy 170.18 24.13))
-    (stroke (width 0) (type default))
-  )
   (wire (pts (xy 78.74 35.56) (xy 78.74 39.37))
     (stroke (width 0) (type default))
@@
     (stroke (width 0) (type default))
   )
-  (wire (pts (xy 172.72 35.56) (xy 172.72 39.37))
-    (stroke (width 0) (type default))
-  )
   (wire (pts (xy 91.44 52.07) (xy 97.79 52.07))
     (stroke (width 0) (type default))
@@
     (stroke (width 0) (type default))
   )
-  (wire (pts (xy 83.82 35.56) (xy 83.82 39.37))
-    (stroke (width 0) (type default))
-  )
   (wire (pts (xy 144.78 35.56) (xy 144.78 39.37))
     (stroke (width 0) (type default))
@@
     (stroke (width 0) (type default))
   )
-  (wire (pts (xy 172.72 24.13) (xy 172.72 27.94))
-    (stroke (width 0) (type default))
-  )
   (wire (pts (xy 81.28 24.13) (xy 78.74 24.13))
     (stroke (width 0) (type default))
@@
     (stroke (width 0) (type default))
   )
-  (wire (pts (xy 83.82 24.13) (xy 81.28 24.13))
-    (stroke (width 0) (type default))
-  )
   (wire (pts (xy 144.78 24.13) (xy 144.78 27.94))
     (stroke (width 0) (type default))
@@
   )
   (wire (pts (xy 120.65 52.07) (xy 127 52.07))
-    (stroke (width 0) (type default))
-  )
-  (wire (pts (xy 83.82 24.13) (xy 83.82 27.94))
     (stroke (width 0) (type default))
   )
@@
     )
   )
-  (symbol (lib_id "Device:R_Photo") (at 83.82 31.75 0) (unit 1)
-    (in_bom yes) (on_board yes) (dnp no) (fields_autoplaced)
-    (property "Reference" "R?" (at 86.36 30.4799 0)
-      (effects (font (size 1.27 1.27)) (justify left))
-    )
-    (property "Value" "R_Photo" (at 86.36 33.0199 0)
-      (effects (font (size 1.27 1.27)) (justify left))
-    )
-    (property "Footprint" "" (at 85.09 38.1 90)
-      (effects (font (size 1.27 1.27)) (justify left) hide)
-    )
-    (property "Datasheet" "~" (at 83.82 33.02 0)
-      (effects (font (size 1.27 1.27)) hide)
-    )
-    (pin "1")
-    (pin "2")
-    (instances
-      (project "2024l1"
-        (path "/5be543b5-1bdc-438f-a916-f916127c0a2b"
-          (reference "R?") (unit 1)
-        )
-        (path "/5be543b5-1bdc-438f-a916-f916127c0a2b/b3daf402-5eb6-40d4-a766-b970792273e4"
-          (reference "R?") (unit 1)
-        )
-      )
-    )
-  )
   (symbol (lib_id "Device:R_Photo") (at 58.42 31.75 0) (unit 1)
     (in_bom yes) (on_board yes) (dnp no) (fields_autoplaced)
@@
     (in_bom yes) (on_board yes) (dnp no) (fields_autoplaced)
     (property "Reference" "R?" (at 172.72 30.4799 0)
-      (effects (font (size 1.27 1.27)) (justify left))
+      (effects (font (size 1.27 1.27)) (justify left) hide)
     )
     (property "Value" "R_Photo" (at 172.72 33.0199 0)
@@
         )
       )
-    )
-  )
-  (symbol (lib_id "Device:R_Photo") (at 172.72 31.75 0) (unit 1)
-    (in_bom yes) (on_board yes) (dnp no) (fields_autoplaced)
-    (property "Reference" "R?" (at 175.26 30.4799 0)
-      (effects (font (size 1.27 1.27)) (justify left))
-    )
-    (property "Value" "R_Photo" (at 175.26 33.0199 0)
-      (effects (font (size 1.27 1.27)) (justify left))
-    )
-    (property "Footprint" "" (at 173.99 38.1 90)
-      (effects (font (size 1.27 1.27)) (justify left) hide)
-    )
-    (property "Datasheet" "~" (at 172.72 33.02 0)
-      (effects (font (size 1.27 1.27)) hide)
-    )
-    (pin "1")
-    (pin "2")
-    (instances
-      (project "2024l1"
-        (path "/5be543b5-1bdc-438f-a916-f916127c0a2b"
-          (reference "R?") (unit 1)
-        )
-        (path "/5be543b5-1bdc-438f-a916-f916127c0a2b/b3daf402-5eb6-40d4-a766-b970792273e4"
-          (reference "R?") (unit 1)
-        )
-      )
