File: VNH5019.kicad_sch (KiCad schematic)
At the start: 13 parts, among them M3R5 1K, M3R6 1K, M3R7 1K, M3R8 10K

Commit message: vnh5019 - updated mosfet
Parts:
- removed Q?: IPD050N10N5ATMA1, IPD050N10N5ATMA1, symbol vincent:IPD050N10N5ATMA1
- added Q?: IPD050N10N5ATMA1, IPD050N10N5ATMA1, symbol vincent:IPD050N10N5ATMA1
- C?: value C -> 33n
- R?: value R -> 1K5
Connections:
- net VCC: now also Q?.3 (S)
- net at IC?.11 (CP): now also Q?.1 (G)
- net at C?.1, IC?.VCC: now also Q?.2 (D)
Other:
- moved on the sheet: C?, IC?, M3R5, M3R6, M3R7, M3R8, R?
