File: 2024l1.kicad_sch (KiCad schematic)
At the start: 54 parts, among them IC1 SN74LVC2G04DBVTG4, IC2 SN74LVC2G04DBVTG4, M1 VNH5050A-E, M1C1 33n, M1R1 3K3, M1R2 3K3, M1R3 1K, M1R4 1K, M1R5 1K, M1R6 1K, M1R7 1K, M1R8 10K, M1R9 1K5, M1_CONN XT30, M2 VNH5050A-E, M2C1 33n, M2R1 3K3, M2R2 3K3, M2R3 1K, M2R4 1K, M2R5 1K, M2R6 1K, M2R7 1K, M2R8 10K, M2R9 1K5, M2_CONN XT30, M3 VNH5050A-E, M3C1 33n, M3R1 3K3, M3R2 3K3, M3R3 1K, M3R4 1K, M3R5 1K, M3R6 1K, M3R7 1K, M3R8 10K, M3R9 1K5, M3_CONN XT30, M4 VNH5050A-E, M4C1 33n, M4R1 3K3, M4R2 3K3, M4R3 1K, M4R4 1K, M4R5 1K, M4R6 1K, M4R7 1K, M4R8 10K, M4R9 1K5, M4_CONN XT30

Commit message: Motor Driver Capacitors
Parts:
- added M1C1, M2C2, M3C1, M4C1: 680u, symbol vincent:C_Polarized
- renumbered M1C1 to M1C2, M2C1 to M2C2, M3C1 to M3C2, M4C1 to M4C2
Connections:
- net GND: now also M1C1.2, M2C2.2, M3C1.2, M4C1.2
- net VCC: now also M1C1.1, M2C2.1, M3C1.1, M4C1.1

Commit message: buck conv
Parts:
- added C1, C4: 10u, symbol vincent:C
- added C2, C5: 10n, symbol vincent:C
- added C3, C6: 220u, symbol vincent:C_Polarized
- added D1, D2: SS54, symbol vincent:D_Schotty
- added L1, L2: 15u, symbol vincent:L_Iron
- added R1, R3: 10K, symbol vincent:R
- added R2: 3K24, symbol vincent:R
- added R4: 5K9, symbol vincent:R
- added U1: 3V3 Buck, symbol vincent:TPS5430
- added U2: 5V Buck, symbol vincent:TPS5430
Connections:
- net +3V3: now also C6.1, L2.2, R3.2
- net +5V: now also C3.1, L1.2, R1.2
- net GND: now also C1.1, C3.2, C4.1, C6.2, D1.2, D2.2, R2.1, R4.1, U1.6,9 (GND), U2.6,9 (GND)
- new net: R1.1, R2.2, U2.4 (VSENSE)
- new net: C2.2, D1.1, L1.1, U2.8 (PH)
- new net: R3.1, R4.2, U1.4 (VSENSE)
- new net: C5.1, U1.1 (BOOT)
- new net: C5.2, D2.1, L2.1, U1.8 (PH)
- new net: C2.1, U2.1 (BOOT)
- new net +12V: C1.2, C4.2, U1.7 (VIN), U2.7 (VIN)
- new net 3V3_ENA: U1.5 (EN)
- new net 5V_ENA: U2.5 (EN)

Commit message: mux + encoder
Parts:
- added C? (x3): 100n, symbol vincent:C
- added J?: Conn_01x12, symbol Connector_Generic:Conn_01x12
- added R? (x36): R_Photo, symbol Device:R_Photo
- added R? (x3): 3K24, symbol vincent:R
- added R? (x3): 10K, symbol vincent:R
- added SW?: M_SW, symbol Switch:SW_SPDT
- added U? (x3): CD74HC4067SM, Package_SO:SSOP-24_5.3x8.2mm_P0.65mm, symbol 74xx:CD74HC4067SM
Connections:
- net +3V3: now also C?.2, C?.2, C?.2, R?.1, R?.1, R?.1, R?.1, R?.1, R?.1, R?.1, R?.1, R?.1, R?.1, R?.1, R?.1, R?.1, R?.1, R?.1, R?.1, R?.1, R?.1, R?.1, R?.1, R?.1, R?.1, R?.1, R?.1, R?.1, R?.1, R?.1, R?.1, R?.1, R?.1, R?.1, R?.1, R?.1, R?.1, R?.1, R?.1, SW?.1 (A), U?.24 (VCC), U?.24 (VCC), U?.24 (VCC)
- net +5V: now also J?.1 (Pin_1)
- net GND: now also C?.1, C?.1, C?.1, J?.12 (Pin_12), R?.1, R?.1, R?.1, R?.1, R?.1, R?.1, SW?.3 (C), U?.12 (GND), U?.12 (GND), U?.12 (GND)
- net M1E1: now also U?.5 (I4)
- net M1E2: now also U?.4 (I5)
- net M2E1: now also U?.3 (I6)
- net M2E2: now also U?.2 (I7)
- net M3E1: now also U?.23 (I8)
- net M3E2: now also U?.22 (I9)
- net M4E1: now also U?.21 (I10)
- net M4E2: now also U?.20 (I11)
- net M_SW: now also SW?.2 (B)
- new net: R?.2, U?.19 (I12) (x2)
- new net: R?.2, U?.22 (I9) (x2)
- new net: R?.2, U?.1 (COM) (x3)
- new net: R?.2, U?.8 (I1) (x3)
- new net: R?.2, U?.3 (I6) (x2)
- new net: R?.2, U?.15 (~{E}) (x3)
- new net: R?.2, U?.16 (I15) (x2)
- new net: R?.2, U?.17 (I14) (x2)
- new net: R?.2, U?.18 (I13) (x2)
- new net: R?.2, U?.2 (I7) (x2)
- new net: R?.2, U?.20 (I11) (x2)
- new net: R?.2, U?.21 (I10) (x2)
- new net: R?.2, U?.23 (I8) (x2)
- new net: R?.2, U?.4 (I5) (x2)
- new net: R?.2, U?.5 (I4) (x2)
- new net: R?.2, U?.6 (I3) (x3)
- new net: R?.2, U?.7 (I2) (x3)
- new net: R?.2, U?.9 (I0) (x3)
- new net BL DIR: J?.9 (Pin_9)
- new net BL PWM: J?.8 (Pin_8)
- new net BR DIR: J?.11 (Pin_11)
- new net BR PWM: J?.10 (Pin_10)
- new net FL DIR: J?.5 (Pin_5)
- new net FL PWM: J?.4 (Pin_4)
- new net FR DIR: J?.7 (Pin_7)
- new net FR PWM: J?.6 (Pin_6)
- new net RX: J?.3 (Pin_3)
- new net TX: J?.2 (Pin_2)
- no-connect marks 4 -> 8
Other:
- note added: "Connections"

Commit message: split files
Parts:
- removed C1, C4: 10u, symbol vincent:C
- removed C2, C5: 10n, symbol vincent:C
- removed C3, C6: 220u, symbol vincent:C_Polarized
- removed C? (x3): 100n, symbol vincent:C
- removed D1, D2: SS54, symbol vincent:D_Schotty
- removed L1, L2: 15u, symbol vincent:L_Iron
- removed R1, R3, R? (x3): 10K, symbol vincent:R
- removed R2, R? (x3): 3K24, symbol vincent:R
- removed R4: 5K9, symbol vincent:R
- removed R? (x36): R_Photo, symbol Device:R_Photo
- removed U1: 3V3 Buck, symbol vincent:TPS5430
- removed U2: 5V Buck, symbol vincent:TPS5430
- removed U? (x3): CD74HC4067SM, Package_SO:SSOP-24_5.3x8.2mm_P0.65mm, symbol 74xx:CD74HC4067SM
Connections:
- no-connect marks 8 -> 4
Other:
- added sheet Processing (Processing.kicad_sch)
- added sheet Step Down (Step Down.kicad_sch)

Commit message: stm32
Parts:
- removed IC1, IC2: SN74LVC2G04DBVTG4, SOT95P280X145-6N, symbol vincent:SN74LVC2G04DBVTG4
- removed J?: Conn_01x12, symbol Connector_Generic:Conn_01x12
- removed M1, M2, M3, M4: VNH5050A-E, footprints:SOP50P1030X247-39N, symbol vincent:VNH5050A-E
- removed M1C1, M2C2, M3C1, M4C1: 680u, symbol vincent:C_Polarized
- removed M1C2, M2C2, M3C2, M4C2: 33n, symbol vincent:C
- removed M1R1, M1R2, M2R1, M2R2, M3R1, M3R2, M4R1, M4R2: 3K3, symbol vincent:R
- removed M1R3, M1R4, M1R5, M1R6, M1R7, M2R3, M2R4, M2R5, M2R6, M2R7, M3R3, M3R4, M3R5, M3R6, M3R7, M4R3, M4R4, M4R5, M4R6, M4R7: 1K, symbol vincent:R
- removed M1R8, M2R8, M3R8, M4R8: 10K, symbol vincent:R
- removed M1R9, M2R9, M3R9, M4R9: 1K5, symbol vincent:R
- removed M1_CONN, M2_CONN, M3_CONN, M4_CONN: XT30, symbol Connector_Generic:Conn_01x02
- removed ME1, ME2, ME3, ME4: Conn_01x04, symbol Connector_Generic:Conn_01x04
- removed SW?: M_SW, symbol Switch:SW_SPDT
Connections:
- no-connect marks 4 -> 0
Other:
- added sheet Communication (Communication.kicad_sch)
- added sheet Drive (Drive.kicad_sch)
- added sheet Encoders (Encoders.kicad_sch)
- note removed: "Connections"
- note removed: "Motor Encoders"

Commit message: 5050 - ❌ Enc - ❌ CS
Other:
- removed sheet Encoders
Changed lines of the file:
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@@
     (company "Sentinels Robotics")
   )
-  (sheet (at 129.54 106.68) (size 17.78 11.43) (fields_autoplaced)
+  (sheet (at 129.54 142.24) (size 17.78 11.43) (fields_autoplaced)
     (stroke (width 0.1524) (type solid))
     (fill (color 0 0 0 0.0000))
-    (property "Sheetname" "Step Down" (at 129.54 105.9684 0)
+    (property "Sheetname" "Step Down" (at 129.54 141.5284 0)
       (effects (font (size 1.27 1.27)) (justify left bottom))
     )
-    (property "Sheetfile" "Step Down.kicad_sch" (at 129.54 118.6946 0)
+    (property "Sheetfile" "Step Down.kicad_sch" (at 129.54 154.2546 0)
       (effects (font (size 1.27 1.27)) (justify left top))
     )
@@
       )
     )
-  )
-  (sheet (at 153.67 162.56) (size 17.78 11.43) (fields_autoplaced)
-    (stroke (width 0.1524) (type solid))
-    (fill (color 0 0 0 0.0000))
-    (property "Sheetname" "Encoders" (at 153.67 161.8484 0)
-      (effects (font (size 1.27 1.27)) (justify left bottom))
-    )
-    (property "Sheetfile" "Encoders.kicad_sch" (at 153.67 174.5746 0)
-      (effects (font (size 1.27 1.27)) (justify left top))
-    )
-    (instances
-      (project "2024l1"
-        (path "/5be543b5-1bdc-438f-a916-f916127c0a2b" (page "4"))
-      )
-    )

Commit message: vnh5019
Other:
- removed sheet Drive
- added sheet VNH5019 (VNH5019.kicad_sch)
- added sheet VNH5050 (VNH5050.kicad_sch)
Changed lines of the file:
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@@
     (company "Sentinels Robotics")
+  )
+  (sheet (at 153.67 124.46) (size 17.78 11.43) (fields_autoplaced)
+    (stroke (width 0.1524) (type solid))
+    (fill (color 0 0 0 0.0000))
+    (property "Sheetname" "VNH5050" (at 153.67 123.7484 0)
+      (effects (font (size 1.27 1.27)) (justify left bottom))
+    )
+    (property "Sheetfile" "VNH5050.kicad_sch" (at 153.67 136.4746 0)
+      (effects (font (size 1.27 1.27)) (justify left top))
+    )
+    (instances
+      (project "2024l1"
+        (path "/5be543b5-1bdc-438f-a916-f916127c0a2b" (page "5"))
+      )
+    )
   )
   (sheet (at 129.54 142.24) (size 17.78 11.43) (fields_autoplaced)
@@
       (project "2024l1"
         (path "/5be543b5-1bdc-438f-a916-f916127c0a2b" (page "3"))
+      )
+    )
+  )
+  (sheet (at 180.34 124.46) (size 17.78 11.43) (fields_autoplaced)
+    (stroke (width 0.1524) (type solid))
+    (fill (color 0 0 0 0.0000))
+    (property "Sheetname" "VNH5019" (at 180.34 123.7484 0)
+      (effects (font (size 1.27 1.27)) (justify left bottom))
+    )
+    (property "Sheetfile" "VNH5019.kicad_sch" (at 180.34 136.4746 0)
+      (effects (font (size 1.27 1.27)) (justify left top))
+    )
+    (instances
+      (project "2024l1"
+        (path "/5be543b5-1bdc-438f-a916-f916127c0a2b" (page "6"))
       )
     )
@@
       )
     )
-  )
-  (sheet (at 153.67 120.65) (size 17.78 11.43) (fields_autoplaced)
-    (stroke (width 0.1524) (type solid))
-    (fill (color 0 0 0 0.0000))
-    (property "Sheetname" "Drive" (at 153.67 119.9384 0)
-      (effects (font (size 1.27 1.27)) (justify left bottom))
-    )
-    (property "Sheetfile" "Drive.kicad_sch" (at 153.67 132.6646 0)
-      (effects (font (size 1.27 1.27)) (justify left top))
-    )
-    (instances
-      (project "2024l1"
-        (path "/5be543b5-1bdc-438f-a916-f916127c0a2b" (page "6"))
-      )
-    )

Commit message: Rethought L1
Parts:
- added C? (x4): 0.1u, symbol vincent:C
- added C? (x2): 100n, symbol vincent:C
- added C? (x2): 22p, symbol vincent:C
- added C?: 10n, footprints:cap0603, symbol Device:C
- added C?: 10u, footprints:cap0603, symbol Device:C
- added C?: 220u, footprints:EIA-7343-D, symbol Device:C_Polarized
- added D? (x31): LED, symbol Device:LED
- added D?: SS54, footprints:DIOM5025X220N, symbol Diode:B340
- added J?: Conn_01x04, symbol Connector_Generic:Conn_01x04
- added J?: PGMR, symbol Connector_Generic:Conn_01x04
- added L?: 15uH, footprints:0630 One Piece Inductor, symbol Device:L_Iron
- added R? (x30): R_Photo, symbol Device:R_Photo
- added R? (x4): 10K, symbol vincent:R
- added R?: 1K, symbol vincent:R
- added R?: 5K9, footprints:res0603, symbol Device:R
- added R? (x2): 3K24, symbol vincent:R
- added R?: 10K, footprints:res0603, symbol Device:R
- added SW?: SW_Push, symbol Switch:SW_Push
- added SW?: SW_SPDT, symbol Switch:SW_SPDT
- added U?: TPS5430DDA, footprints:TI_SO-PowerPAD-8_ThermalVias, symbol Regulator_Switching:TPS5430DDA
- added U?: STM32F103CBTx, Package_QFP:LQFP-48_7x7mm_P0.5mm, symbol vincent:STM32F103CBTx
- added U? (x2): CD74HC4067SM, Package_SO:SSOP-24_5.3x8.2mm_P0.65mm, symbol 74xx:CD74HC4067SM
- added Y?: 8Mhz, symbol vincent:Crystal
Connections:
- new net: R?.2, U?.9 (I0) (x2)
- new net: R?.2, U?.17 (I14) (x2)
- new net: R?.2, U?.15 (~{E}) (x2)
- new net: R?.2, U?.2 (I7) (x2)
- new net: R?.2, SW?.1
- new net: C?.2, D?.1 (K), L?.1, U?.8 (PH)
- new net: R?.2, U?.8 (I1) (x2)
- new net: R?.2, U?.5 (I4) (x2)
- new net: R?.2, U?.4 (I5) (x2)
- new net: R?.2, U?.22 (I9) (x2)
- new net: R?.2, U?.19 (I12) (x2)
- new net: C?.2, U?.5 (PD0), Y?.2
- new net: R?.2, U?.7 (I2) (x2)
- new net: R?.2, U?.3 (I6) (x2)
- new net: R?.2, U?.18 (I13) (x2)
- new net: R?.1, R?.2, U?.4 (VSENSE)
- new net: C?.2, U?.6 (PD1), Y?.1
- new net: R?.2, U?.23 (I8) (x2)
- new net: C?.1, U?.1 (BOOT)
- new net: R?.2, U?.20 (I11) (x2)
- new net: R?.2, U?.6 (I3) (x2)
- new net: R?.2, U?.21 (I10) (x2)
- new net +3V3: C?.1, C?.2, C?.2, C?.2, C?.2, C?.2, C?.2, D?.2 (A), D?.2 (A), D?.2 (A), D?.2 (A), D?.2 (A), D?.2 (A), D?.2 (A), D?.2 (A), D?.2 (A), D?.2 (A), D?.2 (A), D?.2 (A), D?.2 (A), D?.2 (A), D?.2 (A), D?.2 (A), D?.2 (A), D?.2 (A), D?.2 (A), D?.2 (A), D?.2 (A), D?.2 (A), D?.2 (A), D?.2 (A), D?.2 (A), D?.2 (A), D?.2 (A), D?.2 (A), D?.2 (A), D?.2 (A), L?.2, R?.1, R?.1, R?.1, R?.1, R?.1, R?.1, R?.1, R?.1, R?.1, R?.1, R?.1, R?.1, R?.1, R?.1, R?.1, R?.1, R?.1, R?.1, R?.1, R?.1, R?.1, R?.1, R?.1, R?.1, R?.1, R?.1, R?.1, R?.1, R?.1, R?.1, R?.1, R?.2, SW?.1 (A), U?.24 (VCC), U?.24 (VCC), U?.24 (VDD), U?.36 (VDD), U?.48 (VDD), U?.9 (VDDA)
- new net +5V: C?.1, J?.1 (Pin_1), U?.7 (VIN)
- new net BOOT: R?.2, U?.44 (BOOT0)
- new net GND: C?.1, C?.1, C?.1, C?.1, C?.1, C?.1, C?.1, C?.1, C?.2, C?.2, D?.1 (K), D?.1 (K), D?.1 (K), D?.1 (K), D?.1 (K), D?.1 (K), D?.1 (K), D?.1 (K), D?.1 (K), D?.1 (K), D?.1 (K), D?.1 (K), D?.1 (K), D?.1 (K), D?.1 (K), D?.1 (K), D?.1 (K), D?.1 (K), D?.1 (K), D?.1 (K), D?.1 (K), D?.1 (K), D?.1 (K), D?.1 (K), D?.1 (K), D?.1 (K), D?.1 (K), D?.1 (K), D?.1 (K), D?.1 (K), D?.1 (K), D?.2 (A), J?.4 (Pin_4), J?.4 (Pin_4), R?.1, R?.1, R?.1, R?.1, R?.1, R?.1, R?.2, U?.12 (GND), U?.12 (GND), U?.23 (VSS), U?.35 (VSS), U?.47 (VSS), U?.6 (GND), U?.8 (VSSA), U?.9 (GNDPAD)
- new net LED: D?.2 (A), U?.2 (PC13)
- new net M1: R?.2, U?.1 (COM)
- new net M1_S0: U?.10 (S0), U?.42 (PB6)
- new net M1_S1: U?.11 (S1), U?.43 (PB7)
- new net M1_S2: U?.14 (S2), U?.41 (PB5)
- new net M1_S3: U?.13 (S3), U?.40 (PB4)
- new net M2: R?.2, U?.1 (COM), U?.19 (PB1)
- new net M2_S0: U?.10 (S0), U?.20 (PB2)
- new net M2_S1: U?.11 (S1), U?.21 (PB10)
- new net M2_S2: U?.14 (S2), U?.18 (PB0)
- new net M2_S3: U?.13 (S3), U?.16 (PA6), U?.17 (PA7)
- new net PGMR_3V3: J?.1 (Pin_1), SW?.2 (B)
- new net RST: R?.1, SW?.2, U?.7 (NRST)
- new net RX: J?.3 (Pin_3), U?.13 (PA3)
- new net SWCLK: J?.3 (Pin_3), U?.37 (PA14)
- new net SWDIO: J?.2 (Pin_2), U?.34 (PA13)
- new net Sol: U?.29 (PA8)
- new net TX: J?.2 (Pin_2), U?.12 (PA2)
- no-connect marks 0 -> 23
Other:
- removed sheet Communication
- removed sheet Processing
- removed sheet Step Down
- removed sheet VNH5019
- removed sheet VNH5050
- note added: "Buck 5V -> 3V3"
- note added: "Connection"
- note added: "LED"
- note added: "MUX"
