File: test-pcb/test-pcb.kicad_pcb (KiCad board)
At the start: 4 copper layers, 16 parts, among them IC1 VNH5019ATR-E, J1 Conn_01x06, J2 Conn_01x06, J3 Conn_01x03, Q1 IPD050N10N5ATMA1

Commit message: test - thermal vias for driver
Parts:
- moved IC1 15.3 mm to (30.5, 35.6)

Commit message: test - fixed mdriver sch
Connections:
- IC1 pad GND: (no net) -> GND
- J2 pad 1: VCC -> /M1 OUTA
- J2 pad 6: GND -> /M1 OUTB
Changed lines of the file:
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@@
     (pad "24" smd rect (at -1 -9.15) (size 0.68 1.3) (layers "F.Cu" "F.Paste" "F.Mask"))
     (pad "29" smd rect (at -6 -9.15) (size 0.68 1.3) (layers "F.Cu" "F.Paste" "F.Mask"))
-    (pad "GND" smd rect (at -5 -9.15) (size 0.68 1.3) (layers "F.Cu" "F.Paste" "F.Mask"))
-    (pad "GND" smd rect (at -4 -9.15) (size 0.68 1.3) (layers "F.Cu" "F.Paste" "F.Mask"))
-    (pad "GND" smd rect (at -3 -9.15) (size 0.68 1.3) (layers "F.Cu" "F.Paste" "F.Mask"))
-    (pad "GND" smd rect (at 3 -9.15) (size 0.68 1.3) (layers "F.Cu" "F.Paste" "F.Mask"))
-    (pad "GND" smd rect (at 4 -9.15) (size 0.68 1.3) (layers "F.Cu" "F.Paste" "F.Mask"))
-    (pad "GND" smd rect (at 5 -9.15) (size 0.68 1.3) (layers "F.Cu" "F.Paste" "F.Mask"))
+    (pad "GND" smd rect (at -5 -9.15) (size 0.68 1.3) (layers "F.Cu" "F.Paste" "F.Mask")
+      (net 2 "GND") (pinfunction "GND") (pintype "passive"))
+    (pad "GND" smd rect (at -4 -9.15) (size 0.68 1.3) (layers "F.Cu" "F.Paste" "F.Mask")
+      (net 2 "GND") (pinfunction "GND") (pintype "passive"))
+    (pad "GND" smd rect (at -3 -9.15) (size 0.68 1.3) (layers "F.Cu" "F.Paste" "F.Mask")
+      (net 2 "GND") (pinfunction "GND") (pintype "passive"))
+    (pad "GND" smd rect (at 3 -9.15) (size 0.68 1.3) (layers "F.Cu" "F.Paste" "F.Mask")
+      (net 2 "GND") (pinfunction "GND") (pintype "passive"))
+    (pad "GND" smd rect (at 4 -9.15) (size 0.68 1.3) (layers "F.Cu" "F.Paste" "F.Mask")
+      (net 2 "GND") (pinfunction "GND") (pintype "passive"))
+    (pad "GND" smd rect (at 5 -9.15) (size 0.68 1.3) (layers "F.Cu" "F.Paste" "F.Mask")
+      (net 2 "GND") (pinfunction "GND") (pintype "passive"))
     (pad "OUTA" smd rect (at -7 -9.15) (size 0.68 1.3) (layers "F.Cu" "F.Paste" "F.Mask")
       (net 12 "/M1 OUTA") (pinfunction "OUTA") (pintype "passive"))
@@
       (stroke (width 0.1) (type solid)) (layer "F.Fab"))
     (pad "1" thru_hole rect (at 0 0) (size 1.7 1.7) (drill 1) (layers "*.Cu" "*.Mask")
-      (net 11 "VCC") (pinfunction "Pin_1") (pintype "passive"))
+      (net 12 "/M1 OUTA") (pinfunction "Pin_1") (pintype "passive"))
     (pad "2" thru_hole oval (at 0 2.54) (size 1.7 1.7) (drill 1) (layers "*.Cu" "*.Mask")
       (net 2 "GND") (pinfunction "Pin_2") (pintype "passive"))
@@
       (net 20 "+3V3") (pinfunction "Pin_5") (pintype "passive"))
     (pad "6" thru_hole oval (at 0 12.7) (size 1.7 1.7) (drill 1) (layers "*.Cu" "*.Mask")
-      (net 2 "GND") (pinfunction "Pin_6") (pintype "passive"))
+      (net 13 "/M1 OUTB") (pinfunction "Pin_6") (pintype "passive"))
     (model "${KICAD6_3DMODEL_DIR}/Connector_PinSocket_2.54mm.3dshapes/PinSocket_1x06_P2.54mm_Vertical.wrl"
       (offset (xyz 0 0 0))

Commit message: Test PCB Boost
Parts:
- added C3: 100uF, Capacitor_Tantalum_SMD:CP_EIA-7343-31_Kemet-D_Pad2.25x2.55mm_HandSolder, F.Cu at (88.1, 61.8)
- added C4: 1000uF, test-pcb:CAPAE1030X1270N, F.Cu at (75.6, 36.3)
- added C5: 1500pF, test-pcb:cap0603, F.Cu at (65.9, 31.8)
- added C6: 1uF, test-pcb:cap0603, F.Cu at (65.9, 34.7)
- added C7: 1000u, test-pcb:CAPAE1030X1270N, F.Cu at (75.6, 48.1)
- added D1: SS510-HF, Robocup:DIOM5025X220N, F.Cu at (97.1, 61.0)
- added D2: 1N5401, Diode_THT:D_DO-201AD_P15.24mm_Horizontal, F.Cu at (85.3, 43.4)
- added IC2: LM2587S-ADJ_NOPB, test-pcb:TO170P1435X465-6N, F.Cu at (91.3, 52.8)
- added J2: XT60, Robocup:AMASS_XT60-M, F.Cu at (93.0, 35.2)
- added L1: 56uH, test-pcb:0630 One Piece Inductor, F.Cu at (72.8, 58.6)
- added R11: 57k, test-pcb:res0603, F.Cu at (65.9, 37.6)
- added R12: 20, test-pcb:res0603, F.Cu at (65.9, 40.5)
- added R13: 2.94k, test-pcb:res0603, F.Cu at (65.9, 43.4)
- added R14: 1K, test-pcb:res0603, F.Cu at (65.9, 46.3)
- added R15: 10K, test-pcb:res0603, F.Cu at (65.9, 49.2)
- added R16: 1.5k, test-pcb:res0603, F.Cu at (65.9, 52.1)
- added R17: 10K, test-pcb:res0603, F.Cu at (65.9, 55.0)
- renumbered C1 to C2, R3 to R1, R8 to R2, R1 to R3, R2 to R4, R4 to R5, R5 to R6, R6 to R7, R7 to R8
