File: test-pcb/test-pcb.kicad_sch (KiCad schematic)
At the start: 14 parts, among them IC1 VNH5019ATR-E, Q1 IPD050N10N5ATMA1

Commit message: test-pcb added connectors
Parts:
- added J? (x2): Conn_01x06, symbol Connector_Generic:Conn_01x06
- added J?: Conn_01x03, symbol Connector_Generic:Conn_01x03
Connections:
- net +3V3: now also J?.2 (Pin_2), J?.3 (Pin_3)
- net GND: now also J?.2 (Pin_2), J?.5 (Pin_5), J?.6 (Pin_6)
- net M1 CS: now also J?.4 (Pin_4)
- net M1 INA: now also J?.1 (Pin_1)
- net M1 INB: now also J?.2 (Pin_2)
- net M1 PWM: now also J?.3 (Pin_3)
- net VCC: now also J?.1 (Pin_1), J?.1 (Pin_1)
- new net ENC 1: J?.3 (Pin_3), J?.5 (Pin_5)
- new net ENC 2: J?.4 (Pin_4), J?.6 (Pin_6)
Other:
- moved on the sheet: C1, C2, IC1, Q1, R1, R10, R2, R3, R4, R5, R6, R7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

Commit message: test-pcb fix enc
Connections:
- net +3V3: now also J?.5 (Pin_5); no longer J?.2 (Pin_2)
- net GND: now also J?.2 (Pin_2); no longer J?.5 (Pin_5)
Changed lines of the file:
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@@
   (junction (at 45.72 80.01) (diameter 0) (color 0 0 0 0)
   )
-  (junction (at 132.08 73.66) (diameter 0) (color 0 0 0 0)
-  )
   (junction (at 101.6 57.15) (diameter 0) (color 0 0 0 0)
   )
@@
   (junction (at 101.6 39.37) (diameter 0) (color 0 0 0 0)
   )
-  (wire (pts (xy 130.81 73.66) (xy 132.08 73.66))
+  (wire (pts (xy 130.81 73.66) (xy 135.89 73.66))
     (stroke (width 0) (type default))
   )
@@
     (stroke (width 0) (type default))
   )
+  (wire (pts (xy 130.81 63.5) (xy 135.89 63.5))
+    (stroke (width 0) (type default))
+  )
   (wire (pts (xy 101.6 26.67) (xy 101.6 39.37))
     (stroke (width 0) (type default))
@@
     (stroke (width 0) (type default))
   )
-  (wire (pts (xy 132.08 73.66) (xy 135.89 73.66))
-    (stroke (width 0) (type default))
-  )
   (wire (pts (xy 41.91 44.45) (xy 45.72 44.45))
     (stroke (width 0) (type default))
@@
     (stroke (width 0) (type default))
   )
-  (wire (pts (xy 132.08 71.12) (xy 132.08 73.66))
-    (stroke (width 0) (type default))
-  )
   (wire (pts (xy 82.55 48.26) (xy 93.98 48.26))
     (stroke (width 0) (type default))
@@
     (stroke (width 0) (type default))
   )
-  (wire (pts (xy 135.89 71.12) (xy 132.08 71.12))
-    (stroke (width 0) (type default))
-  )
   (wire (pts (xy 82.55 60.96) (xy 95.25 60.96))
     (stroke (width 0) (type default))
@@
     (stroke (width 0) (type default))
   )
-  (wire (pts (xy 130.81 63.5) (xy 135.89 63.5))
-    (stroke (width 0) (type default))
-  )
   (wire (pts (xy 38.1 80.01) (xy 45.72 80.01))
     (stroke (width 0) (type default))
@@
   )
   (wire (pts (xy 50.8 57.15) (xy 58.42 57.15))
+    (stroke (width 0) (type default))
+  )
+  (wire (pts (xy 130.81 71.12) (xy 135.89 71.12))
     (stroke (width 0) (type default))
   )
@@
     )
   )
-  (symbol (lib_id "power:+3V3") (at 130.81 63.5 90) (unit 1)
-    (in_bom yes) (on_board yes) (dnp no) (fields_autoplaced)
-    (property "Reference" "#PWR011" (at 134.62 63.5 0)
-      (effects (font (size 1.27 1.27)) hide)
-    )
-    (property "Value" "+3V3" (at 127 63.4999 90)
-      (effects (font (size 1.27 1.27)) (justify left))
+  (symbol (lib_id "power:GND") (at 130.81 63.5 270) (mirror x) (unit 1)
+    (in_bom yes) (on_board yes) (dnp no) (fields_autoplaced)
+    (property "Reference" "#PWR013" (at 124.46 63.5 0)
+      (effects (font (size 1.27 1.27)) hide)
+    )
+    (property "Value" "GND" (at 127 63.4999 90)
+      (effects (font (size 1.27 1.27)) (justify right))
     )
     (property "Footprint" "" (at 130.81 63.5 0)
@@
       (project "test-pcb"
         (path "/1cd04cc7-ac63-4801-a234-4389545ae7cf"
-          (reference "#PWR011") (unit 1)
+          (reference "#PWR013") (unit 1)
         )
       )
@@
         )
       )
+    )
+  )
+  (symbol (lib_id "power:+3V3") (at 130.81 71.12 90) (mirror x) (unit 1)
+    (in_bom yes) (on_board yes) (dnp no) (fields_autoplaced)
+    (property "Reference" "#PWR011" (at 134.62 71.12 0)
+      (effects (font (size 1.27 1.27)) hide)
+    )
+    (property "Value" "+3V3" (at 127 71.1201 90)
+      (effects (font (size 1.27 1.27)) (justify left))
+    )
+    (property "Footprint" "" (at 130.81 71.12 0)
+      (effects (font (size 1.27 1.27)) hide)
+    )
+    (property "Datasheet" "" (at 130.81 71.12 0)
+      (effects (font (size 1.27 1.27)) hide)
+    )
+    (pin "1")
+    (instances
+      (project "test-pcb"
+        (path "/1cd04cc7-ac63-4801-a234-4389545ae7cf"
+          (reference "#PWR011") (unit 1)
+        )
+      )

Commit message: test - footprint & 3dmodels
Parts:
- C1: footprint (none) -> test-pcb:cap0603
- IC1: footprint VNH5019A-E_1 -> test-pcb:VNH5019A-E
- J1, J2: renamed from J?; footprint (none) -> Connector_PinSocket_2.54mm:PinSocket_1x06_P2.54mm_Vertical
- J3: renamed from J?; footprint (none) -> Connector_PinSocket_2.54mm:PinSocket_1x03_P2.54mm_Vertical
- Q1: footprint IPD050N10N5ATMA1 -> test-pcb:IPD050N10N5ATMA1
- R1, R10, R2, R3, R4, R5, R6, R7, R8, R9: footprint (none) -> test-pcb:res0603
Changed lines of the file:
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@@
       (effects (font (size 1.27 1.27)) (justify left))
     )
-    (property "Footprint" "" (at 55.372 77.47 90)
+    (property "Footprint" "test-pcb:res0603" (at 55.372 77.47 90)
       (effects (font (size 1.27 1.27)) hide)
     )
@@
       (effects (font (size 1.27 1.27)) (justify left))
     )
-    (property "Footprint" "" (at 55.118 73.66 90)
+    (property "Footprint" "test-pcb:res0603" (at 55.118 73.66 90)
       (effects (font (size 1.27 1.27)) hide)
     )
@@
       (effects (font (size 1.27 1.27)))
     )
-    (property "Footprint" "" (at 36.83 44.45 0)
+    (property "Footprint" "test-pcb:res0603" (at 36.83 44.45 0)
       (effects (font (size 1.27 1.27)) hide)
     )
@@
   (symbol (lib_id "Connector_Generic:Conn_01x06") (at 140.97 45.72 0) (unit 1)
     (in_bom yes) (on_board yes) (dnp no) (fields_autoplaced)
-    (property "Reference" "J?" (at 143.51 45.7199 0)
+    (property "Reference" "J1" (at 143.51 45.7199 0)
       (effects (font (size 1.27 1.27)) (justify left))
     )
@@
       (effects (font (size 1.27 1.27)) (justify left))
     )
-    (property "Footprint" "" (at 140.97 45.72 0)
+    (property "Footprint" "Connector_PinSocket_2.54mm:PinSocket_1x06_P2.54mm_Vertical" (at 140.97 45.72 0)
       (effects (font (size 1.27 1.27)) hide)
     )
@@
       (project "test-pcb"
         (path "/1cd04cc7-ac63-4801-a234-4389545ae7cf"
-          (reference "J?") (unit 1)
+          (reference "J1") (unit 1)
         )
       )
@@
       (effects (font (size 1.27 1.27)))
     )
-    (property "Footprint" "" (at 36.83 48.26 0)
+    (property "Footprint" "test-pcb:res0603" (at 36.83 48.26 0)
       (effects (font (size 1.27 1.27)) hide)
     )
@@
       (effects (font (size 1.27 1.27)) (justify left))
     )
-    (property "Footprint" "" (at 49.022 35.56 90)
+    (property "Footprint" "test-pcb:res0603" (at 49.022 35.56 90)
       (effects (font (size 1.27 1.27)) hide)
     )
@@
       (effects (font (size 1.27 1.27)))
     )
-    (property "Footprint" "" (at 45.72 57.15 0)
+    (property "Footprint" "test-pcb:res0603" (at 45.72 57.15 0)
       (effects (font (size 1.27 1.27)) hide)
     )
@@
       (effects (font (size 1.27 1.27)) (justify left))
     )
-    (property "Footprint" "" (at 47.498 35.56 90)
+    (property "Footprint" "test-pcb:res0603" (at 47.498 35.56 90)
       (effects (font (size 1.27 1.27)) hide)
     )
@@
       (effects (font (size 1.27 1.27)) (justify left))
     )
-    (property "Footprint" "" (at 39.0652 77.47 0)
+    (property "Footprint" "test-pcb:cap0603" (at 39.0652 77.47 0)
       (effects (font (size 1.27 1.27)) hide)
     )
@@
       (effects (font (size 1.27 1.27)))
     )
-    (property "Footprint" "" (at 45.72 67.31 0)
+    (property "Footprint" "test-pcb:res0603" (at 45.72 67.31 0)
       (effects (font (size 1.27 1.27)) hide)
     )
@@
       (effects (font (size 1.27 1.27)))
     )
-    (property "Footprint" "" (at 45.72 53.34 0)
+    (property "Footprint" "test-pcb:res0603" (at 45.72 53.34 0)
       (effects (font (size 1.27 1.27)) hide)
     )
@@
       (effects (font (size 1.27 1.27)))
     )
-    (property "Footprint" "VNH5019A-E_1" (at 90.17 139.37 0)
+    (property "Footprint" "test-pcb:VNH5019A-E" (at 90.17 139.37 0)
       (effects (font (size 1.27 1.27)) (justify left top) hide)
     )
@@
       (effects (font (size 1.27 1.27)) (justify left))
     )
-    (property "Footprint" "IPD050N10N5ATMA1" (at 105.41 -50.47 0)
+    (property "Footprint" "test-pcb:IPD050N10N5ATMA1" (at 105.41 -50.47 0)
       (effects (font (size 1.27 1.27)) (justify left top) hide)
     )
@@
   (symbol (lib_id "Connector_Generic:Conn_01x03") (at 189.23 30.48 0) (mirror y) (unit 1)
     (in_bom yes) (on_board yes) (dnp no) (fields_autoplaced)
-    (property "Reference" "J?" (at 189.23 21.59 0)
+    (property "Reference" "J3" (at 189.23 21.59 0)
       (effects (font (size 1.27 1.27)))
     )
@@
       (effects (font (size 1.27 1.27)))
     )
-    (property "Footprint" "" (at 189.23 30.48 0)
+    (property "Footprint" "Connector_PinSocket_2.54mm:PinSocket_1x03_P2.54mm_Vertical" (at 189.23 30.48 0)
       (effects (font (size 1.27 1.27)) hide)
     )
@@
       (project "test-pcb"
         (path "/1cd04cc7-ac63-4801-a234-4389545ae7cf"
-          (reference "J?") (unit 1)
+          (reference "J3") (unit 1)
         )
       )
@@
       (effects (font (size 1.27 1.27)))
     )
-    (property "Footprint" "" (at 45.72 62.23 0)
+    (property "Footprint" "test-pcb:res0603" (at 45.72 62.23 0)
       (effects (font (size 1.27 1.27)) hide)
     )
@@
   (symbol (lib_id "Connector_Generic:Conn_01x06") (at 140.97 66.04 0) (unit 1)
     (in_bom yes) (on_board yes) (dnp no) (fields_autoplaced)
-    (property "Reference" "J?" (at 143.51 66.0399 0)
+    (property "Reference" "J2" (at 143.51 66.0399 0)
       (effects (font (size 1.27 1.27)) (justify left))
     )
@@
       (effects (font (size 1.27 1.27)) (justify left))
     )
-    (property "Footprint" "" (at 140.97 66.04 0)
+    (property "Footprint" "Connector_PinSocket_2.54mm:PinSocket_1x06_P2.54mm_Vertical" (at 140.97 66.04 0)
       (effects (font (size 1.27 1.27)) hide)
     )
@@
       (project "test-pcb"
         (path "/1cd04cc7-ac63-4801-a234-4389545ae7cf"
-          (reference "J?") (unit 1)
-        )
-      )
+          (reference "J2") (unit 1)
+        )
+      )

Commit message: test - fixed mdriver sch
Connections:
- net GND: no longer J2.6 (Pin_6)
- net M1 OUTA: now also J2.1 (Pin_1)
- net M1 OUTB: now also J2.6 (Pin_6)
- net VCC: no longer J2.1 (Pin_1)
Changed lines of the file:
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@@
   (junction (at 101.6 39.37) (diameter 0) (color 0 0 0 0)
   )
-  (wire (pts (xy 130.81 73.66) (xy 135.89 73.66))
+  (wire (pts (xy 125.73 73.66) (xy 135.89 73.66))
     (stroke (width 0) (type default))
   )
@@
     (stroke (width 0) (type default))
   )
-  (wire (pts (xy 130.81 63.5) (xy 135.89 63.5))
-    (stroke (width 0) (type default))
-  )
   (wire (pts (xy 101.6 26.67) (xy 101.6 39.37))
     (stroke (width 0) (type default))
@@
     (stroke (width 0) (type default))
   )
-  (wire (pts (xy 129.54 66.04) (xy 135.89 66.04))
-    (stroke (width 0) (type default))
-  )
-  (wire (pts (xy 129.54 68.58) (xy 135.89 68.58))
+  (wire (pts (xy 125.73 66.04) (xy 135.89 66.04))
+    (stroke (width 0) (type default))
+  )
+  (wire (pts (xy 125.73 68.58) (xy 135.89 68.58))
     (stroke (width 0) (type default))
   )
@@
     (stroke (width 0) (type default))
   )
+  (wire (pts (xy 127 63.5) (xy 135.89 63.5))
+    (stroke (width 0) (type default))
+  )
   (wire (pts (xy 25.4 44.45) (xy 31.75 44.45))
     (stroke (width 0) (type default))
@@
     (stroke (width 0) (type default))
   )
-  (wire (pts (xy 130.81 60.96) (xy 135.89 60.96))
+  (wire (pts (xy 125.73 60.96) (xy 135.89 60.96))
     (stroke (width 0) (type default))
   )
@@
     (stroke (width 0) (type default))
   )
-  (wire (pts (xy 130.81 71.12) (xy 135.89 71.12))
+  (wire (pts (xy 127 71.12) (xy 135.89 71.12))
     (stroke (width 0) (type default))
   )
@@
     (effects (font (size 1.27 1.27)) (justify right bottom))
   )
-  (label "ENC 1" (at 130.81 66.04 0) (fields_autoplaced)
+  (label "ENC 1" (at 127 66.04 0) (fields_autoplaced)
     (effects (font (size 1.27 1.27)) (justify left bottom))
   )
@@
     (effects (font (size 1.27 1.27)) (justify left bottom))
   )
-  (label "ENC 2" (at 130.81 68.58 0) (fields_autoplaced)
+  (label "ENC 2" (at 127 68.58 0) (fields_autoplaced)
     (effects (font (size 1.27 1.27)) (justify left bottom))
   )
@@
     (effects (font (size 1.27 1.27)) (justify left bottom))
   )
+  (label "M1 OUTA" (at 127 60.96 0) (fields_autoplaced)
+    (effects (font (size 1.27 1.27)) (justify left bottom))
+  )
   (label "M1 PWM" (at 26.67 62.23 0) (fields_autoplaced)
     (effects (font (size 1.27 1.27)) (justify left bottom))
   )
   (label "ENC 2" (at 127 53.34 0) (fields_autoplaced)
+    (effects (font (size 1.27 1.27)) (justify left bottom))
+  )
+  (label "M1 OUTB" (at 127 73.66 0) (fields_autoplaced)
     (effects (font (size 1.27 1.27)) (justify left bottom))
   )
@@
     )
   )
-  (symbol (lib_id "power:GND") (at 130.81 63.5 270) (mirror x) (unit 1)
-    (in_bom yes) (on_board yes) (dnp no) (fields_autoplaced)
-    (property "Reference" "#PWR013" (at 124.46 63.5 0)
-      (effects (font (size 1.27 1.27)) hide)
-    )
-    (property "Value" "GND" (at 127 63.4999 90)
+  (symbol (lib_id "power:GND") (at 127 63.5 270) (mirror x) (unit 1)
+    (in_bom yes) (on_board yes) (dnp no) (fields_autoplaced)
+    (property "Reference" "#PWR013" (at 120.65 63.5 0)
+      (effects (font (size 1.27 1.27)) hide)
+    )
+    (property "Value" "GND" (at 123.19 63.4999 90)
       (effects (font (size 1.27 1.27)) (justify right))
     )
-    (property "Footprint" "" (at 130.81 63.5 0)
-      (effects (font (size 1.27 1.27)) hide)
-    )
-    (property "Datasheet" "" (at 130.81 63.5 0)
+    (property "Footprint" "" (at 127 63.5 0)
+      (effects (font (size 1.27 1.27)) hide)
+    )
+    (property "Datasheet" "" (at 127 63.5 0)
       (effects (font (size 1.27 1.27)) hide)
     )
@@
     )
   )
-  (symbol (lib_id "power:+3V3") (at 130.81 71.12 90) (mirror x) (unit 1)
-    (in_bom yes) (on_board yes) (dnp no) (fields_autoplaced)
-    (property "Reference" "#PWR011" (at 134.62 71.12 0)
-      (effects (font (size 1.27 1.27)) hide)
-    )
-    (property "Value" "+3V3" (at 127 71.1201 90)
-      (effects (font (size 1.27 1.27)) (justify left))
-    )
-    (property "Footprint" "" (at 130.81 71.12 0)
-      (effects (font (size 1.27 1.27)) hide)
-    )
-    (property "Datasheet" "" (at 130.81 71.12 0)
+  (symbol (lib_id "power:+3V3") (at 127 71.12 90) (mirror x) (unit 1)
+    (in_bom yes) (on_board yes) (dnp no) (fields_autoplaced)
+    (property "Reference" "#PWR011" (at 130.81 71.12 0)
+      (effects (font (size 1.27 1.27)) hide)
+    )
+    (property "Value" "+3V3" (at 123.19 71.1201 90)
+      (effects (font (size 1.27 1.27)) (justify left))
+    )
+    (property "Footprint" "" (at 127 71.12 0)
+      (effects (font (size 1.27 1.27)) hide)
+    )
+    (property "Datasheet" "" (at 127 71.12 0)
       (effects (font (size 1.27 1.27)) hide)
     )
@@
     )
   )
-  (symbol (lib_id "power:VCC") (at 130.81 60.96 90) (mirror x) (unit 1)
-    (in_bom yes) (on_board yes) (dnp no) (fields_autoplaced)
-    (property "Reference" "#PWR09" (at 134.62 60.96 0)
-      (effects (font (size 1.27 1.27)) hide)
-    )
-    (property "Value" "VCC" (at 127 60.9599 90)
-      (effects (font (size 1.27 1.27)) (justify left))
-    )
-    (property "Footprint" "" (at 130.81 60.96 0)
-      (effects (font (size 1.27 1.27)) hide)
-    )
-    (property "Datasheet" "" (at 130.81 60.96 0)
-      (effects (font (size 1.27 1.27)) hide)
-    )
-    (pin "1")
-    (instances
-      (project "test-pcb"
-        (path "/1cd04cc7-ac63-4801-a234-4389545ae7cf"
-          (reference "#PWR09") (unit 1)
-        )
-      )
-    )
-  )
   (symbol (lib_id "power:GND") (at 101.6 82.55 0) (unit 1)
     (in_bom yes) (on_board yes) (dnp no) (fields_autoplaced)
@@
         )
       )
-    )
-  )
-  (symbol (lib_id "power:GND") (at 130.81 73.66 270) (mirror x) (unit 1)
-    (in_bom yes) (on_board yes) (dnp no) (fields_autoplaced)
-    (property "Reference" "#PWR010" (at 124.46 73.66 0)
-      (effects (font (size 1.27 1.27)) hide)
-    )
-    (property "Value" "GND" (at 127 73.6599 90)
-      (effects (font (size 1.27 1.27)) (justify right))
-    )
-    (property "Footprint" "" (at 130.81 73.66 0)
-      (effects (font (size 1.27 1.27)) hide)
-    )
-    (property "Datasheet" "" (at 130.81 73.66 0)
-      (effects (font (size 1.27 1.27)) hide)
-    )
-    (pin "1")
-    (instances
-      (project "test-pcb"
-        (path "/1cd04cc7-ac63-4801-a234-4389545ae7cf"
-          (reference "#PWR010") (unit 1)
-        )
-      )

Commit message: test - fixed mdriver sch
Connections:
- net GND: now also IC1.GND; no longer IC1.26 (GND)
Changed lines of the file:
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@@
     (pin "11")
     (pin "12")
-    (pin "26")
     (pin "4")
     (pin "5")
@@
     (pin "8")
     (pin "9")
+    (pin "GND")
     (pin "OUTA")
     (pin "OUTB")

Commit message: l2&test - activation circuit
Parts:
- added C?: 1000u, footprints:CAPAE1030X1270N, symbol Device:C_Polarized
- added C?: 1500pF, footprints:cap0603, symbol Device:C
- added D?: 1N5401, Diode_THT:D_DO-201AD_P15.24mm_Horizontal, symbol Diode:1N5401
- added J?: XT30, symbol Connector_Generic:Conn_01x02
- added Q?: STP75NF75, IPD050N10N5ATMA1, symbol vincent:IPD050N10N5ATMA1
- added Q?: AO34OO, IPD050N10N5ATMA1, symbol vincent:IPD050N10N5ATMA1
- added R?: 20, footprints:res0603, symbol Device:R
- added R? (x2): 10K, footprints:res0603, symbol Device:R
- added R?: 1K, footprints:res0603, symbol Device:R
Connections:
- net GND: now also C?.2, Q?.3 (S), R?.2
- new net: Q?.1 (G), R?.2
- new net: D?.2 (A), J?.2 (Pin_2), Q?.2 (D), R?.1
- new net: C?.2, Q?.2 (D), Q?.3 (S), R?.2
- new net: C?.1, R?.2
- new net +12V: R?.1, R?.1
- new net +48V: C?.1, D?.1 (K), J?.1 (Pin_1)
- new net Sol: Q?.1 (G), R?.1
Other:
- note added: "Activation Circuit"

Commit message: test - switch
Parts:
- removed C?: 1000u, footprints:CAPAE1030X1270N, symbol Device:C_Polarized
- removed C?: 1500pF, footprints:cap0603, symbol Device:C
- removed D?: 1N5401, Diode_THT:D_DO-201AD_P15.24mm_Horizontal, symbol Diode:1N5401
- removed J1, J2: Conn_01x06, Connector_PinSocket_2.54mm:PinSocket_1x06_P2.54mm_Vertical, symbol Connector_Generic:Conn_01x06
- removed J3: Conn_01x03, Connector_PinSocket_2.54mm:PinSocket_1x03_P2.54mm_Vertical, symbol Connector_Generic:Conn_01x03
- removed J?: XT30, symbol Connector_Generic:Conn_01x02
- removed Q?: STP75NF75, IPD050N10N5ATMA1, symbol vincent:IPD050N10N5ATMA1
- removed Q?: AO34OO, IPD050N10N5ATMA1, symbol vincent:IPD050N10N5ATMA1
- removed R?: 20, footprints:res0603, symbol Device:R
- removed R? (x2): 10K, footprints:res0603, symbol Device:R
- removed R?: 1K, footprints:res0603, symbol Device:R
- added C?: 1500pF, footprints:cap0603, symbol Device:C
- added C?: 1000u, footprints:CAPAE1030X1270N, symbol Device:C_Polarized
- added D?: 1N5401, Diode_THT:D_DO-201AD_P15.24mm_Horizontal, symbol Diode:1N5401
- added J?: XT30, symbol Connector_Generic:Conn_01x02
- added Q?: AO3400A, symbol vincent:IPD050N10N5ATMA1
- added Q?: STP75NF75, symbol vincent:IPD050N10N5ATMA1
- added R? (x2): 10K, footprints:res0603, symbol Device:R
- added R?: 1K, footprints:res0603, symbol Device:R
- added R?: 20, footprints:res0603, symbol Device:R
- IC1: footprint test-pcb:VNH5019A-E -> 2024l2:VNH5019A-E
- Q1: footprint test-pcb:IPD050N10N5ATMA1 -> IPD050N10N5ATMA1
Connections:
- net +12V: now also R?.1, R?.1
- net +48V: now also C?.1, D?.1 (K), J?.1 (Pin_1)
- net GND: now also C?.2, Q?.3 (S), R?.2
- net Sol: now also Q?.1 (G), R?.1
- new net: D?.2 (A), J?.2 (Pin_2), Q?.2 (D), R?.1
- new net: C?.1, R?.2
- new net: C?.2, Q?.2 (D), Q?.3 (S), R?.2
- new net: Q?.1 (G), R?.2

Commit message: Test PCB Boost
Parts:
- added C10, C3, C8, C9: 100uF, test-pcb:EIA-7343-D, symbol Device:C_Polarized
- added C4: 1000uF, test-pcb:CAPAE1030X1270N, symbol Device:C_Polarized
- added C6: 1uF, test-pcb:cap0603, symbol Device:C
- added D1: SS510-HF, Robocup:DIOM5025X220N, symbol SS510-HF:SS510-HF
- added IC2: LM2587S-ADJ_NOPB, test-pcb:TO170P1435X465-6N, symbol LM2587S-ADJ_NOPB:LM2587S-ADJ_NOPB
- added J2: XT60, test-pcb:AMASS_XT60-M, symbol XT60-M:XT60
- added J3: Conn_01x02_Pin, Connector_PinHeader_2.54mm:PinHeader_1x02_P2.54mm_Vertical, symbol Connector:Conn_01x02_Pin
- added L1: 56uH, test-pcb:0630 One Piece Inductor, symbol Device:L
- added R11: 57k, test-pcb:res0603, symbol Device:R
- added R13: 2.94k, test-pcb:res0603, symbol Device:R
- added R16: 1.5k, test-pcb:res0603, symbol Device:R
- added RV1: 10k, test-pcb:TRIM_3362W-1-203LF, symbol Device:R_Potentiometer_Trim
- C1: renamed from C2; footprint (none) -> test-pcb:TRIM_3362W-1-203LF
- C5: renamed from C?; footprint footprints:cap0603 -> test-pcb:cap0603
- C7: renamed from C?; footprint footprints:CAPAE1030X1270N -> test-pcb:CAPAE1030X1270N
- IC1: footprint 2024l2:VNH5019A-E -> test-pcb:VNH5019A-E
- J1: renamed from J?; footprint (none) -> test-pcb:AMASS_XT30-F
- Q1: footprint IPD050N10N5ATMA1 -> test-pcb:IPD050N10N5ATMA1
- Q2: renamed from Q?; footprint (none) -> test-pcb:TO255P1040X460X2890-3
- R12, R14, R15, R17: renamed from R?; footprint footprints:res0603 -> test-pcb:res0603
- gave numbers to parts that had none: 2
- renumbered C1 to C2, R3 to R1, R8 to R2, R1 to R3, R2 to R4, R4 to R5, R5 to R6, R6 to R7, R7 to R8
Connections:
- net +12V: now also C3.1, IC2.5 (VIN), J2.2 (POS), L1.1
- net +3V3: now also J3.2 (Pin_2)
- net +48V: now also C10.1, C4.1, C8.1, C9.1, D1.1 (K), R11.1
- net GND: now also C10.2, C3.2, C4.2, C6.2, C8.2, C9.2, IC2.3 (GND), IC2.6 (TAB), J2.1 (NEG), J3.1 (Pin_1), R16.2
- new net: D1.2 (A), IC2.4 (SW), L1.2
- new net: IC2.2 (FDBK), R16.1, RV1.1, RV1.2
- new net: R11.2, RV1.3
- new net: C6.1, R13.2
- new net: IC2.1 (COMP), R13.1
Other:
- note added: "Boost"
