File: 2024l1/2024l1.kicad_pcb (KiCad board)
At the start: 2 copper layers, 176 x 167.3 mm, 117 parts, among them J1 Conn_01x04, J2 Conn_01x04, J3 XT30, J5 Conn_01x04, Q1 STP75NF75, Q2 AO3400A, SW1 SW_Push, SW2 SW_SPDT, U1 CD74HC4067SM, U2 CD74HC4067SM, U3 STM32F103CBTx, Y1 8Mhz

Commit message: l1 - MTH & silkscrn
Parts:
- removed ? (x14): , 
- removed REF**: SEN Logo Pad 2cm, Logo:SEN Logo Pad 2cm
- added MTH10: MountingHole_Pad, MountingHole:MountingHole_3.2mm_M3_Pad_Via, F.Cu at (156.8, 102.0)
- added MTH11: MountingHole_Pad, MountingHole:MountingHole_3.2mm_M3_Pad_Via, F.Cu at (25.7, 98.1)
- added MTH12: MountingHole_Pad, MountingHole:MountingHole_3.2mm_M3_Pad_Via, F.Cu at (189.3, 98.1)
- added MTH13: MountingHole_Pad, MountingHole:MountingHole_3.2mm_M3_Pad_Via, F.Cu at (77.8, 73.0)
- added MTH14: MountingHole_Pad, MountingHole:MountingHole_3.2mm_M3_Pad_Via, F.Cu at (137.2, 73.0)
- added MTH15: MountingHole_Pad, MountingHole:MountingHole_3.2mm_M3_Pad_Via, F.Cu at (61.0, 43.5)
- added MTH16: MountingHole_Pad, MountingHole:MountingHole_3.2mm_M3_Pad_Via, F.Cu at (154.0, 43.5)
- added MTH3: MountingHole_Pad, MountingHole:MountingHole_3.2mm_M3_Pad_Via, F.Cu at (77.8, 151.5)
- added MTH4: MountingHole_Pad, MountingHole:MountingHole_3.2mm_M3_Pad_Via, F.Cu at (137.2, 151.5)
- added MTH5: MountingHole_Pad, MountingHole:MountingHole_3.2mm_M3_Pad_Via, F.Cu at (25.7, 126.4)
- added MTH6: MountingHole_Pad, MountingHole:MountingHole_3.2mm_M3_Pad_Via, F.Cu at (189.3, 126.4)
- added MTH7: MountingHole_Pad, MountingHole:MountingHole_3.2mm_M3_Pad_Via, F.Cu at (58.2, 122.5)
- added MTH8: MountingHole_Pad, MountingHole:MountingHole_3.2mm_M3_Pad_Via, F.Cu at (156.8, 122.5)
- added MTH9: MountingHole_Pad, MountingHole:MountingHole_3.2mm_M3_Pad_Via, F.Cu at (58.2, 102.0)
- MTH1, MTH2: renamed from REF**; value MountingHole_3.2mm_M3_Pad_Via -> MountingHole_Pad
- moved R43 12.4 mm to (145.8, 187.0), turned to -90 degrees
- moved MTH2 0.12 mm to (149.9, 183.6)
Connections:
- MTH1 pad 1: (no net) -> unconnected-(MTH1-Pad1)
- MTH2 pad 1: (no net) -> unconnected-(MTH2-Pad1)
Other:
- outline, holes or cut-outs redrawn
- board text added: "@sentinelsrobotics"

Commit message: L1-Routed Light Gate
Routing:
- net /LG: track 0.00 -> 102.5 mm, vias 0 -> 1
- net +3V3: track 587.6 -> 621.0 mm
- net Net-(D32-A): track 0.00 -> 14.3 mm
- net Net-(Q1-S): track 10.1 -> 11.9 mm
- net /SWCLK: track 83.6 -> 82.4 mm
- net GND: vias 0 -> 2
Changed lines of the file:
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@@
   (segment (start 48.194308 86.041186) (end 45.91 92.41) (width 1) (layer "B.Cu") (net 1))
   (segment (start 144.3 109.4) (end 172.165826 109.4) (width 0.3) (layer "B.Cu") (net 1))
+  (segment (start 142.8 180.264509) (end 142.8 184.21) (width 0.3) (layer "B.Cu") (net 1))
   (segment (start 150.822751 160.62909) (end 155.5 155.74) (width 1) (layer "B.Cu") (net 1))
   (segment (start 172.391805 112.283656) (end 172.175826 109.39) (width 1) (layer "B.Cu") (net 1))
@@
   (segment (start 155.58147 68.95725) (end 150.69238 64.280001) (width 1) (layer "B.Cu") (net 1))
   (segment (start 59.41853 155.54275) (end 64.30762 160.219999) (width 1) (layer "B.Cu") (net 1))
+  (segment (start 72.125 184.19) (end 72.125 180.339509) (width 0.3) (layer "B.Cu") (net 1))
   (segment (start 69.470294 59.9066) (end 64.307618 64.280001) (width 1) (layer "B.Cu") (net 1))
   (segment (start 106.25 110.926041) (end 104.823959 109.5) (width 0.3) (layer "B.Cu") (net 1))
@@
   (segment (start 43.154433 105.487008) (end 42.949999 112.25) (width 1) (layer "B.Cu") (net 1))
   (segment (start 116 46.167425) (end 114.262991 47.904434) (width 1) (layer "B.Cu") (net 1))
+  (segment (start 133.75485 171.219359) (end 142.8 180.264509) (width 0.3) (layer "B.Cu") (net 1))
   (segment (start 81.184139 53.143609) (end 75.224999 56.34806) (width 1) (layer "B.Cu") (net 1))
   (segment (start 87.441452 50.586003) (end 81.18 53.15) (width 1) (layer "B.Cu") (net 1))
@@
   (segment (start 72.65 115.84) (end 72.8 115.85) (width 0.3) (layer "B.Cu") (net 1))
   (segment (start 100.698504 176.807783) (end 107.461496 177.012217) (width 1) (layer "B.Cu") (net 1))
+  (segment (start 72.125 180.339509) (end 81.24515 171.219359) (width 0.3) (layer "B.Cu") (net 1))
   (segment (start 72.82 115.85) (end 72.65 115.84) (width 0.3) (layer "B.Cu") (net 1))
   (segment (start 145.529706 59.9066) (end 139.775 56.348059) (width 1) (layer "B.Cu") (net 1))
@@
   (segment (start 106 36.322) (end 106 49.83) (width 0.3) (layer "F.Cu") (net 5))
   (via (at 108.8 52.68) (size 0.8) (drill 0.4) (layers "F.Cu" "B.Cu") (net 5))
+  (segment (start 119.19 61.979339) (end 119.19 96.007106) (width 0.3) (layer "B.Cu") (net 5))
+  (segment (start 111.6625 103.534606) (end 111.6625 109.5) (width 0.3) (layer "B.Cu") (net 5))
   (segment (start 109.890661 52.68) (end 119.19 61.979339) (width 0.3) (layer "B.Cu") (net 5))
-  (segment (start 119.19 104.08) (end 113.77 109.5) (width 0.3) (layer "B.Cu") (net 5))
+  (segment (start 119.19 96.007106) (end 111.6625 103.534606) (width 0.3) (layer "B.Cu") (net 5))
   (segment (start 108.8 52.68) (end 109.890661 52.68) (width 0.3) (layer "B.Cu") (net 5))
-  (segment (start 113.77 109.5) (end 111.6625 109.5) (width 0.3) (layer "B.Cu") (net 5))
-  (segment (start 119.19 61.979339) (end 119.19 104.08) (width 0.3) (layer "B.Cu") (net 5))
   (segment (start 73.925 108.65) (end 73.925 109.825) (width 0.3) (layer "B.Cu") (net 6))
   (segment (start 73.5 110.25) (end 73.925 109.825) (width 0.3) (layer "B.Cu") (net 6))
@@
   (segment (start 103.3375 112) (end 81.25 112) (width 0.3) (layer "B.Cu") (net 14))
   (segment (start 81.25 112) (end 80.425 112.825) (width 0.3) (layer "B.Cu") (net 14))
+  (via (at 110.744 102.87) (size 0.8) (drill 0.4) (layers "F.Cu" "B.Cu") (free) (net 15))
+  (via (at 111.76 100.838) (size 0.8) (drill 0.4) (layers "F.Cu" "B.Cu") (free) (net 15))
   (segment (start 108.25 122.15) (end 109.55 123.45) (width 0.3) (layer "B.Cu") (net 16))
   (segment (start 109.55 123.45) (end 110.5 124.4) (width 0.3) (layer "B.Cu") (net 16))
@@
   (segment (start 106.75 107.248959) (end 106.75 108.0875) (width 0.3) (layer "B.Cu") (net 33))
   (segment (start 104.7 78) (end 104.7 80.321) (width 0.3) (layer "B.Cu") (net 33))
+  (segment (start 142.8 186.75) (end 119.099987 163.049987) (width 0.3) (layer "F.Cu") (net 34))
+  (segment (start 119.099987 116.813987) (end 107.188 105.156) (width 0.3) (layer "F.Cu") (net 34))
+  (segment (start 119.099987 163.049987) (end 119.099987 116.813987) (width 0.3) (layer "F.Cu") (net 34))
+  (via (at 107.188 105.156) (size 0.8) (drill 0.4) (layers "F.Cu" "B.Cu") (net 34))
+  (segment (start 107.25 108.0875) (end 107.25 105.218) (width 0.3) (layer "B.Cu") (net 34))
+  (segment (start 145.2 186.75) (end 142.8 186.75) (width 0.3) (layer "B.Cu") (net 34))
+  (segment (start 145.75 186.2) (end 145.2 186.75) (width 0.3) (layer "B.Cu") (net 34))
+  (segment (start 110.41 82.49) (end 110.42 82.49) (width 0.3) (layer "B.Cu") (net 41))
+  (segment (start 107.55 85.5) (end 107.55 85.35) (width 0.3) (layer "B.Cu") (net 41))
+  (segment (start 101.8 91.25) (end 99.88 91.25) (width 1) (layer "B.Cu") (net 41))
+  (segment (start 107.55 85.5) (end 101.8 91.25) (width 1) (layer "B.Cu") (net 41))
+  (segment (start 107.55 85.35) (end 110.41 82.49) (width 0.5) (layer "B.Cu") (net 41))
   (segment (start 110.42 80.89) (end 108.42 80.89) (width 1) (layer "B.Cu") (net 42))
   (segment (start 137 112.75) (end 135.75 111.5) (width 0.3) (layer "B.Cu") (net 44))
@@
   (segment (start 135.875 125.625) (end 135.875 115.85) (width 0.3) (layer "B.Cu") (net 81))
   (segment (start 107.5 154) (end 135.875 125.625) (width 0.3) (layer "B.Cu") (net 81))
-  (segment (start 105.536 82.945) (end 107.965 82.945) (width 1) (layer "B.Cu") (net 82))
+  (segment (start 106.486 80.887371) (end 106.486 80.435) (width 1) (layer "B.Cu") (net 82))
+  (segment (start 105 85.5) (end 108.01 82.49) (width 1) (layer "B.Cu") (net 82))
+  (segment (start 108.088629 82.49) (end 106.486 80.887371) (width 1) (layer "B.Cu") (net 82))
   (segment (start 100.85 85.5) (end 100.8 85.55) (width 0.3) (layer "B.Cu") (net 82))
-  (segment (start 105 85.5) (end 105 83.481) (width 1) (layer "B.Cu") (net 82))
-  (segment (start 107.965 82.945) (end 108.42 82.49) (width 1) (layer "B.Cu") (net 82))
-  (segment (start 105 83.481) (end 105.536 82.945) (width 1) (layer "B.Cu") (net 82))
+  (segment (start 108.01 82.49) (end 108.42 82.49) (width 1) (layer "B.Cu") (net 82))
   (segment (start 105 85.5) (end 100.85 85.5) (width 1) (layer "B.Cu") (net 82))
+  (segment (start 108.42 82.49) (end 108.088629 82.49) (width 1) (layer "B.Cu") (net 82))
   (segment (start 110.1 85.5) (end 114.2 85.5) (width 1) (layer "B.Cu") (net 83))
   (zone (net 45) (net_name "+48V") (layer "F.Cu") (hatch edge 0.5)

Commit message: L1-Updated DXF and Routed 12v
Parts:
- moved MTH3 3.07 mm to (75.3, 153.3)
- moved MTH7 3.07 mm to (55.7, 124.3)
- moved MTH 3.03 mm to (139.7, 153.3)
- moved MTH8 3.03 mm to (159.2, 124.3)
- moved MTH13 2.98 mm to (75.3, 71.4)
- moved MTH9 2.98 mm to (55.7, 100.4)
- moved MTH14 2.93 mm to (139.7, 71.4)
- moved MTH10 2.93 mm to (159.2, 100.4)
- moved MTH6 0.09 mm to (189.3, 126.5)
- moved MTHe 0.09 mm to (189.3, 98.2)
- moved MTH15 0.09 mm to (60.9, 43.6)
- moved MTH11 0.09 mm to (25.7, 98.2)
- moved MTH5 0.09 mm to (25.7, 126.5)
- moved MTH 0.09 mm to (149.8, 183.7)
- moved MTH16 0.09 mm to (154.0, 43.6)
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- renumbered MTH4 to MTH, MTH2 to MTH, MTH12 to MTHe
Routing:
- net +12V: track 0.00 -> 116.3 mm, vias 0 -> 1
- net /Sol: track 40.8 -> 44.7 mm
- net /SWDIO: track 81.4 -> 82.1 mm
- net /SWCLK: track 82.4 -> 83.0 mm
Other:
- outline, holes or cut-outs redrawn

Commit message: l1 - MTH Desginators
Parts:
- renumbered MTHe to MTH12, MTH to MTH2, MTH to MTH4
Routing:
- net GND: vias 2 -> 3
Changed lines of the file:
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@@
     (pad_to_mask_clearance 0)
     (aux_axis_origin 107.5 112.25)
+    (grid_origin 107.5 112.25)
     (pcbplotparams
       (layerselection 0x00010fc_ffffffff)
@@
     (property "ki_keywords" "mounting hole")
     (attr exclude_from_pos_files)
-    (fp_text reference "MTH" (at 0 -4.2) (layer "F.SilkS") hide
+    (fp_text reference "MTH4" (at 0 -4.2) (layer "F.SilkS") hide
         (effects (font (size 1 1) (thickness 0.15)))
     )
@@
     (property "ki_keywords" "mounting hole")
     (attr exclude_from_pos_files)
-    (fp_text reference "MTHe" (at 0 -4.2) (layer "F.SilkS") hide
+    (fp_text reference "MTH12" (at 0 -4.2) (layer "F.SilkS") hide
         (effects (font (size 1 1) (thickness 0.15)))
     )
@@
     (property "ki_keywords" "mounting hole")
     (attr exclude_from_pos_files)
-    (fp_text reference "MTH" (at 0 -4.2) (layer "F.SilkS") hide
+    (fp_text reference "MTH2" (at 0 -4.2) (layer "F.SilkS") hide
         (effects (font (size 1 1) (thickness 0.15)))
     )
@@
   (segment (start 81.25 112) (end 80.425 112.825) (width 0.3) (layer "B.Cu") (net 14))
   (via (at 110.744 102.87) (size 0.8) (drill 0.4) (layers "F.Cu" "B.Cu") (free) (net 15))
+  (via (at 124.5 102) (size 0.8) (drill 0.4) (layers "F.Cu" "B.Cu") (free) (net 15))
   (via (at 111.76 100.838) (size 0.8) (drill 0.4) (layers "F.Cu" "B.Cu") (free) (net 15))
   (segment (start 108.25 122.15) (end 109.55 123.45) (width 0.3) (layer "B.Cu") (net 16))

Commit message: L1-Reworked Activation routing, Locked all MTH
Parts:
- moved R39 0.90 mm to (114.1, 85.5), turned to 90 degrees
- moved R38 0.83 mm to (101.2, 85.5), turned to 90 degrees
Routing:
- net +12V: track 116.3 -> 104.0 mm
- net /Sol: track 44.7 -> 39.0 mm
- net /SWCLK: track 83.0 -> 82.2 mm
- net GND: vias 3 -> 0

Commit message: L1-Via Size TBD
Routing:
- net +12V: track 104.0 -> 114.1 mm
- net /Sol: track 39.0 -> 43.6 mm
- net /SWDIO: track 81.6 -> 83.9 mm
- net /SWCLK: track 82.2 -> 83.0 mm
Changed lines of the file:
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@@
       (stroke (width 0.1) (type solid)) (layer "F.Fab"))
     (pad "1" thru_hole circle (at 2.5 0 180) (size 3.8 3.8) (drill 2.5) (layers "*.Cu" "*.Mask")
-      (net 45 "+48V") (pinfunction "Pin_1") (pintype "passive"))
+      (net 45 "+48V") (pinfunction "Pin_1") (pintype "passive") (clearance 0.6))
     (pad "2" thru_hole roundrect (at -2.5 0 180) (size 3.8 3.8) (drill 2.5) (layers "*.Cu" "*.Mask") (roundrect_rratio 0.1)
-      (net 41 "Net-(D32-A)") (pinfunction "Pin_2") (pintype "passive"))
+      (net 41 "Net-(D32-A)") (pinfunction "Pin_2") (pintype "passive") (clearance 0.3))
     (model "${KIPRJMOD}/3dmodels/XT30UPB-F.step"
       (offset (xyz 0 0 0))
@@
       (stroke (width 0.1) (type solid)) (layer "F.Fab"))
     (pad "1" thru_hole rect (at 0 0 180) (size 3.2 3.2) (drill 1.6) (layers "*.Cu" "*.Mask")
-      (net 45 "+48V") (pinfunction "K") (pintype "passive"))
+      (net 45 "+48V") (pinfunction "K") (pintype "passive") (clearance 0.6))
     (pad "2" thru_hole oval (at 15.24 0 180) (size 3.2 3.2) (drill 1.6) (layers "*.Cu" "*.Mask")
-      (net 41 "Net-(D32-A)") (pinfunction "A") (pintype "passive"))
+      (net 41 "Net-(D32-A)") (pinfunction "A") (pintype "passive") (clearance 0.3))
     (model "${KICAD6_3DMODEL_DIR}/Diode_THT.3dshapes/D_DO-201AD_P15.24mm_Horizontal.wrl"
       (offset (xyz 0 0 0))
@@
       (stroke (width 0.1) (type solid)) (fill none) (layer "F.Fab"))
     (pad "1" thru_hole rect (at 0 0 180) (size 2.4 2.4) (drill 1.2) (layers "*.Cu" "*.Mask")
-      (net 45 "+48V") (pintype "passive"))
+      (net 45 "+48V") (pintype "passive") (clearance 0.6))
     (pad "2" thru_hole circle (at 7.5 0 180) (size 2.4 2.4) (drill 1.2) (layers "*.Cu" "*.Mask")
       (net 15 "GND") (pintype "passive"))
@@
   (segment (start 109.88 53.73) (end 109.9 53.71) (width 0.3) (layer "F.Cu") (net 4))
   (via (at 109.88 53.73) (size 0.8) (drill 0.4) (layers "F.Cu" "B.Cu") (net 4))
-  (segment (start 109.25 107.248959) (end 109.25 108.0875) (width 0.3) (layer "B.Cu") (net 4))
-  (segment (start 117.406 99.042) (end 114.578 101.87) (width 0.3) (layer "B.Cu") (net 4))
+  (segment (start 109.542 102.598) (end 108.97 103.17) (width 0.3) (layer "B.Cu") (net 4))
+  (segment (start 118.422 62.272) (end 118.422 100.566) (width 0.3) (layer "B.Cu") (net 4))
   (segment (start 108.97 106.968959) (end 109.25 107.248959) (width 0.3) (layer "B.Cu") (net 4))
-  (segment (start 110.27 101.87) (end 108.97 103.17) (width 0.3) (layer "B.Cu") (net 4))
-  (segment (start 117.406 61.256) (end 117.406 99.042) (width 0.3) (layer "B.Cu") (net 4))
+  (segment (start 109.88 53.73) (end 118.422 62.272) (width 0.3) (layer "B.Cu") (net 4))
+  (segment (start 109.25 107.248959) (end 109.25 108.0875) (width 0.3) (layer "B.Cu") (net 4))
   (segment (start 108.97 103.17) (end 108.97 106.968959) (width 0.3) (layer "B.Cu") (net 4))
-  (segment (start 114.578 101.87) (end 110.27 101.87) (width 0.3) (layer "B.Cu") (net 4))
-  (segment (start 109.88 53.73) (end 117.406 61.256) (width 0.3) (layer "B.Cu") (net 4))
+  (segment (start 118.422 100.566) (end 116.39 102.598) (width 0.3) (layer "B.Cu") (net 4))
+  (segment (start 116.39 102.598) (end 109.542 102.598) (width 0.3) (layer "B.Cu") (net 4))
   (segment (start 108.476 52.306) (end 106 49.83) (width 0.3) (layer "F.Cu") (net 5))
   (segment (start 108.8 52.306) (end 108.476 52.306) (width 0.3) (layer "F.Cu") (net 5))
   (segment (start 106 49.83) (end 106 36.322) (width 0.3) (layer "F.Cu") (net 5))
   (via (at 108.8 52.306) (size 0.8) (drill 0.4) (layers "F.Cu" "B.Cu") (net 5))
-  (segment (start 110.294 52.306) (end 118.422 60.434) (width 0.3) (layer "B.Cu") (net 5))
-  (segment (start 118.422 60.434) (end 118.422 102.7405) (width 0.3) (layer "B.Cu") (net 5))
+  (segment (start 110.294 52.306) (end 119.438 61.45) (width 0.3) (layer "B.Cu") (net 5))
+  (segment (start 119.438 101.7245) (end 111.6625 109.5) (width 0.3) (layer "B.Cu") (net 5))
   (segment (start 108.8 52.306) (end 110.294 52.306) (width 0.3) (layer "B.Cu") (net 5))
-  (segment (start 118.422 102.7405) (end 111.6625 109.5) (width 0.3) (layer "B.Cu") (net 5))
+  (segment (start 119.438 61.45) (end 119.438 101.7245) (width 0.3) (layer "B.Cu") (net 5))
   (segment (start 73.925 108.65) (end 73.925 109.825) (width 0.3) (layer "B.Cu") (net 6))
   (segment (start 73.5 110.25) (end 73.925 109.825) (width 0.3) (layer "B.Cu") (net 6))
@@
   (segment (start 111.6625 113) (end 110.823959 113) (width 0.3) (layer "B.Cu") (net 21))
   (segment (start 110.575 115.325) (end 112.01959 116.76959) (width 0.3) (layer "B.Cu") (net 21))
-  (segment (start 106.75 105.778661) (end 97.93 96.958661) (width 0.3) (layer "B.Cu") (net 33))
-  (segment (start 97.93 84.77) (end 104.7 78) (width 0.3) (layer "B.Cu") (net 33))
-  (segment (start 106.75 108.0875) (end 106.75 105.778661) (width 0.3) (layer "B.Cu") (net 33))
-  (segment (start 97.93 96.958661) (end 97.93 84.77) (width 0.3) (layer "B.Cu") (net 33))
+  (segment (start 106.75 107.248959) (end 106.501041 107) (width 0.3) (layer "B.Cu") (net 33))
+  (segment (start 96.324 100.566) (end 96.324 84.564) (width 0.3) (layer "B.Cu") (net 33))
+  (segment (start 106.75 108.0875) (end 106.75 107.248959) (width 0.3) (layer "B.Cu") (net 33))
+  (segment (start 96.324 84.564) (end 102.888 78) (width 0.3) (layer "B.Cu") (net 33))
+  (segment (start 102.758 107) (end 96.324 100.566) (width 0.3) (layer "B.Cu") (net 33))
+  (segment (start 102.888 78) (end 104.7 78) (width 0.3) (layer "B.Cu") (net 33))
+  (segment (start 106.501041 107) (end 102.758 107) (width 0.3) (layer "B.Cu") (net 33))
   (segment (start 104.7 78) (end 104.7 80.321) (width 0.3) (layer "B.Cu") (net 33))
   (segment (start 104.7 80.321) (end 104.586 80.435) (width 0.3) (layer "B.Cu") (net 33))
@@
   (segment (start 135.75 111.5) (end 111.6625 111.5) (width 0.3) (layer "B.Cu") (net 44))
   (segment (start 182.5 112.25) (end 182.5 114.75) (width 1) (layer "F.Cu") (net 46))
-  (segment (start 114.358 99.296) (end 119.347293 104.285293) (width 1) (layer "F.Cu") (net 46))
-  (segment (start 168.853004 104.490996) (end 176.612009 112.25) (width 1) (layer "F.Cu") (net 46))
+  (segment (start 115.882 100.82) (end 119.347293 104.285293) (width 1) (layer "F.Cu") (net 46))
   (segment (start 119.347293 104.285293) (end 168.647301 104.285293) (width 1) (layer "F.Cu") (net 46))
-  (segment (start 168.647301 104.285293) (end 168.853004 104.490996) (width 1) (layer "F.Cu") (net 46))
   (segment (start 176.612009 112.25) (end 182.5 112.25) (width 1) (layer "F.Cu") (net 46))
-  (via (at 114.358 99.296) (size 0.8) (drill 0.4) (layers "F.Cu" "B.Cu") (net 46))
+  (segment (start 168.647301 104.285293) (end 176.612009 112.25) (width 1) (layer "F.Cu") (net 46))
+  (via (at 115.882 100.82) (size 1.4) (drill 0.7) (layers "F.Cu" "B.Cu") (net 46))
   (segment (start 102.674 87.358) (end 102.208 87.358) (width 1) (layer "B.Cu") (net 46))
+  (segment (start 102.3 87.45) (end 102.208 87.358) (width 1) (layer "B.Cu") (net 46))
   (segment (start 113.046 87.358) (end 114.104 86.3) (width 1) (layer "B.Cu") (net 46))
+  (segment (start 115.882 100.82) (end 103.436 100.82) (width 1) (layer "B.Cu") (net 46))
   (segment (start 102.674 87.358) (end 113.046 87.358) (width 1) (layer "B.Cu") (net 46))
   (segment (start 102.208 87.358) (end 101.15 86.3) (width 1) (layer "B.Cu") (net 46))
-  (segment (start 114.104 86.3) (end 112.82 87.584) (width 1) (layer "B.Cu") (net 46))
-  (segment (start 112.82 97.758) (end 114.358 99.296) (width 1) (layer "B.Cu") (net 46))
-  (segment (start 112.82 87.584) (end 112.82 97.758) (width 1) (layer "B.Cu") (net 46))
+  (segment (start 103.436 100.82) (end 102.3 99.684) (width 1) (layer "B.Cu") (net 46))
+  (segment (start 102.3 99.684) (end 102.3 87.45) (width 1) (layer "B.Cu") (net 46))
   (segment (start 71.55 112.25) (end 77.35 112.25) (width 0.3) (layer "B.Cu") (net 50))
   (segment (start 77.35 112.25) (end 79.775 114.675) (width 0.3) (layer "B.Cu") (net 50))

Commit message: l1 - PGMR 3V3
Parts:
- removed SW2: SW_SPDT, 2024l1:SS12D00G3
- renumbered J5 to J4
Connections:
- J1 pad 2: /TX -> /RX
- J1 pad 3: /RX -> /TX
- J2 pad 1: /PGMR_3V3 -> +3V3
Routing:
- net +3V3: track 621.0 -> 622.6 mm
- removed copper zone on F.Cu, net /PGMR_3V3
