File: 2024l1/2024l1.kicad_pcb (KiCad board)
At the start: 2 copper layers, 176 x 167.3 mm, 115 parts, among them J1 Conn_01x04, J2 Conn_01x04, J3 XT30, J4 Conn_01x04, Q1 STP75NF75, Q2 AO3400A, SW1 SW_Push, U1 CD74HC4067SM, U2 CD74HC4067SM, U3 STM32F103CBTx, Y1 8Mhz

Commit message: l1 - XH Conn Centered
Parts:
- moved J1 1.25 mm to (32.5, 108.5)
- moved J4 1.25 mm to (182.5, 116.0)
Routing:
- net /TX: track 75.6 -> 73.5 mm
- net /RX: track 70.9 -> 72.5 mm
- net +3V3: track 622.6 -> 623.1 mm
Changed lines of the file:
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@@
   )
   (footprint "Connector_JST:JST_XH_B4B-XH-A_1x04_P2.50mm_Vertical" (layer "F.Cu")
-    (at 182.5 114.75 90)
+    (at 182.5 116 90)
     (descr "JST XH series connector, B4B-XH-A (http://www.jst-mfg.com/product/pdf/eng/eXH.pdf), generated with kicad-footprint-generator")
     (tags "connector JST XH vertical")
@@
   )
   (footprint "Connector_JST:JST_XH_B4B-XH-A_1x04_P2.50mm_Vertical" (layer "F.Cu")
-    (at 32.5 109.75 -90)
+    (at 32.5 108.5 -90)
     (descr "JST XH series connector, B4B-XH-A (http://www.jst-mfg.com/product/pdf/eng/eXH.pdf), generated with kicad-footprint-generator")
     (tags "connector JST XH vertical")
@@
     )
   )
+  (gr_line (start 189.260843 98.223764) (end 189.260843 126.452036)
+    (stroke (width 0.2) (type default)) (layer "F.Cu"))
   (gr_arc (start 177.519455 127.579004) (mid 179.115027 126.522919) (end 180.990031 126.904393)
     (stroke (width 0.2) (type solid)) (layer "Edge.Cuts"))
@@
   (segment (start 114.211496 47.762217) (end 107.448504 47.557783) (width 1) (layer "B.Cu") (net 1))
   (segment (start 171.845567 119.012992) (end 172.050001 112.25) (width 1) (layer "B.Cu") (net 1))
+  (segment (start 39.05 108.5) (end 42.8 112.25) (width 1) (layer "B.Cu") (net 1))
   (segment (start 71.55 114.3) (end 70.1 115.75) (width 0.3) (layer "B.Cu") (net 1))
   (segment (start 113.9 124.1) (end 113.75 124.25) (width 0.3) (layer "B.Cu") (net 1))
@@
   (segment (start 69.470294 164.5934) (end 75.225 168.151941) (width 1) (layer "B.Cu") (net 1))
   (segment (start 139.90423 168.474898) (end 145.495769 164.665102) (width 1) (layer "B.Cu") (net 1))
-  (segment (start 40.3 109.75) (end 42.8 112.25) (width 1) (layer "B.Cu") (net 1))
   (segment (start 110.25 105.85) (end 110.25 108.0875) (width 0.3) (layer "B.Cu") (net 1))
   (segment (start 105.9 118.65) (end 104.86 118.65) (width 0.25) (layer "B.Cu") (net 1))
   (segment (start 73.925 114.765) (end 73.925 115.85) (width 0.3) (layer "B.Cu") (net 1))
-  (segment (start 32.5 109.75) (end 40.3 109.75) (width 1) (layer "B.Cu") (net 1))
   (segment (start 74.882425 168.371241) (end 80.977575 171.308758) (width 1) (layer "B.Cu") (net 1))
+  (segment (start 32.5 108.5) (end 39.05 108.5) (width 1) (layer "B.Cu") (net 1))
   (segment (start 63.884394 160.309711) (end 69.235606 164.450289) (width 1) (layer "B.Cu") (net 1))
   (segment (start 51.435102 144.77823) (end 55.244898 150.369769) (width 1) (layer "B.Cu") (net 1))
@@
   (segment (start 145.529706 59.9066) (end 139.775 56.348059) (width 1) (layer "B.Cu") (net 1))
   (segment (start 145.529706 164.5934) (end 150.692382 160.219999) (width 1) (layer "B.Cu") (net 1))
-  (segment (start 97.5 116.25) (end 97.5 113.5) (width 0.3) (layer "F.Cu") (net 2))
-  (segment (start 96.25 112.25) (end 32.5 112.25) (width 0.3) (layer "F.Cu") (net 2))
-  (segment (start 97.5 113.5) (end 96.25 112.25) (width 0.3) (layer "F.Cu") (net 2))
+  (segment (start 75.5 116.25) (end 72.75 113.5) (width 0.3) (layer "F.Cu") (net 2))
+  (segment (start 72.75 113.5) (end 32.5 113.5) (width 0.3) (layer "F.Cu") (net 2))
+  (segment (start 97.5 116.25) (end 75.5 116.25) (width 0.3) (layer "F.Cu") (net 2))
   (via (at 97.5 116.25) (size 0.8) (drill 0.4) (layers "F.Cu" "B.Cu") (net 2))
   (segment (start 97.6625 116.4125) (end 104.75 116.4125) (width 0.3) (layer "B.Cu") (net 2))
   (segment (start 97.5 116.25) (end 97.6625 116.4125) (width 0.3) (layer "B.Cu") (net 2))
-  (segment (start 96.25 115) (end 96 114.75) (width 0.3) (layer "F.Cu") (net 3))
-  (segment (start 96 114.75) (end 32.5 114.75) (width 0.3) (layer "F.Cu") (net 3))
+  (segment (start 92.25 111) (end 96.25 115) (width 0.3) (layer "F.Cu") (net 3))
+  (segment (start 32.5 111) (end 92.25 111) (width 0.3) (layer "F.Cu") (net 3))
   (via (at 96.25 115) (size 0.8) (drill 0.4) (layers "F.Cu" "B.Cu") (net 3))
   (segment (start 103.3375 115) (end 96.25 115) (width 0.3) (layer "B.Cu") (net 3))
@@
   (segment (start 139.15 112.75) (end 137 112.75) (width 0.3) (layer "B.Cu") (net 43))
   (segment (start 135.75 111.5) (end 111.6625 111.5) (width 0.3) (layer "B.Cu") (net 43))
-  (segment (start 182.5 112.25) (end 182.5 114.75) (width 1) (layer "F.Cu") (net 45))
-  (segment (start 115.882 100.82) (end 119.347293 104.285293) (width 1) (layer "F.Cu") (net 45))
+  (segment (start 182.5 113.5) (end 182.5 115.775) (width 1) (layer "F.Cu") (net 45))
+  (segment (start 168.647301 104.285293) (end 177.862008 113.5) (width 1) (layer "F.Cu") (net 45))
   (segment (start 119.347293 104.285293) (end 168.647301 104.285293) (width 1) (layer "F.Cu") (net 45))
-  (segment (start 176.612009 112.25) (end 182.5 112.25) (width 1) (layer "F.Cu") (net 45))
-  (segment (start 168.647301 104.285293) (end 176.612009 112.25) (width 1) (layer "F.Cu") (net 45))
+  (segment (start 115.882 100.82) (end 119.347293 104.285293) (width 1) (layer "F.Cu") (net 45))
+  (segment (start 177.862008 113.5) (end 182.5 113.5) (width 1) (layer "F.Cu") (net 45))
   (via (at 115.882 100.82) (size 1.4) (drill 0.7) (layers "F.Cu" "B.Cu") (net 45))
   (segment (start 102.674 87.358) (end 102.208 87.358) (width 1) (layer "B.Cu") (net 45))
