File: 2024l2/Power.kicad_sch (KiCad schematic)
At the start: 16 parts

Commit message: l1 - xt30 12v gnd
Parts:
- added J?: Conn_01x02, symbol Connector_Generic:Conn_01x02
Connections:
- net GND: now also J?.2 (Pin_2)
- net +12V renamed VCC
- net VCC: now also J?.1 (Pin_1)
