File: 2024l2/2024l2.kicad_pcb (KiCad board)
At the start: 2 copper layers, 174 x 141 mm, 101 parts, among them IC1 LM2587S-ADJ, IC2 VNH5019ATR-E, IC3 VNH5019ATR-E, IC4 VNH5019ATR-E, IC5 VNH5019ATR-E, J1 Conn_01x02, J2 Conn_01x02, J3 Conn_01x03, J4 Conn_01x03, J5 Conn_01x04, J6 Conn_01x06, Q1 AON6354, Q2 AON6354, Q3 AON6354, Q4 AON6354, SW1 SW_SPDT, U1 TPS5430DDA, U2 TPS5430DDA, U3 Teensy 4.0

Commit message: Production files
Parts:
- moved R18 0.05 mm to (142.5, 171.8)
Routing:
- net /CPM2: track 0.00 -> 25.6 mm
- net /CPM1: track 0.00 -> 25.6 mm
Changed lines of the file:
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@@
   )
   (footprint "2024l2:res0603" (layer "F.Cu")
-    (at 142.45 171.75 -90)
+    (at 142.5 171.75 -90)
     (property "Sheetfile" "2024l2.kicad_sch")
     (property "Sheetname" "")
@@
     (fp_arc (start -4.3 2.4) (mid -4.512132 2.312132) (end -4.6 2.1)
       (stroke (width 0.1) (type default)) (layer "B.SilkS"))
-    (fp_arc (start 4.3 -2.393934) (mid 4.512109 -2.306062) (end 4.6 -2.093934)
+    (fp_arc (start 4.3 -2.393934) (mid 4.512144 -2.306068) (end 4.6 -2.093934)
       (stroke (width 0.1) (type default)) (layer "B.SilkS"))
-    (fp_arc (start 4.6 2.093934) (mid 4.512116 2.306049) (end 4.3 2.393934)
+    (fp_arc (start 4.6 2.093934) (mid 4.512117 2.306052) (end 4.3 2.393934)
       (stroke (width 0.1) (type default)) (layer "B.SilkS"))
     (fp_line (start -4.6 -2.4) (end -4.6 2.4)
@@
     (fp_arc (start -4.3 2.4) (mid -4.512132 2.312132) (end -4.6 2.1)
       (stroke (width 0.1) (type default)) (layer "B.SilkS"))
-    (fp_arc (start 4.3 -2.393934) (mid 4.512109 -2.306062) (end 4.6 -2.093934)
+    (fp_arc (start 4.3 -2.393934) (mid 4.512144 -2.306068) (end 4.6 -2.093934)
       (stroke (width 0.1) (type default)) (layer "B.SilkS"))
-    (fp_arc (start 4.6 2.093934) (mid 4.512116 2.306049) (end 4.3 2.393934)
+    (fp_arc (start 4.6 2.093934) (mid 4.512117 2.306052) (end 4.3 2.393934)
       (stroke (width 0.1) (type default)) (layer "B.SilkS"))
     (fp_line (start -4.6 -2.4) (end -4.6 2.4)
@@
     (fp_arc (start -5.56211 5.20026) (mid -5.86263 5.07578) (end -5.98711 4.77526)
       (stroke (width 0.1) (type default)) (layer "B.SilkS"))
-    (fp_arc (start 5.57474 -5.20026) (mid 5.875231 -5.075751) (end 5.99974 -4.77526)
+    (fp_arc (start 5.57474 -5.20026) (mid 5.875191 -5.075735) (end 5.99974 -4.77526)
       (stroke (width 0.1) (type default)) (layer "B.SilkS"))
     (fp_arc (start 6.01237 4.77526) (mid 5.887903 5.075796) (end 5.58737 5.20026)
@@
   (via (at 142.15 158.8) (size 0.8) (drill 0.4) (layers "F.Cu" "B.Cu") (net 63))
   (segment (start 142.15 157.04) (end 142.15 158.8) (width 0.25) (layer "B.Cu") (net 63))
-  (segment (start 114.1 175.05) (end 114.1 174.41) (width 0.25) (layer "F.Cu") (net 64))
-  (segment (start 114.1 174.41) (end 113.39 173.7) (width 0.25) (layer "F.Cu") (net 64))
-  (segment (start 111.65 168.45) (end 114.85 165.25) (width 0.25) (layer "F.Cu") (net 64))
-  (segment (start 112.85 173.7) (end 111.65 172.5) (width 0.25) (layer "F.Cu") (net 64))
+  (segment (start 112.85 173.7) (end 111.75 172.6) (width 0.25) (layer "F.Cu") (net 64))
   (segment (start 113.39 173.7) (end 112.85 173.7) (width 0.25) (layer "F.Cu") (net 64))
+  (segment (start 114.1 174.41) (end 113.39 173.7) (width 0.25) (layer "F.Cu") (net 64))
+  (segment (start 111.75 172.6) (end 111.75 168.35) (width 0.25) (layer "F.Cu") (net 64))
+  (segment (start 114.1 175.05) (end 114.1 174.41) (width 0.25) (layer "F.Cu") (net 64))
+  (segment (start 111.75 168.35) (end 114.85 165.25) (width 0.25) (layer "F.Cu") (net 64))
   (segment (start 133.16 165.25) (end 139.61 158.8) (width 0.25) (layer "F.Cu") (net 64))
   (segment (start 114.85 165.25) (end 133.16 165.25) (width 0.25) (layer "F.Cu") (net 64))
-  (segment (start 111.65 172.5) (end 111.65 168.45) (width 0.25) (layer "F.Cu") (net 64))
   (via (at 139.61 158.8) (size 0.8) (drill 0.4) (layers "F.Cu" "B.Cu") (net 64))
   (segment (start 139.61 157.04) (end 139.61 158.8) (width 0.25) (layer "B.Cu") (net 64))
@@
   (segment (start 142.15 152.62) (end 142.15 155.44) (width 0.25) (layer "B.Cu") (net 66))
   (segment (start 137.07 155.44) (end 137.07 152.62) (width 0.25) (layer "B.Cu") (net 68))
+  (segment (start 95.95 173.05) (end 95.95 180.75) (width 0.25) (layer "F.Cu") (net 69))
+  (segment (start 96.45 172.55) (end 95.95 173.05) (width 0.25) (layer "F.Cu") (net 69))
+  (segment (start 110.1 175.05) (end 110.1 173.15) (width 0.25) (layer "F.Cu") (net 69))
+  (segment (start 95.95 180.75) (end 96.185001 180.985001) (width 0.25) (layer "F.Cu") (net 69))
+  (segment (start 110.1 173.15) (end 109.5 172.55) (width 0.25) (layer "F.Cu") (net 69))
+  (segment (start 109.5 172.55) (end 96.45 172.55) (width 0.25) (layer "F.Cu") (net 69))
+  (segment (start 96.185001 180.985001) (end 97.225 180.985001) (width 0.25) (layer "F.Cu") (net 69))
   (segment (start 116.1 175.05) (end 116.1 174.563604) (width 0.25) (layer "F.Cu") (net 71))
   (segment (start 149.77 155.44) (end 149.77 152.62) (width 0.25) (layer "B.Cu") (net 75))
@@
   (segment (start 152.31 155.44) (end 152.31 152.62) (width 0.25) (layer "B.Cu") (net 87))
   (segment (start 159.93 155.44) (end 159.93 152.62) (width 0.25) (layer "B.Cu") (net 88))
+  (segment (start 136.5 172.95) (end 135.9 172.35) (width 0.25) (layer "F.Cu") (net 112))
+  (segment (start 122.35 180.55) (end 122.585001 180.785001) (width 0.25) (layer "F.Cu") (net 112))
+  (segment (start 135.9 172.35) (end 122.85 172.35) (width 0.25) (layer "F.Cu") (net 112))
+  (segment (start 122.35 172.85) (end 122.35 180.55) (width 0.25) (layer "F.Cu") (net 112))
+  (segment (start 136.5 174.85) (end 136.5 172.95) (width 0.25) (layer "F.Cu") (net 112))
+  (segment (start 122.585001 180.785001) (end 123.625 180.785001) (width 0.25) (layer "F.Cu") (net 112))
+  (segment (start 122.85 172.35) (end 122.35 172.85) (width 0.25) (layer "F.Cu") (net 112))
   (zone (net 18) (net_name "+12V") (layer "F.Cu") (hatch edge 0.5)
     (priority 4)

Commit message: removed boost cap on l2
Parts:
- removed C13, C14: 220u, Capacitor_SMD:CP_Elec_10x10.5
Connections:
- U3 pad 10: /M4 IN B -> /M4 IN A
- U3 pad 12: /M4 IN A -> /M4 IN B
- U3 pad 7: /M3 IN B -> /M3 IN A
- U3 pad 9: /M3 IN A -> /M3 IN B

Commit message: Rehaul Motor Driver
Parts:
- moved C1 23.0 mm to (99.8, 214.7)
- moved C3 23.0 mm to (96.0, 209.8)
- moved C5 23.0 mm to (91.5, 203.2)
- moved C7 23.0 mm to (97.8, 204.1)
- moved D1 23.0 mm to (90.9, 216.1)
- moved L1 23.0 mm to (90.9, 209.9)
- moved R1 23.0 mm to (99.8, 204.1)
- moved R2 23.0 mm to (101.7, 204.1)
- moved U1 23.0 mm to (99.8, 209.9)
- moved C2 22.0 mm to (206.8, 214.8)
- moved C4 22.0 mm to (203.0, 209.9)
- moved C6 22.0 mm to (198.5, 203.3)
- moved C8 22.0 mm to (204.8, 204.2)
- moved D2 22.0 mm to (197.9, 216.2)
- moved L2 22.0 mm to (197.9, 209.9)
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Other:
- outline, holes or cut-outs redrawn

Commit message: Rehaul Motor Driver
Parts:
- moved J2 91.5 mm to (201.7, 234.6)
- moved J1 81.4 mm to (196.5, 234.6)
Routing:
- net +12V: track 0.00 -> 22.9 mm
Changed lines of the file:
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@@
   )
   (footprint "2024l2:14 AWG" (layer "F.Cu")
-    (at 110.52 226.48 -90)
+    (at 201.7 234.6 -90)
     (property "Sheetfile" "2024l2.kicad_sch")
     (property "Sheetname" "")
@@
   )
   (footprint "2024l2:14 AWG" (layer "F.Cu")
-    (at 115.52 226.48 -90)
+    (at 196.5 234.61 -90)
     (property "LCSC" "C98733")
     (property "Sheetfile" "2024l2.kicad_sch")
@@
     (fp_arc (start -4.3 2.4) (mid -4.512132 2.312132) (end -4.6 2.1)
       (stroke (width 0.1) (type default)) (layer "B.SilkS"))
-    (fp_arc (start 4.3 -2.393934) (mid 4.512144 -2.306068) (end 4.6 -2.093934)
+    (fp_arc (start 4.3 -2.393934) (mid 4.512109 -2.306062) (end 4.6 -2.093934)
       (stroke (width 0.1) (type default)) (layer "B.SilkS"))
-    (fp_arc (start 4.6 2.093934) (mid 4.512117 2.306052) (end 4.3 2.393934)
+    (fp_arc (start 4.6 2.093934) (mid 4.512116 2.306049) (end 4.3 2.393934)
       (stroke (width 0.1) (type default)) (layer "B.SilkS"))
     (fp_line (start -4.6 -2.4) (end -4.6 2.4)
@@
     (fp_arc (start -4.3 2.4) (mid -4.512132 2.312132) (end -4.6 2.1)
       (stroke (width 0.1) (type default)) (layer "B.SilkS"))
-    (fp_arc (start 4.3 -2.393934) (mid 4.512144 -2.306068) (end 4.6 -2.093934)
+    (fp_arc (start 4.3 -2.393934) (mid 4.512109 -2.306062) (end 4.6 -2.093934)
       (stroke (width 0.1) (type default)) (layer "B.SilkS"))
-    (fp_arc (start 4.6 2.093934) (mid 4.512117 2.306052) (end 4.3 2.393934)
+    (fp_arc (start 4.6 2.093934) (mid 4.512116 2.306049) (end 4.3 2.393934)
       (stroke (width 0.1) (type default)) (layer "B.SilkS"))
     (fp_line (start -4.6 -2.4) (end -4.6 2.4)
@@
     (fp_arc (start -5.56211 5.20026) (mid -5.86263 5.07578) (end -5.98711 4.77526)
       (stroke (width 0.1) (type default)) (layer "B.SilkS"))
-    (fp_arc (start 5.57474 -5.20026) (mid 5.875162 -5.075705) (end 5.99974 -4.77526)
+    (fp_arc (start 5.57474 -5.20026) (mid 5.875173 -5.075693) (end 5.99974 -4.77526)
       (stroke (width 0.1) (type default)) (layer "B.SilkS"))
     (fp_arc (start 6.01237 4.77526) (mid 5.887903 5.075796) (end 5.58737 5.20026)
@@
   (via (at 134.95 173.4) (size 0.8) (drill 0.4) (layers "F.Cu" "B.Cu") (free) (net 18))
   (via (at 123.65 173.45) (size 0.8) (drill 0.4) (layers "F.Cu" "B.Cu") (free) (net 18))
+  (segment (start 105.5 209.35985) (end 106.21485 208.645) (width 2) (layer "B.Cu") (net 18))
+  (segment (start 98.98985 217.07) (end 101.31485 219.395) (width 2) (layer "B.Cu") (net 18))
+  (segment (start 101.31485 219.395) (end 103.705 219.395) (width 2) (layer "B.Cu") (net 18))
+  (segment (start 98.98985 215.97) (end 98.98985 214.745) (width 1) (layer "B.Cu") (net 18))
+  (segment (start 109.18985 208.645) (end 109.019266 208.645) (width 1.5) (layer "B.Cu") (net 18))
+  (segment (start 105.5 217.6) (end 105.5 209.35985) (width 2) (layer "B.Cu") (net 18))
+  (segment (start 98.98985 217.07) (end 98.98985 215.97) (width 1.5) (layer "B.Cu") (net 18))
+  (segment (start 103.705 219.395) (end 105.5 217.6) (width 2) (layer "B.Cu") (net 18))
+  (segment (start 106.21485 208.645) (end 109.18985 208.645) (width 2) (layer "B.Cu") (net 18))
   (segment (start 155.7 205.6) (end 154.7 206.6) (width 0.25) (layer "B.Cu") (net 25))
   (segment (start 155.7 204.6) (end 155.7 205.6) (width 0.25) (layer "B.Cu") (net 25))

Commit message: L2 Driver Major Edits
Parts:
- added R10: 1K, 2024l2:res0603, F.Cu at (141.0, 167.8)
- added R11: 1K, 2024l2:res0603, F.Cu at (138.3, 167.8)
- added R16: 3K3, 2024l2:res0603, F.Cu at (145.9, 163.8)
- added R17: 3K3, 2024l2:res0603, F.Cu at (148.6, 163.8)
- added R19: 1K, 2024l2:res0603, F.Cu at (145.9, 167.8)
- added R24: 3K3, 2024l2:res0603, F.Cu at (163.8, 163.8)
- added R25: 3K3, 2024l2:res0603, F.Cu at (161.1, 163.8)
- added R26: 3K3, 2024l2:res0603, F.Cu at (156.2, 163.8)
- added R27: 3K3, 2024l2:res0603, F.Cu at (153.5, 163.8)
- added R28: 1K, 2024l2:res0603, F.Cu at (156.2, 167.8)
- added R29: 1K, 2024l2:res0603, F.Cu at (163.8, 167.8)
- added R31: 1K, 2024l2:res0603, F.Cu at (161.1, 167.8)
- added R8: 3K3, 2024l2:res0603, F.Cu at (138.3, 163.8)
- added R9: 3K3, 2024l2:res0603, F.Cu at (141.0, 163.8)
- moved R18 7.29 mm to (148.6, 167.8)
- moved R30 5.04 mm to (153.5, 167.8)
- moved Q2 0.95 mm to (126.3, 179.8)
- moved Q3 0.95 mm to (170.7, 179.8)
- moved C17 0.95 mm to (126.3, 189.3)
- moved C18 0.95 mm to (126.3, 183.9)
- moved C19 0.95 mm to (170.7, 189.3)
- moved C20 0.95 mm to (170.7, 183.9)
- moved IC3 0.95 mm to (139.5, 184.9)
- moved IC4 0.95 mm to (157.5, 184.9)
- moved C15 0.75 mm to (99.9, 189.3)
- moved C16 0.75 mm to (99.9, 183.9)
- moved C21 0.75 mm to (197.1, 189.3)
- moved C22 0.75 mm to (197.1, 183.9)
- moved IC2 0.75 mm to (113.1, 184.9)
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Connections:
- U3 pad 10: /M4 IN A -> /M4 IN B
- U3 pad 12: /M4 IN B -> /M4 IN A
- U3 pad 7: /M3 IN A -> /M3 IN B
- U3 pad 9: /M3 IN B -> /M3 IN A
Routing:
- net +12V: track 22.9 -> 191.6 mm
- net +3V3: track 0.00 -> 165.2 mm, vias 0 -> 1
- net /ESC: track 0.00 -> 131.1 mm
- net +5V: track 5.39 -> 119.7 mm
- net /L1 TX: track 0.00 -> 109.0 mm
- net /L1 RX: track 0.00 -> 104.1 mm
- net +48V: track 0.00 -> 71.8 mm, vias 0 -> 1
- net Net-(IC5-INB): track 0.00 -> 41.3 mm, vias 0 -> 1
- net Net-(IC5-PWM): track 0.00 -> 41.0 mm, vias 0 -> 1
- net Net-(IC5-INA): track 0.00 -> 38.4 mm, vias 0 -> 1
- net Net-(IC2-ENB/DIAGB): track 0.00 -> 33.0 mm, vias 0 -> 2
- net Net-(IC2-ENA/DIAGA): track 0.49 -> 32.3 mm, vias 0 -> 2
- net Net-(IC5-ENA/DIAGA): track 0.00 -> 29.8 mm, vias 0 -> 2
- net Net-(IC5-ENB/DIAGB): track 0.00 -> 29.1 mm, vias 0 -> 2
- net Net-(IC3-INB): track 0.00 -> 25.1 mm, vias 0 -> 1
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- added copper zone on F.Cu, net /M SW
Other:
- outline, holes or cut-outs redrawn

Commit message: Minor trace adjustment
Parts:
- moved J5 0.11 mm to (109.3, 213.6)
- moved J3 0.11 mm to (187.7, 207.4)
Changed lines of the file:
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@@
   )
   (footprint "Connector_JST:JST_XH_B4B-XH-A_1x04_P2.50mm_Vertical" (layer "B.Cu")
-    (at 109.18985 213.645 90)
+    (at 109.3 213.645 90)
     (descr "JST XH series connector, B4B-XH-A (http://www.jst-mfg.com/product/pdf/eng/eXH.pdf), generated with kicad-footprint-generator")
     (tags "connector JST XH vertical")
@@
   )
   (footprint "Connector_JST:JST_XH_B3B-XH-A_1x03_P2.50mm_Vertical" (layer "B.Cu")
-    (at 187.58985 207.395 -90)
+    (at 187.7 207.395 -90)
     (descr "JST XH series connector, B3B-XH-A (http://www.jst-mfg.com/product/pdf/eng/eXH.pdf), generated with kicad-footprint-generator")
     (tags "connector JST XH vertical")
@@
   (segment (start 124.125 151.975) (end 124.125 156.75) (width 1) (layer "F.Cu") (net 4))
   (via (at 124.125 151.975) (size 0.8) (drill 0.4) (layers "F.Cu" "B.Cu") (net 4))
+  (segment (start 99.58485 201.6) (end 102.475 201.6) (width 1) (layer "B.Cu") (net 4))
   (segment (start 124.125 139.3) (end 128.7 134.725) (width 1) (layer "B.Cu") (net 4))
+  (segment (start 92.8 183.3) (end 92.8 201.35515) (width 1) (layer "B.Cu") (net 4))
+  (segment (start 103.95 204.35) (end 105.775 206.175) (width 1) (layer "B.Cu") (net 4))
+  (segment (start 94.68985 203.245) (end 94.251637 202.806787) (width 0.25) (layer "B.Cu") (net 4))
+  (segment (start 124.125 151.975) (end 92.8 183.3) (width 1) (layer "B.Cu") (net 4))
+  (segment (start 103.95 203.075) (end 103.95 204.35) (width 1) (layer "B.Cu") (net 4))
+  (segment (start 144.6 132.025) (end 144.6 130.4) (width 1) (layer "B.Cu") (net 4))
+  (segment (start 105.775 206.175) (end 109.15985 206.175) (width 1) (layer "B.Cu") (net 4))
+  (segment (start 128.7 134.725) (end 141.9 134.725) (width 1) (layer "B.Cu") (net 4))
+  (segment (start 97.83985 203.345) (end 99.58485 201.6) (width 1) (layer "B.Cu") (net 4))
   (segment (start 102.475 201.6) (end 103.95 203.075) (width 1) (layer "B.Cu") (net 4))
-  (segment (start 103.95 203.075) (end 103.95 204.35) (width 1) (layer "B.Cu") (net 4))
-  (segment (start 105.775 206.175) (end 109.15985 206.175) (width 1) (layer "B.Cu") (net 4))
-  (segment (start 103.95 204.35) (end 105.775 206.175) (width 1) (layer "B.Cu") (net 4))
-  (segment (start 92.8 183.3) (end 92.8 201.35515) (width 1) (layer "B.Cu") (net 4))
-  (segment (start 94.68985 203.245) (end 94.251637 202.806787) (width 0.25) (layer "B.Cu") (net 4))
-  (segment (start 99.58485 201.6) (end 102.475 201.6) (width 1) (layer "B.Cu") (net 4))
-  (segment (start 97.83985 203.345) (end 99.58485 201.6) (width 1) (layer "B.Cu") (net 4))
+  (segment (start 124.125 151.975) (end 124.125 139.3) (width 1) (layer "B.Cu") (net 4))
   (segment (start 109.15985 206.175) (end 109.18985 206.145) (width 1) (layer "B.Cu") (net 4))
-  (segment (start 124.125 151.975) (end 92.8 183.3) (width 1) (layer "B.Cu") (net 4))
-  (segment (start 144.6 132.025) (end 144.6 130.4) (width 1) (layer "B.Cu") (net 4))
-  (segment (start 128.7 134.725) (end 141.9 134.725) (width 1) (layer "B.Cu") (net 4))
-  (segment (start 124.125 151.975) (end 124.125 139.3) (width 1) (layer "B.Cu") (net 4))
   (segment (start 141.9 134.725) (end 144.6 132.025) (width 1) (layer "B.Cu") (net 4))
   (segment (start 92.8 201.35515) (end 94.68985 203.245) (width 1) (layer "B.Cu") (net 4))
+  (segment (start 162.47 137.38) (end 162.47 139.67) (width 0.25) (layer "F.Cu") (net 16))
+  (segment (start 202.55 176.25) (end 202.55 181.25) (width 0.25) (layer "F.Cu") (net 16))
+  (segment (start 205.875 205) (end 198.48 212.395) (width 0.25) (layer "F.Cu") (net 16))
+  (segment (start 198.48 212.395) (end 187.7 212.395) (width 0.25) (layer "F.Cu") (net 16))
+  (segment (start 196.80559 170.50559) (end 202.55 176.25) (width 0.25) (layer "F.Cu") (net 16))
+  (segment (start 205.875 184.575) (end 205.875 205) (width 0.25) (layer "F.Cu") (net 16))
+  (segment (start 162.47 139.67) (end 193.30559 170.50559) (width 0.25) (layer "F.Cu") (net 16))
   (segment (start 193.30559 170.50559) (end 196.80559 170.50559) (width 0.25) (layer "F.Cu") (net 16))
   (segment (start 202.55 181.25) (end 205.875 184.575) (width 0.25) (layer "F.Cu") (net 16))
-  (segment (start 205.875 205) (end 198.48 212.395) (width 0.25) (layer "F.Cu") (net 16))
-  (segment (start 162.47 139.67) (end 193.30559 170.50559) (width 0.25) (layer "F.Cu") (net 16))
-  (segment (start 162.47 137.38) (end 162.47 139.67) (width 0.25) (layer "F.Cu") (net 16))
-  (segment (start 198.48 212.395) (end 187.58985 212.395) (width 0.25) (layer "F.Cu") (net 16))
-  (segment (start 196.80559 170.50559) (end 202.55 176.25) (width 0.25) (layer "F.Cu") (net 16))
-  (segment (start 202.55 176.25) (end 202.55 181.25) (width 0.25) (layer "F.Cu") (net 16))
-  (segment (start 205.875 184.575) (end 205.875 205) (width 0.25) (layer "F.Cu") (net 16))
-  (segment (start 159.93 137.38) (end 159.93 139.705) (width 0.25) (layer "F.Cu") (net 17))
+  (segment (start 159.93 139.705) (end 192.55 172.325) (width 0.25) (layer "F.Cu") (net 17))
   (segment (start 203.85 185.4) (end 203.85 201.525) (width 0.25) (layer "F.Cu") (net 17))
   (segment (start 201.825 183.375) (end 203.85 185.4) (width 0.25) (layer "F.Cu") (net 17))
+  (segment (start 203.85 201.525) (end 197.98 207.395) (width 0.25) (layer "F.Cu") (net 17))
+  (segment (start 192.55 172.325) (end 197.825 172.325) (width 0.25) (layer "F.Cu") (net 17))
+  (segment (start 201.825 176.325) (end 201.825 183.375) (width 0.25) (layer "F.Cu") (net 17))
+  (segment (start 159.93 137.38) (end 159.93 139.705) (width 0.25) (layer "F.Cu") (net 17))
   (segment (start 197.98 207.395) (end 187.58985 207.395) (width 0.25) (layer "F.Cu") (net 17))
-  (segment (start 192.55 172.325) (end 197.825 172.325) (width 0.25) (layer "F.Cu") (net 17))
-  (segment (start 159.93 139.705) (end 192.55 172.325) (width 0.25) (layer "F.Cu") (net 17))
-  (segment (start 203.85 201.525) (end 197.98 207.395) (width 0.25) (layer "F.Cu") (net 17))
   (segment (start 197.825 172.325) (end 201.825 176.325) (width 0.25) (layer "F.Cu") (net 17))
-  (segment (start 201.825 176.325) (end 201.825 183.375) (width 0.25) (layer "F.Cu") (net 17))
   (via (at 131.1 200.775) (size 0.8) (drill 0.4) (layers "F.Cu" "B.Cu") (free) (net 18))
   (via (at 104.625 199.3) (size 0.8) (drill 0.4) (layers "F.Cu" "B.Cu") (free) (net 18))
@@
   (segment (start 190.525 237.4) (end 196.5 237.4) (width 2) (layer "B.Cu") (net 18))
   (segment (start 205.925 217.480075) (end 205.925 216.269925) (width 1.5) (layer "B.Cu") (net 18))
-  (segment (start 105.5 209.35985) (end 106.21485 208.645) (width 2) (layer "B.Cu") (net 18))
+  (segment (start 105.5 217.6) (end 103.705 219.395) (width 2) (layer "B.Cu") (net 18))
   (segment (start 98.98985 217.07) (end 101.31485 219.395) (width 2) (layer "B.Cu") (net 18))
   (segment (start 201.7 237.39) (end 203.335 237.39) (width 2) (layer "B.Cu") (net 18))
   (segment (start 126.075 204.55) (end 126.075 200.5) (width 1.5) (layer "B.Cu") (net 18))
+  (segment (start 109.3 208.645) (end 106.21485 208.645) (width 2) (layer "B.Cu") (net 18))
   (segment (start 101.31485 219.395) (end 103.705 219.395) (width 2) (layer "B.Cu") (net 18))
   (segment (start 98.98985 215.97) (end 98.98985 214.745) (width 1) (layer "B.Cu") (net 18))
   (segment (start 201.69 237.4) (end 201.7 237.39) (width 2) (layer "B.Cu") (net 18))
+  (segment (start 106.21485 208.645) (end 105.5 209.35985) (width 2) (layer "B.Cu") (net 18))
+  (segment (start 105.5 209.35985) (end 105.5 217.6) (width 2) (layer "B.Cu") (net 18))
   (segment (start 103.705 219.395) (end 111.906162 227.596162) (width 2) (layer "B.Cu") (net 18))
+  (segment (start 109.3 208.645) (end 121.98 208.645) (width 1.5) (layer "B.Cu") (net 18))
   (segment (start 205.98985 214.785) (end 205.98985 216.03985) (width 1) (layer "B.Cu") (net 18))
   (segment (start 196.5 237.4) (end 201.69 237.4) (width 2) (layer "B.Cu") (net 18))
   (segment (start 121.98 208.645) (end 126.075 204.55) (width 1.5) (layer "B.Cu") (net 18))
   (segment (start 121.98 208.645) (end 121.98 216.3) (width 1.5) (layer "B.Cu") (net 18))
-  (segment (start 109.18985 208.645) (end 121.98 208.645) (width 1.5) (layer "B.Cu") (net 18))
   (segment (start 111.906162 227.596162) (end 180.721162 227.596162) (width 2) (layer "B.Cu") (net 18))
-  (segment (start 105.5 217.6) (end 105.5 209.35985) (width 2) (layer "B.Cu") (net 18))
   (segment (start 121.98 216.3) (end 129.9 216.3) (width 1.5) (layer "B.Cu") (net 18))
   (segment (start 98.98985 217.07) (end 98.98985 215.97) (width 1.5) (layer "B.Cu") (net 18))
   (segment (start 180.721162 227.596162) (end 190.525 237.4) (width 2) (layer "B.Cu") (net 18))
-  (segment (start 103.705 219.395) (end 105.5 217.6) (width 2) (layer "B.Cu") (net 18))
   (segment (start 206.025 234.7) (end 206.025 217.48515) (width 2) (layer "B.Cu") (net 18))
   (segment (start 203.335 237.39) (end 206.025 234.7) (width 2) (layer "B.Cu") (net 18))
-  (segment (start 106.21485 208.645) (end 109.18985 208.645) (width 2) (layer "B.Cu") (net 18))
+  (segment (start 166.525 203.45) (end 122.875 203.45) (width 1) (layer "F.Cu") (net 23))
+  (segment (start 115.18 211.145) (end 109.3 211.145) (width 1) (layer "F.Cu") (net 23))
   (segment (start 172.225 209.15) (end 166.525 203.45) (width 1) (layer "F.Cu") (net 23))
-  (segment (start 115.18 211.145) (end 109.18985 211.145) (width 1) (layer "F.Cu") (net 23))
   (segment (start 122.875 203.45) (end 115.18 211.145) (width 1) (layer "F.Cu") (net 23))
-  (segment (start 166.525 203.45) (end 122.875 203.45) (width 1) (layer "F.Cu") (net 23))
   (via (at 172.225 209.15) (size 0.8) (drill 0.4) (layers "F.Cu" "B.Cu") (net 23))
   (segment (start 171.15 211.95) (end 171.15 210.225) (width 1) (layer "B.Cu") (net 23))

Commit message: Jesus wires
Parts:
- moved C11 3.79 mm to (151.2, 203.4), turned to 180 degrees
Routing:
- net +12V: track 191.6 -> 257.6 mm
- net /CPM2: track 23.7 -> 25.3 mm
- net +3V3: track 165.2 -> 164.5 mm
- net Net-(C11-Pad1): track 2.00 -> 2.60 mm
- net GND: vias 0 -> 149

Commit message: L2 Motor Output
Parts:
- added J10: Conn_01x02, 2024l2:18 AWG, F.Cu at (183.9, 196.5)
- added J7: Conn_01x02, 2024l2:18 AWG, F.Cu at (113.1, 196.5)
- added J8: Conn_01x02, 2024l2:18 AWG, F.Cu at (139.5, 196.5)
- added J9: Conn_01x02, 2024l2:18 AWG, F.Cu at (157.5, 196.5)
- added SW2: SW_SPST, Connector_JST:JST_XH_B2B-XH-A_1x02_P2.50mm_Vertical, F.Cu at (170.3, 164.5)
Routing:
- net +12V: track 257.6 -> 179.6 mm, vias 6 -> 27
- net +3V3: track 164.5 -> 149.8 mm, vias 1 -> 3
- net /M SW: track 0.00 -> 6.55 mm
- net GND: vias 149 -> 77
- added copper zone on F.Cu, net +3V3
