File: lightweight/2024l3/2024l3.kicad_sch (KiCad schematic)
At the start: 14 parts, among them J1 0526101433, J2 Conn_01x03_Pin, SW1 SW_DIP_x02, U28 xiao-esp32c3

Commit message: lw - l3 - fixed serial
Parts:
- removed J2: Conn_01x03_Pin, Connector_PinHeader_2.54mm:PinHeader_1x03_P2.54mm_Vertical, symbol Connector:Conn_01x03_Pin
- added J?: LED, LED_THT:LED_D3.0mm_Horizontal_O1.27mm_Z2.0mm_Clear, symbol Connector_Generic:Conn_01x02
Connections:
- net +5V: now also J?.1 (Pin_1)
- net GND: now also J?.2 (Pin_2)
- no-connect marks 37 -> 36
Changed lines of the file:
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@@
   (no_connect (at 97.79 93.98))
   (no_connect (at 128.27 91.44))
-  (no_connect (at 190.5 91.44))
   (no_connect (at 77.47 46.99))
   (wire (pts (xy 123.19 36.83) (xy 132.08 36.83))
@@
     (stroke (width 0) (type default))
   )
-  (wire (pts (xy 190.5 93.98) (xy 199.39 93.98))
+  (wire (pts (xy 190.5 91.44) (xy 199.39 91.44))
     (stroke (width 0) (type default))
   )
@@
     (effects (font (size 1.27 1.27)) (justify left bottom))
   )
-  (label "ESC" (at 194.31 88.9 0) (fields_autoplaced)
+  (label "+5V" (at 194.31 88.9 0) (fields_autoplaced)
     (effects (font (size 1.27 1.27)) (justify left bottom))
   )
@@
     (effects (font (size 1.27 1.27)) (justify left bottom))
   )
-  (label "GND" (at 194.31 93.98 0) (fields_autoplaced)
+  (label "GND" (at 194.31 91.44 0) (fields_autoplaced)
     (effects (font (size 1.27 1.27)) (justify left bottom))
   )
@@
     (property "Intersheetrefs" "${INTERSHEET_REFS}" (at 182.4983 49.53 0)
       (effects (font (size 1.27 1.27)) hide)
+    )
+  )
+  (symbol (lib_id "Connector_Generic:Conn_01x02") (at 185.42 88.9 0) (mirror y) (unit 1)
+    (in_bom yes) (on_board yes) (dnp no) (fields_autoplaced)
+    (property "Reference" "J?" (at 185.42 82.55 0)
+      (effects (font (size 1.27 1.27)))
+    )
+    (property "Value" "LED" (at 185.42 85.09 0)
+      (effects (font (size 1.27 1.27)))
+    )
+    (property "Footprint" "LED_THT:LED_D3.0mm_Horizontal_O1.27mm_Z2.0mm_Clear" (at 185.42 88.9 0)
+      (effects (font (size 1.27 1.27)) hide)
+    )
+    (property "Datasheet" "~" (at 185.42 88.9 0)
+      (effects (font (size 1.27 1.27)) hide)
+    )
+    (pin "1")
+    (pin "2")
+    (instances
+      (project "2024l3"
+        (path "/91e7b1c2-b009-4d84-9159-ee8884a12474"
+          (reference "J?") (unit 1)
+        )
+      )
     )
   )
@@
         )
       )
-      (project "2023l3-int"
+      (project "2024l3"
         (path "/91e7b1c2-b009-4d84-9159-ee8884a12474"
           (reference "U2") (unit 1)
@@
     (pin "MP2")
     (instances
-      (project "2023l3-int"
+      (project "2024l3"
         (path "/91e7b1c2-b009-4d84-9159-ee8884a12474"
           (reference "J1") (unit 1)
@@
     (pin "1")
     (instances
-      (project "2023l3-int"
+      (project "2024l3"
         (path "/91e7b1c2-b009-4d84-9159-ee8884a12474"
           (reference "#PWR09") (unit 1)
@@
         )
       )
-      (project "2023l3-int"
+      (project "2024l3"
         (path "/91e7b1c2-b009-4d84-9159-ee8884a12474/b6f041e8-1c4e-4d5e-bf26-3f97c4703dae"
           (reference "R3") (unit 1)
@@
         )
       )
-      (project "2023l3-int"
+      (project "2024l3"
         (path "/91e7b1c2-b009-4d84-9159-ee8884a12474"
           (reference "#PWR0118") (unit 1)
@@
     (pin "1")
     (instances
-      (project "2023l3-int"
+      (project "2024l3"
         (path "/91e7b1c2-b009-4d84-9159-ee8884a12474"
           (reference "#PWR0104") (unit 1)
@@
         )
       )
-      (project "2023l3-int"
+      (project "2024l3"
         (path "/91e7b1c2-b009-4d84-9159-ee8884a12474"
           (reference "#PWR03") (unit 1)
@@
         )
       )
-      (project "2023l3-int"
+      (project "2024l3"
         (path "/91e7b1c2-b009-4d84-9159-ee8884a12474"
           (reference "#PWR014") (unit 1)
@@
         )
       )
-      (project "2023l3-int"
+      (project "2024l3"
         (path "/91e7b1c2-b009-4d84-9159-ee8884a12474"
           (reference "U1") (unit 1)
@@
     (pin "1")
     (instances
-      (project "2023l3-int"
+      (project "2024l3"
         (path "/91e7b1c2-b009-4d84-9159-ee8884a12474"
           (reference "#PWR0105") (unit 1)
@@
         )
       )
-      (project "2023l3-int"
+      (project "2024l3"
         (path "/91e7b1c2-b009-4d84-9159-ee8884a12474/b6f041e8-1c4e-4d5e-bf26-3f97c4703dae"
           (reference "R5") (unit 1)
@@
         )
       )
-      (project "2023l3-int"
+      (project "2024l3"
         (path "/91e7b1c2-b009-4d84-9159-ee8884a12474/b6f041e8-1c4e-4d5e-bf26-3f97c4703dae"
           (reference "#PWR0167") (unit 1)
@@
     (pin "1")
     (instances
-      (project "2023l3-int"
+      (project "2024l3"
         (path "/91e7b1c2-b009-4d84-9159-ee8884a12474"
           (reference "#PWR05") (unit 1)
-        )
-      )
-    )
-  )
-  (symbol (lib_id "Connector:Conn_01x03_Pin") (at 185.42 91.44 0) (unit 1)
-    (in_bom yes) (on_board yes) (dnp no) (fields_autoplaced)
-    (property "Reference" "J2" (at 186.055 85.09 0)
-      (effects (font (size 1.27 1.27)))
-    )
-    (property "Value" "Conn_01x03_Pin" (at 186.055 87.63 0)
-      (effects (font (size 1.27 1.27)))
-    )
-    (property "Footprint" "Connector_PinHeader_2.54mm:PinHeader_1x03_P2.54mm_Vertical" (at 185.42 91.44 0)
-      (effects (font (size 1.27 1.27)) hide)
-    )
-    (property "Datasheet" "~" (at 185.42 91.44 0)
-      (effects (font (size 1.27 1.27)) hide)
-    )
-    (pin "1")
-    (pin "2")
-    (pin "3")
-    (instances
-      (project "2023l3-int"
-        (path "/91e7b1c2-b009-4d84-9159-ee8884a12474"
-          (reference "J2") (unit 1)
         )
       )
@@
     (pin "1")
     (instances
-      (project "2023l3-int"
+      (project "2024l3"
         (path "/91e7b1c2-b009-4d84-9159-ee8884a12474"
           (reference "H1") (unit 1)
@@
     (pin "1")
     (instances
-      (project "2023l3-int"
+      (project "2024l3"
         (path "/91e7b1c2-b009-4d84-9159-ee8884a12474"
           (reference "H4") (unit 1)
@@
         )
       )
-      (project "2023l3-int"
+      (project "2024l3"
         (path "/91e7b1c2-b009-4d84-9159-ee8884a12474"
           (reference "#PWR04") (unit 1)
@@
     (pin "1")
     (instances
-      (project "2023l3-int"
+      (project "2024l3"
         (path "/91e7b1c2-b009-4d84-9159-ee8884a12474"
           (reference "#PWR06") (unit 1)
@@
     (pin "4")
     (instances
-      (project "2023l3-int"
+      (project "2024l3"
         (path "/91e7b1c2-b009-4d84-9159-ee8884a12474"
           (reference "SW1") (unit 1)
@@
     (pin "1")
     (instances
-      (project "2023l3-int"
+      (project "2024l3"
         (path "/91e7b1c2-b009-4d84-9159-ee8884a12474"
           (reference "#PWR01") (unit 1)
@@
         )
       )
-      (project "2023l3-int"
+      (project "2024l3"
         (path "/91e7b1c2-b009-4d84-9159-ee8884a12474"
           (reference "#PWR02") (unit 1)
@@
         )
       )
-      (project "2023l3-int"
+      (project "2024l3"
         (path "/91e7b1c2-b009-4d84-9159-ee8884a12474"
           (reference "#PWR08") (unit 1)
@@
     (pin "1")
     (instances
-      (project "2023l3-int"
+      (project "2024l3"
         (path "/91e7b1c2-b009-4d84-9159-ee8884a12474"
           (reference "H2") (unit 1)
@@
         )
       )
-      (project "2023l3-int"
+      (project "2024l3"
         (path "/91e7b1c2-b009-4d84-9159-ee8884a12474/b6f041e8-1c4e-4d5e-bf26-3f97c4703dae"
           (reference "SW2") (unit 1)
@@
         )
       )
-      (project "2023l3-int"
+      (project "2024l3"
         (path "/91e7b1c2-b009-4d84-9159-ee8884a12474"
           (reference "#PWR0117") (unit 1)
@@
         )
       )
-      (project "2023l3-int"
+      (project "2024l3"
         (path "/91e7b1c2-b009-4d84-9159-ee8884a12474"
           (reference "U3") (unit 1)
@@
         )
       )
-      (project "2023l3-int"
+      (project "2024l3"
         (path "/91e7b1c2-b009-4d84-9159-ee8884a12474"
           (reference "#PWR0115") (unit 1)
@@
     (pin "9")
     (instances
-      (project "2023l3-int"
+      (project "2024l3"
         (path "/91e7b1c2-b009-4d84-9159-ee8884a12474"
           (reference "U28") (unit 1)
@@
         )
       )
-      (project "2023l3-int"
+      (project "2024l3"
         (path "/91e7b1c2-b009-4d84-9159-ee8884a12474/b6f041e8-1c4e-4d5e-bf26-3f97c4703dae"
           (reference "#PWR0171") (unit 1)
@@
     (pin "1")
     (instances
-      (project "2023l3-int"
+      (project "2024l3"
         (path "/91e7b1c2-b009-4d84-9159-ee8884a12474"
           (reference "H3") (unit 1)
@@
     )
     (instances
-      (project "2023l3-int"
+      (project "2024l3"
         (path "/91e7b1c2-b009-4d84-9159-ee8884a12474" (page "3"))
       )
