File: open/2024l2/Power.kicad_sch (KiCad schematic)
At the start: 17 parts

Commit message: open - l1,l2 - 3v3 buck to l1
Parts:
- removed C?: 220u, footprints:EIA-7343-D, symbol Device:C_Polarized
- removed C?: 10n, footprints:cap0603, symbol Device:C
- removed C?: 10u, footprints:cap0603, symbol Device:C
- removed D?: SS54, Diode_SMD:D_SMC, symbol Diode:B340
- removed L?: 15uH, footprints:0630 One Piece Inductor, symbol Device:L_Iron
- removed R?: 5K9, footprints:res0603, symbol Device:R
- removed R?: 10K, footprints:res0603, symbol Device:R
- removed U?: TPS5430DDA, footprints:TI_SO-PowerPAD-8_ThermalVias, symbol Regulator_Switching:TPS5430DDA
