File: open/2024l2/2024l2.kicad_pcb (KiCad board)
At the start: 2 copper layers, 176 x 167.3 mm, 77 parts, among them J1 Conn_01x02, J2 Conn_01x04, J3 Conn_01x06, J4 Conn_01x03, J5 Conn_01x02, J6 Conn_01x02, J7 Conn_01x02, J8 Conn_01x02, SW1 SW_DIP_x02, SW2 SW_SPDT, U1 TPS5430DDA, U2 Teensy 4.0, U3 VNH5050A-E, U4 VNH5050A-E, U5 VNH5050A-E, U6 VNH5050A-E

Commit message: open - l2 - changed XH Conn + RM Cutout
Parts:
- J2: value Conn_01x04 -> Conn_01x06; footprint Connector_JST:JST_XH_B4B-XH-A_1x04_P2.50mm_Vertical -> Connector_JST:JST_XH_B6B-XH-A_1x06_P2.50mm_Vertical
- moved J2 2.21 mm to (73.8, 106.5)
- renumbered He to H1, He to H2
Connections:
- J2 pad 1: +5V -> VCC
- J2 pad 2: /L1 TX -> VCC
- J2 pad 3: /L1 RX -> /L1 TX
- J2 pad 4: GND -> /L1 RX
Other:
- outline, holes or cut-outs redrawn

Commit message: open - l3 - 3d models
Parts:
- turned D1 to 90 degrees
- turned J1 to 0 degrees
Changed lines of the file:
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@@
     (fp_arc (start -4.3 2.387868) (mid -4.512132 2.3) (end -4.6 2.087868)
       (stroke (width 0.1) (type default)) (layer "F.SilkS"))
-    (fp_arc (start 4.3 -2.393934) (mid 4.512109 -2.306062) (end 4.6 -2.093934)
-      (stroke (width 0.1) (type default)) (layer "F.SilkS"))
-    (fp_arc (start 4.6 2.093934) (mid 4.512131 2.306067) (end 4.3 2.393934)
+    (fp_arc (start 4.3 -2.393934) (mid 4.512144 -2.306068) (end 4.6 -2.093934)
+      (stroke (width 0.1) (type default)) (layer "F.SilkS"))
+    (fp_arc (start 4.6 2.093934) (mid 4.512131 2.306063) (end 4.3 2.393934)
       (stroke (width 0.1) (type default)) (layer "F.SilkS"))
     (fp_line (start -4.6 -2.4) (end 4.6 -2.4)
@@
   )
   (footprint "2024l2:SMA (DO-214AC)" (layer "F.Cu")
-    (at 179.15 120.65 -90)
+    (at 179.15 120.65 90)
     (descr "SMA (DO-214AC)")
     (tags "Schottky Diode")
@@
     (fp_line (start 2.475 1.25) (end -2.475 1.25)
       (stroke (width 0.1) (type solid)) (layer "F.Fab"))
-    (pad "1" smd roundrect (at -2 0) (size 1.5 2) (layers "F.Cu" "F.Paste" "F.Mask") (roundrect_rratio 0.1)
+    (pad "1" smd roundrect (at -2 0 180) (size 1.5 2) (layers "F.Cu" "F.Paste" "F.Mask") (roundrect_rratio 0.1)
       (net 62 "Net-(D1-K)") (pinfunction "K") (pintype "passive"))
-    (pad "2" smd roundrect (at 2 0) (size 1.5 2) (layers "F.Cu" "F.Paste" "F.Mask") (roundrect_rratio 0.1)
+    (pad "2" smd roundrect (at 2 0 180) (size 1.5 2) (layers "F.Cu" "F.Paste" "F.Mask") (roundrect_rratio 0.1)
       (net 1 "GND") (pinfunction "A") (pintype "passive"))
     (model "${KIPRJMOD}/3dmodels/SS5X.stp"
@@
   )
   (footprint "2024l2:AMASS_XT60-M" (layer "F.Cu")
-    (at 188.75 128.25 180)
+    (at 188.75 128.25)
     (property "Sheetfile" "2024l2.kicad_sch")
     (property "Sheetname" "")
@@
     (fp_line (start 7.75 1.6) (end 4.95 4.05)
       (stroke (width 0.127) (type solid)) (layer "F.Fab"))
-    (pad "1" thru_hole circle (at 3.6 0 180) (size 6 6) (drill 4.55) (layers "*.Cu" "*.Mask")
+    (pad "1" thru_hole circle (at 3.6 0) (size 6 6) (drill 4.55) (layers "*.Cu" "*.Mask")
       (net 1 "GND") (pinfunction "Pin_1") (pintype "passive"))
-    (pad "2" thru_hole rect (at -3.6 0 180) (size 6 6) (drill 4.55) (layers "*.Cu" "*.Mask")
+    (pad "2" thru_hole rect (at -3.6 0) (size 6 6) (drill 4.55) (layers "*.Cu" "*.Mask")
       (net 4 "VCC") (pinfunction "Pin_2") (pintype "passive"))
     (model "${KIPRJMOD}/3dmodels/XT60UPB-M.step"

Commit message: L2- basic Mdriver Routing
Parts:
- moved U4 15.0 mm to (156.9, 68.5)
- moved U5 15.0 mm to (141.9, 68.5)
Connections:
- J6 pad 1: /M2 OUTB -> /M2 OUTA
- J6 pad 2: /M2 OUTA -> /M2 OUTB
- J7 pad 1: /M3 OUTB -> /M3 OUTA
- J7 pad 2: /M3 OUTA -> /M3 OUTB
Routing:
- net VCC: track 0.00 -> 45.0 mm
- added copper zone on B.Cu, net /M1 OUTA
- added copper zone on B.Cu, net /M1 OUTB
- added copper zone on B.Cu, net /M2 OUTA
- added copper zone on B.Cu, net /M2 OUTB
- added copper zone on B.Cu, net /M3 OUTA
- added copper zone on B.Cu, net /M3 OUTB
- added copper zone on B.Cu, net /M4 OUTA
- added copper zone on B.Cu, net /M4 OUTB

Commit message: open - l2 - brd
Parts:
- removed H15, H16: MountingHole_Pad, MountingHole:MountingHole_3.2mm_M3_Pad_Via
Other:
- board size 176 x 167.3 mm -> 176 x 132.7 mm

Commit message: open - l2 - silkscrn
Parts:
- added kibuzzard-64CDC36A: G***, kibuzzard-64CDC36A, B.Cu at (68.0, 100.5)
- added kibuzzard-64CDC3D3: G***, kibuzzard-64CDC3D3, F.Cu at (78.0, 96.5)
- added kibuzzard-64CDC3D7: G***, kibuzzard-64CDC3D7, F.Cu at (78.0, 94.0)
- added kibuzzard-64CDC3DB: G***, kibuzzard-64CDC3DB, F.Cu at (77.3, 99.0)
- added kibuzzard-64CDC3E9: G***, kibuzzard-64CDC3E9, F.Cu at (77.3, 101.7)
- added kibuzzard-64CDC3FE: G***, kibuzzard-64CDC3FE, F.Cu at (78.3, 106.7)
- added kibuzzard-64CDC403: G***, kibuzzard-64CDC403, F.Cu at (78.3, 104.2)
Other:
- outline, holes or cut-outs redrawn

Commit message: open - l2 - silkscrn
Parts:
- moved C4 57.7 mm to (215.5, 99.0)
- moved C1 57.7 mm to (231.8, 105.5)
- moved D1 57.7 mm to (231.8, 97.0)
- moved U1 57.7 mm to (225.9, 105.5)
- moved kibuzzard-64CCD310 57.7 mm to (214.2, 95.5)
- moved C2 57.7 mm to (226.0, 101.5)
- moved C3 57.7 mm to (219.2, 98.7)
- moved L1 57.7 mm to (225.9, 96.2)
- moved R1 57.7 mm to (219.2, 104.8)
- moved R2 57.7 mm to (219.2, 107.2)
- moved J1 16.1 mm to (174.2, 121.5)
- moved C5 6.00 mm to (127.0, 50.3)
- moved C6 6.00 mm to (141.9, 50.3)
- moved C7 6.00 mm to (156.9, 50.3)
- moved C8 6.00 mm to (171.9, 50.3)
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Routing:
- net VCC: track 45.0 -> 0.00 mm
- net /FL INBD: track 31.1 -> 0.00 mm, vias 1 -> 0
- net /M2 OUTB: track 4.39 -> 0.00 mm
- net /M2 OUTA: track 4.39 -> 0.00 mm
- net /M1 OUTB: track 4.39 -> 0.00 mm
- net /M3 OUTB: track 4.39 -> 0.00 mm
- net /M3 OUTA: track 4.39 -> 0.00 mm
- net /M1 OUTA: track 4.39 -> 0.00 mm
- net /M4 OUTB: track 4.39 -> 0.00 mm
- net /M4 OUTA: track 4.39 -> 0.00 mm
- net /BL PWMD: track 3.93 -> 0.00 mm, vias 1 -> 0
- net /FR PWMD: track 3.93 -> 0.00 mm, vias 1 -> 0
- net /FL PWMD: track 3.93 -> 0.00 mm, vias 1 -> 0
- net /FL PWMC: track 3.74 -> 0.00 mm
- net /FR PWMC: track 3.58 -> 0.00 mm
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
Commit message: L2- Stitching Vias
Parts:
- R15, R16, R19, R23: moved to B.Cu
- moved R19 51.7 mm to (130.4, 75.8), turned to 90 degrees
- moved R23 49.7 mm to (125.5, 75.8), turned to 90 degrees
- moved R15 49.2 mm to (128.4, 75.8), turned to 90 degrees
- moved R16 47.5 mm to (123.5, 75.8), turned to 90 degrees
Routing:
- net VCC: track 0.00 -> 45.0 mm
- net Net-(U3-ENB): track 0.00 -> 26.4 mm, vias 0 -> 1
- net /FR INBD: track 0.00 -> 4.85 mm, vias 0 -> 1
- net /BR INBD: track 0.00 -> 4.85 mm, vias 0 -> 1
- net /BL INBD: track 0.00 -> 4.85 mm, vias 0 -> 1
- net /FL INBD: track 0.00 -> 4.85 mm, vias 0 -> 1
- net Net-(U6-ENB): track 0.00 -> 3.88 mm, vias 0 -> 1
- net Net-(U5-ENB): track 0.00 -> 3.88 mm, vias 0 -> 1
- net Net-(U4-ENB): track 0.00 -> 3.88 mm, vias 0 -> 1
- net /FL PWMC: track 0.00 -> 3.74 mm
- net /FR PWMC: track 0.00 -> 3.58 mm
- net /FL INBC: track 0.00 -> 3.51 mm
- net /BL PWMC: track 0.00 -> 3.42 mm
- net /FR INBC: track 0.00 -> 3.36 mm
- net /FL INAC: track 0.00 -> 3.29 mm
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
Commit message: l2-Added VCC line
Routing:
- net VCC: track 45.0 -> 232.3 mm
Changed lines of the file:
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@@
   (via (at 133.75 94.25) (size 0.8) (drill 0.4) (layers "F.Cu" "B.Cu") (free) (net 1))
   (via (at 88.75 94.25) (size 0.8) (drill 0.4) (layers "F.Cu" "B.Cu") (free) (net 1))
+  (segment (start 75.45 106.55) (end 90.35 121.45) (width 2) (layer "F.Cu") (net 4))
+  (segment (start 73.75 104.05) (end 73.75 106.55) (width 2) (layer "F.Cu") (net 4))
+  (segment (start 73.75 104.05) (end 80.35 104.05) (width 2) (layer "F.Cu") (net 4))
+  (segment (start 90.35 121.45) (end 170.55 121.45) (width 2) (layer "F.Cu") (net 4))
   (segment (start 126.95 54.450001) (end 171.95 54.450001) (width 2) (layer "F.Cu") (net 4))
+  (segment (start 84.4 86.15) (end 116.099999 54.450001) (width 2) (layer "F.Cu") (net 4))
+  (segment (start 73.75 106.55) (end 75.45 106.55) (width 2) (layer "F.Cu") (net 4))
+  (segment (start 80.35 104.05) (end 84.4 100) (width 2) (layer "F.Cu") (net 4))
+  (segment (start 116.099999 54.450001) (end 126.95 54.450001) (width 2) (layer "F.Cu") (net 4))
+  (segment (start 84.4 100) (end 84.4 86.15) (width 2) (layer "F.Cu") (net 4))
   (segment (start 134.95 40.9) (end 136.18 39.67) (width 0.25) (layer "B.Cu") (net 8))
   (segment (start 134.95 42.45) (end 134.95 40.9) (width 0.25) (layer "B.Cu") (net 8))
