File: open/2024l2/2024l2.kicad_sch (KiCad schematic)
At the start: 92 parts, among them IC1 LM2587S-ADJ, J1 Conn_01x03, J10 Conn_01x03, J2 Conn_01x02, J3 Conn_01x02, J4 Conn_01x02, J5 Conn_01x02, J6 Conn_01x02, J7 Conn_01x03, J8 Conn_01x06, J9 Conn_01x02, SW1 SW_SPST, U1 DRV8873SPWPRQ1, U2 DRV8873SPWPRQ1, U3 TPS5430DDA, U4 TPS5430DDA, U5 DRV8873SPWPRQ1, U6 DRV8873SPWPRQ1, U7 Teensy 4.0

Commit message: Boost on L2 and additional resistors
Parts:
- added J11: Conn_01x02, 2024l2:14 AWG, symbol Connector_Generic:Conn_01x02
Connections:
- net +48V: now also J11.2 (Pin_2)
- net GND: now also J11.1 (Pin_1)
Changed lines of the file:
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@@
+    )
+  )
+  (symbol (lib_id "power:GND") (at 365.1124 193.9372 0) (unit 1)
+    (in_bom yes) (on_board yes) (dnp no) (fields_autoplaced)
+    (property "Reference" "#PWR081" (at 365.1124 200.2872 0)
+      (effects (font (size 1.27 1.27)) hide)
+    )
+    (property "Value" "GND" (at 365.1124 199.5252 0)
+      (effects (font (size 1.27 1.27)))
+    )
+    (property "Footprint" "" (at 365.1124 193.9372 0)
+      (effects (font (size 1.27 1.27)) hide)
+    )
+    (property "Datasheet" "" (at 365.1124 193.9372 0)
+      (effects (font (size 1.27 1.27)) hide)
+    )
+    (pin "1")
+    (instances
+      (project "2024l2"
+        (path "/36f2ccec-186b-4304-87fe-6495d5655b87"
+          (reference "#PWR081") (unit 1)
+        )
+      )
+      (project "2024l1"
+        (path "/5be543b5-1bdc-438f-a916-f916127c0a2b"
+          (reference "#PWR013") (unit 1)
+        )
+      )
     )
   )
@@
         (path "/df3073b9-8d60-44a4-89ea-71f9aa763c80"
           (reference "#PWR?") (unit 1)
+        )
+      )
+    )
+  )
+  (symbol (lib_id "Connector_Generic:Conn_01x02") (at 370.1924 193.9372 0) (mirror x) (unit 1)
+    (in_bom yes) (on_board yes) (dnp no)
+    (property "Reference" "J11" (at 370.1924 182.5072 0)
+      (effects (font (size 1.27 1.27)))
+    )
+    (property "Value" "Conn_01x02" (at 370.1924 185.0472 0)
+      (effects (font (size 1.27 1.27)))
+    )
+    (property "Footprint" "2024l2:14 AWG" (at 370.1924 193.9372 0)
+      (effects (font (size 1.27 1.27)) hide)
+    )
+    (property "Datasheet" "~" (at 370.1924 193.9372 0)
+      (effects (font (size 1.27 1.27)) hide)
+    )
+    (pin "1")
+    (pin "2")
+    (instances
+      (project "2024l2"
+        (path "/36f2ccec-186b-4304-87fe-6495d5655b87"
+          (reference "J11") (unit 1)
         )
       )
@@
         )
       )
+    )
+  )
+  (symbol (lib_id "power:+48V") (at 365.1124 191.3972 0) (unit 1)
+    (in_bom yes) (on_board yes) (dnp no)
+    (property "Reference" "#PWR080" (at 365.1124 195.2072 0)
+      (effects (font (size 1.27 1.27)) hide)
+    )
+    (property "Value" "+48V" (at 365.1124 188.0952 0)
+      (effects (font (size 1.27 1.27)))
+    )
+    (property "Footprint" "" (at 365.1124 191.3972 0)
+      (effects (font (size 1.27 1.27)) hide)
+    )
+    (property "Datasheet" "" (at 365.1124 191.3972 0)
+      (effects (font (size 1.27 1.27)) hide)
+    )
+    (pin "1")
+    (instances
+      (project "2024l2"
+        (path "/36f2ccec-186b-4304-87fe-6495d5655b87"
+          (reference "#PWR080") (unit 1)
+        )
+      )
+      (project "2024l1"
+        (path "/5be543b5-1bdc-438f-a916-f916127c0a2b"
+          (reference "#PWR06") (unit 1)
+        )
+      )

Commit message: L3 DXF change
Parts:
- J11: footprint 2024l2:14 AWG -> 2024l2:AMASS_XT30-F
Changed lines of the file:
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@@
       (effects (font (size 1.27 1.27)))
     )
-    (property "Footprint" "2024l2:14 AWG" (at 370.1924 193.9372 0)
+    (property "Footprint" "2024l2:AMASS_XT30-F" (at 370.1924 193.9372 0)
       (effects (font (size 1.27 1.27)) hide)
     )

Commit message: L2 Rework
Parts:
- removed J1: Conn_01x03, Connector_JST:JST_XH_B3B-XH-A_1x03_P2.50mm_Vertical, symbol Connector_Generic:Conn_01x03
- added J1: Conn_01x02, 2024l2:AMASS_XT30-F, symbol Connector_Generic:Conn_01x02
Connections:
- net +3V3: now also J1.2 (Pin_2)
- net GND: now also J1.1 (Pin_1)
Changed lines of the file:
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@@
     (stroke (width 0) (type default))
   )
-  (wire (pts (xy 59.69 121.92) (xy 54.61 121.92))
-    (stroke (width 0) (type default))
-  )
   (wire (pts (xy 160.02 44.45) (xy 151.13 44.45))
     (stroke (width 0) (type default))
@@
     )
   )
-  (symbol (lib_id "power:+12V") (at 59.69 121.92 270) (mirror x) (unit 1)
-    (in_bom yes) (on_board yes) (dnp no)
-    (property "Reference" "#PWR062" (at 55.88 121.92 0)
-      (effects (font (size 1.27 1.27)) hide)
-    )
-    (property "Value" "+12V" (at 60.9864 123.7643 90)
-      (effects (font (size 1.27 1.27)) (justify left))
-    )
-    (property "Footprint" "" (at 59.69 121.92 0)
-      (effects (font (size 1.27 1.27)) hide)
-    )
-    (property "Datasheet" "" (at 59.69 121.92 0)
-      (effects (font (size 1.27 1.27)) hide)
-    )
-    (pin "1")
-    (instances
-      (project "2024l2"
-        (path "/36f2ccec-186b-4304-87fe-6495d5655b87"
-          (reference "#PWR062") (unit 1)
-        )
-      )
-      (project "2024l1"
-        (path "/5be543b5-1bdc-438f-a916-f916127c0a2b"
-          (reference "#PWR?") (unit 1)
-        )
-      )
-    )
-  )
   (symbol (lib_id "Device:C") (at 370.84 100.33 0) (mirror y) (unit 1)
     (in_bom yes) (on_board yes) (dnp no)
@@
     )
   )
-  (symbol (lib_id "Connector_Generic:Conn_01x03") (at 49.53 119.38 180) (unit 1)
-    (in_bom yes) (on_board yes) (dnp no) (fields_autoplaced)
-    (property "Reference" "J1" (at 49.53 111.5403 0)
-      (effects (font (size 1.27 1.27)))
-    )
-    (property "Value" "Conn_01x03" (at 49.53 114.0803 0)
-      (effects (font (size 1.27 1.27)))
-    )
-    (property "Footprint" "Connector_JST:JST_XH_B3B-XH-A_1x03_P2.50mm_Vertical" (at 49.53 119.38 0)
-      (effects (font (size 1.27 1.27)) hide)
-    )
-    (property "Datasheet" "~" (at 49.53 119.38 0)
-      (effects (font (size 1.27 1.27)) hide)
-    )
-    (pin "1")
-    (pin "2")
-    (pin "3")
-    (instances
-      (project "2024l2"
-        (path "/36f2ccec-186b-4304-87fe-6495d5655b87"
-          (reference "J1") (unit 1)
-        )
-      )
-      (project "2024l1"
-        (path "/5be543b5-1bdc-438f-a916-f916127c0a2b"
-          (reference "J?") (unit 1)
-        )
-      )
-    )
-  )
   (symbol (lib_id "Device:R") (at 154.4634 113.03 270) (unit 1)
     (in_bom yes) (on_board yes) (dnp no)
@@
     )
   )
+  (symbol (lib_id "Connector_Generic:Conn_01x02") (at 49.53 119.38 180) (unit 1)
+    (in_bom yes) (on_board yes) (dnp no) (fields_autoplaced)
+    (property "Reference" "J1" (at 49.53 111.1795 0)
+      (effects (font (size 1.27 1.27)))
+    )
+    (property "Value" "Conn_01x02" (at 49.53 113.7195 0)
+      (effects (font (size 1.27 1.27)))
+    )
+    (property "Footprint" "2024l2:AMASS_XT30-F" (at 49.53 119.38 0)
+      (effects (font (size 1.27 1.27)) hide)
+    )
+    (property "Datasheet" "~" (at 49.53 119.38 0)
+      (effects (font (size 1.27 1.27)) hide)
+    )
+    (pin "1")
+    (pin "2")
+    (instances
+      (project "2024l2"
+        (path "/36f2ccec-186b-4304-87fe-6495d5655b87"
+          (reference "J1") (unit 1)
+        )
+      )
+    )
+  )
   (symbol (lib_id "power:GND") (at 210.82 138.43 0) (unit 1)
     (in_bom yes) (on_board yes) (dnp no) (fields_autoplaced)
@@
     )
   )
-  (symbol (lib_id "power:GND") (at 59.69 119.38 90) (unit 1)
-    (in_bom yes) (on_board yes) (dnp no)
-    (property "Reference" "#PWR?" (at 66.04 119.38 0)
-      (effects (font (size 1.27 1.27)) hide)
-    )
-    (property "Value" "GND" (at 64.135 121.285 0)
-      (effects (font (size 1.27 1.27)) (justify left))
-    )
-    (property "Footprint" "" (at 59.69 119.38 0)
-      (effects (font (size 1.27 1.27)) hide)
-    )
-    (property "Datasheet" "" (at 59.69 119.38 0)
-      (effects (font (size 1.27 1.27)) hide)
-    )
-    (pin "1")
-    (instances
-      (project "2024l2"
-        (path "/24bb1a41-3dfa-48eb-8eef-57082ba6082b"
-          (reference "#PWR?") (unit 1)
-        )
-      )
-      (project "2024l2"
-        (path "/36f2ccec-186b-4304-87fe-6495d5655b87"
-          (reference "#PWR060") (unit 1)
-        )
-      )
-      (project "2024l1"
-        (path "/5be543b5-1bdc-438f-a916-f916127c0a2b"
-          (reference "#PWR?") (unit 1)
-        )
-      )
-      (project "2023l3-int"
-        (path "/91e7b1c2-b009-4d84-9159-ee8884a12474"
-          (reference "#PWR?") (unit 1)
-        )
-      )
-      (project "2023l1-int"
-        (path "/dd82140d-c14c-4d8d-8674-edeceaca486e"
-          (reference "#PWR?") (unit 1)
-        )
-      )
-    )
-  )
   (symbol (lib_id "Mechanical:MountingHole_Pad") (at 165.1 204.47 0) (unit 1)
     (in_bom no) (on_board yes) (dnp no) (fields_autoplaced)
@@
         )
       )
+    )
+  )
+  (symbol (lib_id "power:GND") (at 59.69 119.38 0) (unit 1)
+    (in_bom yes) (on_board yes) (dnp no) (fields_autoplaced)
+    (property "Reference" "#PWR060" (at 59.69 125.73 0)
+      (effects (font (size 1.27 1.27)) hide)
+    )
+    (property "Value" "GND" (at 59.69 124.8655 0)
+      (effects (font (size 1.27 1.27)))
+    )
+    (property "Footprint" "" (at 59.69 119.38 0)
+      (effects (font (size 1.27 1.27)) hide)
+    )
+    (property "Datasheet" "" (at 59.69 119.38 0)
+      (effects (font (size 1.27 1.27)) hide)
+    )
+    (pin "1")
+    (instances
+      (project "2024l2"
+        (path "/36f2ccec-186b-4304-87fe-6495d5655b87"
+          (reference "#PWR060") (unit 1)
+        )
+      )

Commit message: Boost I think XT hitting
Parts:
- IC1: footprint 2024l1:TO170P1435X465-6N -> 2024l2:TO170P1435X465-6N
- J1: footprint 2024l2:AMASS_XT30-F -> Connector_JST:JST_XH_B2B-XH-A_1x02_P2.50mm_Vertical
- L3: footprint 2024l1:1040 One Piece Inductor -> 2024l2:1040 One Piece Inductor
- RV1: footprint 2024l1:TRIM_3362W-1-203LF -> 2024l2:TRIM_3362W-1-203LF
Changed lines of the file:
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@@
       (effects (font (size 1.27 1.27)))
     )
-    (property "Footprint" "2024l1:TO170P1435X465-6N" (at 308.7005 284.6175 0)
+    (property "Footprint" "2024l2:TO170P1435X465-6N" (at 308.7005 284.6175 0)
       (effects (font (size 1.27 1.27)) (justify left top) hide)
     )
@@
       (effects (font (size 1.27 1.27)))
     )
-    (property "Footprint" "2024l2:AMASS_XT30-F" (at 49.53 119.38 0)
+    (property "Footprint" "Connector_JST:JST_XH_B2B-XH-A_1x02_P2.50mm_Vertical" (at 49.53 119.38 0)
       (effects (font (size 1.27 1.27)) hide)
     )
@@
       (effects (font (size 1.27 1.27)))
     )
-    (property "Footprint" "2024l1:1040 One Piece Inductor" (at 279.4905 175.7275 0)
+    (property "Footprint" "2024l2:1040 One Piece Inductor" (at 279.4905 175.7275 0)
       (effects (font (size 1.27 1.27)) hide)
     )
@@
       (effects (font (size 1.27 1.27)))
     )
-    (property "Footprint" "2024l1:TRIM_3362W-1-203LF" (at 304.8905 193.5075 0)
-      (effects (font (size 1.27 1.27)) hide)
-    )
+    (property "Footprint" "2024l2:TRIM_3362W-1-203LF" (at 304.8905 193.5075 0)
+      (effects (font (size 1.27 1.27)) hide)
+    )

Commit message: Battery Indicator need parts
Parts:
- added D?: 1n4735a, symbol Device:D
- added D?: RED, symbol Device:LED
- added Q? (x2): Q_NPN_BEC, symbol Device:Q_NPN_BEC
- added R? (x4): 1K, symbol Device:R
- added RV?: 50K, symbol Device:R_Potentiometer
- added SW?: SW_SPDT, symbol Switch:SW_SPDT
Connections:
- net +12V: now also SW?.2 (B)
- net GND: now also Q?.2 (E), Q?.2 (E), RV?.3
- new net: R?.1, R?.1, SW?.3 (C)
- new net: R?.1, R?.1, R?.2
- new net: Q?.1 (B), Q?.3 (C), R?.2
- new net: D?.2 (A), R?.2
- new net: D?.1 (K), RV?.2
- new net: D?.2 (A), Q?.1 (B)
- new net: D?.1 (K), Q?.3 (C)
- new net: R?.2, RV?.1
- no-connect marks 12 -> 13

Commit message: Low Voltage Indicator
Parts:
- C29, C31, C32: footprint 2024l1:cap0603 -> 2024l2:cap0603
- D3: footprint 2024l1:SMA (DO-214AC) -> 2024l2:SMA (DO-214AC)
- D4: renamed from D?; footprint (none) -> 2024l2:led0603
- D5: renamed from D?; footprint (none) -> Diode_THT:D_DO-41_SOD81_P7.62mm_Horizontal
- Q1, Q2: renamed from Q?; value Q_NPN_BEC -> SMBT2222A; footprint (none) -> Package_TO_SOT_SMD:SOT-23
- R21, R22, R23, R24: renamed from R?; footprint (none) -> 2024l2:res0603
- RV2: renamed from RV?; footprint (none) -> 2024l2:TRIM_3362W-1-203LF
- SW2: renamed from SW?; footprint (none) -> 2024l2:SS12D00G3
Changed lines of the file:
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@@
   (symbol (lib_id "Device:R") (at 55.88 236.22 90) (unit 1)
     (in_bom yes) (on_board yes) (dnp no) (fields_autoplaced)
-    (property "Reference" "R?" (at 55.88 229.87 90)
+    (property "Reference" "R21" (at 55.88 229.87 90)
       (effects (font (size 1.27 1.27)))
     )
@@
       (effects (font (size 1.27 1.27)))
     )
-    (property "Footprint" "" (at 55.88 237.998 90)
+    (property "Footprint" "2024l2:res0603" (at 55.88 237.998 90)
       (effects (font (size 1.27 1.27)) hide)
     )
@@
       (project "2024l2"
         (path "/36f2ccec-186b-4304-87fe-6495d5655b87"
-          (reference "R?") (unit 1)
+          (reference "R21") (unit 1)
         )
       )
@@
   (symbol (lib_id "Device:R") (at 69.85 242.57 0) (unit 1)
     (in_bom yes) (on_board yes) (dnp no) (fields_autoplaced)
-    (property "Reference" "R?" (at 72.39 241.2999 0)
+    (property "Reference" "R22" (at 72.39 241.2999 0)
       (effects (font (size 1.27 1.27)) (justify left))
     )
@@
       (effects (font (size 1.27 1.27)) (justify left))
     )
-    (property "Footprint" "" (at 68.072 242.57 90)
+    (property "Footprint" "2024l2:res0603" (at 68.072 242.57 90)
       (effects (font (size 1.27 1.27)) hide)
     )
@@
       (project "2024l2"
         (path "/36f2ccec-186b-4304-87fe-6495d5655b87"
-          (reference "R?") (unit 1)
+          (reference "R22") (unit 1)
         )
       )
@@
       (effects (font (size 1.27 1.27)) (justify left))
     )
-    (property "Footprint" "2024l1:cap0603" (at 332.5257 196.0475 0)
+    (property "Footprint" "2024l2:cap0603" (at 332.5257 196.0475 0)
       (effects (font (size 1.27 1.27)) hide)
     )
@@
   (symbol (lib_id "Device:R") (at 90.17 242.57 0) (unit 1)
     (in_bom yes) (on_board yes) (dnp no) (fields_autoplaced)
-    (property "Reference" "R?" (at 92.71 241.2999 0)
+    (property "Reference" "R23" (at 92.71 241.2999 0)
       (effects (font (size 1.27 1.27)) (justify left))
     )
@@
       (effects (font (size 1.27 1.27)) (justify left))
     )
-    (property "Footprint" "" (at 88.392 242.57 90)
+    (property "Footprint" "2024l2:res0603" (at 88.392 242.57 90)
       (effects (font (size 1.27 1.27)) hide)
     )
@@
       (project "2024l2"
         (path "/36f2ccec-186b-4304-87fe-6495d5655b87"
-          (reference "R?") (unit 1)
+          (reference "R23") (unit 1)
         )
       )
@@
   (symbol (lib_id "Device:D") (at 55.88 260.35 0) (unit 1)
     (in_bom yes) (on_board yes) (dnp no) (fields_autoplaced)
-    (property "Reference" "D?" (at 55.88 254 0)
+    (property "Reference" "D5" (at 55.88 254 0)
       (effects (font (size 1.27 1.27)))
     )
@@
       (effects (font (size 1.27 1.27)))
     )
-    (property "Footprint" "" (at 55.88 260.35 0)
+    (property "Footprint" "Diode_THT:D_DO-41_SOD81_P7.62mm_Horizontal" (at 55.88 260.35 0)
       (effects (font (size 1.27 1.27)) hide)
     )
@@
       (project "2024l2"
         (path "/36f2ccec-186b-4304-87fe-6495d5655b87"
-          (reference "D?") (unit 1)
+          (reference "D5") (unit 1)
         )
       )
@@
   (symbol (lib_id "Device:Q_NPN_BEC") (at 87.63 264.16 0) (unit 1)
     (in_bom yes) (on_board yes) (dnp no) (fields_autoplaced)
-    (property "Reference" "Q?" (at 92.71 262.8899 0)
+    (property "Reference" "Q2" (at 92.71 262.8899 0)
       (effects (font (size 1.27 1.27)) (justify left))
     )
-    (property "Value" "Q_NPN_BEC" (at 92.71 265.4299 0)
+    (property "Value" "SMBT2222A" (at 92.71 265.4299 0)
       (effects (font (size 1.27 1.27)) (justify left))
     )
-    (property "Footprint" "" (at 92.71 261.62 0)
+    (property "Footprint" "Package_TO_SOT_SMD:SOT-23" (at 92.71 261.62 0)
       (effects (font (size 1.27 1.27)) hide)
     )
@@
       (project "2024l2"
         (path "/36f2ccec-186b-4304-87fe-6495d5655b87"
-          (reference "Q?") (unit 1)
+          (reference "Q2") (unit 1)
         )
       )
@@
   (symbol (lib_id "Device:LED") (at 90.17 252.73 90) (unit 1)
     (in_bom yes) (on_board yes) (dnp no) (fields_autoplaced)
-    (property "Reference" "D?" (at 93.98 253.0474 90)
+    (property "Reference" "D4" (at 93.98 253.0474 90)
       (effects (font (size 1.27 1.27)) (justify right))
     )
@@
       (effects (font (size 1.27 1.27)) (justify right))
     )
-    (property "Footprint" "" (at 90.17 252.73 0)
+    (property "Footprint" "2024l2:led0603" (at 90.17 252.73 0)
       (effects (font (size 1.27 1.27)) hide)
     )
@@
       (project "2024l2"
         (path "/36f2ccec-186b-4304-87fe-6495d5655b87"
-          (reference "D?") (unit 1)
+          (reference "D4") (unit 1)
         )
       )
@@
   (symbol (lib_id "Switch:SW_SPDT") (at 38.1 233.68 0) (unit 1)
     (in_bom yes) (on_board yes) (dnp no) (fields_autoplaced)
-    (property "Reference" "SW?" (at 38.1 226.06 0)
+    (property "Reference" "SW2" (at 38.1 226.06 0)
       (effects (font (size 1.27 1.27)))
     )
@@
       (effects (font (size 1.27 1.27)))
     )
-    (property "Footprint" "" (at 38.1 233.68 0)
+    (property "Footprint" "2024l2:SS12D00G3" (at 38.1 233.68 0)
       (effects (font (size 1.27 1.27)) hide)
     )
@@
       (project "2024l2"
         (path "/36f2ccec-186b-4304-87fe-6495d5655b87"
-          (reference "SW?") (unit 1)
+          (reference "SW2") (unit 1)
         )
       )
@@
   (symbol (lib_id "Device:Q_NPN_BEC") (at 67.31 260.35 0) (unit 1)
     (in_bom yes) (on_board yes) (dnp no) (fields_autoplaced)
-    (property "Reference" "Q?" (at 72.39 259.0799 0)
+    (property "Reference" "Q1" (at 72.39 259.0799 0)
       (effects (font (size 1.27 1.27)) (justify left))
     )
-    (property "Value" "Q_NPN_BEC" (at 72.39 261.6199 0)
+    (property "Value" "SMBT2222A" (at 72.39 261.6199 0)
       (effects (font (size 1.27 1.27)) (justify left))
     )
-    (property "Footprint" "" (at 72.39 257.81 0)
+    (property "Footprint" "Package_TO_SOT_SMD:SOT-23" (at 72.39 257.81 0)
       (effects (font (size 1.27 1.27)) hide)
     )
@@
       (project "2024l2"
         (path "/36f2ccec-186b-4304-87fe-6495d5655b87"
-          (reference "Q?") (unit 1)
+          (reference "Q1") (unit 1)
         )
       )
@@
       (effects (font (size 1.27 1.27)))
     )
-    (property "Footprint" "2024l1:SMA (DO-214AC)" (at 303.6205 175.7275 0)
+    (property "Footprint" "2024l2:SMA (DO-214AC)" (at 303.6205 175.7275 0)
       (effects (font (size 1.27 1.27)) hide)
     )
@@
   (symbol (lib_id "Device:R") (at 45.72 246.38 0) (unit 1)
     (in_bom yes) (on_board yes) (dnp no) (fields_autoplaced)
-    (property "Reference" "R?" (at 48.26 245.1099 0)
+    (property "Reference" "R24" (at 48.26 245.1099 0)
       (effects (font (size 1.27 1.27)) (justify left))
     )
@@
       (effects (font (size 1.27 1.27)) (justify left))
     )
-    (property "Footprint" "" (at 43.942 246.38 90)
+    (property "Footprint" "2024l2:res0603" (at 43.942 246.38 90)
       (effects (font (size 1.27 1.27)) hide)
     )
@@
       (project "2024l2"
         (path "/36f2ccec-186b-4304-87fe-6495d5655b87"
-          (reference "R?") (unit 1)
+          (reference "R24") (unit 1)
         )
       )
@@
       (effects (font (size 1.27 1.27)) (justify left))
     )
-    (property "Footprint" "2024l1:cap0603" (at 257.5957 208.7475 0)
+    (property "Footprint" "2024l2:cap0603" (at 257.5957 208.7475 0)
       (effects (font (size 1.27 1.27)) hide)
     )
@@
       (effects (font (size 1.27 1.27)) (justify left))
     )
-    (property "Footprint" "2024l1:cap0603" (at 233.4657 196.0475 0)
+    (property "Footprint" "2024l2:cap0603" (at 233.4657 196.0475 0)
       (effects (font (size 1.27 1.27)) hide)
     )
@@
   (symbol (lib_id "Device:R_Potentiometer") (at 45.72 260.35 0) (unit 1)
     (in_bom yes) (on_board yes) (dnp no) (fields_autoplaced)
-    (property "Reference" "RV?" (at 43.18 259.0799 0)
+    (property "Reference" "RV2" (at 43.18 259.0799 0)
       (effects (font (size 1.27 1.27)) (justify right))
     )
@@
       (effects (font (size 1.27 1.27)) (justify right))
     )
-    (property "Footprint" "" (at 45.72 260.35 0)
+    (property "Footprint" "2024l2:TRIM_3362W-1-203LF" (at 45.72 260.35 0)
       (effects (font (size 1.27 1.27)) hide)
     )
@@
       (project "2024l2"
         (path "/36f2ccec-186b-4304-87fe-6495d5655b87"
-          (reference "RV?") (unit 1)
+          (reference "RV2") (unit 1)
         )
       )

Commit message: Power Routing Done
Parts:
- removed D4: RED, 2024l2:led0603, symbol Device:LED
- removed D5: 1n4735a, Diode_THT:D_DO-41_SOD81_P7.62mm_Horizontal, symbol Device:D
- removed J1: Conn_01x02, Connector_JST:JST_XH_B2B-XH-A_1x02_P2.50mm_Vertical, symbol Connector_Generic:Conn_01x02
- removed J11: Conn_01x02, 2024l2:AMASS_XT30-F, symbol Connector_Generic:Conn_01x02
- removed Q1, Q2: SMBT2222A, Package_TO_SOT_SMD:SOT-23, symbol Device:Q_NPN_BEC
- removed R21, R22, R23, R24: 1K, 2024l2:res0603, symbol Device:R
- removed RV2: 50K, 2024l2:TRIM_3362W-1-203LF, symbol Device:R_Potentiometer
- removed SW2: SW_SPDT, 2024l2:SS12D00G3, symbol Switch:SW_SPDT
- added J11: Conn_01x04, Connector_JST:JST_XH_B4B-XH-A_1x04_P2.50mm_Vertical, symbol Connector_Generic:Conn_01x04
Connections:
- net +12V: now also J11.3 (Pin_3)
- net +3V3: now also J11.4 (Pin_4)
- net +48V: now also J11.2 (Pin_2)
- net GND: now also J11.1 (Pin_1)
- no-connect marks 13 -> 12
