File: open/2024l1/2024l1.kicad_pcb (KiCad board)
At the start: 2 copper layers, 176 x 167.3 mm, 135 parts, among them IC1 LM2587S-ADJ, J1 Conn_01x04, J2 Conn_01x04, J3 Conn_01x02, J4 XT30, Q1 STP75NF75, SW1 STM RST, U1 CD74HC4067SM, U2 CD74HC4067SM, U3 STM32F103CBTx, U4 PC817, U5 TPS5430DDA, Y1 8Mhz

Commit message: open - l1 - silkscreen UI
Parts:
- added kibuzzard-64C26A52: G***, kibuzzard-64C26A52, F.Cu at (107.5, 103.0)
- added kibuzzard-64C26B0D: G***, kibuzzard-64C26B0D, F.Cu at (55.1, 117.5)
- added kibuzzard-64C26B8C: G***, kibuzzard-64C26B8C, F.Cu at (138.1, 120.2)
- C10: value 1m -> 1000u
- C11: footprint Capacitor_SMD:CP_Elec_6.3x7.7 -> Capacitor_SMD:CP_Elec_10x10.5
- C12: value 1uF -> 1u
- C18, C19: value 0u1 -> 0.1u
- R39: value 2.94k -> 2k94
- R40: value 1.5k -> 1k5
- moved C19 6.44 mm to (139.4, 108.7), turned to -90 degrees
- moved C12 4.27 mm to (144.3, 105.0)
- moved D19 4.20 mm to (146.3, 107.8)
- moved R39 4.04 mm to (148.3, 105.0)
- moved C18 3.68 mm to (174.7, 120.2)
- moved IC1 3.40 mm to (159.5, 112.2)
- moved L1 3.40 mm to (146.2, 115.7)
- moved C11 1.80 mm to (173.9, 112.2)
- moved C17 0.45 mm to (53.3, 114.0)
Routing:
- net +12V: track 122.3 -> 97.2 mm
- net +48V: track 103.7 -> 114.3 mm
- net Net-(IC1-FDBK): track 41.0 -> 45.4 mm
- net +3V3: track 605.3 -> 607.3 mm
- net Net-(IC1-COMP): track 5.87 -> 7.06 mm

Commit message: L1-Added Test Pads
Routing:
- net +3V3: track 607.3 -> 652.2 mm

Commit message: L1- Moved Trace A bit further
Parts:
- added 12V: Test Pad, 2024l1:Test Pad, F.Cu at (123.2, 44.2)
- added 3V3: Test Pad, 2024l1:Test Pad, F.Cu at (117.2, 38.2)
- added 48V: Test Pad, 2024l1:Test Pad, F.Cu at (117.2, 44.2)
- added 5V: Test Pad, 2024l1:Test Pad, F.Cu at (123.2, 38.2)
- added GND: Test Pad, 2024l1:Test Pad, F.Cu at (97.7, 38.3)
Routing:
- net +5V: track 0.00 -> 132.5 mm, vias 0 -> 1
- net +48V: track 114.3 -> 235.0 mm
- net +12V: track 97.2 -> 130.5 mm
- net +3V3: track 652.2 -> 658.3 mm
- net GND: track 0.00 -> 5.98 mm

Commit message: L1-Changed Test Pad Position
Parts:
- removed the 5V at (123.2, 38.2)
- added 3V3: Test Pad, 2024l1:Test Pad, F.Cu at (91.7, 38.2)
- added GND: Test Pad, 2024l1:Test Pad, F.Cu at (97.7, 38.2)
- moved 48V 13.4 mm to (129.2, 38.2)
- moved 5V 12.0 mm to (85.7, 38.2)
- moved 12V 6.00 mm to (123.2, 38.2)
- renumbered GND to 5V, 3V3 to GND
Connections:
- 5V pad 1: GND -> +5V
- GND pad 1: +3V3 -> GND
Routing:
- net +5V: track 132.5 -> 96.9 mm
- net +3V3: track 658.3 -> 674.2 mm
- net +48V: track 235.0 -> 226.0 mm
- net +12V: track 130.5 -> 136.5 mm
- net GND: track 5.98 -> 0.01 mm, vias 0 -> 1

Commit message: open - l1 - silkscreen
Parts:
- added kibuzzard-64C35411: G***, kibuzzard-64C35411, F.Cu at (107.4, 45.8)

Commit message: L1-Edited Silkscreen
Parts:
- added D37: PESD2USB3UX-T, 2024l1:PESD2USB3UXT-QR, F.Cu at (54.3, 107.5)
Routing:
- net +3V3: track 674.2 -> 677.0 mm

Commit message: open - l1 - silkscreen
Parts:
- C1: footprint 2024l1:cap0603 -> 2024l1:Test Pad
- TP1, TP2: renamed from GND; value Test Pad -> Conn_01x01
- TP3: renamed from 3V3; value Test Pad -> Conn_01x01
- TP4: renamed from 5V; value Test Pad -> Conn_01x01
- TP5: renamed from 48V; value Test Pad -> Conn_01x01
- TP6: renamed from 12V; value Test Pad -> Conn_01x01
Connections:
- TP5 pad 1: +48V -> +12V
- TP6 pad 1: +12V -> +48V
Routing:
- net +48V: track 226.0 -> 158.6 mm
- net +5V: track 96.9 -> 108.7 mm
- net /Sol: track 52.7 -> 59.5 mm
- net +12V: track 136.5 -> 142.7 mm
- net Net-(U1-I0): track 70.9 -> 77.1 mm
- net +3V3: track 677.0 -> 679.2 mm
- net GND: vias 1 -> 268

Commit message: L1-correct Vincent's mistakes
Parts:
- removed D37: PESD2USB3UX-T, 2024l1:PESD2USB3UXT-QR
- C1: footprint 2024l1:Test Pad -> 2024l1:cap0603
- C10: footprint Capacitor_THT:CP_Radial_D16.0mm_P7.50mm -> 2024l1:CP_Radial_D16.0mm_P7.50mm
Routing:
- net Net-(U2-I0): track 70.9 -> 76.6 mm
- net +3V3: track 679.2 -> 676.3 mm
- net Net-(U2-I6): track 35.4 -> 34.7 mm
- net Net-(U2-I4): track 44.7 -> 45.2 mm
- net Net-(U1-I0): track 77.1 -> 76.6 mm
- net GND: vias 268 -> 248
