File: open/2024l1/2024l1.kicad_sch (KiCad schematic)
At the start: 129 parts, among them IC1 LM2587S-ADJ, J1 Conn_01x04, J2 Conn_01x04, J3 Conn_01x02, SW1 STM RST, U1 CD74HC4067SM, U2 CD74HC4067SM, U3 STM32F103CBTx, U4 PC817, Y1 8Mhz

Commit message: L1-Changed Boost Inductor, Shifted L2 Connector
Parts:
- L1: footprint 2024l1:0630 One Piece Inductor -> 2024l1:1040 One Piece Inductor
Changed lines of the file:
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@@
       (effects (font (size 1.27 1.27)))
     )
-    (property "Footprint" "2024l1:0630 One Piece Inductor" (at 205.74 152.4 0)
+    (property "Footprint" "2024l1:1040 One Piece Inductor" (at 205.74 152.4 0)
       (effects (font (size 1.27 1.27)) hide)
     )

Commit message: open - l1 - ceramic caps
Parts:
- added C17, C18, C19: 0u1, 2024l1:cap0603, symbol Device:C
- C10: value 1000uF -> 1m
- C11: value 100uF -> 100u
Connections:
- net +12V: now also C18.1
- net +3V3: now also C17.1
- net +48V: now also C19.1
- net GND: now also C17.2, C18.2, C19.2
Other:
- moved on the sheet: C10, C11, C12, C?, D19, D?, IC1, L1, L?, R38, R39, R40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

Commit message: open - l1 - silkscreen UI
Parts:
- C10: value 1m -> 1000u
- C11: footprint Capacitor_SMD:CP_Elec_6.3x7.7 -> Capacitor_SMD:CP_Elec_10x10.5
- C12: value 1uF -> 1u
- C18, C19: value 0u1 -> 0.1u
- R39: value 2.94k -> 2k94
- R40: value 1.5k -> 1k5
Other:
- moved on the sheet: C10, C11, C12, C18, C19, D19, IC1, J3, KM1, KM2, L1, MTH1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

Commit message: L1 - Reorganised Schematic Folder
Other:
- note added: "3V3 Buck"
- note added: "MTH"
- note added: "STM32"
- moved on the sheet: C10, C11, C12, C17, C18, C19, C?, D19, D?, IC1, L1, L?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

Commit message: L1-Edited Silkscreen
Parts:
- added D37: PESD2USB3UX-T, 2024l1:PESD2USB3UXT-QR, symbol Device:D_Dual_CommonAnode_AKK
Connections:
- net +3V3: now also D37.2 (K)
- net GND: now also D37.1 (A)
- no-connect marks 20 -> 21
Changed lines of the file:
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@@
   (no_connect (at 353.06 83.82))
   (no_connect (at 320.04 114.3))
+  (no_connect (at 391.16 85.09))
   (no_connect (at 137.16 60.96))
   (no_connect (at 320.04 104.14))
@@
     )
   )
+  (symbol (lib_id "Device:D_Dual_CommonAnode_AKK") (at 383.54 85.09 0) (unit 1)
+    (in_bom yes) (on_board yes) (dnp no) (fields_autoplaced)
+    (property "Reference" "D37" (at 383.54 80.01 0)
+      (effects (font (size 1.27 1.27)))
+    )
+    (property "Value" "PESD2USB3UX-T" (at 383.54 82.55 0)
+      (effects (font (size 1.27 1.27)))
+    )
+    (property "Footprint" "2024l1:PESD2USB3UXT-QR" (at 383.54 85.09 0)
+      (effects (font (size 1.27 1.27)) hide)
+    )
+    (property "Datasheet" "~" (at 383.54 85.09 0)
+      (effects (font (size 1.27 1.27)) hide)
+    )
+    (pin "1")
+    (pin "2")
+    (pin "3")
+    (instances
+      (project "2024l1"
+        (path "/5be543b5-1bdc-438f-a916-f916127c0a2b"
+          (reference "D37") (unit 1)
+        )
+      )
+    )
+  )
   (symbol (lib_id "power:GND") (at 299.72 142.24 0) (unit 1)
     (in_bom yes) (on_board yes) (dnp no) (fields_autoplaced)
@@
     )
   )
+  (symbol (lib_id "power:GND") (at 383.54 90.17 0) (unit 1)
+    (in_bom yes) (on_board yes) (dnp no) (fields_autoplaced)
+    (property "Reference" "#PWR049" (at 383.54 96.52 0)
+      (effects (font (size 1.27 1.27)) hide)
+    )
+    (property "Value" "GND" (at 383.54 94.996 0)
+      (effects (font (size 1.27 1.27)))
+    )
+    (property "Footprint" "" (at 383.54 90.17 0)
+      (effects (font (size 1.27 1.27)) hide)
+    )
+    (property "Datasheet" "" (at 383.54 90.17 0)
+      (effects (font (size 1.27 1.27)) hide)
+    )
+    (pin "1")
+    (instances
+      (project "2024l1"
+        (path "/5be543b5-1bdc-438f-a916-f916127c0a2b"
+          (reference "#PWR049") (unit 1)
+        )
+      )
+    )
+  )
   (symbol (lib_id "power:GND") (at 149.86 73.66 90) (unit 1)
     (in_bom yes) (on_board yes) (dnp no) (fields_autoplaced)
@@
         )
       )
+    )
+  )
+  (symbol (lib_id "power:+3V3") (at 375.92 85.09 90) (unit 1)
+    (in_bom yes) (on_board yes) (dnp no) (fields_autoplaced)
+    (property "Reference" "#PWR048" (at 379.73 85.09 0)
+      (effects (font (size 1.27 1.27)) hide)
+    )
+    (property "Value" "+3V3" (at 371.856 85.725 90)
+      (effects (font (size 1.27 1.27)) (justify left))
+    )
+    (property "Footprint" "" (at 375.92 85.09 0)
+      (effects (font (size 1.27 1.27)) hide)
+    )
+    (property "Datasheet" "" (at 375.92 85.09 0)
+      (effects (font (size 1.27 1.27)) hide)
+    )
+    (pin "1")
+    (instances
+      (project "2024l1"
+        (path "/5be543b5-1bdc-438f-a916-f916127c0a2b"
+          (reference "#PWR048") (unit 1)
+        )
+      )

Commit message: open - l1 - silkscreen
Parts:
- added TP1, TP2, TP3, TP4, TP5, TP6: Conn_01x01, 2024l1:Test Pad, symbol Connector_Generic:Conn_01x01
- C1: footprint 2024l1:cap0603 -> 2024l1:Test Pad
Connections:
- net +12V: now also TP5.1 (Pin_1)
- net +3V3: now also TP3.1 (Pin_1)
- net +48V: now also TP6.1 (Pin_1)
- net +5V: now also TP4.1 (Pin_1)
- net GND: now also TP1.1 (Pin_1), TP2.1 (Pin_1)

Commit message: L1-correct Vincent's mistakes
Parts:
- removed D37: PESD2USB3UX-T, 2024l1:PESD2USB3UXT-QR, symbol Device:D_Dual_CommonAnode_AKK
- C1: footprint 2024l1:Test Pad -> 2024l1:cap0603
- C10: footprint Capacitor_THT:CP_Radial_D16.0mm_P7.50mm -> 2024l1:CP_Radial_D16.0mm_P7.50mm
Connections:
- no-connect marks 21 -> 20
Changed lines of the file:
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@@
   (no_connect (at 353.06 83.82))
   (no_connect (at 320.04 114.3))
-  (no_connect (at 391.16 85.09))
   (no_connect (at 137.16 60.96))
   (no_connect (at 320.04 104.14))
@@
       (effects (font (size 1.27 1.27)))
     )
-    (property "Footprint" "2024l1:Test Pad" (at 297.815 46.6598 0)
+    (property "Footprint" "2024l1:cap0603" (at 297.815 46.6598 0)
       (effects (font (size 1.27 1.27)) hide)
     )
@@
       (effects (font (size 1.27 1.27)) (justify left))
     )
-    (property "Footprint" "Capacitor_THT:CP_Radial_D16.0mm_P7.50mm" (at 384.2512 196.469 0)
+    (property "Footprint" "2024l1:CP_Radial_D16.0mm_P7.50mm" (at 384.2512 196.469 0)
       (effects (font (size 1.27 1.27)) hide)
     )
@@
     )
   )
-  (symbol (lib_id "Device:D_Dual_CommonAnode_AKK") (at 383.54 85.09 0) (unit 1)
-    (in_bom yes) (on_board yes) (dnp no) (fields_autoplaced)
-    (property "Reference" "D37" (at 383.54 80.01 0)
-      (effects (font (size 1.27 1.27)))
-    )
-    (property "Value" "PESD2USB3UX-T" (at 383.54 82.55 0)
-      (effects (font (size 1.27 1.27)))
-    )
-    (property "Footprint" "2024l1:PESD2USB3UXT-QR" (at 383.54 85.09 0)
-      (effects (font (size 1.27 1.27)) hide)
-    )
-    (property "Datasheet" "~" (at 383.54 85.09 0)
-      (effects (font (size 1.27 1.27)) hide)
-    )
-    (pin "1")
-    (pin "2")
-    (pin "3")
-    (instances
-      (project "2024l1"
-        (path "/5be543b5-1bdc-438f-a916-f916127c0a2b"
-          (reference "D37") (unit 1)
-        )
-      )
-    )
-  )
   (symbol (lib_id "power:GND") (at 299.72 142.24 0) (unit 1)
     (in_bom yes) (on_board yes) (dnp no) (fields_autoplaced)
@@
     )
   )
-  (symbol (lib_id "power:GND") (at 383.54 90.17 0) (unit 1)
-    (in_bom yes) (on_board yes) (dnp no) (fields_autoplaced)
-    (property "Reference" "#PWR049" (at 383.54 96.52 0)
-      (effects (font (size 1.27 1.27)) hide)
-    )
-    (property "Value" "GND" (at 383.54 94.996 0)
-      (effects (font (size 1.27 1.27)))
-    )
-    (property "Footprint" "" (at 383.54 90.17 0)
-      (effects (font (size 1.27 1.27)) hide)
-    )
-    (property "Datasheet" "" (at 383.54 90.17 0)
-      (effects (font (size 1.27 1.27)) hide)
-    )
-    (pin "1")
-    (instances
-      (project "2024l1"
-        (path "/5be543b5-1bdc-438f-a916-f916127c0a2b"
-          (reference "#PWR049") (unit 1)
-        )
-      )
-    )
-  )
   (symbol (lib_id "power:GND") (at 149.86 73.66 90) (unit 1)
     (in_bom yes) (on_board yes) (dnp no) (fields_autoplaced)
@@
         )
       )
-    )
-  )
-  (symbol (lib_id "power:+3V3") (at 375.92 85.09 90) (unit 1)
-    (in_bom yes) (on_board yes) (dnp no) (fields_autoplaced)
-    (property "Reference" "#PWR048" (at 379.73 85.09 0)
-      (effects (font (size 1.27 1.27)) hide)
-    )
-    (property "Value" "+3V3" (at 371.856 85.725 90)
-      (effects (font (size 1.27 1.27)) (justify left))
-    )
-    (property "Footprint" "" (at 375.92 85.09 0)
-      (effects (font (size 1.27 1.27)) hide)
-    )
-    (property "Datasheet" "" (at 375.92 85.09 0)
-      (effects (font (size 1.27 1.27)) hide)
-    )
-    (pin "1")
-    (instances
-      (project "2024l1"
-        (path "/5be543b5-1bdc-438f-a916-f916127c0a2b"
-          (reference "#PWR048") (unit 1)
-        )
-      )

Commit message: open - l1 - redid schematic
Parts:
- C6, C7, C8, C9: value 0.1u -> 0u1
- J1: value Conn_01x04 -> PGMR
- KM1, KM2: value MountingHole_Pad -> M4
- R33: value 1k -> 3k24
Connections:
- no-connect marks 20 -> 21
Other:
- note added: "48V Boost"
- note added: "MTH and Testpoints"
- note removed: "Boost"
- note removed: "MTH"
- moved on the sheet: C1, C10, C11, C12, C17, C18, C19, C2, C3, C4, C5, C6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
