File: open/2024l3/2024l3.kicad_pcb (KiCad board)
At the start: 2 copper layers, 173.6 x 90 mm, 2 parts, among them U1 OpenMV, U2 xiao-esp32c3

Commit message: open - l3 - 3d models
Parts:
- added J1: Conn_01x08, Connector_JST:JST_XH_S8B-XH-A_1x08_P2.50mm_Horizontal, F.Cu at (166.8, 79.6)
- added U3: xiao-esp32c3, 2024l3:xiao-esp32c3, F.Cu at (187.4, 99.3)
- U2: value xiao-esp32c3 -> 4754; footprint 2024l3:xiao-esp32c3 -> 2024l3:bno085
- moved U2 1.50 mm to (157.2, 127.9), turned to 180 degrees
Other:
- board size 173.6 x 90 mm -> 173.6 x 100 mm

Commit message: L3-Updated Edge Cuts and added MTH
Parts:
- added H1: MountingHole_Pad, MountingHole:MountingHole_3.2mm_M3_Pad, F.Cu at (75.8, 92.2)
- added H2: MountingHole_Pad, MountingHole:MountingHole_3.2mm_M3_Pad, F.Cu at (75.8, 120.4)
- added H3: MountingHole_Pad, MountingHole:MountingHole_3.2mm_M3_Pad, F.Cu at (125.6, 74.3)
- added H4: MountingHole_Pad, MountingHole:MountingHole_3.2mm_M3_Pad, F.Cu at (125.6, 138.3)
- added H5: MountingHole_Pad, MountingHole:MountingHole_3.2mm_M3_Pad, F.Cu at (189.6, 138.3)
- added H6: MountingHole_Pad, MountingHole:MountingHole_3.2mm_M3_Pad, F.Cu at (189.6, 74.3)
- added H7: MountingHole_Pad, MountingHole:MountingHole_3.2mm_M3_Pad, F.Cu at (239.4, 92.2)
- added He: MountingHole_Pad, MountingHole:MountingHole_3.2mm_M3_Pad, F.Cu at (239.4, 120.4)
Other:
- board size 173.6 x 100 mm -> 173.6 x 90 mm

Commit message: L3-Updated DXF
Parts:
- H1, H2, H3, H4, H5, H6, H7: footprint MountingHole:MountingHole_3.2mm_M3_Pad -> MountingHole:MountingHole_3.2mm_M3_Pad_Via
- H8: renamed from He; footprint MountingHole:MountingHole_3.2mm_M3_Pad -> MountingHole:MountingHole_3.2mm_M3_Pad_Via
- moved H4 0.51 mm to (125.2, 138.7)
- moved H3 0.51 mm to (125.2, 74.0)
- moved H5 0.51 mm to (189.9, 138.7)
- moved H6 0.51 mm to (189.9, 74.0)

Commit message: L3- Changed DXF L1- Routed PWR again L2-Redid Enable Resistors
Parts:
- added H9: MountingHole_Pad, MountingHole:MountingHole_3.2mm_M3_Pad_Via, F.Cu at (204.1, 37.6)
- added He: MountingHole_Pad, MountingHole:MountingHole_3.2mm_M3_Pad_Via, F.Cu at (111.1, 37.6)
- J1: moved to B.Cu
- moved J1 17.1 mm to (149.7, 80.9), turned to 0 degrees
Other:
- board size 173.6 x 90 mm -> 173.6 x 125.5 mm

Commit message: Basic L3 routing
Parts:
- added U4: Adafruit Featherwing, 2024l3:Adafruit Feather OLED, F.Cu at (160.2, 54.0)
- renumbered He to H10
Connections:
- U1 pad 10: unconnected-(U1-VIN_(3V6-5V)-Pad10) -> +5V
- U1 pad 9: unconnected-(U1-GND-Pad9) -> GND
- U2 pad JP1_1: unconnected-(U2-VIN-PadJP1_1) -> +5V
- U2 pad JP1_3: unconnected-(U2-GND-PadJP1_3) -> GND
- U2 pad JP1_4: unconnected-(U2-SCL-PadJP1_4) -> /COM SCL
- U2 pad JP1_5: unconnected-(U2-SDA-PadJP1_5) -> /COM SDA
- U3 pad 11: unconnected-(U3-3V3-Pad11) -> +3V3
- U3 pad 12: unconnected-(U3-GND-Pad12) -> GND
- U3 pad 13: unconnected-(U3-5V-Pad13) -> +5V

Commit message: All Layers: Major revisions
Parts:
- added C1: 0u1, 2024l2:cap0603, F.Cu at (215.9, 42.0)
- added C2: 0u1, 2024l2:cap0603, F.Cu at (215.9, 44.9)
- added C3: 0u1, 2024l2:cap0603, F.Cu at (215.9, 47.8)
- added C4: 0u1, 2024l2:cap0603, F.Cu at (215.9, 50.7)
- added C5: 100n, 2024l2:cap0603, F.Cu at (215.9, 53.6)
- added C6: 22p, 2024l2:cap0603, F.Cu at (215.9, 56.5)
- added C7: 22p, 2024l2:cap0603, F.Cu at (215.9, 59.4)
- added D1: LED, 2024l2:led0603, F.Cu at (215.9, 62.3)
- added J2: Conn_01x06, Connector_PinSocket_2.54mm:PinSocket_1x06_P2.54mm_Vertical, F.Cu at (113.3, 63.1)
- added J3: Conn_01x06, Connector_PinSocket_2.54mm:PinSocket_1x06_P2.54mm_Vertical, F.Cu at (117.9, 63.1)
- added J4: Conn_01x06, Connector_PinSocket_2.54mm:PinSocket_1x06_P2.54mm_Vertical, F.Cu at (122.5, 63.1)
- added J5: Conn_01x06, Connector_PinSocket_2.54mm:PinSocket_1x06_P2.54mm_Vertical, F.Cu at (127.1, 63.1)
- added J6: PGMR, Connector_JST:JST_XH_B4B-XH-A_1x04_P2.50mm_Vertical, F.Cu at (114.5, 80.4)
- added R1: 10K, 2024l2:res0603, F.Cu at (215.9, 65.2)
- added SW1: STM RST, 2024l2:SW_PUSH_SPST, F.Cu at (221.7, 59.0)
- added U5: STM32F103CBTx, Package_QFP:LQFP-48_7x7mm_P0.5mm, F.Cu at (223.9, 46.3)
- added Y1: 8Mhz, 2024l1:Crystal, F.Cu at (221.8, 54.4)
- moved U2 43.8 mm to (124.6, 98.7)
- moved U4 18.8 mm to (142.4, 47.9)
- moved H4 8.99 mm to (131.6, 132.3)
- moved H3 8.99 mm to (131.6, 80.3)
- moved H5 8.99 mm to (183.6, 132.3)
- moved H6 8.99 mm to (183.6, 80.3)
Connections:
- U1 pad 5: unconnected-(U1-P4-UART_TX/I2C2_SCL-Pad5) -> /CAM TX
- U1 pad 6: unconnected-(U1-P5-UART_RX/I2C_SDA-Pad6) -> /CAM RX
- U2 pad JP2_4: unconnected-(U2-~{RST}-PadJP2_4) -> /COM RST
- U3 pad 11: +3V3 -> unconnected-(U3-3V3-Pad11)
- U3 pad 6: unconnected-(U3-TX-Pad6) -> /ESP TX
- U3 pad 7: unconnected-(U3-RX-Pad7) -> /ESP RX
- U4 pad 17: unconnected-(U4-SDA-Pad17) -> /OLED SDA
- U4 pad 18: unconnected-(U4-SCL-Pad18) -> /OLED SCL
Other:
- board size 173.6 x 125.5 mm -> 173.6 x 119.5 mm

Commit message: L3-Updated DXF
Parts:
- moved U5 29.8 mm to (196.5, 58.1)
- moved U1 0.07 mm to (157.6, 112.0)
Other:
- board size 173.6 x 119.5 mm -> 176 x 119.5 mm

Commit message: L1- Redid Boost Placement
Parts:
- C1, C2, C3, C4: value 0u1 -> 0.1uF
- J2: value Conn_01x06 -> TOF 0
- J3: value Conn_01x06 -> TOF 1
- J4: value Conn_01x06 -> TOF 2
- J5: value Conn_01x06 -> TOF 3
Connections:
- J2 pad 1: unconnected-(J2-Pin_1-Pad1) -> /XSHUT 0
- J2 pad 3: unconnected-(J2-Pin_3-Pad3) -> /SDA TOF
- J2 pad 4: unconnected-(J2-Pin_4-Pad4) -> /SCL TOF
- J2 pad 5: unconnected-(J2-Pin_5-Pad5) -> GND
- J2 pad 6: unconnected-(J2-Pin_6-Pad6) -> +5V
- J3 pad 1: unconnected-(J3-Pin_1-Pad1) -> /XSHUT 1
- J3 pad 3: unconnected-(J3-Pin_3-Pad3) -> /SDA TOF
- J3 pad 4: unconnected-(J3-Pin_4-Pad4) -> /SCL TOF
- J3 pad 5: unconnected-(J3-Pin_5-Pad5) -> GND
- J3 pad 6: unconnected-(J3-Pin_6-Pad6) -> +5V
- J4 pad 1: unconnected-(J4-Pin_1-Pad1) -> /XSHUT 2
- J4 pad 3: unconnected-(J4-Pin_3-Pad3) -> /SDA TOF
- J4 pad 4: unconnected-(J4-Pin_4-Pad4) -> /SCL TOF
- J4 pad 5: unconnected-(J4-Pin_5-Pad5) -> GND
- J4 pad 6: unconnected-(J4-Pin_6-Pad6) -> +5V
- J5 pad 1: unconnected-(J5-Pin_1-Pad1) -> /XSHUT 3
- J5 pad 3: unconnected-(J5-Pin_3-Pad3) -> /SDA TOF
- J5 pad 4: unconnected-(J5-Pin_4-Pad4) -> /SCL TOF
- J5 pad 5: unconnected-(J5-Pin_5-Pad5) -> GND
- J5 pad 6: unconnected-(J5-Pin_6-Pad6) -> +5V
- U3 pad 0: unconnected-(U3-A0-Pad0) -> /XSHUT 0
- U3 pad 1: unconnected-(U3-A1-Pad1) -> /XSHUT 1
- U3 pad 2: unconnected-(U3-A2-Pad2) -> /XSHUT 2
- U3 pad 3: unconnected-(U3-A3-Pad3) -> /XSHUT 3
- U3 pad 4: unconnected-(U3-SDA-Pad4) -> /SDA TOF
- U3 pad 5: unconnected-(U3-SCL-Pad5) -> /SCL TOF
- U4 pad 19: unconnected-(U4-C-Pad19) -> /C
- U4 pad 20: unconnected-(U4-B-Pad20) -> /B
- U4 pad 21: unconnected-(U4-A-Pad21) -> /A
