File: open/2024l3/2024l3.kicad_sch (KiCad schematic)
At the start: 26 parts, among them J1 Conn_01x10, J2 TOF 0, J3 TOF 1, J4 TOF 2, J5 TOF 3, U1 OpenMV, U2 4754, U3 xiao-esp32c3, U4 Adafruit Featherwing, U5 Seeed Studio XIAO SAMD21, U6 C5199435

Commit message: small adjustment
Connections:
- net COM SCL: now also J1.4 (Pin_4); no longer J1.5 (Pin_5)
- net COM SDA: now also J1.5 (Pin_5); no longer J1.4 (Pin_4)
Changed lines of the file:
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@@
     (stroke (width 0) (type default))
   )
-  (wire (pts (xy 64.376 39.1273) (xy 73.266 39.1273))
+  (wire (pts (xy 64.376 41.6673) (xy 73.266 41.6673))
     (stroke (width 0) (type default))
   )
@@
     (stroke (width 0) (type default))
   )
-  (wire (pts (xy 64.376 41.6673) (xy 73.266 41.6673))
+  (wire (pts (xy 64.376 39.1273) (xy 73.266 39.1273))
     (stroke (width 0) (type default))
   )
@@
     (effects (font (size 1.27 1.27)) (justify left bottom))
   )
-  (label "COM SDA" (at 65.646 41.6673 0) (fields_autoplaced)
+  (label "COM SDA" (at 65.646 39.1273 0) (fields_autoplaced)
     (effects (font (size 1.27 1.27)) (justify left bottom))
   )
@@
     (effects (font (size 1.27 1.27)) (justify left bottom))
   )
-  (label "COM SCL" (at 65.646 39.1273 0) (fields_autoplaced)
+  (label "COM SCL" (at 65.646 41.6673 0) (fields_autoplaced)
     (effects (font (size 1.27 1.27)) (justify left bottom))
   )
