File: open/2024l1  (Single Mux)/2024l1 Single.kicad_pcb (KiCad board)
At the start: 2 copper layers, 176 x 169.5 mm, 103 parts, among them IC1 LM2587S-ADJ, J1 Conn_01x03, J2 Conn_01x03, J3 Conn_01x02, J4 Conn_01x02, J5 XT30, J6 Conn_01x04, Q1 STP75NF75, Q2 STP75NF75, SW1 SW_SPDT, U1 Seeed Studio XIAO SAMD21, U2 CD74HC4067SM

Commit message: L1 Single Mux - A bit more routing
Parts:
- moved R23 146.3 mm to (97.1, 114.9)
- moved C7 144.5 mm to (97.1, 109.6)
- moved R24 142.2 mm to (97.1, 112.2)
Connections:
- U1 pad 10: /S3 -> /S0
- U1 pad 3: /S0 -> /S3
- U1 pad 4: /S1 -> /S2
- U1 pad 9: /S2 -> /S1
Routing:
- net /M1: track 31.8 -> 85.1 mm, vias 1 -> 3
- net /S0: track 29.4 -> 78.3 mm, vias 1 -> 0
- net /S1: track 28.0 -> 71.4 mm, vias 1 -> 0
- net /S2: track 38.6 -> 69.2 mm, vias 0 -> 1
- net Net-(U2-~{E}): track 0.00 -> 17.2 mm
- net +3V3: track 491.5 -> 507.4 mm
- net /S3: track 78.5 -> 69.5 mm, vias 0 -> 1
- added copper zone on F.Cu, net Net-(C8-Pad1)
- removed copper zone on F.Cu, net Net-(C6-Pad1)

Commit message: L1 - Single MUX Version done
Connections:
- R10 pad 2: Net-(U2-I13) -> Net-(U2-I1)
- R11 pad 2: Net-(U2-I12) -> Net-(U2-I0)
- R12 pad 2: Net-(U2-I11) -> Net-(U2-I14)
- R13 pad 2: Net-(U2-I10) -> Net-(U2-I13)
- R14 pad 2: Net-(U2-I9) -> Net-(U2-I12)
- R15 pad 2: Net-(U2-I8) -> Net-(U2-I11)
- R16 pad 2: Net-(U2-I7) -> Net-(U2-I10)
- R17 pad 2: Net-(U2-I6) -> Net-(U2-I9)
- R18 pad 2: Net-(U2-I5) -> Net-(U2-I8)
- R19 pad 2: Net-(U2-I4) -> Net-(U2-I7)
- R20 pad 2: Net-(U2-I3) -> Net-(U2-I6)
- R21 pad 2: Net-(U2-I2) -> Net-(U2-I5)
- R22 pad 2: Net-(U2-I1) -> Net-(U2-I4)
- R8 pad 2: Net-(U2-I0) -> Net-(U2-I3)
- R9 pad 2: Net-(U2-I14) -> Net-(U2-I2)
Routing:
- net Net-(U2-I11): track 0.00 -> 77.6 mm, vias 0 -> 1
- net Net-(U2-I3): track 0.00 -> 76.1 mm, vias 0 -> 1
- net Net-(U2-I10): track 0.00 -> 74.6 mm, vias 0 -> 1
- net Net-(U2-I12): track 0.00 -> 70.5 mm, vias 0 -> 1
- net Net-(U2-I9): track 0.00 -> 66.1 mm, vias 0 -> 1
- net Net-(U2-I13): track 0.00 -> 63.7 mm, vias 0 -> 1
- net Net-(U2-I7): track 0.00 -> 61.1 mm, vias 0 -> 1
- net Net-(U2-I0): track 0.00 -> 61.1 mm, vias 0 -> 1
- net Net-(U2-I14): track 0.00 -> 60.7 mm, vias 0 -> 1
- net Net-(U2-I2): track 0.00 -> 60.7 mm, vias 0 -> 1
- net Net-(U2-I4): track 0.00 -> 60.2 mm, vias 0 -> 1
- net Net-(U2-I6): track 0.00 -> 59.8 mm, vias 0 -> 1
- net Net-(U2-I1): track 0.00 -> 59.2 mm, vias 0 -> 1
- net Net-(U2-I8): track 0.00 -> 58.1 mm, vias 0 -> 1
- net Net-(U2-I5): track 0.00 -> 57.9 mm, vias 0 -> 1
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
Commit message: L1- Almost Production version
Parts:
- moved D4 13.0 mm to (190.8, 112.2), turned to 90 degrees
Connections:
- SW1 pad 1: +3V3 -> Net-(SW1-A)
- SW1 pad 2: Net-(D4-A) -> +3V3
- SW1 pad 3: unconnected-(SW1-C-Pad3) -> Net-(D4-A)
- U1 pad 12: Net-(D4-A) -> Net-(SW1-A)
Routing:
- net Net-(SW1-A): track 0.00 -> 5.98 mm
- net +3V3: track 564.8 -> 566.0 mm
- net Net-(D4-A): track 11.3 -> 12.3 mm
- net /S2: track 69.2 -> 70.0 mm

Commit message: L1 and Single - Flipped Connector
Parts:
- moved J2 5.03 mm to (159.5, 114.8), turned to 90 degrees
Connections:
- J2 pad 1: /L1 TX -> /L1 RX
- J2 pad 3: /L1 RX -> /L1 TX
Routing:
- net /L1 RX: track 14.4 -> 14.9 mm
- net /L1 TX: track 18.3 -> 18.8 mm
Changed lines of the file:
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@@
   )
   (footprint "Connector_JST:JST_XH_B3B-XH-A_1x03_P2.50mm_Vertical" (layer "F.Cu")
-    (at 160.02 109.76 -90)
+    (at 159.495 114.76 90)
     (descr "JST XH series connector, B3B-XH-A (http://www.jst-mfg.com/product/pdf/eng/eXH.pdf), generated with kicad-footprint-generator")
     (tags "connector JST XH vertical")
@@
     (fp_line (start 7.45 3.4) (end 7.45 -2.35)
       (stroke (width 0.1) (type solid)) (layer "F.Fab"))
-    (pad "1" thru_hole roundrect (at 0 0 270) (size 1.7 1.95) (drill 0.95) (layers "*.Cu" "*.Mask") (roundrect_rratio 0.1470588235)
-      (net 53 "/L1 TX") (pinfunction "Pin_1") (pintype "passive"))
-    (pad "2" thru_hole oval (at 2.5 0 270) (size 1.7 1.95) (drill 0.95) (layers "*.Cu" "*.Mask")
+    (pad "1" thru_hole roundrect (at 0 0 90) (size 1.7 1.95) (drill 0.95) (layers "*.Cu" "*.Mask") (roundrect_rratio 0.1470588235)
+      (net 52 "/L1 RX") (pinfunction "Pin_1") (pintype "passive"))
+    (pad "2" thru_hole oval (at 2.5 0 90) (size 1.7 1.95) (drill 0.95) (layers "*.Cu" "*.Mask")
       (net 14 "GND") (pinfunction "Pin_2") (pintype "passive"))
-    (pad "3" thru_hole oval (at 5 0 270) (size 1.7 1.95) (drill 0.95) (layers "*.Cu" "*.Mask")
-      (net 52 "/L1 RX") (pinfunction "Pin_3") (pintype "passive"))
+    (pad "3" thru_hole oval (at 5 0 90) (size 1.7 1.95) (drill 0.95) (layers "*.Cu" "*.Mask")
+      (net 53 "/L1 TX") (pinfunction "Pin_3") (pintype "passive"))
     (model "${KICAD6_3DMODEL_DIR}/Connector_JST.3dshapes/JST_XH_B3B-XH-A_1x03_P2.50mm_Vertical.wrl"
       (offset (xyz 0 0 0))
@@
   (segment (start 171 105.9) (end 171.08 105.82) (width 0.3) (layer "B.Cu") (net 51))
   (segment (start 171.08 105.82) (end 179.42 105.82) (width 0.3) (layer "B.Cu") (net 51))
-  (segment (start 164.02 114.76) (end 169.5925 120.3325) (width 0.3) (layer "F.Cu") (net 52))
-  (segment (start 160.02 114.76) (end 164.02 114.76) (width 0.3) (layer "F.Cu") (net 52))
   (segment (start 169.5925 120.3325) (end 172.08 120.3325) (width 0.3) (layer "F.Cu") (net 52))
-  (segment (start 160.02 109.76) (end 161.17 108.61) (width 0.3) (layer "F.Cu") (net 53))
+  (segment (start 159.495 114.76) (end 164.02 114.76) (width 0.3) (layer "F.Cu") (net 52))
+  (segment (start 164.02 114.76) (end 169.5925 120.3325) (width 0.3) (layer "F.Cu") (net 52))
   (segment (start 173.37 105.4575) (end 172.08 104.1675) (width 0.3) (layer "F.Cu") (net 53))
-  (segment (start 173.37 107.67) (end 173.37 105.4575) (width 0.3) (layer "F.Cu") (net 53))
   (segment (start 172.43 108.61) (end 173.37 107.67) (width 0.3) (layer "F.Cu") (net 53))
-  (segment (start 161.17 108.61) (end 172.43 108.61) (width 0.3) (layer "F.Cu") (net 53))
+  (segment (start 160.645 108.61) (end 172.43 108.61) (width 0.3) (layer "F.Cu") (net 53))
+  (segment (start 173.37 107.67) (end 173.37 105.4575) (width 0.3) (layer "F.Cu") (net 53))
+  (segment (start 159.495 109.76) (end 160.645 108.61) (width 0.3) (layer "F.Cu") (net 53))
   (segment (start 182.24 117.51) (end 182.24 120.3325) (width 0.5) (layer "F.Cu") (net 54))
   (segment (start 180.01 115.28) (end 182.24 117.51) (width 0.5) (layer "F.Cu") (net 54))

Commit message: L1-Production files
Parts:
- removed D4: LED, 2024l1:led0603
- removed SW1: SW_SPDT, 2024l1:SS12F21
- added kibuzzard-64F35836: G***, kibuzzard-64F35836, F.Cu at (117.0, 112.2)
- D3, R4, R5: moved to B.Cu
- J3, J4: moved to F.Cu
- moved J3 2.54 mm to (115.7, 191.7)
- moved J4 2.54 mm to (97.4, 191.7)
- turned R4 to 180 degrees
- turned D10 to 42 degrees
- turned D11 to 66 degrees
- turned D12 to 90 degrees
- turned D14 to 114 degrees
- turned D15 to 138 degrees
- turned D16 to 162 degrees
- turned D17 to -174 degrees
- turned D18 to -150 degrees
- turned D19 to -126 degrees
- turned D20 to -102 degrees
- turned D5 to -78 degrees
- turned D6 to -54 degrees
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Connections:
- U1 pad 12: Net-(SW1-A) -> unconnected-(U1-3V3-Pad12)
- U1 pad 14: unconnected-(U1-5V-Pad14) -> +3V3
Routing:
- net Net-(D4-A): track 12.3 -> 0.00 mm
- net +3V3: track 566.0 -> 558.5 mm
- net Net-(SW1-A): track 5.98 -> 0.00 mm
- net /L1 TX: track 18.8 -> 17.7 mm
- added copper zone on B.Cu, net +3.3VA
- removed copper zone on F.Cu, net +3.3VA
Other:
- board text added: "JLCJLCJLCJLC"

Commit message: fixed some traces
Parts:
- removed mouse-bite-2mm-slot (x2): VAL**, 2024l1:mouse-bite-2mm-slot
- moved kibuzzard-64F1C247 2.03 mm to (155.3, 114.8), turned to 180 degrees
- moved kibuzzard-64F1BF81 2.00 mm to (155.3, 109.8), turned to 180 degrees
- moved kibuzzard-64F1954C 0.32 mm to (154.8, 112.2), turned to 180 degrees
Connections:
- U1 pad 2: /Sol -> unconnected-(U1-PA4_A1_D1-Pad2)
- U1 pad 3: /S3 -> /Sol
- U1 pad 4: /S2 -> /S3
- U1 pad 5: unconnected-(U1-PA8_A4_D4_SDA-Pad5) -> /S2
Routing:
- net /M1: track 109.7 -> 85.7 mm, vias 1 -> 0
- net /S0: track 77.9 -> 69.8 mm
- net /S1: track 71.5 -> 64.9 mm
- net /Sol: track 165.6 -> 163.1 mm, vias 1 -> 0
- net /S2: track 70.0 -> 67.6 mm
- net /S3: track 69.5 -> 67.4 mm
- net /LG: track 81.5 -> 81.7 mm, vias 1 -> 0

Commit message: L1- Fixed edge cuts
Parts:
- added mouse-bite-2mm-slot: VAL**, 2024l1:mouse-bite-2mm-slot, F.Cu at (117.0, 179.9)
- added mouse-bite-2mm-slot: VAL**, 2024l1:mouse-bite-2mm-slot, F.Cu at (98.6, 179.9)
