File: open/2024l1  (Single Mux)/2024l1 Single.kicad_sch (KiCad schematic)
At the start: 92 parts, among them IC1 LM2587S-ADJ, J1 Conn_01x03, J2 Conn_01x03, J3 Conn_01x02, J4 Conn_01x02, J6 Conn_01x04, SW1 SW_SPDT, U1 Seeed Studio XIAO SAMD21, U2 CD74HC4067SM

Commit message: L1 Single Mux - A bit more routing
Connections:
- net S0: now also U1.10 (PA5_A9_D9_MISO); no longer U1.3 (PA10_A2_D2)
- net S1: now also U1.9 (PA7_A8_D8_SCK); no longer U1.4 (PA11_A3_D3)
- net S2: now also U1.4 (PA11_A3_D3); no longer U1.9 (PA7_A8_D8_SCK)
- net S3: now also U1.3 (PA10_A2_D2); no longer U1.10 (PA5_A9_D9_MISO)
Changed lines of the file:
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@@
+    (stroke (width 0) (type default))
+  )
+  (wire (pts (xy 242.555 84.7232) (xy 232.395 84.7232))
     (stroke (width 0) (type default))
   )
@@
     (stroke (width 0) (type default))
   )
+  (wire (pts (xy 294.625 88.5332) (xy 284.465 88.5332))
+    (stroke (width 0) (type default))
+  )
   (wire (pts (xy 184.297 54.1855) (xy 184.297 54.3563))
     (stroke (width 0) (type default))
@@
     (stroke (width 0) (type default))
   )
-  (wire (pts (xy 242.555 84.7232) (xy 232.395 84.7232))
-    (stroke (width 0) (type default))
-  )
   (wire (pts (xy 44.5964 194.4606) (xy 44.5964 194.5114))
     (stroke (width 0) (type default))
@@
     (stroke (width 0) (type default))
   )
-  (wire (pts (xy 294.625 88.5332) (xy 284.465 88.5332))
-    (stroke (width 0) (type default))
-  )
   (polyline (pts (xy 142.9799 75.6918) (xy 142.9799 12.0131))
     (stroke (width 0) (type dash))
@@
     (stroke (width 0) (type default))
   )
+  (wire (pts (xy 294.625 92.3432) (xy 284.465 92.3432))
+    (stroke (width 0) (type default))
+  )
   (wire (pts (xy 187.8517 24.0797) (xy 192.7322 24.0797))
     (stroke (width 0) (type default))
@@
     (stroke (width 0) (type default))
   )
+  (wire (pts (xy 242.555 80.9132) (xy 232.395 80.9132))
+    (stroke (width 0) (type default))
+  )
   (wire (pts (xy 291.3515 168.9828) (xy 281.1915 168.9828))
     (stroke (width 0) (type default))
@@
     (stroke (width 0) (type default))
   )
-  (wire (pts (xy 294.625 92.3432) (xy 284.465 92.3432))
-    (stroke (width 0) (type default))
-  )
   (wire (pts (xy 57.0177 83.9214) (xy 59.5577 83.9214))
     (stroke (width 0) (type default))
@@
     (stroke (width 0) (type default))
   )
-  (wire (pts (xy 242.555 80.9132) (xy 232.395 80.9132))
-    (stroke (width 0) (type default))
-  )
   (wire (pts (xy 53.489 218.6414) (xy 61.109 218.6414))
     (stroke (width 0) (type default))
@@
     (effects (font (size 1.27 1.27)) (justify left bottom))
   )
+  (label "S1" (at 292.085 92.3432 180) (fields_autoplaced)
+    (effects (font (size 1.27 1.27)) (justify right bottom))
+  )
   (label "S1" (at 69.7177 127.0973 270) (fields_autoplaced)
     (effects (font (size 1.27 1.27)) (justify right bottom))
@@
     (effects (font (size 1.27 1.27)) (justify left bottom))
   )
-  (label "S2" (at 292.085 92.3432 180) (fields_autoplaced)
-    (effects (font (size 1.27 1.27)) (justify right bottom))
-  )
   (label "Sol" (at 237.5505 77.1032 0) (fields_autoplaced)
     (effects (font (size 1.27 1.27)) (justify left bottom))
   )
+  (label "S2" (at 240.015 84.7232 180) (fields_autoplaced)
+    (effects (font (size 1.27 1.27)) (justify right bottom))
+  )
   (label "S0" (at 67.1777 127.0973 270) (fields_autoplaced)
     (effects (font (size 1.27 1.27)) (justify right bottom))
@@
     (effects (font (size 1.27 1.27)) (justify left bottom))
   )
-  (label "S1" (at 240.015 84.7232 180) (fields_autoplaced)
+  (label "S3" (at 240.015 80.9132 180) (fields_autoplaced)
+    (effects (font (size 1.27 1.27)) (justify right bottom))
+  )
+  (label "S0" (at 292.085 88.5332 180) (fields_autoplaced)
     (effects (font (size 1.27 1.27)) (justify right bottom))
   )
@@
     (effects (font (size 1.27 1.27)) (justify left bottom))
   )
-  (label "S0" (at 240.015 80.9132 180) (fields_autoplaced)
-    (effects (font (size 1.27 1.27)) (justify right bottom))
-  )
-  (label "S3" (at 292.085 88.5332 180) (fields_autoplaced)
-    (effects (font (size 1.27 1.27)) (justify right bottom))
-  )
   (label "L1 RX" (at 284.465 96.1532 0) (fields_autoplaced)

Commit message: L1 - Single MUX Version done
Connections:
- net at R13.2: now also U2.18 (I13); no longer U2.21 (I10)
- net at R20.2: now also U2.3 (I6); no longer U2.6 (I3)
- net at R15.2: now also U2.20 (I11); no longer U2.23 (I8)
- net at R9.2: now also U2.7 (I2); no longer U2.17 (I14)
- net at R19.2: now also U2.2 (I7); no longer U2.5 (I4)
- net at R17.2: now also U2.22 (I9); no longer U2.3 (I6)
- net at R8.2: now also U2.6 (I3); no longer U2.9 (I0)
- net at R16.2: now also U2.21 (I10); no longer U2.2 (I7)
- net at R22.2: now also U2.5 (I4); no longer U2.8 (I1)
- net at R18.2: now also U2.23 (I8); no longer U2.4 (I5)
- net at R14.2: now also U2.19 (I12); no longer U2.22 (I9)
- net at R12.2: now also U2.17 (I14); no longer U2.20 (I11)
- net at R21.2: now also U2.4 (I5); no longer U2.7 (I2)
- net at R10.2: now also U2.8 (I1); no longer U2.18 (I13)
- net at R11.2: now also U2.9 (I0); no longer U2.19 (I12)
Other:
- moved on the sheet: R10, R11, R12, R13, R14, R15, R16, R17, R18, R19, R20, R21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

Commit message: L1- Almost Production version
Connections:
- net +3V3: now also SW1.2 (B); no longer SW1.1 (A)
- net at SW1.3 (C): now also D4.2 (A)
- new net: SW1.1 (A), U1.12 (3V3)
Other:
- moved on the sheet: D4, SW1
Changed lines of the file:
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@@
   (junction (at 57.0177 83.9173) (diameter 0) (color 0 0 0 0)
   )
-  (junction (at 293.408 80.9151) (diameter 0) (color 0 0 0 0)
-  )
   (junction (at 260.8715 194.3828) (diameter 0) (color 0 0 0 0)
   )
@@
     (stroke (width 0) (type default))
   )
-  (wire (pts (xy 298.556 80.9151) (xy 293.408 80.9151))
-    (stroke (width 0) (type default))
-  )
   (wire (pts (xy 230.3915 191.8428) (xy 230.3915 194.3828))
     (stroke (width 0) (type default))
@@
     (stroke (width 0) (type default))
   )
-  (wire (pts (xy 293.408 80.9151) (xy 293.2371 80.9151))
-    (stroke (width 0) (type default))
-  )
   (wire (pts (xy 184.297 54.3563) (xy 184.297 54.3676))
     (stroke (width 0) (type default))
@@
     (stroke (width 0) (type default))
   )
+  (wire (pts (xy 298.556 75.8351) (xy 298.556 70.267))
+    (stroke (width 0) (type default))
+  )
   (wire (pts (xy 184.297 46.5655) (xy 197.8114 46.5655))
     (stroke (width 0) (type default))
@@
     (stroke (width 0) (type default))
   )
+  (wire (pts (xy 293.2371 80.9151) (xy 298.556 80.9151))
+    (stroke (width 0) (type default))
+  )
   (wire (pts (xy 281.1915 180.4128) (xy 291.3515 180.4128))
     (stroke (width 0) (type default))
@@
     )
   )
-  (symbol (lib_id "Switch:SW_SPDT") (at 303.636 80.9151 0) (unit 1)
+  (symbol (lib_id "Switch:SW_SPDT") (at 303.636 78.3751 180) (unit 1)
     (in_bom yes) (on_board yes) (dnp no) (fields_autoplaced)
-    (property "Reference" "SW1" (at 303.636 74.6309 0)
+    (property "Reference" "SW1" (at 303.636 71.12 0)
       (effects (font (size 1.27 1.27)))
     )
-    (property "Value" "SW_SPDT" (at 303.636 77.1709 0)
+    (property "Value" "SW_SPDT" (at 303.636 73.66 0)
       (effects (font (size 1.27 1.27)))
     )
-    (property "Footprint" "2024l1:SS12F21" (at 303.636 80.9151 0)
+    (property "Footprint" "2024l1:SS12F21" (at 303.636 78.3751 0)
       (effects (font (size 1.27 1.27)) hide)
     )
-    (property "Datasheet" "~" (at 303.636 80.9151 0)
+    (property "Datasheet" "~" (at 303.636 78.3751 0)
       (effects (font (size 1.27 1.27)) hide)
     )
@@
     )
   )
-  (symbol (lib_id "Device:LED") (at 293.408 77.1051 270) (unit 1)
+  (symbol (lib_id "Device:LED") (at 298.556 66.457 270) (unit 1)
     (in_bom yes) (on_board yes) (dnp no) (fields_autoplaced)
-    (property "Reference" "D4" (at 295.576 74.8826 90)
+    (property "Reference" "D4" (at 300.724 64.2345 90)
       (effects (font (size 1.27 1.27)) (justify left))
     )
-    (property "Value" "LED" (at 295.576 77.4226 90)
+    (property "Value" "LED" (at 300.724 66.7745 90)
       (effects (font (size 1.27 1.27)) (justify left))
     )
-    (property "Footprint" "2024l1:led0603" (at 293.408 77.1051 0)
+    (property "Footprint" "2024l1:led0603" (at 298.556 66.457 0)
       (effects (font (size 1.27 1.27)) hide)
     )
-    (property "Datasheet" "~" (at 293.408 77.1051 0)
+    (property "Datasheet" "~" (at 298.556 66.457 0)
       (effects (font (size 1.27 1.27)) hide)
     )
@@
     )
   )
-  (symbol (lib_id "power:GND") (at 293.408 73.2951 180) (unit 1)
+  (symbol (lib_id "power:GND") (at 298.556 62.647 180) (unit 1)
     (in_bom yes) (on_board yes) (dnp no) (fields_autoplaced)
-    (property "Reference" "#PWR016" (at 293.408 66.9451 0)
+    (property "Reference" "#PWR016" (at 298.556 56.297 0)
       (effects (font (size 1.27 1.27)) hide)
     )
-    (property "Value" "GND" (at 293.408 69.7657 0)
+    (property "Value" "GND" (at 298.556 59.1176 0)
       (effects (font (size 1.27 1.27)))
     )
-    (property "Footprint" "" (at 293.408 73.2951 0)
+    (property "Footprint" "" (at 298.556 62.647 0)
       (effects (font (size 1.27 1.27)) hide)
     )
-    (property "Datasheet" "" (at 293.408 73.2951 0)
+    (property "Datasheet" "" (at 298.556 62.647 0)
       (effects (font (size 1.27 1.27)) hide)
     )

Commit message: L1 and Single - Flipped Connector
Connections:
- net L1 RX: now also J2.1 (Pin_1); no longer J2.3 (Pin_3)
- net L1 TX: now also J2.3 (Pin_3); no longer J2.1 (Pin_1)

Commit message: L1-Production files
Parts:
- removed D4: LED, 2024l1:led0603, symbol Device:LED
- removed SW1: SW_SPDT, 2024l1:SS12F21, symbol Switch:SW_SPDT
- C1, C5, C7: LCSC (none) -> C5128349
- C2: LCSC (none) -> C5355007
- C3, C4: LCSC (none) -> C1669545
- C6: LCSC (none) -> C59782
- C?: LCSC (none) -> C5463924
- D1, R1: LCSC (none) -> C2935896
- D10, D11, D12, D14, D15, D16, D17, D18, D19, D20, D3, D5, D6, D7, D8, D9: LCSC (none) -> C5440714
- D2: LCSC (none) -> C908682
- D?: LCSC (none) -> C179506
- IC1: LCSC (none) -> C1355343
- J1, J2: LCSC (none) -> C144394
- J?: LCSC (none) -> C108769
- L1: LCSC (none) -> C7461383
- Q? (x2): LCSC (none) -> C13678
- R10, R11, R12, R13, R14, R15, R16, R17, R18, R19, R20, R21, R22, R4, R8, R9: LCSC (none) -> C146233
- R2, R23: LCSC (none) -> C22994
- R24, R25: LCSC (none) -> C25804
- R27: LCSC (none) -> C21190
- R3: LCSC (none) -> C23082
- R6: LCSC (none) -> C22909
- R7: LCSC (none) -> C22843
- R?: LCSC (none) -> C22950
- RV1: LCSC (none) -> C124590
- U2: LCSC (none) -> C1545936
Connections:
- net +3V3: now also U1.14 (5V)

Commit message: L1- Production files and l3 routing
Parts:
- J3, J4: LCSC (none) -> C492410
Changed lines of the file:
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@@
+      (effects (font (size 1.27 1.27)) hide)
+    )
+    (property "LCSC" "C492410" (at 159.2298 63.2296 0)
       (effects (font (size 1.27 1.27)) hide)
     )
@@
       (effects (font (size 1.27 1.27)) hide)
     )
+    (property "LCSC" "C492410" (at 171.5915 51.8647 0)
+      (effects (font (size 1.27 1.27)) hide)
+    )

Commit message: fixed some traces
Connections:
- net S2: now also U1.5 (PA8_A4_D4_SDA); no longer U1.4 (PA11_A3_D3)
- net S3: now also U1.4 (PA11_A3_D3); no longer U1.3 (PA10_A2_D2)
- net Sol: now also U1.3 (PA10_A2_D2); no longer U1.2 (PA4_A1_D1)
- no-connect marks 1 -> 4
Changed lines of the file:
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@@
   (junction (at 61.109 205.9414) (diameter 0) (color 0 0 0 0)
   )
+  (no_connect (at 242.57 73.406))
+  (no_connect (at 284.48 81.026))
+  (no_connect (at 242.57 77.216))
   (no_connect (at 90.0377 99.1573))
   (wire (pts (xy 74.7977 83.9173) (xy 74.7977 91.5373))
@@
     (stroke (width 0) (type default))
   )
-  (wire (pts (xy 242.555 92.3432) (xy 232.395 92.3432))
+  (wire (pts (xy 242.57 92.456) (xy 232.41 92.456))
     (stroke (width 0) (type default))
   )
@@
     (stroke (width 0) (type default))
   )
+  (wire (pts (xy 242.57 88.646) (xy 232.41 88.646))
+    (stroke (width 0) (type default))
+  )
   (wire (pts (xy 291.3515 179.1428) (xy 291.3515 180.4128))
     (stroke (width 0) (type default))
@@
     (stroke (width 0) (type default))
   )
+  (wire (pts (xy 242.57 81.026) (xy 232.41 81.026))
+    (stroke (width 0) (type default))
+  )
   (wire (pts (xy 164.3098 58.0984) (xy 164.3098 60.6896))
     (stroke (width 0) (type default))
@@
     (stroke (width 0) (type default))
   )
-  (wire (pts (xy 242.555 84.7232) (xy 232.395 84.7232))
-    (stroke (width 0) (type default))
-  )
   (wire (pts (xy 197.8188 54.3563) (xy 184.297 54.3563))
     (stroke (width 0) (type default))
@@
     (stroke (width 0) (type default))
   )
-  (wire (pts (xy 294.625 88.5332) (xy 284.465 88.5332))
+  (wire (pts (xy 294.64 88.646) (xy 284.48 88.646))
     (stroke (width 0) (type default))
   )
@@
     (stroke (width 0) (type default))
   )
-  (wire (pts (xy 284.465 96.1532) (xy 290.8617 96.1532))
+  (wire (pts (xy 284.48 96.266) (xy 290.83 96.266))
     (stroke (width 0) (type default))
   )
@@
     (stroke (width 0) (type default))
   )
+  (wire (pts (xy 242.57 84.836) (xy 232.41 84.836))
+    (stroke (width 0) (type default))
+  )
   (polyline (pts (xy 12.0065 155.975) (xy 12.0065 155.9813))
     (stroke (width 0) (type default))
@@
     (stroke (width 0) (type default))
   )
-  (wire (pts (xy 294.625 84.7232) (xy 284.465 84.7232))
+  (wire (pts (xy 294.64 84.836) (xy 284.48 84.836))
     (stroke (width 0) (type default))
   )
@@
     (stroke (width 0) (type default))
   )
-  (wire (pts (xy 294.625 92.3432) (xy 284.465 92.3432))
+  (wire (pts (xy 294.64 92.456) (xy 284.48 92.456))
     (stroke (width 0) (type default))
   )
@@
     (stroke (width 0) (type default))
   )
-  (wire (pts (xy 242.555 80.9132) (xy 232.395 80.9132))
-    (stroke (width 0) (type default))
-  )
   (wire (pts (xy 291.3515 168.9828) (xy 281.1915 168.9828))
     (stroke (width 0) (type default))
@@
     (stroke (width 0) (type default))
   )
-  (wire (pts (xy 236.1583 96.1532) (xy 242.555 96.1532))
+  (wire (pts (xy 236.22 96.266) (xy 242.57 96.266))
     (stroke (width 0) (type default))
   )
@@
     (stroke (width 0) (type default))
   )
-  (wire (pts (xy 242.555 77.1032) (xy 232.395 77.1032))
-    (stroke (width 0) (type default))
-  )
   (wire (pts (xy 230.3915 171.5228) (xy 230.3915 168.9828))
     (stroke (width 0) (type default))
@@
     (effects (font (size 1.27 1.27)) (justify left bottom))
   )
-  (label "M1" (at 237.7597 92.3432 0) (fields_autoplaced)
+  (label "Sol" (at 237.49 81.026 0) (fields_autoplaced)
+    (effects (font (size 1.27 1.27)) (justify left bottom))
+  )
+  (label "M1" (at 237.744 92.456 0) (fields_autoplaced)
     (effects (font (size 1.27 1.27)) (justify left bottom))
   )
@@
     (effects (font (size 1.27 1.27)) (justify left bottom))
   )
-  (label "S1" (at 292.085 92.3432 180) (fields_autoplaced)
+  (label "S1" (at 292.1 92.456 180) (fields_autoplaced)
     (effects (font (size 1.27 1.27)) (justify right bottom))
   )
@@
     (effects (font (size 1.27 1.27)) (justify right bottom))
   )
-  (label "LG" (at 291.159 84.7232 0) (fields_autoplaced)
+  (label "LG" (at 291.084 84.836 0) (fields_autoplaced)
     (effects (font (size 1.27 1.27)) (justify left bottom))
   )
-  (label "L1 TX" (at 236.1583 96.1532 0) (fields_autoplaced)
+  (label "L1 TX" (at 236.22 96.266 0) (fields_autoplaced)
     (effects (font (size 1.27 1.27)) (justify left bottom))
   )
-  (label "Sol" (at 237.5505 77.1032 0) (fields_autoplaced)
-    (effects (font (size 1.27 1.27)) (justify left bottom))
-  )
-  (label "S2" (at 240.015 84.7232 180) (fields_autoplaced)
+  (label "S0" (at 67.1777 127.0973 270) (fields_autoplaced)
     (effects (font (size 1.27 1.27)) (justify right bottom))
   )
-  (label "S0" (at 67.1777 127.0973 270) (fields_autoplaced)
+  (label "S2" (at 240.03 88.646 180) (fields_autoplaced)
     (effects (font (size 1.27 1.27)) (justify right bottom))
   )
-  (label "S3" (at 240.015 80.9132 180) (fields_autoplaced)
+  (label "S3" (at 240.03 84.836 180) (fields_autoplaced)
     (effects (font (size 1.27 1.27)) (justify right bottom))
   )
-  (label "S0" (at 292.085 88.5332 180) (fields_autoplaced)
+  (label "S0" (at 292.1 88.646 180) (fields_autoplaced)
     (effects (font (size 1.27 1.27)) (justify right bottom))
   )
@@
     (effects (font (size 1.27 1.27)) (justify left bottom))
   )
-  (label "L1 RX" (at 284.465 96.1532 0) (fields_autoplaced)
+  (label "L1 RX" (at 284.48 96.266 0) (fields_autoplaced)
     (effects (font (size 1.27 1.27)) (justify left bottom))
   )
@@
     )
   )
-  (symbol (lib_id "power:GND") (at 270.495 61.8632 180) (unit 1)
+  (symbol (lib_id "power:GND") (at 270.51 61.976 180) (unit 1)
     (in_bom yes) (on_board yes) (dnp no) (fields_autoplaced)
-    (property "Reference" "#PWR013" (at 270.495 55.5132 0)
+    (property "Reference" "#PWR013" (at 270.51 55.626 0)
       (effects (font (size 1.27 1.27)) hide)
     )
-    (property "Value" "GND" (at 270.495 58.419 0)
+    (property "Value" "GND" (at 270.51 58.5318 0)
       (effects (font (size 1.27 1.27)))
     )
-    (property "Footprint" "" (at 270.495 61.8632 0)
+    (property "Footprint" "" (at 270.51 61.976 0)
       (effects (font (size 1.27 1.27)) hide)
     )
-    (property "Datasheet" "" (at 270.495 61.8632 0)
+    (property "Datasheet" "" (at 270.51 61.976 0)
       (effects (font (size 1.27 1.27)) hide)
     )
@@
     )
   )
-  (symbol (lib_id "power:GND") (at 266.685 106.3132 0) (unit 1)
+  (symbol (lib_id "power:GND") (at 266.7 106.426 0) (unit 1)
     (in_bom yes) (on_board yes) (dnp no) (fields_autoplaced)
-    (property "Reference" "#PWR020" (at 266.685 112.6632 0)
+    (property "Reference" "#PWR020" (at 266.7 112.776 0)
       (effects (font (size 1.27 1.27)) hide)
     )
-    (property "Value" "GND" (at 266.685 111.76 0)
+    (property "Value" "GND" (at 266.7 111.8728 0)
       (effects (font (size 1.27 1.27)))
     )
-    (property "Footprint" "" (at 266.685 106.3132 0)
+    (property "Footprint" "" (at 266.7 106.426 0)
       (effects (font (size 1.27 1.27)) hide)
     )
-    (property "Datasheet" "" (at 266.685 106.3132 0)
+    (property "Datasheet" "" (at 266.7 106.426 0)
       (effects (font (size 1.27 1.27)) hide)
     )
@@
     )
   )
-  (symbol (lib_id "power:+3V3") (at 284.465 73.2932 270) (unit 1)
+  (symbol (lib_id "power:+3V3") (at 284.48 73.406 270) (unit 1)
     (in_bom yes) (on_board yes) (dnp no) (fields_autoplaced)
-    (property "Reference" "#PWR016" (at 280.655 73.2932 0)
+    (property "Reference" "#PWR016" (at 280.67 73.406 0)
       (effects (font (size 1.27 1.27)) hide)
     )
-    (property "Value" "+3V3" (at 288.351 73.9282 90)
+    (property "Value" "+3V3" (at 288.366 74.041 90)
       (effects (font (size 1.27 1.27)) (justify left))
     )
-    (property "Footprint" "" (at 284.465 73.2932 0)
+    (property "Footprint" "" (at 284.48 73.406 0)
       (effects (font (size 1.27 1.27)) hide)
     )
-    (property "Datasheet" "" (at 284.465 73.2932 0)
+    (property "Datasheet" "" (at 284.48 73.406 0)
       (effects (font (size 1.27 1.27)) hide)
     )
@@
     )
   )
-  (symbol (lib_id "power:GND") (at 284.465 77.1032 90) (unit 1)
+  (symbol (lib_id "power:GND") (at 284.48 77.216 90) (unit 1)
     (in_bom yes) (on_board yes) (dnp no) (fields_autoplaced)
-    (property "Reference" "#PWR017" (at 290.815 77.1032 0)
+    (property "Reference" "#PWR017" (at 290.83 77.216 0)
       (effects (font (size 1.27 1.27)) hide)
     )
-    (property "Value" "GND" (at 287.6716 77.7382 90)
+    (property "Value" "GND" (at 287.6866 77.851 90)
       (effects (font (size 1.27 1.27)) (justify right))
     )
-    (property "Footprint" "" (at 284.465 77.1032 0)
+    (property "Footprint" "" (at 284.48 77.216 0)
       (effects (font (size 1.27 1.27)) hide)
     )
-    (property "Datasheet" "" (at 284.465 77.1032 0)
+    (property "Datasheet" "" (at 284.48 77.216 0)
       (effects (font (size 1.27 1.27)) hide)
     )
@@
     )
   )
-  (symbol (lib_id "Seeed_Studio_XIAO_Series:Seeed Studio XIAO SAMD21") (at 264.145 84.7232 0) (unit 1)
+  (symbol (lib_id "Seeed_Studio_XIAO_Series:Seeed Studio XIAO SAMD21") (at 264.16 84.836 0) (unit 1)
     (in_bom yes) (on_board yes) (dnp no) (fields_autoplaced)
-    (property "Reference" "U1" (at 268.6409 106.68 0)
+    (property "Reference" "U1" (at 268.6559 106.7928 0)
       (effects (font (size 1.27 1.27)) (justify left))
     )
-    (property "Value" "Seeed Studio XIAO SAMD21" (at 268.6409 109.22 0)
+    (property "Value" "Seeed Studio XIAO SAMD21" (at 268.6559 109.3328 0)
       (effects (font (size 1.27 1.27)) (justify left))
     )
-    (property "Footprint" "2024l1:Seeeduino XIAO SAMD 21 TFT" (at 255.255 79.6432 0)
+    (property "Footprint" "2024l1:Seeeduino XIAO SAMD 21 TFT" (at 255.27 79.756 0)
       (effects (font (size 1.27 1.27)) hide)
     )
-    (property "Datasheet" "" (at 255.255 79.6432 0)
+    (property "Datasheet" "" (at 255.27 79.756 0)
       (effects (font (size 1.27 1.27)) hide)
     )
