File: open/2024l1  (Single Mux)/2024l1 Single.kicad_sch (KiCad schematic)
At the start: 90 parts, among them IC1 LM2587S-ADJ, J1 Conn_01x03, J2 Conn_01x03, J3 Conn_01x02, J4 Conn_01x02, J6 Conn_01x04, U1 Seeed Studio XIAO SAMD21, U2 CD74HC4067SM

Commit message: L1- Added QR code
Parts:
- D10, D11, D12, D14, D15, D16, D17, D18, D19, D20, D3, D5, D6, D7, D8, D9: footprint 2024l1:LED5050 -> 2024l1:C2843867
- R10, R11, R12, R13, R14, R15, R16, R17, R18, R19, R20, R21, R22, R4, R8, R9: footprint 2024l1:ALS-PT19 -> 2024l1:C146233
Changed lines of the file:
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@@
       (effects (font (size 1.27 1.27)) (justify left))
     )
-    (property "Footprint" "2024l1:ALS-PT19" (at 86.2277 101.6973 90)
+    (property "Footprint" "2024l1:C146233" (at 86.2277 101.6973 90)
       (effects (font (size 1.27 1.27)) (justify left) hide)
     )
@@
       (effects (font (size 1.27 1.27)) (justify left))
     )
-    (property "Footprint" "2024l1:ALS-PT19" (at 185.567 56.7255 90)
+    (property "Footprint" "2024l1:C146233" (at 185.567 56.7255 90)
       (effects (font (size 1.27 1.27)) (justify left) hide)
     )
@@
       (effects (font (size 1.27 1.27)) (justify left))
     )
-    (property "Footprint" "2024l1:ALS-PT19" (at 68.4477 101.6973 90)
+    (property "Footprint" "2024l1:C146233" (at 68.4477 101.6973 90)
       (effects (font (size 1.27 1.27)) (justify left) hide)
     )
@@
       (effects (font (size 1.27 1.27)) (justify left))
     )
-    (property "Footprint" "2024l1:ALS-PT19" (at 81.1477 101.6973 90)
+    (property "Footprint" "2024l1:C146233" (at 81.1477 101.6973 90)
       (effects (font (size 1.27 1.27)) (justify left) hide)
     )
@@
       (effects (font (size 1.27 1.27)) (justify right))
     )
-    (property "Footprint" "2024l1:LED5050" (at 260.8715 188.0328 0)
+    (property "Footprint" "2024l1:C2843867" (at 260.8715 188.0328 0)
       (effects (font (size 1.27 1.27)) hide)
     )
@@
       (effects (font (size 1.27 1.27)) (justify right))
     )
-    (property "Footprint" "2024l1:LED5050" (at 230.3915 175.3328 0)
+    (property "Footprint" "2024l1:C2843867" (at 230.3915 175.3328 0)
       (effects (font (size 1.27 1.27)) hide)
     )
@@
       (effects (font (size 1.27 1.27)) (justify right))
     )
-    (property "Footprint" "2024l1:LED5050" (at 240.5515 188.0328 0)
+    (property "Footprint" "2024l1:C2843867" (at 240.5515 188.0328 0)
       (effects (font (size 1.27 1.27)) hide)
     )
@@
       (effects (font (size 1.27 1.27)) (justify left))
     )
-    (property "Footprint" "2024l1:ALS-PT19" (at 58.2877 101.6973 90)
+    (property "Footprint" "2024l1:C146233" (at 58.2877 101.6973 90)
       (effects (font (size 1.27 1.27)) (justify left) hide)
     )
@@
       (effects (font (size 1.27 1.27)) (justify left))
     )
-    (property "Footprint" "2024l1:ALS-PT19" (at 70.9877 101.6973 90)
+    (property "Footprint" "2024l1:C146233" (at 70.9877 101.6973 90)
       (effects (font (size 1.27 1.27)) (justify left) hide)
     )
@@
       (effects (font (size 1.27 1.27)) (justify right) hide)
     )
-    (property "Footprint" "2024l1:LED5050" (at 170.6396 62.0739 0)
+    (property "Footprint" "2024l1:C2843867" (at 170.6396 62.0739 0)
       (effects (font (size 1.27 1.27)) hide)
     )
@@
       (effects (font (size 1.27 1.27)) (justify left))
     )
-    (property "Footprint" "2024l1:ALS-PT19" (at 76.0677 101.6973 90)
+    (property "Footprint" "2024l1:C146233" (at 76.0677 101.6973 90)
       (effects (font (size 1.27 1.27)) (justify left) hide)
     )
@@
       (effects (font (size 1.27 1.27)) (justify right))
     )
-    (property "Footprint" "2024l1:LED5050" (at 230.3915 188.0328 0)
+    (property "Footprint" "2024l1:C2843867" (at 230.3915 188.0328 0)
       (effects (font (size 1.27 1.27)) hide)
     )
@@
       (effects (font (size 1.27 1.27)) (justify right))
     )
-    (property "Footprint" "2024l1:LED5050" (at 281.1915 188.0328 0)
+    (property "Footprint" "2024l1:C2843867" (at 281.1915 188.0328 0)
       (effects (font (size 1.27 1.27)) hide)
     )
@@
       (effects (font (size 1.27 1.27)) (justify left))
     )
-    (property "Footprint" "2024l1:ALS-PT19" (at 60.8277 101.6973 90)
+    (property "Footprint" "2024l1:C146233" (at 60.8277 101.6973 90)
       (effects (font (size 1.27 1.27)) (justify left) hide)
     )
@@
       (effects (font (size 1.27 1.27)) (justify left))
     )
-    (property "Footprint" "2024l1:ALS-PT19" (at 78.6077 101.6973 90)
+    (property "Footprint" "2024l1:C146233" (at 78.6077 101.6973 90)
       (effects (font (size 1.27 1.27)) (justify left) hide)
     )
@@
       (effects (font (size 1.27 1.27)) (justify right))
     )
-    (property "Footprint" "2024l1:LED5050" (at 260.8715 175.3328 0)
+    (property "Footprint" "2024l1:C2843867" (at 260.8715 175.3328 0)
       (effects (font (size 1.27 1.27)) hide)
     )
@@
       (effects (font (size 1.27 1.27)) (justify right))
     )
-    (property "Footprint" "2024l1:LED5050" (at 250.7115 175.3328 0)
+    (property "Footprint" "2024l1:C2843867" (at 250.7115 175.3328 0)
       (effects (font (size 1.27 1.27)) hide)
     )
@@
       (effects (font (size 1.27 1.27)) (justify right))
     )
-    (property "Footprint" "2024l1:LED5050" (at 271.0315 188.0328 0)
+    (property "Footprint" "2024l1:C2843867" (at 271.0315 188.0328 0)
       (effects (font (size 1.27 1.27)) hide)
     )
@@
       (effects (font (size 1.27 1.27)) (justify right))
     )
-    (property "Footprint" "2024l1:LED5050" (at 291.3515 188.0328 0)
+    (property "Footprint" "2024l1:C2843867" (at 291.3515 188.0328 0)
       (effects (font (size 1.27 1.27)) hide)
     )
@@
       (effects (font (size 1.27 1.27)) (justify left))
     )
-    (property "Footprint" "2024l1:ALS-PT19" (at 63.3677 101.6973 90)
+    (property "Footprint" "2024l1:C146233" (at 63.3677 101.6973 90)
       (effects (font (size 1.27 1.27)) (justify left) hide)
     )
@@
       (effects (font (size 1.27 1.27)) (justify left) hide)
     )
-    (property "Footprint" "2024l1:ALS-PT19" (at 73.5277 101.6973 90)
+    (property "Footprint" "2024l1:C146233" (at 73.5277 101.6973 90)
       (effects (font (size 1.27 1.27)) (justify left) hide)
     )
@@
       (effects (font (size 1.27 1.27)) (justify right))
     )
-    (property "Footprint" "2024l1:LED5050" (at 291.3515 175.3328 0)
+    (property "Footprint" "2024l1:C2843867" (at 291.3515 175.3328 0)
       (effects (font (size 1.27 1.27)) hide)
     )
@@
       (effects (font (size 1.27 1.27)) (justify right))
     )
-    (property "Footprint" "2024l1:LED5050" (at 271.0315 175.3328 0)
+    (property "Footprint" "2024l1:C2843867" (at 271.0315 175.3328 0)
       (effects (font (size 1.27 1.27)) hide)
     )
@@
       (effects (font (size 1.27 1.27)) (justify left))
     )
-    (property "Footprint" "2024l1:ALS-PT19" (at 83.6877 101.6973 90)
+    (property "Footprint" "2024l1:C146233" (at 83.6877 101.6973 90)
       (effects (font (size 1.27 1.27)) (justify left) hide)
     )
@@
       (effects (font (size 1.27 1.27)) (justify right))
     )
-    (property "Footprint" "2024l1:LED5050" (at 281.1915 175.3328 0)
+    (property "Footprint" "2024l1:C2843867" (at 281.1915 175.3328 0)
       (effects (font (size 1.27 1.27)) hide)
     )
@@
       (effects (font (size 1.27 1.27)) (justify right))
     )
-    (property "Footprint" "2024l1:LED5050" (at 250.7115 188.0328 0)
+    (property "Footprint" "2024l1:C2843867" (at 250.7115 188.0328 0)
       (effects (font (size 1.27 1.27)) hide)
     )
@@
       (effects (font (size 1.27 1.27)) (justify left))
     )
-    (property "Footprint" "2024l1:ALS-PT19" (at 88.7677 101.6973 90)
+    (property "Footprint" "2024l1:C146233" (at 88.7677 101.6973 90)
       (effects (font (size 1.27 1.27)) (justify left) hide)
     )
@@
       (effects (font (size 1.27 1.27)) (justify left))
     )
-    (property "Footprint" "2024l1:ALS-PT19" (at 65.9077 101.6973 90)
+    (property "Footprint" "2024l1:C146233" (at 65.9077 101.6973 90)
       (effects (font (size 1.27 1.27)) (justify left) hide)
     )
@@
       (effects (font (size 1.27 1.27)) (justify left))
     )
-    (property "Footprint" "2024l1:ALS-PT19" (at 55.7477 101.6973 90)
+    (property "Footprint" "2024l1:C146233" (at 55.7477 101.6973 90)
       (effects (font (size 1.27 1.27)) (justify left) hide)
     )
@@
       (effects (font (size 1.27 1.27)) (justify left))
     )
-    (property "Footprint" "2024l1:ALS-PT19" (at 53.2077 101.6973 90)
+    (property "Footprint" "2024l1:C146233" (at 53.2077 101.6973 90)
       (effects (font (size 1.27 1.27)) (justify left) hide)
     )
@@
       (effects (font (size 1.27 1.27)) (justify right))
     )
-    (property "Footprint" "2024l1:LED5050" (at 301.5115 175.3328 0)
+    (property "Footprint" "2024l1:C2843867" (at 301.5115 175.3328 0)
       (effects (font (size 1.27 1.27)) hide)
     )
@@
       (effects (font (size 1.27 1.27)) (justify right))
     )
-    (property "Footprint" "2024l1:LED5050" (at 240.5515 175.3328 0)
-      (effects (font (size 1.27 1.27)) hide)
-    )
+    (property "Footprint" "2024l1:C2843867" (at 240.5515 175.3328 0)
+      (effects (font (size 1.27 1.27)) hide)
+    )
