File: open/2024l1-single/2024l1-single.kicad_pcb (KiCad board)
At the start: 2 copper layers, 176 x 169.5 mm, 100 parts, among them IC1 LM2587S-ADJ, J1 Conn_01x03, J2 Conn_01x03, J3 Conn_01x02, J4 Conn_01x02, J5 XT30, J6 Conn_01x04, Q1 STP75NF75, Q2 STP75NF75, U1 Seeed Studio XIAO SAMD21, U2 CD74HC4067SM

Commit message: Connector movements
Parts:
- moved J1 0.20 mm to (75.6, 48.8)

Commit message: reformatted
Parts:
- removed MTH17, MTH18, MTH19, MTH20: MountingHole_Pad, MountingHole:MountingHole_3.2mm_M3_Pad_Via
- R27: moved to B.Cu
- moved R27 95.6 mm to (182.2, 107.5), turned to -90 degrees
Routing:
- net Net-(U2-I3): track 74.8 -> 56.1 mm
- net /Sol: track 163.1 -> 161.3 mm
- net GND: vias 173 -> 167

Commit message: L1 Minor adjust and l2 still need to add stitching vias
Routing:
- net /S3: track 67.4 -> 66.8 mm
Changed lines of the file:
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@@
   )
   (footprint "Connector_JST:JST_XH_B3B-XH-A_1x03_P2.50mm_Vertical" (layer "F.Cu")
-    (at 159.495 114.76 90)
+    (at 159.5 114.75 90)
     (descr "JST XH series connector, B3B-XH-A (http://www.jst-mfg.com/product/pdf/eng/eXH.pdf), generated with kicad-footprint-generator")
     (tags "connector JST XH vertical")
@@
   (segment (start 114.495 107.6) (end 114.485 107.61) (width 0.3) (layer "F.Cu") (net 44))
   (via (at 127.5 107.6) (size 0.8) (drill 0.4) (layers "F.Cu" "B.Cu") (net 44))
-  (segment (start 128.46 108.56) (end 127.5 107.6) (width 0.3) (layer "B.Cu") (net 44))
-  (segment (start 179.7 104.1675) (end 175.3075 108.56) (width 0.3) (layer "B.Cu") (net 44))
-  (segment (start 175.3075 108.56) (end 128.46 108.56) (width 0.3) (layer "B.Cu") (net 44))
-  (segment (start 113.215 106.405) (end 113.215 107.61) (width 0.3) (layer "F.Cu") (net 45))
-  (segment (start 114.19 105.43) (end 113.215 106.405) (width 0.3) (layer "F.Cu") (net 45))
-  (segment (start 143.9 106.65) (end 142.68 105.43) (width 0.3) (layer "F.Cu") (net 45))
+  (segment (start 127.75 107.85) (end 127.5 107.6) (width 0.3) (layer "B.Cu") (net 44))
+  (segment (start 176.0175 107.85) (end 127.75 107.85) (width 0.3) (layer "B.Cu") (net 44))
+  (segment (start 179.7 104.1675) (end 176.0175 107.85) (width 0.3) (layer "B.Cu") (net 44))
   (segment (start 142.68 105.43) (end 114.19 105.43) (width 0.3) (layer "F.Cu") (net 45))
-  (via (at 143.9 106.65) (size 0.8) (drill 0.4) (layers "F.Cu" "B.Cu") (net 45))
-  (segment (start 174.0775 107.25) (end 173.3 107.25) (width 0.3) (layer "B.Cu") (net 45))
-  (segment (start 143.9 106.65) (end 144.5 107.25) (width 0.3) (layer "B.Cu") (net 45))
-  (segment (start 144.5 107.25) (end 173.3 107.25) (width 0.3) (layer "B.Cu") (net 45))
-  (segment (start 177.16 104.1675) (end 174.0775 107.25) (width 0.3) (layer "B.Cu") (net 45))
+  (segment (start 143.6 106.35) (end 142.68 105.43) (width 0.3) (layer "F.Cu") (net 45))
+  (segment (start 114.19 105.43) (end 113.215 106.405) (width 0.3) (layer "F.Cu") (net 45))
+  (segment (start 113.215 106.405) (end 113.215 107.61) (width 0.3) (layer "F.Cu") (net 45))
+  (via (at 143.6 106.35) (size 0.8) (drill 0.4) (layers "F.Cu" "B.Cu") (net 45))
+  (segment (start 174.1075 107.22) (end 177.16 104.1675) (width 0.3) (layer "B.Cu") (net 45))
+  (segment (start 143.6 106.35) (end 144.47 107.22) (width 0.3) (layer "B.Cu") (net 45))
+  (segment (start 144.47 107.22) (end 174.1075 107.22) (width 0.3) (layer "B.Cu") (net 45))
   (segment (start 169.5925 120.3325) (end 172.08 120.3325) (width 0.3) (layer "F.Cu") (net 46))
   (segment (start 159.495 114.76) (end 164.02 114.76) (width 0.3) (layer "F.Cu") (net 46))

Commit message: Restored L1 Footprint Library
Parts:
- C1, C5, C6, C7, C8: footprint 2024l1:cap0603 -> 2024l1 Single:cap0603
- D10: renamed from D11; footprint 2024l1:C2843867 -> 2024l1 Single:C2843867
- D11: renamed from D12; footprint 2024l1:C2843867 -> 2024l1 Single:C2843867
- D13: renamed from D14; footprint 2024l1:C2843867 -> 2024l1 Single:C2843867
- D14: renamed from D15; footprint 2024l1:C2843867 -> 2024l1 Single:C2843867
- D15: renamed from D16; footprint 2024l1:C2843867 -> 2024l1 Single:C2843867
- D16: renamed from D17; footprint 2024l1:C2843867 -> 2024l1 Single:C2843867
- D17: renamed from D18; footprint 2024l1:C2843867 -> 2024l1 Single:C2843867
- D18: renamed from D19; footprint 2024l1:C2843867 -> 2024l1 Single:C2843867
- D19: renamed from D20; footprint 2024l1:C2843867 -> 2024l1 Single:C2843867
- D2: footprint 2024l1:SMA (DO-214AC) -> 2024l1 Single:SMA (DO-214AC)
- D3: footprint 2024l1:C2843867 -> 2024l1 Single:C2843867
- D4: renamed from D5; footprint 2024l1:C2843867 -> 2024l1 Single:C2843867
- D5: renamed from D6; footprint 2024l1:C2843867 -> 2024l1 Single:C2843867
- D6: renamed from D7; footprint 2024l1:C2843867 -> 2024l1 Single:C2843867
- D7: renamed from D8; footprint 2024l1:C2843867 -> 2024l1 Single:C2843867
- D8: renamed from D9; footprint 2024l1:C2843867 -> 2024l1 Single:C2843867
- D9: renamed from D10; footprint 2024l1:C2843867 -> 2024l1 Single:C2843867
- H1: footprint 2024l1:SEN Logo Mini -> 2024l1 Single:SEN Logo Mini
- IC1: footprint 2024l1:TO170P1435X465-6N -> 2024l1 Single:TO170P1435X465-6N
- J5: footprint 2024l1:AMASS_XT30-F -> 2024l1 Single:AMASS_XT30-F
- J6: footprint 2024l1:14 AWG 4 Holes -> 2024l1 Single:14 AWG 4 Holes
- L1: footprint 2024l1:1040 One Piece Inductor -> 2024l1 Single:1040 One Piece Inductor
- Q1: footprint 2024l1:TO255P1040X460X2890-3 -> 2024l1 Single:TO255P1040X460X2890-3
- Q2: value STP75NF75 -> IRLML6344TRPBF; footprint 2024l1:TO255P1040X460X2890-3 -> 2024l1 Single:SOT95P237X112-3N
- R10: renamed from R8; footprint 2024l1:C146233 -> 2024l1 Single:C146233
- R11: renamed from R22; footprint 2024l1:C146233 -> 2024l1 Single:C146233
- R12: renamed from R21; footprint 2024l1:C146233 -> 2024l1 Single:C146233
- R13: renamed from R20; footprint 2024l1:C146233 -> 2024l1 Single:C146233
- R14: renamed from R19; footprint 2024l1:C146233 -> 2024l1 Single:C146233
- R15: renamed from R18; footprint 2024l1:C146233 -> 2024l1 Single:C146233
- R16: renamed from R17; footprint 2024l1:C146233 -> 2024l1 Single:C146233
- R17: renamed from R16; footprint 2024l1:C146233 -> 2024l1 Single:C146233
- R18: renamed from R15; footprint 2024l1:C146233 -> 2024l1 Single:C146233
- R19: renamed from R14; footprint 2024l1:C146233 -> 2024l1 Single:C146233
- R2: renamed from R3; footprint 2024l1:res0603 -> 2024l1 Single:res0603
- R20: renamed from R13; footprint 2024l1:C146233 -> 2024l1 Single:C146233
- R21: renamed from R12; footprint 2024l1:C146233 -> 2024l1 Single:C146233
- R22: renamed from R23; footprint 2024l1:res0603 -> 2024l1 Single:res0603
- R23: renamed from R24; footprint 2024l1:res0603 -> 2024l1 Single:res0603
- R24: renamed from R25; footprint 2024l1:res0603 -> 2024l1 Single:res0603
- R25: renamed from R26; footprint 2024l1:res0603 -> 2024l1 Single:res0603
- R26: renamed from R27; footprint 2024l1:res0603 -> 2024l1 Single:res0603
- R3: renamed from R6; footprint 2024l1:res0603 -> 2024l1 Single:res0603
- R4, R9: footprint 2024l1:C146233 -> 2024l1 Single:C146233
- R5: footprint 2024l1:Through Hole LDR -> 2024l1 Single:Through Hole LDR
- R6: renamed from R7; footprint 2024l1:res0603 -> 2024l1 Single:res0603
- R7: renamed from R11; footprint 2024l1:C146233 -> 2024l1 Single:C146233
- R8: renamed from R10; footprint 2024l1:C146233 -> 2024l1 Single:C146233
- RV1: footprint 2024l1:TRIM_3362W-1-203LF -> 2024l1 Single:TRIM_3362W-1-203LF
- U1: footprint 2024l1:Seeeduino XIAO SAMD 21 TFT -> 2024l1 Single:Seeeduino XIAO SAMD 21 TFT
- U2: footprint 2024l1:CD74HC4067M -> 2024l1 Single:CD74HC4067M
- moved Q2 2.55 mm to (107.5, 57.5), turned to 90 degrees
- renumbered D13 to D12
Routing:
- net Net-(Q1-S): track 30.4 -> 29.7 mm, vias 0 -> 1
- net /Sol: track 161.3 -> 161.8 mm
- net Net-(U2-I7): track 62.3 -> 61.8 mm

Commit message: L3 - SCH
Parts:
- C2: footprint Capacitor_SMD:CP_Elec_10x10.5 -> Capacitor_SMD:CP_Elec_8x10.5
Routing:
- net GND: vias 167 -> 163
Changed lines of the file:
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@@
     )
   )
-  (footprint "Capacitor_SMD:CP_Elec_10x10.5" (layer "F.Cu")
+  (footprint "Capacitor_SMD:CP_Elec_8x10.5" (layer "F.Cu")
     (at 87.5875 41.65 -90)
-    (descr "SMD capacitor, aluminum electrolytic, Vishay 1010, 10.0x10.5mm, http://www.vishay.com/docs/28395/150crz.pdf")
+    (descr "SMD capacitor, aluminum electrolytic, Vishay 0810, 8.0x10.5mm, http://www.vishay.com/docs/28395/150crz.pdf")
     (tags "capacitor electrolytic")
     (property "LCSC" "C5355007")
@@
     (property "ki_keywords" "cap capacitor")
     (attr smd)
-    (fp_text reference "C2" (at 0 -6.3 90) (layer "F.SilkS") hide
+    (fp_text reference "C2" (at 0 -5.3 -90) (layer "F.SilkS") hide
         (effects (font (size 1 1) (thickness 0.15)))
     )
-    (fp_text value "100u" (at 0 0 90) (layer "F.Fab")
+    (fp_text value "100u" (at 0 5.3 -90) (layer "F.Fab")
         (effects (font (size 1 1) (thickness 0.15)))
     )
-    (fp_text user "${REFERENCE}" (at 0 0 90) (layer "F.Fab")
+    (fp_text user "${REFERENCE}" (at 0 0 -90) (layer "F.Fab")
         (effects (font (size 1 1) (thickness 0.15)))
     )
-    (fp_line (start -6.85 -2.76) (end -5.6 -2.76)
+    (fp_line (start -5.6 -2.51) (end -4.6 -2.51)
       (stroke (width 0.12) (type solid)) (layer "F.SilkS"))
-    (fp_line (start -6.225 -3.385) (end -6.225 -2.135)
+    (fp_line (start -5.1 -3.01) (end -5.1 -2.01)
       (stroke (width 0.12) (type solid)) (layer "F.SilkS"))
-    (fp_line (start -5.36 -4.295563) (end -5.36 -1.51)
+    (fp_line (start -4.36 -3.295563) (end -4.36 -1.51)
       (stroke (width 0.12) (type solid)) (layer "F.SilkS"))
-    (fp_line (start -5.36 -4.295563) (end -4.295563 -5.36)
+    (fp_line (start -4.36 -3.295563) (end -3.295563 -4.36)
       (stroke (width 0.12) (type solid)) (layer "F.SilkS"))
-    (fp_line (start -5.36 4.295563) (end -5.36 1.51)
+    (fp_line (start -4.36 3.295563) (end -4.36 1.51)
       (stroke (width 0.12) (type solid)) (layer "F.SilkS"))
-    (fp_line (start -5.36 4.295563) (end -4.295563 5.36)
+    (fp_line (start -4.36 3.295563) (end -3.295563 4.36)
       (stroke (width 0.12) (type solid)) (layer "F.SilkS"))
-    (fp_line (start -4.295563 -5.36) (end 5.36 -5.36)
+    (fp_line (start -3.295563 -4.36) (end 4.36 -4.36)
       (stroke (width 0.12) (type solid)) (layer "F.SilkS"))
-    (fp_line (start -4.295563 5.36) (end 5.36 5.36)
+    (fp_line (start -3.295563 4.36) (end 4.36 4.36)
       (stroke (width 0.12) (type solid)) (layer "F.SilkS"))
-    (fp_line (start 5.36 -5.36) (end 5.36 -1.51)
+    (fp_line (start 4.36 -4.36) (end 4.36 -1.51)
       (stroke (width 0.12) (type solid)) (layer "F.SilkS"))
-    (fp_line (start 5.36 5.36) (end 5.36 1.51)
+    (fp_line (start 4.36 4.36) (end 4.36 1.51)
       (stroke (width 0.12) (type solid)) (layer "F.SilkS"))
-    (fp_line (start -6.65 -1.5) (end -6.65 1.5)
+    (fp_line (start -6.15 -1.5) (end -6.15 1.5)
       (stroke (width 0.05) (type solid)) (layer "F.CrtYd"))
-    (fp_line (start -6.65 1.5) (end -5.5 1.5)
+    (fp_line (start -6.15 1.5) (end -4.5 1.5)
       (stroke (width 0.05) (type solid)) (layer "F.CrtYd"))
-    (fp_line (start -5.5 -4.35) (end -5.5 -1.5)
+    (fp_line (start -4.5 -3.35) (end -4.5 -1.5)
       (stroke (width 0.05) (type solid)) (layer "F.CrtYd"))
-    (fp_line (start -5.5 -4.35) (end -4.35 -5.5)
+    (fp_line (start -4.5 -3.35) (end -3.35 -4.5)
       (stroke (width 0.05) (type solid)) (layer "F.CrtYd"))
-    (fp_line (start -5.5 -1.5) (end -6.65 -1.5)
+    (fp_line (start -4.5 -1.5) (end -6.15 -1.5)
       (stroke (width 0.05) (type solid)) (layer "F.CrtYd"))
-    (fp_line (start -5.5 1.5) (end -5.5 4.35)
+    (fp_line (start -4.5 1.5) (end -4.5 3.35)
       (stroke (width 0.05) (type solid)) (layer "F.CrtYd"))
-    (fp_line (start -5.5 4.35) (end -4.35 5.5)
+    (fp_line (start -4.5 3.35) (end -3.35 4.5)
       (stroke (width 0.05) (type solid)) (layer "F.CrtYd"))
-    (fp_line (start -4.35 -5.5) (end 5.5 -5.5)
+    (fp_line (start -3.35 -4.5) (end 4.5 -4.5)
       (stroke (width 0.05) (type solid)) (layer "F.CrtYd"))
-    (fp_line (start -4.35 5.5) (end 5.5 5.5)
+    (fp_line (start -3.35 4.5) (end 4.5 4.5)
       (stroke (width 0.05) (type solid)) (layer "F.CrtYd"))
-    (fp_line (start 5.5 -5.5) (end 5.5 -1.5)
+    (fp_line (start 4.5 -4.5) (end 4.5 -1.5)
       (stroke (width 0.05) (type solid)) (layer "F.CrtYd"))
-    (fp_line (start 5.5 -1.5) (end 6.65 -1.5)
+    (fp_line (start 4.5 -1.5) (end 6.15 -1.5)
       (stroke (width 0.05) (type solid)) (layer "F.CrtYd"))
-    (fp_line (start 5.5 1.5) (end 5.5 5.5)
+    (fp_line (start 4.5 1.5) (end 4.5 4.5)
       (stroke (width 0.05) (type solid)) (layer "F.CrtYd"))
-    (fp_line (start 6.65 -1.5) (end 6.65 1.5)
+    (fp_line (start 6.15 -1.5) (end 6.15 1.5)
       (stroke (width 0.05) (type solid)) (layer "F.CrtYd"))
-    (fp_line (start 6.65 1.5) (end 5.5 1.5)
+    (fp_line (start 6.15 1.5) (end 4.5 1.5)
       (stroke (width 0.05) (type solid)) (layer "F.CrtYd"))
-    (fp_line (start -5.25 -4.25) (end -5.25 4.25)
+    (fp_line (start -4.25 -3.25) (end -4.25 3.25)
       (stroke (width 0.1) (type solid)) (layer "F.Fab"))
-    (fp_line (start -5.25 -4.25) (end -4.25 -5.25)
+    (fp_line (start -4.25 -3.25) (end -3.25 -4.25)
       (stroke (width 0.1) (type solid)) (layer "F.Fab"))
-    (fp_line (start -5.25 4.25) (end -4.25 5.25)
+    (fp_line (start -4.25 3.25) (end -3.25 4.25)
       (stroke (width 0.1) (type solid)) (layer "F.Fab"))
-    (fp_line (start -4.558325 -1.7) (end -3.558325 -1.7)
+    (fp_line (start -3.562278 -1.5) (end -2.762278 -1.5)
       (stroke (width 0.1) (type solid)) (layer "F.Fab"))
-    (fp_line (start -4.25 -5.25) (end 5.25 -5.25)
+    (fp_line (start -3.25 -4.25) (end 4.25 -4.25)
       (stroke (width 0.1) (type solid)) (layer "F.Fab"))
-    (fp_line (start -4.25 5.25) (end 5.25 5.25)
+    (fp_line (start -3.25 4.25) (end 4.25 4.25)
       (stroke (width 0.1) (type solid)) (layer "F.Fab"))
-    (fp_line (start -4.058325 -2.2) (end -4.058325 -1.2)
+    (fp_line (start -3.162278 -1.9) (end -3.162278 -1.1)
       (stroke (width 0.1) (type solid)) (layer "F.Fab"))
-    (fp_line (start 5.25 -5.25) (end 5.25 5.25)
+    (fp_line (start 4.25 -4.25) (end 4.25 4.25)
       (stroke (width 0.1) (type solid)) (layer "F.Fab"))
-    (fp_circle (center 0 0) (end 5 0)
+    (fp_circle (center 0 0) (end 4 0)
       (stroke (width 0.1) (type solid)) (fill none) (layer "F.Fab"))
-    (pad "1" smd roundrect (at -4.2 0 270) (size 4.4 2.5) (layers "F.Cu" "F.Paste" "F.Mask") (roundrect_rratio 0.1)
+    (pad "1" smd roundrect (at -3.7 0 270) (size 4.4 2.5) (layers "F.Cu" "F.Paste" "F.Mask") (roundrect_rratio 0.1)
       (net 38 "+12V") (pintype "passive"))
-    (pad "2" smd roundrect (at 4.2 0 270) (size 4.4 2.5) (layers "F.Cu" "F.Paste" "F.Mask") (roundrect_rratio 0.1)
+    (pad "2" smd roundrect (at 3.7 0 270) (size 4.4 2.5) (layers "F.Cu" "F.Paste" "F.Mask") (roundrect_rratio 0.1)
       (net 11 "GND") (pintype "passive"))
-    (model "${KICAD6_3DMODEL_DIR}/Capacitor_SMD.3dshapes/CP_Elec_10x10.5.wrl"
+    (model "${KICAD6_3DMODEL_DIR}/Capacitor_SMD.3dshapes/CP_Elec_8x10.5.wrl"
       (offset (xyz 0 0 0))
       (scale (xyz 1 1 1))
@@
   (via (at 112.62 146.94) (size 0.8) (drill 0.4) (layers "F.Cu" "B.Cu") (free) (net 11))
   (via (at 105 136.78) (size 0.8) (drill 0.4) (layers "F.Cu" "B.Cu") (free) (net 11))
-  (via (at 92.1 42.82) (size 0.8) (drill 0.4) (layers "F.Cu" "B.Cu") (free) (net 11))
   (via (at 111.47 48.25) (size 0.8) (drill 0.4) (layers "F.Cu" "B.Cu") (free) (net 11))
   (via (at 89.92 47.9) (size 0.8) (drill 0.4) (layers "F.Cu" "B.Cu") (free) (net 11))
@@
   (via (at 119.03 78.05) (size 0.8) (drill 0.4) (layers "F.Cu" "B.Cu") (free) (net 11))
   (via (at 126.65 88.19) (size 0.8) (drill 0.4) (layers "F.Cu" "B.Cu") (free) (net 11))
-  (via (at 82.9 42.85) (size 0.8) (drill 0.4) (layers "F.Cu" "B.Cu") (free) (net 11))
   (via (at 102.619998 35.19) (size 0.8) (drill 0.4) (layers "F.Cu" "B.Cu") (free) (net 11))
   (via (at 95.88 83.1) (size 0.8) (drill 0.4) (layers "F.Cu" "B.Cu") (free) (net 11))
@@
   (via (at 119.03 75.499998) (size 0.8) (drill 0.4) (layers "F.Cu" "B.Cu") (free) (net 11))
   (via (at 112.62 149.48) (size 0.8) (drill 0.4) (layers "F.Cu" "B.Cu") (free) (net 11))
-  (via (at 82.9 45.39) (size 0.8) (drill 0.4) (layers "F.Cu" "B.Cu") (free) (net 11))
   (via (at 88.26 78.01) (size 0.8) (drill 0.4) (layers "F.Cu" "B.Cu") (free) (net 11))
   (via (at 112.62 154.56) (size 0.8) (drill 0.4) (layers "F.Cu" "B.Cu") (free) (net 11))
@@
   (via (at 99.92 149.48) (size 0.8) (drill 0.4) (layers "F.Cu" "B.Cu") (free) (net 11))
   (via (at 99.92 139.32) (size 0.8) (drill 0.4) (layers "F.Cu" "B.Cu") (free) (net 11))
-  (via (at 92.1 45.36) (size 0.8) (drill 0.4) (layers "F.Cu" "B.Cu") (free) (net 11))
   (via (at 88.26 67.839998) (size 0.8) (drill 0.4) (layers "F.Cu" "B.Cu") (free) (net 11))
   (via (at 88.26 90.7) (size 0.8) (drill 0.4) (layers "F.Cu" "B.Cu") (free) (net 11))

Commit message: L3 change to teensy
Changed lines of the file:
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@@
         (effects (font (size 1 1) (thickness 0.15)))
     )
-    (pad "1" thru_hole circle (at -6.87 0 180) (size 3 3) (drill 2.1) (layers "*.Cu" "*.Mask" "Eco1.User")
+    (pad "1" thru_hole circle (at -6.87 0 180) (size 2.5 2.5) (drill 1.65) (layers "*.Cu" "*.Mask" "Eco1.User")
       (net 11 "GND") (pinfunction "Pin_1") (pintype "passive"))
-    (pad "2" thru_hole circle (at -2.29 0 180) (size 3 3) (drill 2.1) (layers "*.Cu" "*.Mask" "Eco1.User")
+    (pad "2" thru_hole circle (at -2.29 0 180) (size 2.5 2.5) (drill 1.65) (layers "*.Cu" "*.Mask" "Eco1.User")
       (net 38 "+12V") (pinfunction "Pin_2") (pintype "passive"))
-    (pad "3" thru_hole circle (at 2.29 0 180) (size 3 3) (drill 2.1) (layers "*.Cu" "*.Mask" "Eco1.User")
+    (pad "3" thru_hole circle (at 2.29 0 180) (size 2.5 2.5) (drill 1.65) (layers "*.Cu" "*.Mask" "Eco1.User")
       (net 36 "+48V") (pinfunction "Pin_3") (pintype "passive"))
-    (pad "4" thru_hole circle (at 6.87 0 180) (size 3 3) (drill 2.1) (layers "*.Cu" "*.Mask" "Eco1.User")
+    (pad "4" thru_hole circle (at 6.87 0 180) (size 2.5 2.5) (drill 1.65) (layers "*.Cu" "*.Mask" "Eco1.User")
       (net 37 "+3V3") (pinfunction "Pin_4") (pintype "passive"))
   )
@@
     (pad "3" smd rect (at 1.05 0 180) (size 0.6 1.3) (layers "F.Cu" "F.Paste" "F.Mask")
       (net 11 "GND") (pinfunction "S") (pintype "passive"))
-    (model "IRLML6344TRPBF.stp"
+    (model "${KIPRJMOD}/3dmodels/IRLML6344TRPBF.stp"
       (offset (xyz 0 0 0))
       (scale (xyz 1 1 1))
