File: open/2024l3 Cut Off/2024l3 Cut Off.kicad_pcb (KiCad board)
At the start: 2 copper layers, 130 x 95 mm, 24 parts, among them J1 Conn_01x06, J2 TOF 0, J3 TOF 1, J4 TOF 2, J5 TOF 3, U1 OpenMV, U2 4754, U3 >VALUE, U4 Adafruit Featherwing

Commit message: L3
Parts:
- moved H10 8.10 mm to (138.0, 82.5)
- moved H4 7.94 mm to (159.2, 127.6)
- moved U1 0.34 mm to (148.8, 104.8)
- moved H7 0.11 mm to (181.6, 65.3)
- moved H8 0.11 mm to (115.5, 65.3)
- moved H5 0.11 mm to (199.5, 118.3)
- moved H6 0.11 mm to (199.5, 91.9)
- moved H1 0.11 mm to (97.7, 91.9)
- moved H12 0.11 mm to (93.0, 82.6)
- moved H3 0.11 mm to (93.0, 127.6)
- moved H11 0.11 mm to (204.2, 127.6)
- moved H9 0.11 mm to (204.2, 82.6)
- moved H2 0.11 mm to (97.7, 118.3)
Other:
- outline, holes or cut-outs redrawn
Changed lines of the file:
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@@
   )
   (footprint "MountingHole:MountingHole_3.2mm_M3_Pad_Via" (layer "F.Cu")
-    (at 92.874511 127.503998)
+    (at 92.954511 127.573998)
     (descr "Mounting Hole 3.2mm, M3")
     (tags "mounting hole 3.2mm m3")
@@
   )
   (footprint "2024l3:openmv" (layer "F.Cu")
-    (at 148.496 105.004 90)
+    (at 148.776 104.804 90)
     (property "Sheetfile" "2024l3 Cut Off.kicad_sch")
     (property "Sheetname" "")
@@
   )
   (footprint "MountingHole:MountingHole_3.2mm_M3_Pad_Via" (layer "F.Cu")
-    (at 167.135609 127.504)
+    (at 159.197489 127.573998)
     (descr "Mounting Hole 3.2mm, M3")
     (tags "mounting hole 3.2mm m3")
@@
   )
   (footprint "MountingHole:MountingHole_3.2mm_M3_Pad_Via" (layer "F.Cu")
-    (at 97.572619 91.807836)
+    (at 97.65262 91.877835)
     (descr "Mounting Hole 3.2mm, M3")
     (tags "mounting hole 3.2mm m3")
@@
   )
   (footprint "MountingHole:MountingHole_3.2mm_M3_Pad_Via" (layer "F.Cu")
-    (at 115.466792 65.278635)
+    (at 115.546794 65.348633)
     (descr "Mounting Hole 3.2mm, M3")
     (tags "mounting hole 3.2mm m3")
@@
   )
   (footprint "MountingHole:MountingHole_3.2mm_M3_Pad_Via" (layer "F.Cu")
-    (at 92.874511 82.503998)
+    (at 92.954511 82.573998)
     (descr "Mounting Hole 3.2mm, M3")
     (tags "mounting hole 3.2mm m3")
@@
   )
   (footprint "MountingHole:MountingHole_3.2mm_M3_Pad_Via" (layer "F.Cu")
-    (at 204.117489 82.503998)
+    (at 204.197489 82.573998)
     (descr "Mounting Hole 3.2mm, M3")
     (tags "mounting hole 3.2mm m3")
@@
   )
   (footprint "MountingHole:MountingHole_3.2mm_M3_Pad_Via" (layer "F.Cu")
-    (at 181.525205 65.278635)
+    (at 181.605208 65.348633)
     (descr "Mounting Hole 3.2mm, M3")
     (tags "mounting hole 3.2mm m3")
@@
   )
   (footprint "MountingHole:MountingHole_3.2mm_M3_Pad_Via" (layer "F.Cu")
-    (at 204.11749 127.503998)
+    (at 204.19749 127.573998)
     (descr "Mounting Hole 3.2mm, M3")
     (tags "mounting hole 3.2mm m3")
@@
   )
   (footprint "MountingHole:MountingHole_3.2mm_M3_Pad_Via" (layer "F.Cu")
-    (at 129.85639 82.504)
+    (at 137.954511 82.504)
     (descr "Mounting Hole 3.2mm, M3")
     (tags "mounting hole 3.2mm m3")
@@
   )
   (footprint "MountingHole:MountingHole_3.2mm_M3_Pad_Via" (layer "F.Cu")
-    (at 199.41938 91.807837)
+    (at 199.499381 91.877836)
     (descr "Mounting Hole 3.2mm, M3")
     (tags "mounting hole 3.2mm m3")
@@
   )
   (footprint "MountingHole:MountingHole_3.2mm_M3_Pad_Via" (layer "F.Cu")
-    (at 97.572621 118.200162)
+    (at 97.652621 118.270161)
     (descr "Mounting Hole 3.2mm, M3")
     (tags "mounting hole 3.2mm m3")
@@
   )
   (footprint "MountingHole:MountingHole_3.2mm_M3_Pad_Via" (layer "F.Cu")
-    (at 199.41938 118.200162)
+    (at 199.499381 118.270161)
     (descr "Mounting Hole 3.2mm, M3")
     (tags "mounting hole 3.2mm m3")
@@
     )
   )
-  (gr_arc (start 92.060197 135.003998) (mid 91.006107 134.703669) (end 90.268585 133.892887)
+  (gr_arc (start 206.803417 133.962887) (mid 206.065897 134.773671) (end 205.011805 135.073998)
     (stroke (width 0.2) (type solid)) (layer "Edge.Cuts"))
-  (gr_line (start 176.525207 84.807835) (end 176.525208 71.807835)
+  (gr_circle (center 143.376001 90.341998) (end 144.976002 90.341998)
+    (stroke (width 0.2) (type solid)) (fill none) (layer "Edge.Cuts"))
+  (gr_circle (center 143.376001 119.805999) (end 141.776 119.805998)
+    (stroke (width 0.2) (type solid)) (fill none) (layer "Edge.Cuts"))
+  (gr_line (start 198.605207 84.877836) (end 178.605207 84.877835)
     (stroke (width 0.2) (type solid)) (layer "Edge.Cuts"))
-  (gr_line (start 196.525207 71.807837) (end 196.525207 84.807835)
+  (gr_line (start 92.140197 135.073998) (end 205.011805 135.073998)
     (stroke (width 0.2) (type solid)) (layer "Edge.Cuts"))
-  (gr_line (start 196.525207 84.807835) (end 176.525207 84.807835)
+  (gr_line (start 178.605207 84.877835) (end 178.605207 71.877837)
     (stroke (width 0.2) (type solid)) (layer "Edge.Cuts"))
-  (gr_arc (start 206.723417 133.892887) (mid 205.985897 134.703671) (end 204.931805 135.003998)
+  (gr_arc (start 90.348585 133.962887) (mid 148.576 40.074003) (end 206.803417 133.962887)
     (stroke (width 0.2) (type solid)) (layer "Edge.Cuts"))
-  (gr_line (start 92.060197 135.003998) (end 204.931805 135.003998)
+  (gr_line (start 198.605208 71.877835) (end 198.605207 84.877836)
     (stroke (width 0.2) (type solid)) (layer "Edge.Cuts"))
-  (gr_arc (start 90.268585 133.892887) (mid 148.496 40.004003) (end 206.723417 133.892887)
+  (gr_line (start 178.605207 71.877837) (end 198.605208 71.877835)
     (stroke (width 0.2) (type solid)) (layer "Edge.Cuts"))
-  (gr_line (start 176.525208 71.807835) (end 196.525207 71.807837)
+  (gr_arc (start 92.140197 135.073998) (mid 91.086107 134.773669) (end 90.348585 133.962887)
     (stroke (width 0.2) (type solid)) (layer "Edge.Cuts"))
   (gr_text "JLCJLCJLCJLC" (at 140.771 52.054) (layer "F.SilkS")
@@
     )
   )
-  (group "" (id 2f615264-3b2d-4de4-9c8a-13aa1499d07d)
+  (group "" (id df8e8361-70e5-40c9-8f0a-c4c5101bf9d4)
     (members
-      10c34566-5998-46c4-ab72-9566cae8012f
-      227c8610-e846-428c-a9dd-2ed2404093d8
-      2b99fa6d-33e3-4eac-99bf-6c4465eb1167
-      37221c47-1c71-4c02-b7d2-052ff18d907c
-      8e68044b-9d12-4167-8a14-2b39a1a16d04
-      9cbb6dc5-14f8-4b03-9705-eb9d60398a2a
-      a534233a-c49f-42db-91d4-7882bfb0096d
-      dcef2ecc-9f6a-4767-b10a-4d5d58bab9a3
-    )
-  )
+      131535ac-ac54-4c27-b191-ee2b3c7a5d4f
+      6fb4a17d-56b6-45e9-840f-221199200a36
+      83ac8b0f-0a1b-4bb7-92bb-01918d329b01
+      ad85b513-7b98-4402-ab03-95cb763c7690
+      ca071d26-7ffa-41c6-ae9c-f481a61d3928
+      ce18ce6b-698c-4110-86e9-4ec3c2282d6c
+      cec4f7e3-66d7-46a2-933b-83330d78fa87
+      e4ac9aa3-ed09-4b1d-8bdd-2cf37cb86e47
+      e5443bcf-718c-4fc7-a482-24c822743b97
+      f5020c1e-3ffa-4ae6-95fe-a14ddb89bef7
+    )
+  )

Commit message: L3 and L1
Parts:
- removed U4: Adafruit Featherwing, 2024l3:Adafruit Feather OLED
- added REF**: Adafruit Feather OLED, 2024l3:Adafruit Feather OLED, F.Cu at (149.2, 56.3)
- moved J2 46.6 mm to (134.8, 98.2)
- moved U3 44.7 mm to (102.8, 105.5)
- moved J1 37.0 mm to (181.6, 70.6), turned to -90 degrees
- moved J4 31.3 mm to (177.5, 110.5)
- moved R1 28.3 mm to (168.3, 100.2)
- moved R2 28.3 mm to (168.3, 102.7)
- moved Ue 6.71 mm to (159.7, 76.8)
- moved J3 3.00 mm to (116.0, 82.7)
- moved J5 3.00 mm to (181.0, 127.3)
- moved U2 1.59 mm to (125.9, 105.3)
Other:
- outline, holes or cut-outs redrawn
