File: open/2024l3 Cut Off/2024l3 Cut Off.kicad_sch (KiCad schematic)
At the start: 22 parts, among them J1 Conn_01x06, J2 TOF 0, J3 TOF 1, J4 TOF 2, J5 TOF 3, U1 OpenMV, U2 4754, U3 xiao-esp32c3, U4 Adafruit Featherwing, U7 Teensy 4.0

Commit message: L3 DXF change
Parts:
- added H11, H12: MountingHole_Pad, MountingHole:MountingHole_3.2mm_M3_Pad_Via, symbol Mechanical:MountingHole_Pad
Changed lines of the file:
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@@
+    )
+  )
+  (symbol (lib_id "Mechanical:MountingHole_Pad") (at 31.7112 59.5814 0) (unit 1)
+    (in_bom yes) (on_board yes) (dnp no) (fields_autoplaced)
+    (property "Reference" "H11" (at 34.8595 57.6764 0)
+      (effects (font (size 1.27 1.27)) (justify left))
+    )
+    (property "Value" "MountingHole_Pad" (at 34.8595 60.2164 0)
+      (effects (font (size 1.27 1.27)) (justify left))
+    )
+    (property "Footprint" "MountingHole:MountingHole_3.2mm_M3_Pad_Via" (at 31.7112 59.5814 0)
+      (effects (font (size 1.27 1.27)) hide)
+    )
+    (property "Datasheet" "~" (at 31.7112 59.5814 0)
+      (effects (font (size 1.27 1.27)) hide)
+    )
+    (pin "1")
+    (instances
+      (project "2024l3 Cut Off"
+        (path "/d65f20ed-2841-484c-9395-70974a4cd101"
+          (reference "H11") (unit 1)
+        )
+      )
     )
   )
@@
         )
       )
+    )
+  )
+  (symbol (lib_id "Mechanical:MountingHole_Pad") (at 20.3615 59.8508 0) (unit 1)
+    (in_bom yes) (on_board yes) (dnp no) (fields_autoplaced)
+    (property "Reference" "H12" (at 23.4295 57.9458 0)
+      (effects (font (size 1.27 1.27)) (justify left))
+    )
+    (property "Value" "MountingHole_Pad" (at 23.4295 60.4858 0)
+      (effects (font (size 1.27 1.27)) (justify left))
+    )
+    (property "Footprint" "MountingHole:MountingHole_3.2mm_M3_Pad_Via" (at 20.3615 59.8508 0)
+      (effects (font (size 1.27 1.27)) hide)
+    )
+    (property "Datasheet" "~" (at 20.3615 59.8508 0)
+      (effects (font (size 1.27 1.27)) hide)
+    )
+    (pin "1")
+    (instances
+      (project "2024l3 Cut Off"
+        (path "/d65f20ed-2841-484c-9395-70974a4cd101"
+          (reference "H12") (unit 1)
+        )
+      )

Commit message: L3
Parts:
- removed U4: Adafruit Featherwing, 2024l3:Adafruit Feather OLED, symbol OLED:Adafruit_Featherwing
Connections:
- net A: no longer names the net of U7.5
- net B: no longer names the net of U7.4
- net C: no longer names the net of U7.3
- net OLED RST: no longer names the net of U7.2
- net OLED SCL: no longer names the net of U7.19 (19/A5/SCL0)
- net OLED SDA: no longer names the net of U7.18 (18/A4/SDA0)
Changed lines of the file:
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@@
-    (stroke (width 0) (type default))
-  )
-  (wire (pts (xy 187.0651 84.6928) (xy 187.0651 84.6993))
-    (stroke (width 0) (type default))
-  )
-  (wire (pts (xy 183.8018 94.8593) (xy 187.1128 94.8593))
     (stroke (width 0) (type default))
   )
@@
     (stroke (width 0) (type default))
   )
-  (wire (pts (xy 100.4939 101.193) (xy 103.7921 101.193))
-    (stroke (width 0) (type default))
-  )
   (wire (pts (xy 58.42 43.434) (xy 69.85 43.434))
     (stroke (width 0) (type default))
@@
     (stroke (width 0) (type default))
   )
-  (wire (pts (xy 92.3621 96.113) (xy 103.7921 96.113))
-    (stroke (width 0) (type default))
-  )
   (wire (pts (xy 92.3621 91.033) (xy 103.7921 91.033))
     (stroke (width 0) (type default))
   )
   (wire (pts (xy 58.42 45.974) (xy 58.42 43.434))
-    (stroke (width 0) (type default))
-  )
-  (wire (pts (xy 136.8121 106.273) (xy 147.1048 106.273))
     (stroke (width 0) (type default))
   )
@@
     (stroke (width 0) (type default))
   )
-  (wire (pts (xy 187.0651 84.6993) (xy 183.8018 84.6993))
-    (stroke (width 0) (type default))
-  )
   (polyline (pts (xy 81.2697 69.5626) (xy 81.2697 69.5957))
     (stroke (width 0) (type default))
@@
     (stroke (width 0) (type default))
   )
-  (wire (pts (xy 158.2691 87.2393) (xy 168.5618 87.2393))
-    (stroke (width 0) (type default))
-  )
-  (wire (pts (xy 158.2691 97.3993) (xy 168.5618 97.3993))
-    (stroke (width 0) (type default))
-  )
-  (wire (pts (xy 158.2691 84.6993) (xy 168.5618 84.6993))
-    (stroke (width 0) (type default))
-  )
   (wire (pts (xy 95.7319 88.493) (xy 103.7921 88.493))
     (stroke (width 0) (type default))
@@
     (stroke (width 0) (type default))
   )
-  (wire (pts (xy 183.8018 97.3993) (xy 187.1043 97.3993))
-    (stroke (width 0) (type default))
-  )
   (wire (pts (xy 136.8121 111.353) (xy 145.7021 111.353))
     (stroke (width 0) (type default))
@@
     (stroke (width 0) (type default))
   )
-  (wire (pts (xy 100.4939 103.733) (xy 103.7921 103.733))
-    (stroke (width 0) (type default))
-  )
   (wire (pts (xy 143.1158 36.1998) (xy 153.4085 36.1998))
     (stroke (width 0) (type default))
@@
   )
   (wire (pts (xy 14.8002 94.6965) (xy 23.6902 94.6965))
-    (stroke (width 0) (type default))
-  )
-  (wire (pts (xy 136.8121 108.813) (xy 147.1048 108.813))
     (stroke (width 0) (type default))
   )
@@
     (stroke (width 0) (type default))
   )
-  (wire (pts (xy 100.4939 98.653) (xy 103.7921 98.653))
-    (stroke (width 0) (type default))
-  )
   (wire (pts (xy 192.2697 48.3826) (xy 202.5624 48.3826))
-    (stroke (width 0) (type default))
-  )
-  (wire (pts (xy 183.8018 92.3193) (xy 187.1 92.3193))
     (stroke (width 0) (type default))
   )
@@
     (effects (font (size 1.27 1.27)) (justify left bottom))
   )
-  (label "OLED SCL" (at 158.9592 84.6993 0) (fields_autoplaced)
-    (effects (font (size 1.27 1.27)) (justify left bottom))
-  )
-  (label "B" (at 184.9843 94.8593 0) (fields_autoplaced)
-    (effects (font (size 1.27 1.27)) (justify left bottom))
-  )
   (label "SDA TOF" (at 221.833 28.3626 0) (fields_autoplaced)
     (effects (font (size 1.27 1.27)) (justify left bottom))
@@
     (effects (font (size 1.27 1.27)) (justify left bottom))
   )
-  (label "OLED SDA" (at 137.5891 108.813 0) (fields_autoplaced)
-    (effects (font (size 1.27 1.27)) (justify left bottom))
-  )
   (label "SDA TOF" (at 145.7262 41.2798 0) (fields_autoplaced)
     (effects (font (size 1.27 1.27)) (justify left bottom))
@@
     (effects (font (size 1.27 1.27)) (justify left bottom))
   )
-  (label "B" (at 101.6764 101.193 0) (fields_autoplaced)
-    (effects (font (size 1.27 1.27)) (justify left bottom))
-  )
   (label "CAM RX" (at 16.0702 94.6965 0) (fields_autoplaced)
     (effects (font (size 1.27 1.27)) (justify left bottom))
@@
     (effects (font (size 1.27 1.27)) (justify left bottom))
   )
-  (label "OLED RST" (at 159.324 97.3993 0) (fields_autoplaced)
-    (effects (font (size 1.27 1.27)) (justify left bottom))
-  )
-  (label "C" (at 101.6481 98.653 0) (fields_autoplaced)
-    (effects (font (size 1.27 1.27)) (justify left bottom))
-  )
   (label "SCL TOF" (at 194.7418 30.146 0) (fields_autoplaced)
     (effects (font (size 1.27 1.27)) (justify left bottom))
   )
-  (label "A" (at 185.0267 92.3193 0) (fields_autoplaced)
-    (effects (font (size 1.27 1.27)) (justify left bottom))
-  )
   (label "SDA TOF" (at 194.7554 27.606 0) (fields_autoplaced)
     (effects (font (size 1.27 1.27)) (justify left bottom))
@@
     (effects (font (size 1.27 1.27)) (justify left bottom))
   )
-  (label "C" (at 184.956 97.3993 0) (fields_autoplaced)
-    (effects (font (size 1.27 1.27)) (justify left bottom))
-  )
   (label "SCL TOF" (at 221.8194 30.9026 0) (fields_autoplaced)
     (effects (font (size 1.27 1.27)) (justify left bottom))
   )
   (label "XSHUT 1" (at 144.8167 33.6598 0) (fields_autoplaced)
-    (effects (font (size 1.27 1.27)) (justify left bottom))
-  )
-  (label "OLED RST" (at 94.5543 96.113 0) (fields_autoplaced)
     (effects (font (size 1.27 1.27)) (justify left bottom))
   )
@@
     (effects (font (size 1.27 1.27)) (justify left bottom))
   )
-  (label "A" (at 101.7188 103.733 0) (fields_autoplaced)
-    (effects (font (size 1.27 1.27)) (justify left bottom))
-  )
   (label "CAM RX" (at 138.0821 103.733 0) (fields_autoplaced)
     (effects (font (size 1.27 1.27)) (justify left bottom))
@@
     (effects (font (size 1.27 1.27)) (justify left bottom))
   )
-  (label "OLED SCL" (at 137.5022 106.273 0) (fields_autoplaced)
-    (effects (font (size 1.27 1.27)) (justify left bottom))
-  )
   (label "SCL TOF" (at 145.7126 43.8198 0) (fields_autoplaced)
     (effects (font (size 1.27 1.27)) (justify left bottom))
@@
   )
   (label "ESP RX" (at 172.4585 46.3598 0) (fields_autoplaced)
-    (effects (font (size 1.27 1.27)) (justify left bottom))
-  )
-  (label "OLED SDA" (at 159.0461 87.2393 0) (fields_autoplaced)
     (effects (font (size 1.27 1.27)) (justify left bottom))
   )
@@
     )
   )
-  (symbol (lib_id "power:GND") (at 183.8018 87.2393 90) (unit 1)
-    (in_bom yes) (on_board yes) (dnp no) (fields_autoplaced)
-    (property "Reference" "#PWR011" (at 190.1518 87.2393 0)
-      (effects (font (size 1.27 1.27)) hide)
-    )
-    (property "Value" "GND" (at 188.1482 87.8743 90)
-      (effects (font (size 1.27 1.27)) (justify right))
-    )
-    (property "Footprint" "" (at 183.8018 87.2393 0)
-      (effects (font (size 1.27 1.27)) hide)
-    )
-    (property "Datasheet" "" (at 183.8018 87.2393 0)
-      (effects (font (size 1.27 1.27)) hide)
-    )
-    (pin "1")
-    (instances
-      (project "2024l3 Cut Off"
-        (path "/d65f20ed-2841-484c-9395-70974a4cd101"
-          (reference "#PWR011") (unit 1)
-        )
-      )
-    )
-  )
   (symbol (lib_id "Mechanical:MountingHole_Pad") (at 20.32 52.324 0) (unit 1)
     (in_bom yes) (on_board yes) (dnp no) (fields_autoplaced)
@@
     )
   )
-  (symbol (lib_id "power:+3V3") (at 187.0651 84.6928 0) (unit 1)
-    (in_bom yes) (on_board yes) (dnp no) (fields_autoplaced)
-    (property "Reference" "#PWR010" (at 187.0651 88.5028 0)
-      (effects (font (size 1.27 1.27)) hide)
-    )
-    (property "Value" "+3V3" (at 188.6833 84.0578 0)
-      (effects (font (size 1.27 1.27)) (justify left))
-    )
-    (property "Footprint" "" (at 187.0651 84.6928 0)
-      (effects (font (size 1.27 1.27)) hide)
-    )
-    (property "Datasheet" "" (at 187.0651 84.6928 0)
-      (effects (font (size 1.27 1.27)) hide)
-    )
-    (pin "1")
-    (instances
-      (project "2024l3 Cut Off"
-        (path "/d65f20ed-2841-484c-9395-70974a4cd101"
-          (reference "#PWR010") (unit 1)
-        )
-      )
-    )
-  )
   (symbol (lib_id "power:GND") (at 88.8629 88.497 0) (mirror y) (unit 1)
     (in_bom yes) (on_board yes) (dnp no) (fields_autoplaced)
@@
         )
       )
-    )
-  )
-  (symbol (lib_id "OLED:Adafruit_Featherwing") (at 176.1818 91.0493 0) (unit 1)
-    (in_bom yes) (on_board yes) (dnp no) (fields_autoplaced)
-    (property "Reference" "U4" (at 176.1818 77.9265 0)
-      (effects (font (size 1.27 1.27)))
-    )
-    (property "Value" "Adafruit Featherwing" (at 176.1818 80.4665 0)
-      (effects (font (size 1.27 1.27)))
-    )
-    (property "Footprint" "2024l3:Adafruit Feather OLED" (at 176.1818 101.2093 0)
-      (effects (font (size 1.27 1.27)) hide)
-    )
-    (property "Datasheet" "" (at 176.1818 91.0493 0)
-      (effects (font (size 1.27 1.27)) hide)
-    )
-    (pin "1")
-    (pin "17")
-    (pin "18")
-    (pin "19")
-    (pin "2")
-    (pin "20")
-    (pin "21")
-    (pin "4")
-    (instances
-      (project "2024l3 Cut Off"
-        (path "/d65f20ed-2841-484c-9395-70974a4cd101"
-          (reference "U4") (unit 1)
-        )
-      )

Commit message: L3 and L1
Parts:
- added SW1, SW2: SW_SPDT, symbol Switch:SW_SPDT
Connections:
- net +5V: now also SW1.3 (C), SW2.3 (C); no longer U1.10 (VIN_(3V6-5V)), U2.JP1_1 (VIN)
- new net CAM PWR: SW1.2 (B), U1.10 (VIN_(3V6-5V))
- new net COM PWR: SW2.2 (B), U2.JP1_1 (VIN)
Changed lines of the file:
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@@
+    (stroke (width 0) (type default))
+  )
+  (wire (pts (xy 182.3921 95.4988) (xy 182.3921 100.1213))
     (stroke (width 0) (type default))
   )
@@
     (stroke (width 0) (type default))
   )
-  (wire (pts (xy 70.349 97.2365) (xy 68.1402 97.2365))
-    (stroke (width 0) (type default))
-  )
   (wire (pts (xy 143.1158 33.6598) (xy 153.4085 33.6598))
     (stroke (width 0) (type default))
@@
     (stroke (width 0) (type default))
   )
+  (wire (pts (xy 162.6576 94.9068) (xy 162.6576 99.5293))
+    (stroke (width 0) (type default))
+  )
   (wire (pts (xy 95.7319 88.493) (xy 103.7921 88.493))
     (stroke (width 0) (type default))
@@
     (stroke (width 0) (type default))
   )
+  (wire (pts (xy 87.796 24.7874) (xy 96.9446 24.7874))
+    (stroke (width 0) (type default))
+  )
   (wire (pts (xy 136.8121 111.353) (xy 145.7021 111.353))
     (stroke (width 0) (type default))
@@
     (stroke (width 0) (type default))
   )
-  (wire (pts (xy 70.349 97.2525) (xy 70.349 97.2365))
+  (wire (pts (xy 68.1402 97.2365) (xy 77.2888 97.2365))
     (stroke (width 0) (type default))
   )
@@
     (effects (font (size 1.27 1.27)) (justify left bottom))
   )
+  (label "CAM PWR" (at 68.9139 97.2365 0) (fields_autoplaced)
+    (effects (font (size 1.27 1.27)) (justify left bottom))
+  )
   (label "SDA TOF" (at 145.7262 41.2798 0) (fields_autoplaced)
     (effects (font (size 1.27 1.27)) (justify left bottom))
@@
     (effects (font (size 1.27 1.27)) (justify left bottom))
   )
+  (label "CAM PWR" (at 162.6576 97.4621 0) (fields_autoplaced)
+    (effects (font (size 1.27 1.27)) (justify left bottom))
+  )
   (label "CAM RX" (at 16.0702 94.6965 0) (fields_autoplaced)
     (effects (font (size 1.27 1.27)) (justify left bottom))
@@
     (effects (font (size 1.27 1.27)) (justify left bottom))
   )
+  (label "COM PWR" (at 182.3921 98.0541 0) (fields_autoplaced)
+    (effects (font (size 1.27 1.27)) (justify left bottom))
+  )
   (label "ESP TX" (at 145.7885 46.3598 0) (fields_autoplaced)
     (effects (font (size 1.27 1.27)) (justify left bottom))
@@
   )
   (label "SCL TOF" (at 221.8194 30.9026 0) (fields_autoplaced)
+    (effects (font (size 1.27 1.27)) (justify left bottom))
+  )
+  (label "COM PWR" (at 87.796 24.7874 0) (fields_autoplaced)
     (effects (font (size 1.27 1.27)) (justify left bottom))
   )
@@
     )
   )
+  (symbol (lib_id "Switch:SW_SPDT") (at 182.3921 90.4188 90) (unit 1)
+    (in_bom yes) (on_board yes) (dnp no) (fields_autoplaced)
+    (property "Reference" "SW2" (at 186.5836 89.7838 90)
+      (effects (font (size 1.27 1.27)) (justify right))
+    )
+    (property "Value" "SW_SPDT" (at 186.5836 92.3238 90)
+      (effects (font (size 1.27 1.27)) (justify right))
+    )
+    (property "Footprint" "" (at 182.3921 90.4188 0)
+      (effects (font (size 1.27 1.27)) hide)
+    )
+    (property "Datasheet" "~" (at 182.3921 90.4188 0)
+      (effects (font (size 1.27 1.27)) hide)
+    )
+    (pin "1")
+    (pin "2")
+    (pin "3")
+    (instances
+      (project "2024l3 Cut Off"
+        (path "/d65f20ed-2841-484c-9395-70974a4cd101"
+          (reference "SW2") (unit 1)
+        )
+      )
+    )
+  )
   (symbol (lib_id "vincent:xiao-esp32c3") (at 162.2985 28.5798 0) (unit 1)
     (in_bom yes) (on_board yes) (dnp no) (fields_autoplaced)
@@
     )
   )
-  (symbol (lib_id "power:+5V") (at 70.349 97.2525 0) (unit 1)
-    (in_bom yes) (on_board yes) (dnp no)
-    (property "Reference" "#PWR07" (at 70.349 101.0625 0)
-      (effects (font (size 1.27 1.27)) hide)
-    )
-    (property "Value" "+5V" (at 70.3531 92.9236 90)
-      (effects (font (size 1.27 1.27)) (justify left))
-    )
-    (property "Footprint" "" (at 70.349 97.2525 0)
-      (effects (font (size 1.27 1.27)) hide)
-    )
-    (property "Datasheet" "" (at 70.349 97.2525 0)
-      (effects (font (size 1.27 1.27)) hide)
-    )
-    (pin "1")
-    (instances
-      (project "2024l3 Cut Off"
-        (path "/d65f20ed-2841-484c-9395-70974a4cd101"
-          (reference "#PWR07") (unit 1)
-        )
-      )
-    )
-  )
   (symbol (lib_id "Mechanical:MountingHole_Pad") (at 31.3429 34.7998 0) (unit 1)
     (in_bom yes) (on_board yes) (dnp no) (fields_autoplaced)
@@
         (path "/d65f20ed-2841-484c-9395-70974a4cd101"
           (reference "H9") (unit 1)
+        )
+      )
+    )
+  )
+  (symbol (lib_id "Switch:SW_SPDT") (at 162.6576 89.8268 90) (unit 1)
+    (in_bom yes) (on_board yes) (dnp no) (fields_autoplaced)
+    (property "Reference" "SW1" (at 166.8491 89.1918 90)
+      (effects (font (size 1.27 1.27)) (justify right))
+    )
+    (property "Value" "SW_SPDT" (at 166.8491 91.7318 90)
+      (effects (font (size 1.27 1.27)) (justify right))
+    )
+    (property "Footprint" "" (at 162.6576 89.8268 0)
+      (effects (font (size 1.27 1.27)) hide)
+    )
+    (property "Datasheet" "~" (at 162.6576 89.8268 0)
+      (effects (font (size 1.27 1.27)) hide)
+    )
+    (pin "1")
+    (pin "2")
+    (pin "3")
+    (instances
+      (project "2024l3 Cut Off"
+        (path "/d65f20ed-2841-484c-9395-70974a4cd101"
+          (reference "SW1") (unit 1)
         )
       )
@@
     )
   )
+  (symbol (lib_id "power:+5V") (at 165.1976 84.7468 0) (unit 1)
+    (in_bom yes) (on_board yes) (dnp no) (fields_autoplaced)
+    (property "Reference" "#PWR02" (at 165.1976 88.5568 0)
+      (effects (font (size 1.27 1.27)) hide)
+    )
+    (property "Value" "+5V" (at 165.1976 80.3139 0)
+      (effects (font (size 1.27 1.27)))
+    )
+    (property "Footprint" "" (at 165.1976 84.7468 0)
+      (effects (font (size 1.27 1.27)) hide)
+    )
+    (property "Datasheet" "" (at 165.1976 84.7468 0)
+      (effects (font (size 1.27 1.27)) hide)
+    )
+    (pin "1")
+    (instances
+      (project "2024l3 Cut Off"
+        (path "/d65f20ed-2841-484c-9395-70974a4cd101"
+          (reference "#PWR02") (unit 1)
+        )
+      )
+    )
+  )
   (symbol (lib_id "power:GND") (at 122.3446 52.7274 90) (unit 1)
     (in_bom yes) (on_board yes) (dnp no) (fields_autoplaced)
@@
         (path "/d65f20ed-2841-484c-9395-70974a4cd101"
           (reference "J1") (unit 1)
+        )
+      )
+    )
+  )
+  (symbol (lib_id "power:+5V") (at 184.9321 85.3388 0) (unit 1)
+    (in_bom yes) (on_board yes) (dnp no) (fields_autoplaced)
+    (property "Reference" "#PWR05" (at 184.9321 89.1488 0)
+      (effects (font (size 1.27 1.27)) hide)
+    )
+    (property "Value" "+5V" (at 184.9321 80.9059 0)
+      (effects (font (size 1.27 1.27)))
+    )
+    (property "Footprint" "" (at 184.9321 85.3388 0)
+      (effects (font (size 1.27 1.27)) hide)
+    )
+    (property "Datasheet" "" (at 184.9321 85.3388 0)
+      (effects (font (size 1.27 1.27)) hide)
+    )
+    (pin "1")
+    (instances
+      (project "2024l3 Cut Off"
+        (path "/d65f20ed-2841-484c-9395-70974a4cd101"
+          (reference "#PWR05") (unit 1)
         )
       )
@@
         )
       )
-    )
-  )
-  (symbol (lib_id "power:+5V") (at 96.9446 24.7874 0) (unit 1)
-    (in_bom yes) (on_board yes) (dnp no)
-    (property "Reference" "#PWR05" (at 96.9446 28.5974 0)
-      (effects (font (size 1.27 1.27)) hide)
-    )
-    (property "Value" "+5V" (at 96.9487 20.4585 90)
-      (effects (font (size 1.27 1.27)) (justify left))
-    )
-    (property "Footprint" "" (at 96.9446 24.7874 0)
-      (effects (font (size 1.27 1.27)) hide)
-    )
-    (property "Datasheet" "" (at 96.9446 24.7874 0)
-      (effects (font (size 1.27 1.27)) hide)
-    )
-    (pin "1")
-    (instances
-      (project "2024l3 Cut Off"
-        (path "/d65f20ed-2841-484c-9395-70974a4cd101"
-          (reference "#PWR05") (unit 1)
-        )
-      )
