File: test/test.kicad_pcb (KiCad board)
At the start: 2 copper layers, 30.2 x 60.6 mm, 25 parts, among them J1 Conn_01x02, J2 Conn_01x02, J3 Conn_01x10, U1 DRV8873SPWPRQ1

Commit message: Pin Labels
Parts:
- moved H1 2.00 mm to (141.2, 82.6)
- moved H4 2.00 mm to (159.8, 82.6)
Other:
- board size 30.2 x 60.6 mm -> 30.2 x 62.6 mm
- board text added: "3V3"
- board text added: "5V"
- board text added: "CS"
- board text added: "DIS"
- board text added: "EN"
- board text added: "GND"
- board text added: "PH"
- board text added: "SCLK"
- board text added: "SDI"
- board text added: "SDO"
Changed lines of the file:
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@@
   )
   (setup
+    (stackup
+      (layer "F.SilkS" (type "Top Silk Screen"))
+      (layer "F.Paste" (type "Top Solder Paste"))
+      (layer "F.Mask" (type "Top Solder Mask") (color "Purple") (thickness 0.01))
+      (layer "F.Cu" (type "copper") (thickness 0.035))
+      (layer "dielectric 1" (type "core") (color "FR4 natural") (thickness 1.51) (material "FR4") (epsilon_r 4.5) (loss_tangent 0.02))
+      (layer "B.Cu" (type "copper") (thickness 0.035))
+      (layer "B.Mask" (type "Bottom Solder Mask") (color "Purple") (thickness 0.01))
+      (layer "B.Paste" (type "Bottom Solder Paste"))
+      (layer "B.SilkS" (type "Bottom Silk Screen"))
+      (copper_finish "None")
+      (dielectric_constraints no)
+    )
     (pad_to_mask_clearance 0)
     (aux_axis_origin 145 105)
@@
   (net 28 "unconnected-(H4-Pad1)")
   (footprint "MountingHole:MountingHole_3.2mm_M3_Pad_Via" (layer "F.Cu")
-    (at 159.8 84.6)
+    (at 159.8 82.6)
     (descr "Mounting Hole 3.2mm, M3")
     (tags "mounting hole 3.2mm m3")
@@
   )
   (footprint "MountingHole:MountingHole_3.2mm_M3_Pad_Via" (layer "F.Cu")
-    (at 141.2 84.6)
+    (at 141.2 82.6)
     (descr "Mounting Hole 3.2mm, M3")
     (tags "mounting hole 3.2mm m3")
@@
   (gr_line (start 136.4 128.8) (end 136.4 126.9)
     (stroke (width 0.2) (type default)) (layer "F.Cu"))
-  (gr_line (start 165.6 80) (end 165.6 138.2)
+  (gr_line (start 165.6 78) (end 165.6 138.2)
     (stroke (width 0.1) (type default)) (layer "Edge.Cuts"))
-  (gr_line (start 135.4 138.2) (end 135.4 80)
+  (gr_line (start 135.4 138.2) (end 135.4 78)
     (stroke (width 0.1) (type default)) (layer "Edge.Cuts"))
   (gr_line (start 164.4 139.4) (end 136.6 139.4)
     (stroke (width 0.1) (type default)) (layer "Edge.Cuts"))
-  (gr_arc (start 164.4 78.8) (mid 165.248528 79.151472) (end 165.6 80)
+  (gr_arc (start 164.4 76.8) (mid 165.248528 77.151472) (end 165.6 78)
     (stroke (width 0.1) (type default)) (layer "Edge.Cuts"))
-  (gr_line (start 136.6 78.8) (end 164.4 78.8)
+  (gr_line (start 136.6 76.8) (end 164.4 76.8)
     (stroke (width 0.1) (type default)) (layer "Edge.Cuts"))
   (gr_arc (start 136.6 139.4) (mid 135.751472 139.048528) (end 135.4 138.2)
     (stroke (width 0.1) (type default)) (layer "Edge.Cuts"))
-  (gr_arc (start 135.4 80) (mid 135.751472 79.151472) (end 136.6 78.8)
+  (gr_arc (start 135.4 78) (mid 135.751472 77.151472) (end 136.6 76.8)
     (stroke (width 0.1) (type default)) (layer "Edge.Cuts"))
   (gr_arc (start 165.6 138.2) (mid 165.248528 139.048528) (end 164.4 139.4)
     (stroke (width 0.1) (type default)) (layer "Edge.Cuts"))
+  (gr_text "EN" (at 149.55 88.95 90) (layer "F.SilkS")
+    (effects (font (size 1 1) (thickness 0.15)) (justify left bottom))
+  )
+  (gr_text "PH" (at 146.95 88.95 90) (layer "F.SilkS")
+    (effects (font (size 1 1) (thickness 0.15)) (justify left bottom))
+  )
+  (gr_text "SCLK" (at 154.65 88.95 90) (layer "F.SilkS")
+    (effects (font (size 1 1) (thickness 0.15)) (justify left bottom))
+  )
+  (gr_text "SDO" (at 159.75 88.95 90) (layer "F.SilkS")
+    (effects (font (size 1 1) (thickness 0.15)) (justify left bottom))
+  )
+  (gr_text "SDI" (at 157.1 88.95 90) (layer "F.SilkS")
+    (effects (font (size 1 1) (thickness 0.15)) (justify left bottom))
+  )
+  (gr_text "5V" (at 139.3 88.85 90) (layer "F.SilkS")
+    (effects (font (size 1 1) (thickness 0.15)) (justify left bottom))
+  )
+  (gr_text "CS" (at 152.1 88.95 90) (layer "F.SilkS")
+    (effects (font (size 1 1) (thickness 0.15)) (justify left bottom))
+  )
+  (gr_text "GND" (at 162.35 88.95 90) (layer "F.SilkS")
+    (effects (font (size 1 1) (thickness 0.15)) (justify left bottom))
+  )
   (gr_text "JLCJLCJLCJLC" (at 145.4 135) (layer "F.SilkS")
+    (effects (font (size 1 1) (thickness 0.15)) (justify left bottom))
+  )
+  (gr_text "3V3" (at 141.85 88.95 90) (layer "F.SilkS")
+    (effects (font (size 1 1) (thickness 0.15)) (justify left bottom))
+  )
+  (gr_text "DIS" (at 144.55 88.95 90) (layer "F.SilkS")
     (effects (font (size 1 1) (thickness 0.15)) (justify left bottom))
   )
@@
     (polygon
       (pts
-        (xy 135.4 78.8)
-        (xy 165.6 78.8)
+        (xy 135.4 76.85)
+        (xy 165.6 76.85)
         (xy 165.6 139.4)
         (xy 135.4 139.4)
