File: test/test.kicad_sch (KiCad schematic)
At the start: 37 parts

Commit message: Test PCB
Parts:
- removed C? (x3): 0u1, symbol vincent:C
- removed C? (x2): 1000p, symbol vincent:C
- removed C? (x2): 0u01, symbol vincent:C
- removed C? (x2): 150u, symbol vincent:C_Polarized
- removed C?: 22u, symbol vincent:C
- removed C? (x2): 1u, symbol vincent:C
- removed D?: 1N4148WS-7-F, symbol Device:D
- removed D?: LED, symbol Device:LED
- removed IC?: LM9036QMX-3.3_NOPB, SOIC127P600X175-8N, symbol vincent:LM9036QMX-3.3_NOPB
- removed J?: Conn_01x02, symbol Connector_Generic:Conn_01x02
- removed L?: 1u, symbol Device:L
- removed Q?: CSD18543Q3A, CSD18543Q3A, symbol vincent:CSD18543Q3A
- removed Q?: BC846BLT1G, Package_TO_SOT_SMD:SOT-23, symbol Transistor_BJT:MMBTA42
- removed R?: 4K99, symbol Device:R
- removed R? (x2): 10K, symbol Device:R
- removed TP? (x2): TestPoint, symbol Connector:TestPoint
- added H1, H2, H3, H4: MountingHole_Pad, MountingHole:MountingHole_3.2mm_M3_Pad_Via, symbol Mechanical:MountingHole_Pad
- added J1: Conn_01x02, test:AMASS_XT60-M, symbol Connector_Generic:Conn_01x02
- added J2: Conn_01x02, test:AMASS_XT30-F, symbol Connector_Generic:Conn_01x02
- added J3: Conn_01x10, Connector_PinSocket_2.54mm:PinSocket_1x10_P2.54mm_Vertical, symbol Connector_Generic:Conn_01x10
- added R5, R6: 0, test:res0603, symbol Device:R
- C1, C2, C4, C5: renamed from C?; footprint 2024l2:cap0603 -> test:cap0603
- D1: renamed from D?; footprint (none) -> test:led0603
- R1, R2, R7, R8: renamed from R?; footprint (none) -> test:res0603
- R3, R4: renamed from R?; footprint 2024l2:res0603 -> test:res0603
- U1: renamed from U?; footprint 2024l2:SOP65P640X120-25N -> test:SOP65P640X120-25N
- gave numbers to parts that had none: 1
Connections:
- net M2 VCP is gone; now on net VCP: C1.2, U1.21 (VCP)
- net +12V: now also J1.2 (Pin_2)
- net +3V3: now also J3.2 (Pin_2)
- net +5V: now also J3.1 (Pin_1)
- net DISABLE: now also J3.3 (Pin_3)
- net EN/IN1: now also J3.5 (Pin_5)
- net GND: now also J1.1 (Pin_1), J3.10 (Pin_10)
- net M SCLK: now also J3.7 (Pin_7)
- net M SDI: now also J3.8 (Pin_8), R6.1; no longer U1.4 (SDI)
- net M SDO: now also J3.9 (Pin_9), R5.2; no longer U1.3 (SDO)
- net OUT1: now also J2.1 (Pin_1)
- net OUT2: now also J2.2 (Pin_2)
- net PH/IN2: now also J3.4 (Pin_4)
- net M CS 2 renamed M CS
- net M CS: now also J3.6 (Pin_6)
- net M2 IPROPI1 renamed IPROPI1
- net M2 IPROPI2 renamed IPROPI2
- new net: R5.1, U1.3 (SDO)
- new net: R6.2, U1.4 (SDI)
- no-connect marks 0 -> 4
Other:
- moved on the sheet: C3, C4

Commit message: Schematic Formatting
Other:
- note added: "Connectors and Mounts"
- note added: "Motor Driver"
- moved on the sheet: D1, H1, H2, H3, H4, J3, R1
