File: test (Hardware)/test(Hardware).kicad_pcb (KiCad board)
At the start: 2 copper layers, 30.2 x 62.6 mm, 25 parts, among them J1 Conn_01x02, J2 Conn_01x02, J3 Conn_01x10, U1 DRV8873SPWPRQ1

Commit message: Test Hardware PCB
Parts:
- removed kibuzzard-6569A0F7: G***, kibuzzard-6569A0F7
- added D2: LED, test:led0603, F.Cu at (160.3, 93.8)
- added D3: LED, test:led0603, F.Cu at (153.3, 94.1)
- added R3: 330, test:res0603, F.Cu at (160.3, 95.8)
- added R9: 330, test:res0603, F.Cu at (153.3, 96.1)
- added SW1: SW_SPDT, test:SS12D00G3, F.Cu at (151.5, 79.3)
- added SW2: SW_SPDT, test:SS12D00G3, F.Cu at (151.5, 83.1)
- R5, R6: value 0 -> 1k
- U1: value DRV8873SPWPRQ1 -> ~
- moved R5 20.1 mm to (146.1, 79.3)
- moved R6 15.6 mm to (146.1, 83.1), turned to 90 degrees
- moved R1 2.00 mm to (153.3, 100.0)
- moved R2 0.50 mm to (153.3, 98.0)
Connections:
- J3 pad 6: /M CS -> /SR
- J3 pad 7: /M SCLK -> /MODE
- J3 pad 8: /M SDI -> /nSLEEP
- J3 pad 9: /M SDO -> GND
- R5 pad 1: Net-(U1-SDO) -> /nOL
- R5 pad 2: /M SDO -> Net-(SW1-B)
- R6 pad 1: /M SDI -> /nITRIP
- R6 pad 2: Net-(U1-SDI) -> Net-(SW2-B)
- U1 pad 3: Net-(U1-SDO) -> /MODE
- U1 pad 4: Net-(U1-SDI) -> /SR
- U1 pad 5: /M SCLK -> /nITRIP
- U1 pad 6: /M CS -> /nOL
Routing:
- net /nOL: track 0.00 -> 56.6 mm, vias 0 -> 2
- net /nITRIP: track 0.00 -> 47.6 mm, vias 0 -> 2
- net /nSLEEP: track 5.70 -> 47.0 mm, vias 0 -> 1
- net +5V: track 32.9 -> 52.2 mm
- net Net-(U1-SDO): track 15.9 -> 0.00 mm
- net /M SCLK: track 14.7 -> 0.00 mm
- net /MODE: track 0.00 -> 14.1 mm
- net /M CS: track 13.9 -> 0.00 mm
- net Net-(U1-SDI): track 13.8 -> 0.00 mm
- net /SR: track 0.00 -> 13.3 mm
- net /DISABLE: track 11.5 -> 24.8 mm, vias 0 -> 1
- net Net-(SW1-B): track 0.00 -> 6.35 mm
- net Net-(SW2-B): track 0.00 -> 6.35 mm
- net /M SDO: track 3.20 -> 0.00 mm
- net /M SDI: track 3.20 -> 0.00 mm
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Other:
- board text added: "FAULT"
- board text added: "MODE"
- board text added: "SLEEP"
- board text added: "SLP"
- board text added: "SR"
- board text removed: "CS"
- board text removed: "SCLK"
- board text removed: "SDI"
- board text removed: "SDO"

Commit message: Test PCBS
Parts:
- removed the R3 at (138.8, 98.0)
- added kibuzzard-656D5855: G***, kibuzzard-656D5855, F.Cu at (163.9, 106.6)
Routing:
- net +5V: track 52.2 -> 42.0 mm
- net /nSLEEP: track 47.0 -> 44.1 mm

Commit message: Production Files
Parts:
- removed H1, H2, H3, H4: MountingHole_Pad, MountingHole:MountingHole_3.2mm_M3_Pad_Via
- moved SW2 7.71 mm to (143.9, 81.8), turned to 180 degrees
- moved R5 5.77 mm to (151.3, 81.8)
- moved SW1 5.77 mm to (156.7, 81.8)
- moved R6 3.48 mm to (149.3, 81.8)
Routing:
- net /nOL: track 56.6 -> 47.9 mm
- net /nITRIP: track 47.6 -> 45.0 mm
- net Net-(SW2-B): track 6.35 -> 7.07 mm
- net Net-(SW1-B): track 6.35 -> 7.07 mm
- net +5V: track 42.0 -> 42.6 mm
Other:
- board text added: "nOL"
- board text added: "nTRIP"
