File: test (Hardware)/test(Hardware).kicad_sch (KiCad schematic)
At the start: 20 parts, among them J1 Conn_01x02, J2 Conn_01x02, J3 Conn_01x10

Commit message: Test Hardware PCB
Parts:
- added D2, D3: LED, test:led0603, symbol Device:LED
- added R5, R6: 1k, test:res0603, symbol Device:R
- added R9: 330, test:res0603, symbol Device:R
- added SW1, SW2: SW_SPDT, test:SS12D00G3, symbol Switch:SW_SPDT
- R3: value 1k -> 330
- U1: footprint (none) -> test:SOP65P640X120-25N
Connections:
- net M CS is gone; now on net SR: J3.6 (Pin_6)
- net M SCLK is gone; now on net MODE: J3.7 (Pin_7)
- net M SDI is gone; now on net nSLEEP: J3.8 (Pin_8)
- net M SDO is gone; now on net GND: J3.9 (Pin_9)
- net +5V: now also SW1.1 (A), SW2.1 (A); no longer R3.2
- net DISABLE: now also D3.2 (A)
- net GND: now also R3.2, R9.2, SW1.3 (C), SW2.3 (C)
- net nSLEEP: now also D2.2 (A); no longer R3.1
- net MODE: now reaches U1.3 (MODE)
- net SR: now reaches U1.4 (SR)
- net nITRIP: now reaches U1.5 (nITRIP)
- net nITRIP: now also R6.1
- net nOL: now reaches U1.6 (nOL)
- net nOL: now also R5.1
- new net: D3.1 (K), R9.1
- new net: R6.2, SW2.2 (B)
- new net: D2.1 (K), R3.1
- new net: R5.2, SW1.2 (B)
Other:
- note added: "LED"
- note added: "Switches"

Commit message: Production Files
Parts:
- removed H1, H2, H3, H4: MountingHole_Pad, MountingHole:MountingHole_3.2mm_M3_Pad_Via, symbol Mechanical:MountingHole_Pad
- D1, D2, D3: LCSC (none) -> C219228
- R1, R3, R9: LCSC (none) -> C23138
- R2: LCSC (none) -> C25804
- R4: LCSC (none) -> C21189
- R5, R6: LCSC (none) -> C21190
- R7, R8: LCSC (none) -> C23151
Connections:
- no-connect marks 4 -> 0
Changed lines of the file:
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@@
   (junction (at 106.68 125.73) (diameter 0) (color 0 0 0 0)
   )
-  (no_connect (at 74.8602 69.3144))
-  (no_connect (at 96.4502 69.3144))
-  (no_connect (at 96.4502 79.4744))
-  (no_connect (at 74.8602 79.4744))
   (wire (pts (xy 41.3541 63.7527) (xy 51.5141 63.7527))
     (stroke (width 0) (type default))
@@
       (effects (font (size 1.27 1.27)) hide)
     )
+    (property "LCSC" "C23138" (at 156.21 78.486 0)
+      (effects (font (size 1.27 1.27)) hide)
+    )
     (pin "1")
     (pin "2")
@@
         (path "/02e617c3-633b-46b1-afa5-6a0d8b377d88"
           (reference "R9") (unit 1)
-        )
-      )
-    )
-  )
-  (symbol (lib_id "Mechanical:MountingHole_Pad") (at 96.4502 66.7744 0) (unit 1)
-    (in_bom yes) (on_board yes) (dnp no) (fields_autoplaced)
-    (property "Reference" "H2" (at 98.9902 64.8694 0)
-      (effects (font (size 1.27 1.27)) (justify left))
-    )
-    (property "Value" "MountingHole_Pad" (at 98.9902 67.4094 0)
-      (effects (font (size 1.27 1.27)) (justify left))
-    )
-    (property "Footprint" "MountingHole:MountingHole_3.2mm_M3_Pad_Via" (at 96.4502 66.7744 0)
-      (effects (font (size 1.27 1.27)) hide)
-    )
-    (property "Datasheet" "~" (at 96.4502 66.7744 0)
-      (effects (font (size 1.27 1.27)) hide)
-    )
-    (pin "1")
-    (instances
-      (project "test(Hardware)"
-        (path "/02e617c3-633b-46b1-afa5-6a0d8b377d88"
-          (reference "H2") (unit 1)
         )
       )
@@
     )
   )
-  (symbol (lib_id "Mechanical:MountingHole_Pad") (at 74.8602 66.7744 0) (unit 1)
-    (in_bom yes) (on_board yes) (dnp no) (fields_autoplaced)
-    (property "Reference" "H1" (at 77.4002 64.8694 0)
-      (effects (font (size 1.27 1.27)) (justify left))
-    )
-    (property "Value" "MountingHole_Pad" (at 77.4002 67.4094 0)
-      (effects (font (size 1.27 1.27)) (justify left))
-    )
-    (property "Footprint" "MountingHole:MountingHole_3.2mm_M3_Pad_Via" (at 74.8602 66.7744 0)
-      (effects (font (size 1.27 1.27)) hide)
-    )
-    (property "Datasheet" "~" (at 74.8602 66.7744 0)
-      (effects (font (size 1.27 1.27)) hide)
-    )
-    (pin "1")
-    (instances
-      (project "test(Hardware)"
-        (path "/02e617c3-633b-46b1-afa5-6a0d8b377d88"
-          (reference "H1") (unit 1)
-        )
-      )
-    )
-  )
   (symbol (lib_id "Device:LED") (at 156.21 68.326 90) (unit 1)
     (in_bom yes) (on_board yes) (dnp no) (fields_autoplaced)
@@
       (effects (font (size 1.27 1.27)) hide)
     )
+    (property "LCSC" "C219228" (at 156.21 68.326 90)
+      (effects (font (size 1.27 1.27)) hide)
+    )
     (pin "1")
     (pin "2")
@@
     )
     (property "Datasheet" "~" (at 132.08 76.2 0)
+      (effects (font (size 1.27 1.27)) hide)
+    )
+    (property "LCSC" "C23138" (at 132.08 76.2 0)
       (effects (font (size 1.27 1.27)) hide)
     )
@@
       (effects (font (size 1.27 1.27)) hide)
     )
+    (property "LCSC" "C23151" (at 125.73 167.64 0)
+      (effects (font (size 1.27 1.27)) hide)
+    )
     (pin "1")
     (pin "2")
@@
         (path "/02e617c3-633b-46b1-afa5-6a0d8b377d88"
           (reference "R8") (unit 1)
-        )
-      )
-    )
-  )
-  (symbol (lib_id "Mechanical:MountingHole_Pad") (at 74.8602 76.9344 0) (unit 1)
-    (in_bom yes) (on_board yes) (dnp no) (fields_autoplaced)
-    (property "Reference" "H4" (at 77.4002 75.0294 0)
-      (effects (font (size 1.27 1.27)) (justify left))
-    )
-    (property "Value" "MountingHole_Pad" (at 77.4002 77.5694 0)
-      (effects (font (size 1.27 1.27)) (justify left))
-    )
-    (property "Footprint" "MountingHole:MountingHole_3.2mm_M3_Pad_Via" (at 74.8602 76.9344 0)
-      (effects (font (size 1.27 1.27)) hide)
-    )
-    (property "Datasheet" "~" (at 74.8602 76.9344 0)
-      (effects (font (size 1.27 1.27)) hide)
-    )
-    (pin "1")
-    (instances
-      (project "test(Hardware)"
-        (path "/02e617c3-633b-46b1-afa5-6a0d8b377d88"
-          (reference "H4") (unit 1)
         )
       )
@@
       (effects (font (size 1.27 1.27)) hide)
     )
+    (property "LCSC" "C21189" (at 115.57 152.4 90)
+      (effects (font (size 1.27 1.27)) hide)
+    )
     (pin "1")
     (pin "2")
@@
     )
     (property "Datasheet" "~" (at 118.11 167.64 0)
+      (effects (font (size 1.27 1.27)) hide)
+    )
+    (property "LCSC" "C23151" (at 118.11 167.64 0)
       (effects (font (size 1.27 1.27)) hide)
     )
@@
     )
   )
-  (symbol (lib_id "Mechanical:MountingHole_Pad") (at 96.4502 76.9344 0) (unit 1)
-    (in_bom yes) (on_board yes) (dnp no) (fields_autoplaced)
-    (property "Reference" "H3" (at 98.9902 75.0294 0)
-      (effects (font (size 1.27 1.27)) (justify left))
-    )
-    (property "Value" "MountingHole_Pad" (at 98.9902 77.5694 0)
-      (effects (font (size 1.27 1.27)) (justify left))
-    )
-    (property "Footprint" "MountingHole:MountingHole_3.2mm_M3_Pad_Via" (at 96.4502 76.9344 0)
-      (effects (font (size 1.27 1.27)) hide)
-    )
-    (property "Datasheet" "~" (at 96.4502 76.9344 0)
-      (effects (font (size 1.27 1.27)) hide)
-    )
-    (pin "1")
-    (instances
-      (project "test(Hardware)"
-        (path "/02e617c3-633b-46b1-afa5-6a0d8b377d88"
-          (reference "H3") (unit 1)
-        )
-      )
-    )
-  )
   (symbol (lib_id "power:+3V3") (at 132.08 59.69 0) (unit 1)
     (in_bom yes) (on_board yes) (dnp no) (fields_autoplaced)
@@
       (effects (font (size 1.27 1.27)) hide)
     )
+    (property "LCSC" "C25804" (at 24.13 135.89 0)
+      (effects (font (size 1.27 1.27)) hide)
+    )
     (pin "1")
     (pin "2")
@@
       (effects (font (size 1.27 1.27)) hide)
     )
+    (property "LCSC" "C219228" (at 132.08 66.04 90)
+      (effects (font (size 1.27 1.27)) hide)
+    )
     (pin "1")
     (pin "2")
@@
     )
     (property "Datasheet" "~" (at 145.415 78.613 0)
+      (effects (font (size 1.27 1.27)) hide)
+    )
+    (property "LCSC" "C23138" (at 145.415 78.613 0)
       (effects (font (size 1.27 1.27)) hide)
     )
@@
     )
     (property "Datasheet" "~" (at 145.415 68.453 0)
+      (effects (font (size 1.27 1.27)) hide)
+    )
+    (property "LCSC" "C219228" (at 145.415 68.453 90)
       (effects (font (size 1.27 1.27)) hide)
     )
@@
       (effects (font (size 1.27 1.27)) hide)
     )
+    (property "LCSC" "C21190" (at 195.707 62.992 90)
+      (effects (font (size 1.27 1.27)) hide)
+    )
     (pin "1")
     (pin "2")
@@
       (effects (font (size 1.27 1.27)) hide)
     )
+    (property "LCSC" "C21190" (at 195.707 82.042 90)
+      (effects (font (size 1.27 1.27)) hide)
+    )
