File: test (SPI)/test.kicad_pcb (KiCad board)
At the start: 2 copper layers, 30.2 x 62.6 mm, 25 parts, among them J1 Conn_01x02, J2 Conn_01x02, J3 Conn_01x10, U1 DRV8873SPWPRQ1

Commit message: Test PCBS
Parts:
- removed kibuzzard-6569A0F7: G***, kibuzzard-6569A0F7
- added D2: LED, test:led0603, F.Cu at (152.6, 84.0)
- added D3: LED, test:led0603, F.Cu at (148.1, 84.0)
- added R9: 330, test:res0603, F.Cu at (148.1, 82.0)
- added kibuzzard-656D5CE4: G***, kibuzzard-656D5CE4, F.Cu at (164.6, 106.5)
- J3: value Conn_01x10 -> Conn_01x12; footprint Connector_PinSocket_2.54mm:PinSocket_1x10_P2.54mm_Vertical -> Connector_PinSocket_2.54mm:PinSocket_1x12_P2.54mm_Vertical
- R3: value 1k -> 330
- moved R3 21.2 mm to (152.6, 82.0)
- moved J3 2.55 mm to (136.2, 90.7)
Connections:
- J3 pad 1: +5V -> /nSLEEP
- J3 pad 10: GND -> /M SDO
- J3 pad 2: +3V3 -> +5V
- J3 pad 3: /DISABLE -> +3V3
- J3 pad 4: /PH/IN2 -> /DISABLE
- J3 pad 5: /EN/IN1 -> /PH/IN2
- J3 pad 6: /M CS -> /EN/IN1
- J3 pad 7: /M SCLK -> /M CS
- J3 pad 8: /M SDI -> /M SCLK
- J3 pad 9: /M SDO -> /M SDI
- R3 pad 1: /nSLEEP -> Net-(D2-K)
- R3 pad 2: +5V -> GND
Routing:
- net /nSLEEP: track 5.70 -> 30.1 mm, vias 0 -> 1
- net /DISABLE: track 11.5 -> 22.3 mm
- net +5V: track 32.9 -> 22.7 mm
- net Net-(D3-K): track 0.00 -> 2.00 mm
- net Net-(D2-K): track 0.00 -> 2.00 mm
- net /IPROPI1: track 7.88 -> 8.57 mm
Other:
- board size 30.2 x 62.6 mm -> 32.2 x 62.6 mm
- board text added: "FAULT"
- board text added: "SLEEP"
- board text added: "SLP"

Commit message: DRC Check
Update test(SPI) board in JLC
Routing:
- net /nSLEEP: track 30.1 -> 28.4 mm
Other:
- outline, holes or cut-outs redrawn
Changed lines of the file:
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@@
       (stroke (width 0) (type solid)) (fill solid) (layer "F.SilkS"))
   )
+  (gr_line (start 165.4 76.8) (end 135.6 76.8)
+    (stroke (width 0.1) (type default)) (layer "Edge.Cuts"))
+  (gr_line (start 165.4 139.4) (end 135.6 139.4)
+    (stroke (width 0.1) (type default)) (layer "Edge.Cuts"))
+  (gr_arc (start 165.4 76.8) (mid 166.248528 77.151472) (end 166.6 78)
+    (stroke (width 0.1) (type default)) (layer "Edge.Cuts"))
+  (gr_arc (start 135.6 139.4) (mid 134.751472 139.048528) (end 134.4 138.2)
+    (stroke (width 0.1) (type default)) (layer "Edge.Cuts"))
   (gr_line (start 166.6 78) (end 166.6 138.2)
     (stroke (width 0.1) (type default)) (layer "Edge.Cuts"))
   (gr_line (start 134.4 138.2) (end 134.4 78)
-    (stroke (width 0.1) (type default)) (layer "Edge.Cuts"))
-  (gr_line (start 165.4 139.4) (end 136.6 139.4)
-    (stroke (width 0.1) (type default)) (layer "Edge.Cuts"))
-  (gr_arc (start 165.4 76.8) (mid 166.248528 77.151472) (end 166.6 78)
-    (stroke (width 0.1) (type default)) (layer "Edge.Cuts"))
-  (gr_line (start 135.6 76.8) (end 165.4 76.8)
-    (stroke (width 0.1) (type default)) (layer "Edge.Cuts"))
-  (gr_arc (start 135.6 139.4) (mid 134.751472 139.048528) (end 134.4 138.2)
     (stroke (width 0.1) (type default)) (layer "Edge.Cuts"))
   (gr_arc (start 134.4 78) (mid 134.751472 77.151472) (end 135.6 76.8)
@@
   (segment (start 148.85 100.05) (end 150.5 100.05) (width 0.25) (layer "F.Cu") (net 9))
   (segment (start 147.925 102.062) (end 147.925 100.975) (width 0.25) (layer "F.Cu") (net 9))
-  (segment (start 141.33 97.95) (end 141.33 98.68) (width 0.25) (layer "F.Cu") (net 10))
   (segment (start 139.71 87.16) (end 136.17 90.7) (width 0.25) (layer "F.Cu") (net 10))
   (segment (start 147.32 83.95) (end 144.11 87.16) (width 0.25) (layer "F.Cu") (net 10))
   (segment (start 141.33 98.68) (end 142.075 99.425) (width 0.25) (layer "F.Cu") (net 10))
   (segment (start 139.6 98) (end 140.65 98) (width 0.25) (layer "F.Cu") (net 10))
-  (segment (start 141.73 97.55) (end 141.33 97.95) (width 0.25) (layer "F.Cu") (net 10))
   (segment (start 144.11 87.16) (end 139.71 87.16) (width 0.25) (layer "F.Cu") (net 10))
   (segment (start 142.075 99.425) (end 142.075 102.062) (width 0.25) (layer "F.Cu") (net 10))
   (segment (start 140.65 98) (end 141.33 98.68) (width 0.25) (layer "F.Cu") (net 10))
-  (via (at 141.73 97.55) (size 0.8) (drill 0.4) (layers "F.Cu" "B.Cu") (net 10))
-  (segment (start 141.73 97.55) (end 136.17 91.99) (width 0.25) (layer "B.Cu") (net 10))
-  (segment (start 136.17 91.99) (end 136.17 90.7) (width 0.25) (layer "B.Cu") (net 10))
+  (via (at 139.6 98) (size 0.8) (drill 0.4) (layers "F.Cu" "B.Cu") (net 10))
+  (segment (start 139.6 98) (end 139.59 98) (width 0.25) (layer "B.Cu") (net 10))
+  (segment (start 139.59 98) (end 136.17 94.58) (width 0.25) (layer "B.Cu") (net 10))
+  (segment (start 136.17 94.58) (end 136.17 90.7) (width 0.25) (layer "B.Cu") (net 10))
   (segment (start 159.04 93.89) (end 159.05 93.9) (width 0.25) (layer "F.Cu") (net 12))
   (segment (start 159.04 90.7) (end 159.04 93.89) (width 0.25) (layer "F.Cu") (net 12))

Commit message: Production Files
Parts:
- removed H1, H2, H3, H4: MountingHole_Pad, MountingHole:MountingHole_3.2mm_M3_Pad_Via
