File: test (SPI)/test.kicad_sch (KiCad schematic)
At the start: 22 parts, among them J1 Conn_01x02, J2 Conn_01x02, J3 Conn_01x10, U1 DRV8873SPWPRQ1

Commit message: Test PCBS
Parts:
- removed J3: Conn_01x10, Connector_PinSocket_2.54mm:PinSocket_1x10_P2.54mm_Vertical, symbol Connector_Generic:Conn_01x10
- added D2, D3: LED, test:led0603, symbol Device:LED
- added J3: Conn_01x12, Connector_PinSocket_2.54mm:PinSocket_1x12_P2.54mm_Vertical, symbol Connector_Generic:Conn_01x12
- added R9: 330, test:res0603, symbol Device:R
- R3: value 1k -> 330
Connections:
- net +3V3: now also J3.3 (Pin_3)
- net +5V: now also J3.2 (Pin_2); no longer R3.2
- net DISABLE: now also D2.2 (A), J3.4 (Pin_4)
- net EN/IN1: now also J3.6 (Pin_6)
- net GND: now also R3.2, J3.11 (Pin_11), J3.12 (Pin_12), R9.2
- net M CS: now also J3.7 (Pin_7)
- net M SCLK: now also J3.8 (Pin_8)
- net M SDI: now also J3.9 (Pin_9)
- net M SDO: now also J3.10 (Pin_10)
- net PH/IN2: now also J3.5 (Pin_5)
- net nSLEEP: now also D3.2 (A), J3.1 (Pin_1); no longer R3.1
- new net: D2.1 (K), R3.1
- new net: D3.1 (K), R9.1
Other:
- note added: "LED"

Commit message: Production Files
Parts:
- removed H1, H2, H3, H4: MountingHole_Pad, MountingHole:MountingHole_3.2mm_M3_Pad_Via, symbol Mechanical:MountingHole_Pad
- D1, D2, D3: LCSC (none) -> C219228
- R1, R3, R9: LCSC (none) -> C23138
- R2: LCSC (none) -> C25804
- R4, R5, R6: LCSC (none) -> C21189
- R7, R8: LCSC (none) -> C23151
Connections:
- no-connect marks 4 -> 0
Changed lines of the file:
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@@
   (junction (at 106.68 125.73) (diameter 0) (color 0 0 0 0)
   )
-  (no_connect (at 74.8602 69.3144))
-  (no_connect (at 96.4502 69.3144))
-  (no_connect (at 96.4502 79.4744))
-  (no_connect (at 74.8602 79.4744))
   (wire (pts (xy 133.3969 70.6027) (xy 133.3969 73.1427))
     (stroke (width 0) (type default))
@@
   (label "PH{slash}IN2" (at 59.69 146.05 0) (fields_autoplaced)
     (effects (font (size 1.27 1.27)) (justify left bottom))
-  )
-  (symbol (lib_id "Mechanical:MountingHole_Pad") (at 96.4502 66.7744 0) (unit 1)
-    (in_bom yes) (on_board yes) (dnp no) (fields_autoplaced)
-    (property "Reference" "H2" (at 98.9902 64.8694 0)
-      (effects (font (size 1.27 1.27)) (justify left))
-    )
-    (property "Value" "MountingHole_Pad" (at 98.9902 67.4094 0)
-      (effects (font (size 1.27 1.27)) (justify left))
-    )
-    (property "Footprint" "MountingHole:MountingHole_3.2mm_M3_Pad_Via" (at 96.4502 66.7744 0)
-      (effects (font (size 1.27 1.27)) hide)
-    )
-    (property "Datasheet" "~" (at 96.4502 66.7744 0)
-      (effects (font (size 1.27 1.27)) hide)
-    )
-    (pin "1")
-    (instances
-      (project "test"
-        (path "/02e617c3-633b-46b1-afa5-6a0d8b377d88"
-          (reference "H2") (unit 1)
-        )
-      )
-    )
   )
   (symbol (lib_id "power:+3V3") (at 34.6713 61.2127 0) (unit 1)
@@
     )
   )
-  (symbol (lib_id "Mechanical:MountingHole_Pad") (at 74.8602 66.7744 0) (unit 1)
-    (in_bom yes) (on_board yes) (dnp no) (fields_autoplaced)
-    (property "Reference" "H1" (at 77.4002 64.8694 0)
-      (effects (font (size 1.27 1.27)) (justify left))
-    )
-    (property "Value" "MountingHole_Pad" (at 77.4002 67.4094 0)
-      (effects (font (size 1.27 1.27)) (justify left))
-    )
-    (property "Footprint" "MountingHole:MountingHole_3.2mm_M3_Pad_Via" (at 74.8602 66.7744 0)
-      (effects (font (size 1.27 1.27)) hide)
-    )
-    (property "Datasheet" "~" (at 74.8602 66.7744 0)
-      (effects (font (size 1.27 1.27)) hide)
-    )
-    (pin "1")
-    (instances
-      (project "test"
-        (path "/02e617c3-633b-46b1-afa5-6a0d8b377d88"
-          (reference "H1") (unit 1)
-        )
-      )
-    )
-  )
   (symbol (lib_id "power:+12V") (at 46.99 132.08 0) (unit 1)
     (in_bom yes) (on_board yes) (dnp no) (fields_autoplaced)
@@
     )
     (property "Datasheet" "~" (at 54.61 163.83 0)
+      (effects (font (size 1.27 1.27)) hide)
+    )
+    (property "LCSC" "C21189" (at 54.61 163.83 90)
       (effects (font (size 1.27 1.27)) hide)
     )
@@
       (effects (font (size 1.27 1.27)) hide)
     )
+    (property "LCSC" "C23138" (at 133.3969 76.9527 0)
+      (effects (font (size 1.27 1.27)) hide)
+    )
     (pin "1")
     (pin "2")
@@
       (effects (font (size 1.27 1.27)) hide)
     )
+    (property "LCSC" "C23138" (at 157.5269 79.2387 0)
+      (effects (font (size 1.27 1.27)) hide)
+    )
     (pin "1")
     (pin "2")
@@
     )
     (property "Datasheet" "~" (at 146.7319 79.3657 0)
+      (effects (font (size 1.27 1.27)) hide)
+    )
+    (property "LCSC" "C23138" (at 146.7319 79.3657 0)
       (effects (font (size 1.27 1.27)) hide)
     )
@@
       (effects (font (size 1.27 1.27)) hide)
     )
+    (property "LCSC" "C21189" (at 54.61 166.37 90)
+      (effects (font (size 1.27 1.27)) hide)
+    )
     (pin "1")
     (pin "2")
@@
       (effects (font (size 1.27 1.27)) hide)
     )
+    (property "LCSC" "C23151" (at 125.73 167.64 0)
+      (effects (font (size 1.27 1.27)) hide)
+    )
     (pin "1")
     (pin "2")
@@
         (path "/02e617c3-633b-46b1-afa5-6a0d8b377d88"
           (reference "#PWR017") (unit 1)
-        )
-      )
-    )
-  )
-  (symbol (lib_id "Mechanical:MountingHole_Pad") (at 74.8602 76.9344 0) (unit 1)
-    (in_bom yes) (on_board yes) (dnp no) (fields_autoplaced)
-    (property "Reference" "H4" (at 77.4002 75.0294 0)
-      (effects (font (size 1.27 1.27)) (justify left))
-    )
-    (property "Value" "MountingHole_Pad" (at 77.4002 77.5694 0)
-      (effects (font (size 1.27 1.27)) (justify left))
-    )
-    (property "Footprint" "MountingHole:MountingHole_3.2mm_M3_Pad_Via" (at 74.8602 76.9344 0)
-      (effects (font (size 1.27 1.27)) hide)
-    )
-    (property "Datasheet" "~" (at 74.8602 76.9344 0)
-      (effects (font (size 1.27 1.27)) hide)
-    )
-    (pin "1")
-    (instances
-      (project "test"
-        (path "/02e617c3-633b-46b1-afa5-6a0d8b377d88"
-          (reference "H4") (unit 1)
         )
       )
@@
       (effects (font (size 1.27 1.27)) hide)
     )
+    (property "LCSC" "C21189" (at 115.57 152.4 90)
+      (effects (font (size 1.27 1.27)) hide)
+    )
     (pin "1")
     (pin "2")
@@
     )
     (property "Datasheet" "~" (at 118.11 167.64 0)
+      (effects (font (size 1.27 1.27)) hide)
+    )
+    (property "LCSC" "C23151" (at 118.11 167.64 0)
       (effects (font (size 1.27 1.27)) hide)
     )
@@
     )
   )
-  (symbol (lib_id "Mechanical:MountingHole_Pad") (at 96.4502 76.9344 0) (unit 1)
-    (in_bom yes) (on_board yes) (dnp no) (fields_autoplaced)
-    (property "Reference" "H3" (at 98.9902 75.0294 0)
-      (effects (font (size 1.27 1.27)) (justify left))
-    )
-    (property "Value" "MountingHole_Pad" (at 98.9902 77.5694 0)
-      (effects (font (size 1.27 1.27)) (justify left))
-    )
-    (property "Footprint" "MountingHole:MountingHole_3.2mm_M3_Pad_Via" (at 96.4502 76.9344 0)
-      (effects (font (size 1.27 1.27)) hide)
-    )
-    (property "Datasheet" "~" (at 96.4502 76.9344 0)
-      (effects (font (size 1.27 1.27)) hide)
-    )
-    (pin "1")
-    (instances
-      (project "test"
-        (path "/02e617c3-633b-46b1-afa5-6a0d8b377d88"
-          (reference "H3") (unit 1)
-        )
-      )
-    )
-  )
   (symbol (lib_id "Device:C") (at 54.61 132.08 90) (unit 1)
     (in_bom yes) (on_board yes) (dnp no)
@@
       (effects (font (size 1.27 1.27)) hide)
     )
+    (property "LCSC" "C25804" (at 24.13 135.89 0)
+      (effects (font (size 1.27 1.27)) hide)
+    )
     (pin "1")
     (pin "2")
@@
       (effects (font (size 1.27 1.27)) hide)
     )
+    (property "LCSC" "C219228" (at 133.3969 66.7927 90)
+      (effects (font (size 1.27 1.27)) hide)
+    )
     (pin "1")
     (pin "2")
@@
       (effects (font (size 1.27 1.27)) hide)
     )
+    (property "LCSC" "C219228" (at 146.7319 69.2057 90)
+      (effects (font (size 1.27 1.27)) hide)
+    )
     (pin "1")
     (pin "2")
@@
       (effects (font (size 1.27 1.27)) hide)
     )
+    (property "LCSC" "C219228" (at 157.5269 69.0787 90)
+      (effects (font (size 1.27 1.27)) hide)
+    )
