File: 2024l2 (VNH5019)/2024l2 (VNH5019).kicad_pcb (KiCad board)
At the start: 2 copper layers, 174 x 141 mm, 106 parts, among them IC1 LM2587S-ADJ, J10 Conn_01x03, J11 Conn_01x04, J2 Conn_01x02, J3 Conn_01x02, J4 Conn_01x02, J5 Conn_01x02, J6 Conn_01x02, J7 Conn_01x03, J8 Conn_01x06, J9 Conn_01x02, SW1 SW_SPST, U1 DRV8873SPWPRQ1, U2 DRV8873SPWPRQ1, U3 TPS5430DDA, U4 TPS5430DDA, U5 DRV8873SPWPRQ1, U6 DRV8873SPWPRQ1, U7 Teensy 4.0

Commit message: 5019 L2 Routing
Parts:
- removed the C13 at (167.4, 186.8)
- removed the C14 at (137.4, 186.8)
- removed C21, C24: 1u, 2024l2:cap0603
- removed C22, C25: 470u, Capacitor_SMD:CP_Elec_10x10.5
- removed C23, C26: 0u1, 2024l2:cap0603
- removed C27, C28: 47n, 2024l2:cap0603
- removed the C5 at (167.4, 188.8)
- removed the C6 at (137.3, 188.8)
- removed the C7 at (126.0, 191.2)
- removed the C8 at (167.4, 190.7)
- removed the R25 at (172.6, 186.1)
- removed the R4 at (177.3, 177.3)
- removed the R5 at (177.3, 173.4)
- removed the R6 at (161.2, 175.1)
- removed the U1 at (171.0, 180.3)
- removed the U2 at (156.0, 180.3)
- removed kibuzzard-65260DBA: G***, kibuzzard-65260DBA
- added C16: 1uF, 2024l2:cap0603, B.Cu at (132.1, 182.5)
- added C17: 1uF, 2024l2:cap0603, B.Cu at (170.1, 182.5)
- added Q1: AOD482, 2024l2:AOD482, F.Cu at (125.6, 181.9)
- added Q2: AOD482, 2024l2:AOD482, F.Cu at (163.6, 181.9)
- added Q3: AOD482, 2024l2:AOD482, F.Cu at (144.6, 181.9)
- added Q4: AOD482, 2024l2:AOD482, F.Cu at (182.6, 181.9)
- added R18: 1k, 2024l2:res0603, B.Cu at (153.1, 182.5)
- added R19: 1k, 2024l2:res0603, B.Cu at (165.1, 182.5)
- added R20: 1k, 2024l2:res0603, B.Cu at (159.1, 182.5)
- added R31: 1k, 2024l2:res0603, B.Cu at (146.1, 182.5)
- added R32: 1k, 2024l2:res0603, B.Cu at (140.1, 182.5)
- added R33: 1k, 2024l2:res0603, B.Cu at (172.1, 182.5)
- added R34: 1k, 2024l2:res0603, B.Cu at (184.1, 182.5)
- added R35: 1k, 2024l2:res0603, B.Cu at (178.1, 182.5)
- added R8: 1k, 2024l2:res0603, B.Cu at (125.1, 182.5)
- added R9: 1k, 2024l2:res0603, B.Cu at (155.1, 182.5)
- added U4: ~, Package_SO:ST_MultiPowerSO-30, B.Cu at (120.0, 196.0)
- added U7: ~, Package_SO:ST_MultiPowerSO-30, B.Cu at (177.0, 196.0)
- C10, C9: value 1u -> 1uF
- C11: value 470u -> 680uF
- C12: value 0u1 -> 680uF; footprint 2024l2:cap0603 -> Capacitor_SMD:CP_Elec_10x10.5; moved to F.Cu
- C19, C20: value 1u -> 680uF; footprint 2024l2:cap0603 -> Capacitor_SMD:CP_Elec_10x10.5; moved to F.Cu
- R10, R7: value 1K5 -> 1k
- R11, R12, R13: value 1K5 -> 3k3
- R14: value 10k -> 3k3
- R15, R16, R17: value 10k -> 1k
- R21, R22, R23, R24: value 10K -> 1k
- R26, R27, R28: value 0 -> 3k3
- R29: value 0 -> 3k3; moved to B.Cu
- R30: value 0 -> 1k; moved to B.Cu
- U5, U6: value DRV8873SPWPRQ1 -> ~; footprint 2024l2:SOP65P640X120-25N -> Package_SO:ST_MultiPowerSO-30
- moved R15 62.6 mm to (115.1, 182.5), turned to -90 degrees
- moved R24 60.9 mm to (182.1, 182.5), turned to 90 degrees
- moved C9 52.7 mm to (113.1, 182.5), turned to 90 degrees
- moved J7 51.9 mm to (120.1, 209.5)
- moved C20 51.4 mm to (173.3, 181.8), turned to 90 degrees
- moved J10 50.2 mm to (177.1, 209.5)
- moved R7 45.5 mm to (117.1, 182.5), turned to -90 degrees
- moved R30 41.4 mm to (134.1, 182.5), turned to -90 degrees
- moved R27 37.7 mm to (180.1, 182.5), turned to -90 degrees
- moved R21 32.5 mm to (136.1, 182.5), turned to -90 degrees
- moved R12 30.9 mm to (161.1, 182.5), turned to -90 degrees
- moved R29 30.3 mm to (176.1, 182.5), turned to -90 degrees
- moved C11 26.4 mm to (116.3, 181.8)
- moved R11 25.7 mm to (123.1, 182.5), turned to -90 degrees
- moved R23 24.7 mm to (174.1, 182.5), turned to -90 degrees
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- renumbered C4 to C1, C29 to C13, C30 to C14, C32 to C15, C31 to C18, C18 to C2, C1 to C3, C15 to C4, C2 to C5, C16 to C6, C3 to C7, C17 to C8, H14 to H10, H3 to H11, H6 to H12, H9 to H13, H12 to H14, H4 to H2, H7 to H3, H10 to H4, H13 to H5, H2 to H6, H5 to H7, H11 to H9, J4 to J1, J9 to J10, J5 to J2, J7 to J3, J10 to J4, J11 to J5, J8 to J6, J2 to J7, J3 to J8, J6 to J9, R19 to R25, R1 to R3, R20 to R36, R18 to R37, R3 to R38, R2 to R4, R8 to R5, R9 to R6, U3 to U1, U4 to U2, U7 to U3
Connections:
- C10 pad 1: +5V -> Net-(Q2-D)
- C11 pad 1: +12V -> Net-(Q1-D)
- C12 pad 1: +12V -> Net-(Q2-D)
- C19 pad 1: +12V -> Net-(Q3-D)
- C19 pad 2: /M2 VCP -> GND
- C20 pad 1: +12V -> Net-(Q4-D)
- C20 pad 2: /M4 VCP -> GND
- C9 pad 1: +5V -> Net-(Q1-D)
- J10 pad 1: /M4 OUT1 -> /M4 OUTA
- J10 pad 2: /M4 OUT2 -> /M4 OUTB
- J7 pad 1: /M1 OUT1 -> /M1 OUTA
- J7 pad 2: /M1 OUT2 -> /M1 OUTB
- J8 pad 1: /M2 OUT1 -> /M2 OUTA
- J8 pad 2: /M2 OUT2 -> /M2 OUTB
- J9 pad 1: /M3 OUT1 -> /M3 OUTA
- J9 pad 2: /M3 OUT2 -> /M3 OUTB
- R10 pad 1: /M3 IPROPI2 -> Net-(U5-ENB)
- R10 pad 2: GND -> /M SW
- R11 pad 1: /M3 IPROPI1 -> +5V
- R11 pad 2: GND -> Net-(U4-ENB)
- R12 pad 1: /M4 IPROPI2 -> +5V
- R12 pad 2: GND -> Net-(U5-ENB)
- R13 pad 1: /M4 IPROPI1 -> +5V
- R13 pad 2: GND -> Net-(U4-ENA)
- R14 pad 1: Net-(U2-NSLEEP) -> +5V
- R14 pad 2: +5V -> Net-(U5-ENA)
- R15 pad 1: Net-(U1-NSLEEP) -> /M1 INA
- R15 pad 2: +5V -> Net-(U4-INA)
- R16 pad 1: Net-(U5-NSLEEP) -> Net-(U4-INB)
- R16 pad 2: +5V -> /M1 INB
- R17 pad 1: Net-(U6-NSLEEP) -> Net-(R17-Pad1)
- R17 pad 2: +5V -> /M1 PWM
- R21 pad 1: +3V3 -> /M SW
- R21 pad 2: /M1 nFAULT -> Net-(U6-ENA)
- R22 pad 1: +3V3 -> Net-(U6-ENB)
- R22 pad 2: /M3 nFAULT -> /M SW
- R23 pad 1: +3V3 -> /M SW
- R23 pad 2: /M2 nFAULT -> Net-(U7-ENA)
- R24 pad 1: +3V3 -> Net-(U7-ENB)
- R24 pad 2: /M4 nFAULT -> /M SW
- R26 pad 1: GND -> +5V
- R26 pad 2: Net-(U2-SRC_1) -> Net-(U6-ENB)
- R27 pad 1: GND -> +5V
- R27 pad 2: Net-(U5-SRC_1) -> Net-(U7-ENB)
- R28 pad 1: GND -> +5V
- R28 pad 2: Net-(U6-SRC_1) -> Net-(U6-ENA)
- R29 pad 1: /M SDO -> +5V
- R29 pad 2: Net-(U7-11/MOSI) -> Net-(U7-ENA)
- R30 pad 1: /M SDI -> /M2 INA
- R30 pad 2: Net-(U7-12/MISO) -> Net-(U6-INA)
- R7 pad 1: /M2 IPROPI1 -> /M SW
- R7 pad 2: GND -> Net-(U4-ENA)
- U3 pad 0: /M CS 4 -> /M1 INA
- U3 pad 1: /M4 EN -> /M1 PWM
- U3 pad 10: /M1 EN -> /M4 PWM
- U3 pad 11: Net-(U7-11/MOSI) -> /M4 INB
- U3 pad 12: Net-(U7-12/MISO) -> unconnected-(U3-12/MISO-Pad12)
- U3 pad 13: /M SCLK -> unconnected-(U3-13/SCL/LED-Pad13)
- U3 pad 18: /M1 PH -> unconnected-(U3-18/A4/SDA0-Pad18)
- U3 pad 2: /M4 PH -> /M1 INB
- U3 pad 3: /M CS 3 -> /M2 INA
- U3 pad 4: /M3 EN -> /M2 PWM
- U3 pad 5: /M3 PH -> /M2 INB
- U3 pad 6: /M CS 2 -> /M3 INA
- U3 pad 7: /M2 EN -> /M3 PWM
- U3 pad 8: /M2 PH -> /M3 INB
- U3 pad 9: /M CS 1 -> /M4 INA
- U5 pad 1: +5V -> /M3 OUTA
- U5 pad 10: /M3 IPROPI1 -> Net-(U5-INB)
- U5 pad 11: Net-(U5-NSLEEP) -> Net-(Q2-G)
- U5 pad 12: /M3 IPROPI2 -> +12V
- U5 pad 13: +12V -> Net-(Q2-D)
- U5 pad 14: /M3 OUT2 -> (no net)
- U5 pad 15: /M3 OUT2 -> /M3 OUTB
- U5 pad 16: Net-(U5-SRC_1) -> /M3 OUTB
- U5 pad 17: Net-(U5-SRC_1) -> (no net)
- U5 pad 18: /M3 OUT1 -> GND
- U5 pad 19: /M3 OUT1 -> GND
- U5 pad 2: /M3 nFAULT -> (no net)
- U5 pad 20: +12V -> GND
- U5 pad 21: /M3 VCP -> /M3 OUTB
- U5 pad 22: /M3 CPH -> (no net)
- U5 pad 23: /M3 CPL -> Net-(Q2-D)
- U5 pad 24: GND -> (no net)
- U5 pad 25: GND -> /M3 OUTA
- U5 pad 3: /M SDO -> Net-(Q2-D)
- U5 pad 4: /M SDI -> Net-(U5-INA)
- U5 pad 5: /M SCLK -> Net-(U5-ENA)
- U5 pad 6: /M CS 3 -> unconnected-(U5-CS_DIS-Pad6)
- U5 pad 7: /M3 EN -> Net-(R20-Pad1)
- U5 pad 8: /M3 PH -> unconnected-(U5-CS-Pad8)
- U5 pad 9: /M SW -> Net-(U5-ENB)
- U6 pad 1: +5V -> /M2 OUTA
- U6 pad 10: /M4 IPROPI1 -> Net-(U6-INB)
- U6 pad 11: Net-(U6-NSLEEP) -> Net-(Q3-G)
- U6 pad 12: /M4 IPROPI2 -> +12V
- U6 pad 13: +12V -> Net-(Q3-D)
- U6 pad 14: /M4 OUT2 -> (no net)
- U6 pad 15: /M4 OUT2 -> /M2 OUTB
- U6 pad 16: Net-(U6-SRC_1) -> /M2 OUTB
- U6 pad 17: Net-(U6-SRC_1) -> (no net)
- U6 pad 18: /M4 OUT1 -> GND
- U6 pad 19: /M4 OUT1 -> GND
- U6 pad 2: /M4 nFAULT -> (no net)
- U6 pad 20: +12V -> GND
- U6 pad 21: /M4 VCP -> /M2 OUTB
- U6 pad 22: /M4 CPH -> (no net)
- U6 pad 23: /M4 CPL -> Net-(Q3-D)
- U6 pad 24: GND -> (no net)
- U6 pad 25: GND -> /M2 OUTA
- U6 pad 3: /M SDO -> Net-(Q3-D)
- U6 pad 4: /M SDI -> Net-(U6-INA)
- U6 pad 5: /M SCLK -> Net-(U6-ENA)
- U6 pad 6: /M CS 4 -> unconnected-(U6-CS_DIS-Pad6)
- U6 pad 7: /M4 EN -> Net-(R32-Pad1)
- U6 pad 8: /M4 PH -> unconnected-(U6-CS-Pad8)
- U6 pad 9: /M SW -> Net-(U6-ENB)
Routing:
- net /M SW: track 144.4 -> 2.28 mm, vias 4 -> 0
- net +5V: track 282.6 -> 146.2 mm, vias 4 -> 0
- net /M SCLK: track 118.5 -> 0.00 mm, vias 4 -> 0
- net /M SDO: track 114.0 -> 0.00 mm, vias 4 -> 0
- net /M SDI: track 106.8 -> 0.00 mm, vias 4 -> 0
- net +3V3: track 198.6 -> 131.9 mm, vias 5 -> 0
- net /M1 PH: track 48.1 -> 0.00 mm
- net /M CS 1: track 30.2 -> 0.00 mm
- net /M4 PH: track 30.0 -> 0.00 mm
- net /M1 EN: track 29.4 -> 0.00 mm
- net /M4 EN: track 29.2 -> 0.00 mm
- net +12V: track 228.2 -> 199.3 mm, vias 24 -> 4
- net /M CS 4: track 28.4 -> 0.00 mm
- net /M CS 2: track 27.2 -> 0.00 mm
- net /M3 PH: track 26.9 -> 0.00 mm
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- added copper zone on B.Cu, net /M1 OUTA
- added copper zone on B.Cu, net /M1 OUTB
- added copper zone on B.Cu, net /M2 OUTA
- added copper zone on B.Cu, net /M2 OUTB
- added copper zone on B.Cu, net /M3 OUTA
- added copper zone on B.Cu, net /M3 OUTB
- added copper zone on B.Cu, net /M4 OUTA
- added copper zone on B.Cu, net /M4 OUTB
- added copper zone on B.Cu, net Net-(Q1-D)
- added copper zone on F.Cu, net Net-(Q1-D)
- added copper zone on B.Cu, net Net-(Q2-D)
- added copper zone on F.Cu, net Net-(Q2-D)
- added copper zone on B.Cu, net Net-(Q3-D)
- added copper zone on F.Cu, net Net-(Q3-D)
- added copper zone on B.Cu, net Net-(Q4-D)
- added copper zone on F.Cu, net Net-(Q4-D)
- removed copper zone on F.Cu, net +12V
- removed copper zone on B.Cu, net /M1 OUT1
- removed copper zone on B.Cu, net /M1 OUT2
- removed copper zone on B.Cu, net /M2 OUT1
- removed copper zone on B.Cu, net /M2 OUT2
- removed copper zone on B.Cu, net /M3 OUT1
- removed copper zone on B.Cu, net /M3 OUT2
- removed copper zone on B.Cu, net /M4 OUT1
- removed copper zone on B.Cu, net /M4 OUT2
- removed copper zone on B.Cu, net Net-(U1-SRC_1)
- removed copper zone on B.Cu, net Net-(U2-SRC_1)
- removed copper zone on B.Cu, net Net-(U5-SRC_1)
- removed copper zone on B.Cu, net Net-(U6-SRC_1)

Commit message: 5019 L2 routing
Routing:
- net /M SW: track 2.28 -> 244.1 mm, vias 0 -> 8
- net +5V: track 146.2 -> 317.7 mm, vias 0 -> 9
- net /M4 INB: track 0.00 -> 38.0 mm
- net /M4 PWM: track 0.00 -> 37.2 mm
- net /M1 INA: track 0.00 -> 37.1 mm
- net /M4 INA: track 0.00 -> 35.9 mm
- net /M1 PWM: track 0.00 -> 35.7 mm
- net /M1 INB: track 0.00 -> 34.3 mm
- net /M3 INB: track 0.00 -> 33.3 mm
- net /M2 INA: track 0.00 -> 32.4 mm
- net /M3 PWM: track 0.00 -> 31.9 mm
- net /M3 INA: track 0.00 -> 31.3 mm
- net /M2 PWM: track 0.00 -> 31.0 mm
- net /M2 INB: track 0.00 -> 30.4 mm
- net +12V: track 199.3 -> 227.1 mm
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- added copper zone on F.Cu, net +12V

Commit message: Vnh5019
Parts:
- moved R16 3.00 mm to (130.1, 182.5)
- moved R8 3.00 mm to (128.1, 182.5)
- moved C17 3.00 mm to (167.1, 182.5)
- moved C9 3.00 mm to (116.1, 182.5)
- moved R11 3.00 mm to (126.1, 182.5)
- moved R13 3.00 mm to (122.1, 182.5)
- moved R15 3.00 mm to (118.1, 182.5)
- moved R17 3.00 mm to (124.1, 182.5)
- moved R23 3.00 mm to (171.1, 182.5)
- moved R24 3.00 mm to (179.1, 182.5)
- moved R27 3.00 mm to (177.1, 182.5)
- moved R29 3.00 mm to (173.1, 182.5)
- moved R33 3.00 mm to (169.1, 182.5)
- moved R34 3.00 mm to (181.1, 182.5)
- moved R35 3.00 mm to (175.1, 182.5)
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Routing:
- net +12V: track 227.1 -> 213.3 mm
- net +5V: track 317.7 -> 312.6 mm
- net /M SW: track 244.1 -> 239.0 mm
- net Net-(Q4-D): track 4.37 -> 7.60 mm
- net Net-(U4-INB): track 7.10 -> 9.94 mm
- net Net-(U7-INB): track 7.10 -> 4.44 mm
- net Net-(U4-ENB): track 6.44 -> 9.07 mm
- net Net-(R17-Pad1): track 4.44 -> 6.94 mm
- net Net-(U7-INA): track 3.96 -> 6.02 mm
- net /M4 INA: track 35.9 -> 34.6 mm
- net /M1 PWM: track 35.7 -> 34.5 mm
- net /M1 INB: track 34.3 -> 33.0 mm
- net /M1 INA: track 37.1 -> 35.9 mm
- net Net-(U4-ENA): track 5.61 -> 6.85 mm
- net /M4 INB: track 38.0 -> 36.8 mm
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
Commit message: Pull down resistors
Parts:
- added R1: 10k, 2024l2:res0603, B.Cu at (137.1, 149.6)
- added R2: 10k, 2024l2:res0603, B.Cu at (152.3, 149.6)
- added R39: 10k, 2024l2:res0603, B.Cu at (144.7, 149.6)
- added R40: 10k, 2024l2:res0603, B.Cu at (159.9, 149.6)
Routing:
- net /M4 PWM: track 36.2 -> 38.4 mm
- net /M3 PWM: track 31.9 -> 34.1 mm
- net /M2 PWM: track 31.0 -> 33.2 mm
- net /M1 PWM: track 34.5 -> 36.7 mm

Commit message: L3 Redo
Parts:
- added SW2: SW_SPDT, 2024l3:SS12D00G3, F.Cu at (134.7, 131.1)
Connections:
- U3 pad VIN: +5V -> /TEENSY PWR
Routing:
- net +5V: track 312.6 -> 304.8 mm
- net /TEENSY PWR: track 0.00 -> 7.38 mm
Changed lines of the file:
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@@
   (net 106 "unconnected-(U7-CS_DIS-Pad6)")
   (net 107 "unconnected-(U7-CS-Pad8)")
+  (net 108 "/TEENSY PWR")
+  (net 109 "unconnected-(SW2-C-Pad3)")
   (footprint "MountingHole:MountingHole_3.2mm_M3_Pad_Via" (layer "F.Cu")
     (at 181.529207 170.274635)
@@
       (net 3 "unconnected-(H1-Pad1)") (pinfunction "1") (pintype "input+no_connect"))
   )
+  (footprint "2024l3:SS12D00G3" (layer "F.Cu")
+    (at 134.65 131.1 180)
+    (descr "SS12D00G3-1")
+    (tags "Switch")
+    (property "Sheetfile" "2024l2 (VNH5019).kicad_sch")
+    (property "Sheetname" "")
+    (property "ki_description" "Switch, single pole double throw")
+    (property "ki_keywords" "switch single-pole double-throw spdt ON-ON")
+    (attr through_hole)
+    (fp_text reference "SW2" (at 1.3 1.1) (layer "F.SilkS") hide
+        (effects (font (size 0.8 0.8) (thickness 0.1)))
+    )
+    (fp_text value "SW_SPDT" (at 0 0) (layer "F.SilkS") hide
+        (effects (font (size 1.27 1.27) (thickness 0.254)))
+    )
+    (fp_text user "${REFERENCE}" (at 0 0) (layer "F.Fab")
+        (effects (font (size 1.27 1.27) (thickness 0.254)))
+    )
+    (fp_line (start -4.25 -1.75) (end 4.25 -1.75)
+      (stroke (width 0.1) (type solid)) (layer "F.SilkS"))
+    (fp_line (start -4.25 1.75) (end -4.25 -1.75)
+      (stroke (width 0.1) (type solid)) (layer "F.SilkS"))
+    (fp_line (start 4.25 -1.75) (end 4.25 1.75)
+      (stroke (width 0.1) (type solid)) (layer "F.SilkS"))
+    (fp_line (start 4.25 1.75) (end -4.25 1.75)
+      (stroke (width 0.1) (type solid)) (layer "F.SilkS"))
+    (fp_line (start -4.318 -1.778) (end 4.318 -1.778)
+      (stroke (width 0.1) (type solid)) (layer "F.CrtYd"))
+    (fp_line (start -4.318 1.778) (end -4.318 -1.778)
+      (stroke (width 0.1) (type solid)) (layer "F.CrtYd"))
+    (fp_line (start 4.318 -1.778) (end 4.318 1.778)
+      (stroke (width 0.1) (type solid)) (layer "F.CrtYd"))
+    (fp_line (start 4.318 1.778) (end -4.318 1.778)
+      (stroke (width 0.1) (type solid)) (layer "F.CrtYd"))
+    (fp_line (start -4.25 -1.75) (end 4.25 -1.75)
+      (stroke (width 0.2) (type solid)) (layer "F.Fab"))
+    (fp_line (start -4.25 1.75) (end -4.25 -1.75)
+      (stroke (width 0.2) (type solid)) (layer "F.Fab"))
+    (fp_line (start 4.25 -1.75) (end 4.25 1.75)
+      (stroke (width 0.2) (type solid)) (layer "F.Fab"))
+    (fp_line (start 4.25 1.75) (end -4.25 1.75)
+      (stroke (width 0.2) (type solid)) (layer "F.Fab"))
+    (pad "1" thru_hole circle (at -2.5 0 180) (size 1.4 1.4) (drill 0.9) (layers "*.Cu" "*.Mask")
+      (net 2 "+5V") (pinfunction "A") (pintype "passive"))
+    (pad "2" thru_hole circle (at 0 0 180) (size 1.4 1.4) (drill 0.9) (layers "*.Cu" "*.Mask")
+      (net 108 "/TEENSY PWR") (pinfunction "B") (pintype "passive"))
+    (pad "3" thru_hole circle (at 2.5 0 180) (size 1.4 1.4) (drill 0.9) (layers "*.Cu" "*.Mask")
+      (net 109 "unconnected-(SW2-C-Pad3)") (pinfunction "C") (pintype "passive+no_connect"))
+    (model "${KIPRJMOD}/3dmodels/SS12D00G3.stp"
+      (offset (xyz 0 0 0.1800000044))
+      (scale (xyz 1 1 1))
+      (rotate (xyz 0 0 0))
+    )
+  )
   (footprint "MountingHole:MountingHole_3.2mm_M3_Pad_Via" (layer "F.Cu")
     (at 199.42338 223.196162)
@@
       (net 1 "GND") (pinfunction "G3") (pintype "power_in"))
     (pad "VIN" thru_hole circle (at 7.62 -16.51 90) (size 1.53 1.53) (drill 1.02) (layers "*.Cu" "*.Mask")
-      (net 2 "+5V") (pinfunction "VIN") (pintype "power_in"))
+      (net 108 "/TEENSY PWR") (pinfunction "VIN") (pintype "power_in"))
     (model "${KIPRJMOD}/3dmodels/teensy4.step"
       (offset (xyz 0 0 10))
@@
     (fp_arc (start -5.56211 5.20026) (mid -5.86263 5.07578) (end -5.98711 4.77526)
       (stroke (width 0.1) (type default)) (layer "B.SilkS"))
-    (fp_arc (start 5.57474 -5.20026) (mid 5.875103 -5.075647) (end 5.99974 -4.77526)
+    (fp_arc (start 5.57474 -5.20026) (mid 5.875074 -5.075618) (end 5.99974 -4.77526)
       (stroke (width 0.1) (type default)) (layer "B.SilkS"))
     (fp_arc (start 6.01237 4.77526) (mid 5.887903 5.075796) (end 5.58737 5.20026)
@@
   (segment (start 173.08 178.99) (end 166.09 172) (width 0.25) (layer "B.Cu") (net 2))
   (segment (start 177.08 178.7) (end 170.38 172) (width 0.25) (layer "B.Cu") (net 2))
-  (segment (start 142.25 131.1) (end 138.27 131.1) (width 0.75) (layer "B.Cu") (net 2))
   (segment (start 215.3 200.2) (end 214.78 200.72) (width 0.25) (layer "B.Cu") (net 2))
   (segment (start 223.8 201) (end 223.8 203.39) (width 0.75) (layer "B.Cu") (net 2))
@@
   (segment (start 215.3 200.2) (end 223 200.2) (width 0.75) (layer "B.Cu") (net 2))
   (segment (start 189.7 174.6) (end 189.7 156.55) (width 0.75) (layer "B.Cu") (net 2))
+  (segment (start 142.25 131.1) (end 137.15 131.1) (width 0.75) (layer "B.Cu") (net 2))
   (segment (start 157.08 181.7) (end 157.08 179.48) (width 0.25) (layer "B.Cu") (net 2))
   (segment (start 142.25 132.3) (end 142.25 131.1) (width 0.75) (layer "B.Cu") (net 2))
@@
   (segment (start 166.09 172) (end 164.8 172) (width 0.25) (layer "B.Cu") (net 2))
   (segment (start 126.08 178.72) (end 126.08 181.7) (width 0.25) (layer "B.Cu") (net 2))
-  (segment (start 138.27 131.1) (end 131.99 137.38) (width 0.75) (layer "B.Cu") (net 2))
   (segment (start 177.08 181.7) (end 177.08 180.7) (width 0.25) (layer "B.Cu") (net 2))
   (segment (start 215.3 200.2) (end 189.7 174.6) (width 0.75) (layer "B.Cu") (net 2))
@@
   (segment (start 193.94 244.5) (end 195.35 244.5) (width 0.25) (layer "F.Cu") (net 86))
   (segment (start 192.74 243.3) (end 193.94 244.5) (width 0.25) (layer "F.Cu") (net 86))
+  (segment (start 134.65 131.1) (end 131.99 133.76) (width 0.75) (layer "B.Cu") (net 108))
+  (segment (start 131.99 133.76) (end 131.99 137.38) (width 0.75) (layer "B.Cu") (net 108))
   (zone (net 23) (net_name "+12V") (layer "F.Cu") (hatch edge 0.5)
     (priority 12)

Commit message: L2 and L1 Changes
Parts:
- D1, D2: value B340 -> DIOM5336X265N
- moved C18 11.8 mm to (173.1, 229.7)
- moved D3 11.8 mm to (173.1, 222.9)
- moved L3 11.8 mm to (166.1, 225.4)
- moved C13 11.8 mm to (131.6, 228.3)
- moved C14 11.8 mm to (137.4, 225.4)
- moved C15 11.8 mm to (159.8, 219.2)
- moved IC1 11.8 mm to (150.5, 225.4)
- moved R25 11.8 mm to (156.9, 220.0)
- moved J7 5.39 mm to (113.1, 211.5)
- moved J8 5.39 mm to (134.1, 211.5)
- moved J10 5.14 mm to (183.9, 211.5)
- moved J9 5.14 mm to (162.9, 211.5)
Routing:
- net Net-(IC1-FDBK): track 77.4 -> 64.1 mm
- net +12V: track 213.3 -> 216.3 mm

Commit message: L2 Updates
Parts:
- moved C14 14.3 mm to (132.6, 238.9), turned to -90 degrees
- moved C15 6.40 mm to (154.8, 215.2)
- moved C18 6.40 mm to (168.1, 225.7)
- moved D3 6.40 mm to (168.1, 218.9)
- moved IC1 6.40 mm to (145.5, 221.4)
- moved L3 6.40 mm to (161.1, 221.4)
- moved R25 6.40 mm to (151.9, 216.0)
- moved C13 5.30 mm to (126.5, 227.1)
- moved J10 1.50 mm to (183.9, 210.0)
- moved J7 1.50 mm to (113.1, 210.0)
- moved J8 1.50 mm to (134.1, 210.0)
- moved J9 1.50 mm to (162.9, 210.0)
Routing:
- net Net-(IC1-FDBK): track 64.1 -> 69.0 mm
- net +12V: track 216.3 -> 213.8 mm
- net +48V: track 151.0 -> 148.8 mm

Commit message: Motor Connector
Parts:
- added J10: Conn_01x02, 2024l2:16 AWG, F.Cu at (177.0, 210.0)
- added J7: Conn_01x02, 2024l2:16 AWG, F.Cu at (120.0, 210.0)
- added J8: Conn_01x02, 2024l2:16 AWG, F.Cu at (139.0, 210.0)
- added J9: Conn_01x02, 2024l2:16 AWG, F.Cu at (158.0, 210.0)
- added R41: 27k, 2024l2:res0603, F.Cu at (108.5, 199.2)
- added R42: 10k, 2024l2:res0603, F.Cu at (108.5, 197.1)
- D1, D2: value DIOM5336X265N -> B340
- moved SW1 37.5 mm to (191.9, 179.6)
- moved R38 37.0 mm to (194.9, 178.8)
- moved J12 30.8 mm to (103.5, 213.0)
- moved J13 30.8 mm to (193.5, 207.0)
- moved J11 10.1 mm to (103.5, 207.0)
- moved J14 10.1 mm to (193.5, 213.0)
- moved R1 2.54 mm to (139.6, 149.6)
- moved R2 2.54 mm to (154.8, 149.6)
- moved R39 2.54 mm to (147.2, 149.6)
- moved R40 2.54 mm to (162.5, 149.6)
- moved J1 0.08 mm to (110.5, 226.5)
- moved J2 0.08 mm to (105.5, 226.5)
- moved kibuzzard-656013AD 0.08 mm to (108.1, 234.3)
- moved kibuzzard-656013CD 0.08 mm to (108.1, 219.3)
- renumbered J7 to J11, J8 to J12, J9 to J13, J10 to J14
Connections:
- J11 pad 1: /M1 OUTA -> unconnected-(J11-Pin_1-Pad1)
- J11 pad 2: /M1 OUTB -> unconnected-(J11-Pin_2-Pad2)
- J12 pad 1: /M2 OUTA -> unconnected-(J12-Pin_1-Pad1)
- J12 pad 2: /M2 OUTB -> unconnected-(J12-Pin_2-Pad2)
- J13 pad 1: /M3 OUTA -> unconnected-(J13-Pin_1-Pad1)
- J13 pad 2: /M3 OUTB -> unconnected-(J13-Pin_2-Pad2)
- J14 pad 1: /M4 OUTA -> unconnected-(J14-Pin_1-Pad1)
- J14 pad 2: /M4 OUTB -> unconnected-(J14-Pin_2-Pad2)
- U3 pad 0: /M1 INA -> /ESC
- U3 pad 1: /M1 PWM -> /M1 INA
- U3 pad 10: /M4 PWM -> /M4 INA
- U3 pad 11: /M4 INB -> /M4 PWM
- U3 pad 12: unconnected-(U3-12/MISO-Pad12) -> /M4 INB
- U3 pad 2: /M1 INB -> /M1 PWM
- U3 pad 22: /ESC -> unconnected-(U3-22/A8-Pad22)
- U3 pad 23: unconnected-(U3-23/A9-Pad23) -> /BATT LVL
- U3 pad 3: /M2 INA -> /M1 INB
- U3 pad 4: /M2 PWM -> /M2 INA
- U3 pad 5: /M2 INB -> /M2 PWM
- U3 pad 6: /M3 INA -> /M2 INB
- U3 pad 7: /M3 PWM -> /M3 INA
- U3 pad 8: /M3 INB -> /M3 PWM
- U3 pad 9: /M4 INA -> /M3 INB
Routing:
- net /BATT LVL: track 0.00 -> 74.3 mm
- net /M SW: track 239.0 -> 203.9 mm
- net /ESC: track 147.3 -> 121.3 mm, vias 0 -> 1
- net +5V: track 304.8 -> 298.7 mm
- net +12V: track 213.8 -> 217.7 mm
- net /L1 RX: track 110.1 -> 106.3 mm
- net /M1 PWM: track 36.7 -> 37.7 mm
- net /M4 PWM: track 38.4 -> 37.3 mm
- net /M4 INB: track 36.8 -> 35.7 mm
- net /M3 INB: track 33.3 -> 32.3 mm
- net /M2 PWM: track 33.2 -> 34.2 mm
- net /M2 INA: track 32.4 -> 33.5 mm
- net /M1 INB: track 33.0 -> 34.1 mm
- net /M1 INA: track 35.9 -> 36.9 mm
- net /L1 TX: track 114.7 -> 113.7 mm
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