File: LDR Plate/LDR Plate.kicad_pcb (KiCad board)
At the start: 2 copper layers, 9.2 x 12.9 mm, 3 parts, among them J1 Conn_01x02

Commit message: Aesthetic Updates and checks
Changed lines of the file:
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@@
     (property "ki_keywords" "resistor variable light sensitive opto LDR")
     (attr through_hole)
-    (fp_text reference "R2" (at 0 -0.5 90 unlocked) (layer "F.SilkS")
+    (fp_text reference "R2" (at 0 -0.5 90 unlocked) (layer "F.SilkS") hide
         (effects (font (size 1 1) (thickness 0.1)))
     )
