File: LED Plate/LED Plate.kicad_pcb (KiCad board)
At the start: 2 copper layers, 9.2 x 12.9 mm, 2 parts, among them J1 Conn_01x02

Commit message: Aesthetic Updates and checks
Parts:
- added D2: LED, 2024l1:led2835, F.Cu at (146.7, 108.8)
- added D3: LED, 2024l1:led2835, F.Cu at (146.7, 104.2)
- added D4: LED, 2024l1:led2835, F.Cu at (150.3, 104.2)
- D1: footprint 2024l1:LED5050 -> 2024l1:led2835
- moved D1 3.85 mm to (150.3, 108.8), turned to 90 degrees
Routing:
- net +3V3: track 0.00 -> 9.19 mm
