File: LED Plate/LED Plate.kicad_sch (KiCad schematic)
At the start: 2 parts, among them J1 Conn_01x02

Commit message: Aesthetic Updates and checks
Parts:
- added D2, D3, D4: LED, 2024l1:led2835, symbol Device:LED
- D1: footprint 2024l1:LED5050 -> 2024l1:led2835
Connections:
- net +3V3: now also D2.2 (A), D3.2 (A), D4.2 (A)
- net GND: now also D2.1 (K), D3.1 (K), D4.1 (K)
Changed lines of the file:
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@@
 (kicad_sch (version 20230121) (generator eeschema)
   (paper "A4")
+  (junction (at 92.0132 70.8246) (diameter 0) (color 0 0 0 0)
+  )
+  (junction (at 79.3536 78.4446) (diameter 0) (color 0 0 0 0)
+  )
+  (junction (at 85.6834 78.4446) (diameter 0) (color 0 0 0 0)
+  )
+  (junction (at 79.3536 70.8246) (diameter 0) (color 0 0 0 0)
+  )
   (junction (at 73.0238 70.8246) (diameter 0) (color 0 0 0 0)
   )
   (junction (at 73.0238 78.4446) (diameter 0) (color 0 0 0 0)
+  )
+  (junction (at 92.0132 78.4446) (diameter 0) (color 0 0 0 0)
+  )
+  (junction (at 85.6834 70.8246) (diameter 0) (color 0 0 0 0)
+  )
+  (wire (pts (xy 79.3536 70.8246) (xy 85.6834 70.8246))
+    (stroke (width 0) (type default))
   )
   (wire (pts (xy 73.0238 70.8246) (xy 79.3536 70.8246))
@@
   )
   (wire (pts (xy 79.3536 78.4446) (xy 73.0238 78.4446))
+    (stroke (width 0) (type default))
+  )
+  (wire (pts (xy 85.6834 70.8246) (xy 92.0132 70.8246))
+    (stroke (width 0) (type default))
+  )
+  (wire (pts (xy 92.0132 78.4446) (xy 85.6834 78.4446))
+    (stroke (width 0) (type default))
+  )
+  (wire (pts (xy 98.343 78.4446) (xy 92.0132 78.4446))
     (stroke (width 0) (type default))
   )
@@
     (stroke (width 0) (type default))
   )
+  (wire (pts (xy 92.0132 70.8246) (xy 98.343 70.8246))
+    (stroke (width 0) (type default))
+  )
+  (wire (pts (xy 85.6834 78.4446) (xy 79.3536 78.4446))
+    (stroke (width 0) (type default))
+  )
   (wire (pts (xy 73.0238 70.8246) (xy 73.0238 73.2503))
     (stroke (width 0) (type default))
   )
+  (symbol (lib_id "Device:LED") (at 85.6834 74.6346 90) (unit 1)
+    (in_bom yes) (on_board yes) (dnp no)
+    (property "Reference" "D2" (at 87.7633 75.31 90)
+      (effects (font (size 1.27 1.27)) (justify right))
+    )
+    (property "Value" "LED" (at 88.7949 78.1271 90)
+      (effects (font (size 1.27 1.27)) (justify right) hide)
+    )
+    (property "Footprint" "2024l1:led2835" (at 85.6834 74.6346 0)
+      (effects (font (size 1.27 1.27)) hide)
+    )
+    (property "Datasheet" "~" (at 85.6834 74.6346 0)
+      (effects (font (size 1.27 1.27)) hide)
+    )
+    (pin "1")
+    (pin "2")
+    (instances
+      (project "LED Plate"
+        (path "/fcedcb69-8dd9-4ce9-8bf8-c39f35cca66f"
+          (reference "D2") (unit 1)
+        )
+      )
+    )
+  )
+  (symbol (lib_id "Device:LED") (at 92.0132 74.6346 90) (unit 1)
+    (in_bom yes) (on_board yes) (dnp no)
+    (property "Reference" "D3" (at 94.0319 75.3991 90)
+      (effects (font (size 1.27 1.27)) (justify right))
+    )
+    (property "Value" "LED" (at 95.1247 78.1271 90)
+      (effects (font (size 1.27 1.27)) (justify right) hide)
+    )
+    (property "Footprint" "2024l1:led2835" (at 92.0132 74.6346 0)
+      (effects (font (size 1.27 1.27)) hide)
+    )
+    (property "Datasheet" "~" (at 92.0132 74.6346 0)
+      (effects (font (size 1.27 1.27)) hide)
+    )
+    (pin "1")
+    (pin "2")
+    (instances
+      (project "LED Plate"
+        (path "/fcedcb69-8dd9-4ce9-8bf8-c39f35cca66f"
+          (reference "D3") (unit 1)
+        )
+      )
+    )
+  )
+  (symbol (lib_id "Device:LED") (at 98.343 74.6346 90) (unit 1)
+    (in_bom yes) (on_board yes) (dnp no) (fields_autoplaced)
+    (property "Reference" "D4" (at 101.4545 75.5871 90)
+      (effects (font (size 1.27 1.27)) (justify right))
+    )
+    (property "Value" "LED" (at 101.4545 78.1271 90)
+      (effects (font (size 1.27 1.27)) (justify right) hide)
+    )
+    (property "Footprint" "2024l1:led2835" (at 98.343 74.6346 0)
+      (effects (font (size 1.27 1.27)) hide)
+    )
+    (property "Datasheet" "~" (at 98.343 74.6346 0)
+      (effects (font (size 1.27 1.27)) hide)
+    )
+    (pin "1")
+    (pin "2")
+    (instances
+      (project "LED Plate"
+        (path "/fcedcb69-8dd9-4ce9-8bf8-c39f35cca66f"
+          (reference "D4") (unit 1)
+        )
+      )
+    )
+  )
   (symbol (lib_id "Device:LED") (at 79.3536 74.6346 90) (unit 1)
-    (in_bom yes) (on_board yes) (dnp no) (fields_autoplaced)
-    (property "Reference" "D1" (at 82.4651 75.5871 90)
+    (in_bom yes) (on_board yes) (dnp no)
+    (property "Reference" "D1" (at 81.5527 75.3171 90)
       (effects (font (size 1.27 1.27)) (justify right))
     )
@@
       (effects (font (size 1.27 1.27)) (justify right) hide)
     )
-    (property "Footprint" "2024l1:LED5050" (at 79.3536 74.6346 0)
+    (property "Footprint" "2024l1:led2835" (at 79.3536 74.6346 0)
       (effects (font (size 1.27 1.27)) hide)
     )

Commit message: LCSC
Parts:
- D1, D2, D3, D4: LCSC (none) -> C7423447
Changed lines of the file:
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@@
+      (effects (font (size 1.27 1.27)) hide)
+    )
+    (property "LCSC" "C7423447" (at 85.6834 74.6346 90)
       (effects (font (size 1.27 1.27)) hide)
     )
@@
       (effects (font (size 1.27 1.27)) hide)
     )
+    (property "LCSC" "C7423447" (at 92.0132 74.6346 90)
+      (effects (font (size 1.27 1.27)) hide)
+    )
     (pin "1")
     (pin "2")
@@
     )
     (property "Datasheet" "~" (at 98.343 74.6346 0)
+      (effects (font (size 1.27 1.27)) hide)
+    )
+    (property "LCSC" "C7423447" (at 98.343 74.6346 90)
       (effects (font (size 1.27 1.27)) hide)
     )
@@
       (effects (font (size 1.27 1.27)) hide)
     )
+    (property "LCSC" "C7423447" (at 79.3536 74.6346 90)
+      (effects (font (size 1.27 1.27)) hide)
+    )
