File: 2024l3/2024l3.kicad_pcb (KiCad board)
At the start: 2 copper layers, 133 x 90.5 mm, 40 parts, among them J1 Conn_01x06, J2 TOF 0, J3 TOF 1, J4 TOF 2, J5 TOF 3, SW1 SW_SPDT, SW2 SW_SPDT, SW3 SW_SPDT, SW4 SW_SPDT, SW5 SW_SPDT, SW6 SW_SPDT, U1 OpenMV, U2 4754, U3 xiao-esp32c3, U4 Adafruit Featherwing, U5 Teensy 4.0, U6 xiao-esp32c3

Commit message: L1 Revert
Routing:
- net /ESP2 TX: track 64.7 -> 71.8 mm
- net /COM SCL: track 40.8 -> 41.6 mm
- net /COM SDA: track 41.4 -> 42.0 mm
Changed lines of the file:
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@@
   (segment (start 165.735 84.108) (end 165.735 88.244) (width 0.25) (layer "F.Cu") (net 45))
   (segment (start 165.735 88.244) (end 165.683 88.296) (width 0.25) (layer "F.Cu") (net 45))
-  (segment (start 158.115 84.108) (end 146.285 95.938) (width 0.25) (layer "F.Cu") (net 47))
+  (segment (start 132.835 93.388) (end 126.625 93.388) (width 0.25) (layer "F.Cu") (net 47))
+  (segment (start 147.738 95.938) (end 135.385 95.938) (width 0.25) (layer "F.Cu") (net 47))
+  (segment (start 126.625 93.388) (end 124.265 95.748) (width 0.25) (layer "F.Cu") (net 47))
+  (segment (start 158.115 85.561) (end 147.738 95.938) (width 0.25) (layer "F.Cu") (net 47))
   (segment (start 135.385 95.938) (end 132.835 93.388) (width 0.25) (layer "F.Cu") (net 47))
-  (segment (start 132.835 93.388) (end 126.625 93.388) (width 0.25) (layer "F.Cu") (net 47))
-  (segment (start 126.625 93.388) (end 124.265 95.748) (width 0.25) (layer "F.Cu") (net 47))
-  (segment (start 146.285 95.938) (end 135.385 95.938) (width 0.25) (layer "F.Cu") (net 47))
-  (segment (start 155.575 85.198) (end 155.575 84.108) (width 0.25) (layer "F.Cu") (net 48))
-  (segment (start 135.735 94.838) (end 145.935 94.838) (width 0.25) (layer "F.Cu") (net 48))
-  (segment (start 145.935 94.838) (end 155.575 85.198) (width 0.25) (layer "F.Cu") (net 48))
+  (segment (start 158.115 84.108) (end 158.115 85.561) (width 0.25) (layer "F.Cu") (net 47))
   (segment (start 133.235 92.338) (end 135.735 94.838) (width 0.25) (layer "F.Cu") (net 48))
+  (segment (start 146.938 94.838) (end 155.575 86.201) (width 0.25) (layer "F.Cu") (net 48))
+  (segment (start 135.735 94.838) (end 146.938 94.838) (width 0.25) (layer "F.Cu") (net 48))
+  (segment (start 121.725 95.748) (end 125.135 92.338) (width 0.25) (layer "F.Cu") (net 48))
   (segment (start 125.135 92.338) (end 133.235 92.338) (width 0.25) (layer "F.Cu") (net 48))
-  (segment (start 121.725 95.748) (end 125.135 92.338) (width 0.25) (layer "F.Cu") (net 48))
+  (segment (start 155.575 86.201) (end 155.575 84.108) (width 0.25) (layer "F.Cu") (net 48))
   (segment (start 140.835 97.138) (end 140.655 97.138) (width 0.25) (layer "F.Cu") (net 53))
   (segment (start 140.655 97.138) (end 124.265 113.528) (width 0.25) (layer "F.Cu") (net 53))
@@
   (segment (start 121.385 93.138) (end 124.185 90.338) (width 0.25) (layer "F.Cu") (net 91))
   (segment (start 135.535 90.338) (end 140.235 85.638) (width 0.25) (layer "F.Cu") (net 91))
-  (segment (start 147.955 84.108) (end 145.975 86.088) (width 0.25) (layer "F.Cu") (net 92))
-  (segment (start 114.035 110.238) (end 110.335 113.938) (width 0.25) (layer "F.Cu") (net 92))
-  (segment (start 121.785 93.988) (end 115.885 93.988) (width 0.25) (layer "F.Cu") (net 92))
-  (segment (start 110.335 113.938) (end 106.285 113.938) (width 0.25) (layer "F.Cu") (net 92))
-  (segment (start 136.221396 91.188) (end 124.585 91.188) (width 0.25) (layer "F.Cu") (net 92))
-  (segment (start 124.585 91.188) (end 121.785 93.988) (width 0.25) (layer "F.Cu") (net 92))
-  (segment (start 115.885 93.988) (end 114.035 95.838) (width 0.25) (layer "F.Cu") (net 92))
-  (segment (start 141.321396 86.088) (end 136.221396 91.188) (width 0.25) (layer "F.Cu") (net 92))
-  (segment (start 114.035 95.838) (end 114.035 110.238) (width 0.25) (layer "F.Cu") (net 92))
-  (segment (start 145.975 86.088) (end 141.321396 86.088) (width 0.25) (layer "F.Cu") (net 92))
-  (segment (start 106.285 113.938) (end 104.705 112.358) (width 0.25) (layer "F.Cu") (net 92))
+  (segment (start 124.585 91.188) (end 133.714 91.188) (width 0.25) (layer "F.Cu") (net 92))
+  (segment (start 110.335 113.938) (end 114.035 110.238) (width 0.25) (layer "F.Cu") (net 92))
+  (segment (start 121.785 93.988) (end 124.585 91.188) (width 0.25) (layer "F.Cu") (net 92))
+  (segment (start 114.035 110.238) (end 114.035 95.838) (width 0.25) (layer "F.Cu") (net 92))
+  (segment (start 114.035 95.838) (end 115.885 93.988) (width 0.25) (layer "F.Cu") (net 92))
+  (segment (start 147.955 91.821) (end 147.955 84.108) (width 0.25) (layer "F.Cu") (net 92))
+  (segment (start 106.285 113.938) (end 110.335 113.938) (width 0.25) (layer "F.Cu") (net 92))
+  (segment (start 136.826 94.3) (end 145.476 94.3) (width 0.25) (layer "F.Cu") (net 92))
+  (segment (start 115.885 93.988) (end 121.785 93.988) (width 0.25) (layer "F.Cu") (net 92))
+  (segment (start 104.705 112.358) (end 106.285 113.938) (width 0.25) (layer "F.Cu") (net 92))
+  (segment (start 145.476 94.3) (end 147.955 91.821) (width 0.25) (layer "F.Cu") (net 92))
+  (segment (start 133.714 91.188) (end 136.826 94.3) (width 0.25) (layer "F.Cu") (net 92))
   (zone locked (net 1) (net_name "GND") (layers "F&B.Cu") (hatch edge 0.5)
     (connect_pads yes (clearance 0.2))

Commit message: L3 Silk
Parts:
- removed kibuzzard-65630B7E: G***, kibuzzard-65630B7E
- removed kibuzzard-65630B95: G***, kibuzzard-65630B95
- removed kibuzzard-657BF135: G***, kibuzzard-657BF135
- removed kibuzzard-657D3EC8: G***, kibuzzard-657D3EC8
- added kibuzzard-6590F6B4: G***, kibuzzard-6590F6B4, F.Cu at (131.3, 78.0)
- added kibuzzard-6590F77B: G***, kibuzzard-6590F77B, F.Cu at (131.6, 74.1)
- added kibuzzard-6590F814: G***, kibuzzard-6590F814, F.Cu at (113.7, 77.8)
- U3, U6: value xiao-esp32c3 -> >VALUE

Commit message: L3 Silk
Parts:
- removed kibuzzard-65630B66: G***, kibuzzard-65630B66
- removed kibuzzard-657BF16E: G***, kibuzzard-657BF16E
- removed kibuzzard-657BF185: G***, kibuzzard-657BF185
- added kibuzzard-659111B0: G***, kibuzzard-659111B0, F.Cu at (113.9, 70.3)
- added kibuzzard-659111BA: G***, kibuzzard-659111BA, F.Cu at (132.6, 70.3)
- added kibuzzard-65911205: G***, kibuzzard-65911205, F.Cu at (114.0, 74.1)
- moved kibuzzard-6590F814 0.25 mm to (113.7, 78.0)
- moved SW1 0.25 mm to (104.4, 78.0)
- moved SW6 0.15 mm to (104.4, 74.1)
- moved SW3 0.10 mm to (104.4, 70.3)
- moved kibuzzard-6590F77B 0.08 mm to (131.7, 74.1)

Commit message: LCSC Updates
Changed lines of the file:
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@@
     (attr board_only exclude_from_pos_files exclude_from_bom)
     (fp_text reference "kibuzzard-65911205" (at 0 -3.97166 180) (layer "F.SilkS") hide
-        (effects (font (size 0 0)))
+        (effects (font (size 0 0) (thickness 0.15)))
     )
     (fp_text value "G***" (at 0 3.97166 180) (layer "F.SilkS") hide
-        (effects (font (size 0 0)))
+        (effects (font (size 0 0) (thickness 0.15)))
     )
     (fp_poly
@@
     (attr board_only exclude_from_pos_files exclude_from_bom)
     (fp_text reference "kibuzzard-659111BA" (at 0 -3.97166 180) (layer "F.SilkS") hide
-        (effects (font (size 0 0)))
+        (effects (font (size 0 0) (thickness 0.15)))
     )
     (fp_text value "G***" (at 0 3.97166 180) (layer "F.SilkS") hide
-        (effects (font (size 0 0)))
+        (effects (font (size 0 0) (thickness 0.15)))
     )
     (fp_poly
@@
     (attr board_only exclude_from_pos_files exclude_from_bom)
     (fp_text reference "kibuzzard-659111B0" (at 0 -3.97166 180) (layer "F.SilkS") hide
-        (effects (font (size 0 0)))
+        (effects (font (size 0 0) (thickness 0.15)))
     )
     (fp_text value "G***" (at 0 3.97166 180) (layer "F.SilkS") hide
-        (effects (font (size 0 0)))
+        (effects (font (size 0 0) (thickness 0.15)))
     )
     (fp_poly
@@
     )
   )
-  (gr_rect (start 128.585 71.77) (end 136.535 68.91)
+  (gr_rect (start 128.585 68.91) (end 136.535 71.77)
     (stroke (width 0.2) (type default)) (fill none) (layer "F.SilkS"))
   (gr_rect (start 128.585 72.6215) (end 134.73 75.6665)
@@
   (gr_rect (start 110.935 72.6215) (end 117.08 75.6665)
     (stroke (width 0.2) (type default)) (fill none) (layer "F.SilkS"))
-  (gr_rect (start 110.935 71.77) (end 116.855 68.92)
+  (gr_rect (start 110.935 68.92) (end 116.855 71.77)
     (stroke (width 0.2) (type default)) (fill none) (layer "F.SilkS"))
   (gr_rect (start 128.585 76.518) (end 134.105 79.563)

Commit message: Changed OPENMV FOOTPRINT
Parts:
- U1: value OpenMV -> ~; footprint 2024l3:openmv -> 2024l3:OpenMV_RT
- U3, U6: value >VALUE -> xiao-esp32c3
- moved U1 126.6 mm to (22.2, 100.9)
Connections:
- U1 pad 0: (no net) -> unconnected-(U1-P0-MOSI/PWM-Pad0)
- U1 pad 10: /CAM PWR -> /CAM RX
- U1 pad 15: unconnected-(U1-BOOT-Pad15) -> GND
- U1 pad 16: /CAM RST -> unconnected-(U1-NC-Pad16)
- U1 pad 5: /CAM TX -> unconnected-(U1-P2-ETH_RXN-Pad5)
- U1 pad 6: /CAM RX -> unconnected-(U1-P3-SS-Pad6)
- U1 pad 8: unconnected-(U1-3V3(250mA)-Pad8) -> /CAM TX
- U1 pad 9: GND -> unconnected-(U1-P4-ETH_TXP-Pad9)
Routing:
- net /CAM PWR: track 76.0 -> 27.4 mm
- net /CAM RX: track 44.3 -> 0.00 mm
- net /CAM TX: track 42.2 -> 0.00 mm, vias 1 -> 0
- net /CAM RST: track 4.14 -> 0.00 mm

Commit message: Cam Placement
Parts:
- removed kibuzzard-659111BA: G***, kibuzzard-659111BA
- added kibuzzard-6592C7F1: G***, kibuzzard-6592C7F1, F.Cu at (131.8, 70.3)
- U3, U6: value xiao-esp32c3 -> >VALUE
- moved U1 126.6 mm to (148.8, 104.8)

Commit message: L3 Trace Size decrease
Routing:
- net /CAM RX: track 0.00 -> 56.9 mm
- net /CAM TX: track 0.00 -> 51.7 mm
- net /CAM PWR: track 27.4 -> 73.8 mm
- net /CAM RST: track 0.00 -> 4.60 mm
- net /XSHUT 0: track 110.1 -> 109.6 mm
