File: 2024l3/2024l3.kicad_sch (KiCad schematic)
At the start: 26 parts, among them J1 Conn_01x06, J2 TOF 0, J3 TOF 1, J4 TOF 2, J5 TOF 3, SW1 SW_SPDT, SW2 SW_SPDT, U1 OpenMV, U2 4754, U3 xiao-esp32c3, U4 Adafruit Featherwing, U7 Teensy 4.0

Commit message: L3 Schematic
Parts:
- added SW3: SW_SPDT, 2024l3:SS12D00G3, symbol Switch:SW_SPDT
Connections:
- net +3V3: now also SW3.1 (A); no longer U4.2 (VIN)
- new net OLED PWR: SW3.2 (B), U4.2 (VIN)
- no-connect marks 44 -> 45
Other:
- moved on the sheet: SW1, SW2

Commit message: L3 Partial Routing
Connections:
- net A: now also U7.10 (10/CS)
- net B: now also U7.11 (11/MOSI)
- net C: now also U7.12 (12/MISO)
- no-connect marks 45 -> 42
Changed lines of the file:
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@@
   (no_connect (at 104.14 96.52))
   (no_connect (at 137.16 93.98))
-  (no_connect (at 104.14 116.84))
-  (no_connect (at 104.14 121.92))
   (no_connect (at 104.14 114.3))
   (no_connect (at 104.14 101.6))
   (no_connect (at 31.6697 54.5946))
   (no_connect (at 24.13 90.17))
-  (no_connect (at 104.14 119.38))
   (no_connect (at 218.2623 51.4499))
   (no_connect (at 20.2289 45.4226))
@@
     (stroke (width 0) (type default))
   )
+  (wire (pts (xy 100.8418 121.92) (xy 104.14 121.92))
+    (stroke (width 0) (type default))
+  )
   (wire (pts (xy 201.2127 58.5426) (xy 192.2697 58.5426))
     (stroke (width 0) (type default))
@@
     (stroke (width 0) (type default))
   )
+  (wire (pts (xy 100.8418 116.84) (xy 104.14 116.84))
+    (stroke (width 0) (type default))
+  )
   (wire (pts (xy 156.5705 122.2617) (xy 165.4605 122.2617))
     (stroke (width 0) (type default))
@@
     (stroke (width 0) (type default))
   )
+  (wire (pts (xy 100.8418 119.38) (xy 104.14 119.38))
+    (stroke (width 0) (type default))
+  )
   (wire (pts (xy 137.16 109.22) (xy 148.59 109.22))
     (stroke (width 0) (type default))
@@
     (effects (font (size 1.27 1.27)) (justify left bottom))
   )
+  (label "A" (at 102.0667 116.84 0) (fields_autoplaced)
+    (effects (font (size 1.27 1.27)) (justify left bottom))
+  )
   (label "L3 RX" (at 102.87 91.44 180) (fields_autoplaced)
     (effects (font (size 1.27 1.27)) (justify right bottom))
@@
     (effects (font (size 1.27 1.27)) (justify left bottom))
   )
+  (label "B" (at 102.0243 119.38 0) (fields_autoplaced)
+    (effects (font (size 1.27 1.27)) (justify left bottom))
+  )
   (label "ESP TX" (at 101.6 109.22 180) (fields_autoplaced)
     (effects (font (size 1.27 1.27)) (justify right bottom))
   )
+  (label "C" (at 101.996 121.92 0) (fields_autoplaced)
+    (effects (font (size 1.27 1.27)) (justify left bottom))
+  )
   (label "CAM TX" (at 16.51 92.71 0) (fields_autoplaced)

Commit message: L3 Routing
Connections:
- net XSHUT 0: now also U3.3 (A3); no longer U3.0 (A0)
- net XSHUT 1: now also U3.2 (A2); no longer U3.1 (A1)
- net XSHUT 2: now also U3.0 (A0); no longer U3.2 (A2)
- net XSHUT 3: now also U3.1 (A1); no longer U3.3 (A3)
Changed lines of the file:
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@@
+    (stroke (width 0) (type default))
+  )
+  (wire (pts (xy 143.1158 38.7398) (xy 153.4085 38.7398))
     (stroke (width 0) (type default))
   )
@@
     (stroke (width 0) (type default))
   )
-  (wire (pts (xy 143.1158 38.7398) (xy 153.4085 38.7398))
-    (stroke (width 0) (type default))
-  )
   (wire (pts (xy 218.2623 56.5299) (xy 228.555 56.5299))
     (stroke (width 0) (type default))
@@
     (stroke (width 0) (type default))
   )
+  (wire (pts (xy 219.2226 35.9826) (xy 224.1187 35.9826))
+    (stroke (width 0) (type default))
+  )
+  (wire (pts (xy 137.16 104.14) (xy 148.59 104.14))
+    (stroke (width 0) (type default))
+  )
+  (wire (pts (xy 192.145 35.226) (xy 197.0235 35.226))
+    (stroke (width 0) (type default))
+  )
+  (wire (pts (xy 100.8418 121.92) (xy 104.14 121.92))
+    (stroke (width 0) (type default))
+  )
+  (wire (pts (xy 201.2127 58.5426) (xy 192.2697 58.5426))
+    (stroke (width 0) (type default))
+  )
+  (wire (pts (xy 182.88 97.79) (xy 193.1727 97.79))
+    (stroke (width 0) (type default))
+  )
   (wire (pts (xy 143.1158 33.6598) (xy 153.4085 33.6598))
     (stroke (width 0) (type default))
   )
-  (wire (pts (xy 219.2226 35.9826) (xy 224.1187 35.9826))
-    (stroke (width 0) (type default))
-  )
-  (wire (pts (xy 137.16 104.14) (xy 148.59 104.14))
-    (stroke (width 0) (type default))
-  )
-  (wire (pts (xy 192.145 35.226) (xy 197.0235 35.226))
-    (stroke (width 0) (type default))
-  )
-  (wire (pts (xy 100.8418 121.92) (xy 104.14 121.92))
-    (stroke (width 0) (type default))
-  )
-  (wire (pts (xy 201.2127 58.5426) (xy 192.2697 58.5426))
-    (stroke (width 0) (type default))
-  )
-  (wire (pts (xy 182.88 97.79) (xy 193.1727 97.79))
-    (stroke (width 0) (type default))
-  )
   (wire (pts (xy 92.71 91.44) (xy 104.14 91.44))
     (stroke (width 0) (type default))
@@
     (stroke (width 0) (type default))
   )
+  (wire (pts (xy 219.2226 23.2826) (xy 229.5153 23.2826))
+    (stroke (width 0) (type default))
+  )
+  (wire (pts (xy 177.0886 78.6025) (xy 177.0886 81.1425))
+    (stroke (width 0) (type default))
+  )
+  (wire (pts (xy 143.1158 46.3598) (xy 153.4085 46.3598))
+    (stroke (width 0) (type default))
+  )
   (wire (pts (xy 143.1158 31.1198) (xy 153.4085 31.1198))
     (stroke (width 0) (type default))
   )
-  (wire (pts (xy 219.2226 23.2826) (xy 229.5153 23.2826))
-    (stroke (width 0) (type default))
-  )
-  (wire (pts (xy 177.0886 78.6025) (xy 177.0886 81.1425))
-    (stroke (width 0) (type default))
-  )
-  (wire (pts (xy 143.1158 46.3598) (xy 153.4085 46.3598))
-    (stroke (width 0) (type default))
-  )
   (polyline (pts (xy 12.0423 69.565) (xy 81.274 69.565))
     (stroke (width 0) (type dash))
   )
+  (wire (pts (xy 143.1158 36.1998) (xy 153.4085 36.1998))
+    (stroke (width 0) (type default))
+  )
   (wire (pts (xy 218.2623 48.9099) (xy 228.555 48.9099))
     (stroke (width 0) (type default))
@@
     (stroke (width 0) (type default))
   )
-  (wire (pts (xy 143.1158 36.1998) (xy 153.4085 36.1998))
-    (stroke (width 0) (type default))
-  )
   (wire (pts (xy 58.42 45.974) (xy 69.85 45.974))
     (stroke (width 0) (type default))
@@
     (effects (font (size 1.27 1.27)) (justify right bottom))
   )
+  (label "XSHUT 3" (at 144.857 33.6598 0) (fields_autoplaced)
+    (effects (font (size 1.27 1.27)) (justify left bottom))
+  )
   (label "CAM PWR" (at 68.58 97.79 0) (fields_autoplaced)
     (effects (font (size 1.27 1.27)) (justify left bottom))
@@
     (effects (font (size 1.27 1.27)) (justify left bottom))
   )
-  (label "XSHUT 0" (at 144.7679 31.1198 0) (fields_autoplaced)
-    (effects (font (size 1.27 1.27)) (justify left bottom))
-  )
   (label "SDA TOF" (at 194.8801 53.4626 0) (fields_autoplaced)
     (effects (font (size 1.27 1.27)) (justify left bottom))
@@
     (effects (font (size 1.27 1.27)) (justify left bottom))
   )
+  (label "XSHUT 2" (at 144.8583 31.1198 0) (fields_autoplaced)
+    (effects (font (size 1.27 1.27)) (justify left bottom))
+  )
   (label "OLED SCL" (at 183.5701 97.79 0) (fields_autoplaced)
     (effects (font (size 1.27 1.27)) (justify left bottom))
@@
     (effects (font (size 1.27 1.27)) (justify left bottom))
   )
+  (label "XSHUT 0" (at 144.7679 38.7398 0) (fields_autoplaced)
+    (effects (font (size 1.27 1.27)) (justify left bottom))
+  )
   (label "CAM TX" (at 146.05 101.6 180) (fields_autoplaced)
     (effects (font (size 1.27 1.27)) (justify right bottom))
@@
     (effects (font (size 1.27 1.27)) (justify left bottom))
   )
-  (label "XSHUT 3" (at 144.857 38.7398 0) (fields_autoplaced)
-    (effects (font (size 1.27 1.27)) (justify left bottom))
-  )
   (label "OLED SDA" (at 183.657 100.33 0) (fields_autoplaced)
     (effects (font (size 1.27 1.27)) (justify left bottom))
@@
     (effects (font (size 1.27 1.27)) (justify left bottom))
   )
-  (label "XSHUT 1" (at 144.8167 33.6598 0) (fields_autoplaced)
+  (label "XSHUT 1" (at 144.8167 36.1998 0) (fields_autoplaced)
     (effects (font (size 1.27 1.27)) (justify left bottom))
   )
@@
     (effects (font (size 1.27 1.27)) (justify right bottom))
   )
-  (label "XSHUT 2" (at 144.8583 36.1998 0) (fields_autoplaced)
-    (effects (font (size 1.27 1.27)) (justify left bottom))
-  )
   (symbol (lib_id "power:+5V") (at 177.0886 78.6025 0) (unit 1)

Commit message: L3 Routing Complete
Connections:
- net COM RST: now also U7.13 (13/SCL/LED); no longer U7.6
- net OLED RST: now also U7.6
- net CAM RST: now reaches U7.14 (14/A0/TX3)
- net CAM RST: now also U1.16 (RST)
- no-connect marks 42 -> 39
Changed lines of the file:
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@@
   (no_connect (at 192.2697 50.9226))
   (no_connect (at 104.14 99.06))
-  (no_connect (at 137.16 119.38))
-  (no_connect (at 137.16 121.92))
   (no_connect (at 31.3429 37.3398))
   (no_connect (at 137.16 116.84))
@@
   (no_connect (at 24.13 85.09))
   (no_connect (at 24.13 87.63))
-  (no_connect (at 68.58 82.55))
   (no_connect (at 31.246 30.3452))
   (no_connect (at 68.58 85.09))
@@
     (stroke (width 0) (type default))
   )
+  (wire (pts (xy 137.16 119.38) (xy 147.9457 119.38))
+    (stroke (width 0) (type default))
+  )
   (wire (pts (xy 87.796 24.7874) (xy 96.9446 24.7874))
     (stroke (width 0) (type default))
@@
     (stroke (width 0) (type default))
   )
+  (wire (pts (xy 137.16 121.92) (xy 147.9457 121.92))
+    (stroke (width 0) (type default))
+  )
   (wire (pts (xy 174.5486 81.1425) (xy 177.0886 81.1425))
     (stroke (width 0) (type default))
@@
     (stroke (width 0) (type default))
   )
+  (wire (pts (xy 68.58 82.55) (xy 77.47 82.55))
+    (stroke (width 0) (type default))
+  )
   (wire (pts (xy 192.145 30.146) (xy 202.4377 30.146))
     (stroke (width 0) (type default))
@@
     (stroke (width 0) (type default))
   )
-  (wire (pts (xy 92.71 106.68) (xy 104.14 106.68))
-    (stroke (width 0) (type default))
-  )
   (wire (pts (xy 88.0546 34.9474) (xy 96.9446 34.9474))
     (stroke (width 0) (type default))
@@
     (stroke (width 0) (type default))
   )
+  (wire (pts (xy 93.8473 106.68) (xy 104.14 106.68))
+    (stroke (width 0) (type default))
+  )
   (wire (pts (xy 138.1208 41.2798) (xy 153.4085 41.2798))
     (stroke (width 0) (type default))
@@
     (effects (font (size 1.27 1.27)) (justify left bottom))
   )
+  (label "CAM RST" (at 68.58 82.55 0) (fields_autoplaced)
+    (effects (font (size 1.27 1.27)) (justify left bottom))
+  )
   (label "XSHUT 0" (at 144.7679 38.7398 0) (fields_autoplaced)
     (effects (font (size 1.27 1.27)) (justify left bottom))
@@
     (effects (font (size 1.27 1.27)) (justify right bottom))
   )
+  (label "CAM RST" (at 138.9199 119.38 0) (fields_autoplaced)
+    (effects (font (size 1.27 1.27)) (justify left bottom))
+  )
   (label "SCL TOF" (at 194.7418 30.146 0) (fields_autoplaced)
     (effects (font (size 1.27 1.27)) (justify left bottom))
@@
     (effects (font (size 1.27 1.27)) (justify right bottom))
   )
+  (label "OLED RST" (at 94.9022 106.68 0) (fields_autoplaced)
+    (effects (font (size 1.27 1.27)) (justify left bottom))
+  )
   (label "COM PWR" (at 156.7686 83.6825 0) (fields_autoplaced)
     (effects (font (size 1.27 1.27)) (justify left bottom))
@@
     (effects (font (size 1.27 1.27)) (justify left bottom))
   )
-  (label "COM RST" (at 95.25 106.68 0) (fields_autoplaced)
-    (effects (font (size 1.27 1.27)) (justify left bottom))
-  )
   (label "ESP RX" (at 172.4585 46.3598 0) (fields_autoplaced)
     (effects (font (size 1.27 1.27)) (justify left bottom))
@@
     (effects (font (size 1.27 1.27)) (justify right bottom))
   )
+  (label "COM RST" (at 138.9199 121.92 0) (fields_autoplaced)
+    (effects (font (size 1.27 1.27)) (justify left bottom))
+  )
   (symbol (lib_id "power:+5V") (at 177.0886 78.6025 0) (unit 1)

Commit message: L3 Redo
Parts:
- added R3, R4: 1K, 2024l3:res0603, symbol Device:R
- added SW4, SW5, SW6: SW_SPDT, 2024l3:SS12D00G3, symbol Switch:SW_SPDT
- added U6: xiao-esp32c3, 2024l3:xiao-esp32c3, symbol vincent:xiao-esp32c3
Connections:
- net +5V: now also R3.1, R4.2, SW4.1 (A), SW5.1 (A), SW6.1 (A); no longer U3.13 (5V), U7.VIN
- net A: now also U6.8 (SCK); no longer U7.10 (10/CS)
- net B: now also U6.9 (MISO); no longer U7.11 (11/MOSI)
- net C: now also U6.10 (MOSI); no longer U7.12 (12/MISO)
- net CAM RST: now also U7.22 (22/A8); no longer U7.14 (14/A0/TX3)
- net GND: now also U6.12 (GND)
- net OLED RST: now also U6.3 (A3); no longer U7.6
- net OLED SCL: now also R4.1, U6.5 (SCL); no longer U7.16 (16/A2/RX4/SCL1)
- net OLED SDA: now also R3.2, U6.4 (SDA); no longer U7.17 (17/A3/TX4/SDA1)
- net XSHUT 0: now also U3.9 (MISO); no longer U3.3 (A3)
- net XSHUT 1: now also U3.0 (A0); no longer U3.2 (A2)
- net XSHUT 2: now also U3.1 (A1); no longer U3.0 (A0)
- net XSHUT 3: now also U3.8 (SCK); no longer U3.1 (A1)
- net ESP2 TX: now reaches U7.15 (15/A1/RX3)
- net ESP2 TX: now also U6.6 (TX)
- net ESP RX: no longer names the net of U7.8 (8/TX2)
- net ESP RX: no longer U3.7 (RX)
- net ESP TX: no longer names the net of U7.7 (7/RX2)
- net ESP TX: no longer U3.6 (TX)
- new net ESP1 PWR: SW5.2 (B), U3.13 (5V)
- new net ESP1 RX: U3.7 (RX), U7.17 (17/A3/TX4/SDA1)
- new net ESP1 TX: U3.6 (TX), U7.16 (16/A2/RX4/SCL1)
- new net ESP2 PWR: SW6.2 (B), U6.13 (5V)
- new net ESP2 RX: U6.7 (RX), U7.14 (14/A0/TX3)
- new net TEENSY PWR: SW4.2 (B), U7.VIN
- no-connect marks 39 -> 53
Other:
- note added: "OLED"
- moved on the sheet: U4

Commit message: Changed OPENMV FOOTPRINT
Parts:
- removed U1: OpenMV, 2024l3:openmv, symbol vincent:OpenMV
- added U1: ~, 2024l3:OpenMV_RT, symbol vincent:OpenMV_RT
Connections:
- net CAM PWR: now also U1.29 (VIN)
- net CAM RST: now also U1.17 (RST)
- net CAM RX: now also U1.10 (P5-RX/SDA/PWM)
- net CAM TX: now also U1.8 (P4-TX/SCL/PWM)
- net GND: now also U1.15 (GND), U1.31 (GND)
- no-connect marks 53 -> 63
Other:
- moved on the sheet: R3, R4, U4, U6

Commit message: DNP L3 PULLUP
Parts:
- R1, R2: now not fitted
- R3, R4: value 1K -> 10K; LCSC C21190 -> (none); now not fitted
Connections:
- net +5V: now also R4.1; no longer R4.2
- net OLED SCL: now also R3.2; no longer R4.1
- net OLED SDA: now also R4.2; no longer R3.2
Other:
- note removed: "OLED/Screen"
- moved on the sheet: U4, U6
