File: Extras/2024l2 (VNH5019)/2024l2 (VNH5019).kicad_pcb (KiCad board)
At the start: 2 copper layers, 174 x 141 mm, 114 parts, among them IC1 LM2587S-ADJ, J1 Conn_01x02, J10 Conn_01x02, J11 Conn_01x02, J12 Conn_01x02, J13 Conn_01x02, J14 Conn_01x02, J2 Conn_01x02, J3 Conn_01x03, J4 Conn_01x03, J5 Conn_01x04, J6 Conn_01x06, J7 Conn_01x02, J8 Conn_01x02, J9 Conn_01x02, Q1 AOD482, Q2 AOD482, Q3 AOD482, Q4 AOD482, SW1 SW_SPST, SW2 SW_SPDT, U1 TPS5430DDA, U2 TPS5430DDA, U3 Teensy 4.0

Commit message: L2 5019 changes
Parts:
- removed J11, J12, J13, J14: Conn_01x02, 2024l2:AMASS_XT30-F
- moved J3 13.0 mm to (189.7, 207.5)
Routing:
- net /L1 RX: track 106.3 -> 99.0 mm
- net /L1 TX: track 113.7 -> 106.7 mm

Commit message: L2 edits
Parts:
- removed R41: 27k, 2024l2:res0603
- removed R42: 10k, 2024l2:res0603
- removed kibuzzard-656013AD: G***, kibuzzard-656013AD
- removed kibuzzard-656013CD: G***, kibuzzard-656013CD
- added C21: 220u, Capacitor_SMD:CP_Elec_10x10.5, F.Cu at (57.4, 153.1)
- added C22: 220u, Capacitor_SMD:CP_Elec_10x10.5, F.Cu at (57.4, 165.1)
- C14: moved to F.Cu
- D1, D2: value B340 -> SS54; footprint 2024l2:B340 -> 2024l2:SMA (DO-214AC)
- moved C14 106.3 mm to (71.2, 152.1), turned to 0 degrees
- moved J5 14.8 mm to (107.3, 213.8)
- moved R38 5.80 mm to (213.9, 204.8), turned to 180 degrees
- moved SW1 3.78 mm to (214.5, 211.2)
Connections:
- U3 pad 23: /BATT LVL -> unconnected-(U3-23/A9-Pad23)
Routing:
- net /BATT LVL: track 74.3 -> 0.00 mm
- net +48V: track 148.8 -> 119.0 mm
- net +12V: track 217.7 -> 204.8 mm
- net +3V3: track 131.9 -> 143.7 mm
- net /M SW: track 241.0 -> 248.9 mm
- net +5V: track 305.5 -> 300.3 mm
- net Net-(U1-BOOT): track 3.50 -> 0.00 mm
- net /ESC: track 121.3 -> 120.6 mm
Other:
- outline, holes or cut-outs redrawn
