File: Extras/2024l2 (VNH5019)/2024l2 (VNH5019).kicad_sch (KiCad schematic)
At the start: 111 parts, among them IC1 LM2587S-ADJ, J1 Conn_01x02, J10 Conn_01x02, J11 Conn_01x02, J12 Conn_01x02, J13 Conn_01x02, J14 Conn_01x02, J2 Conn_01x02, J3 Conn_01x03, J4 Conn_01x03, J5 Conn_01x04, J6 Conn_01x06, J7 Conn_01x02, J8 Conn_01x02, J9 Conn_01x02, Q1 AOD482, Q2 AOD482, Q3 AOD482, Q4 AOD482, SW1 SW_SPST, SW2 SW_SPDT, U1 TPS5430DDA, U2 TPS5430DDA, U3 Teensy 4.0

Commit message: L2 5019 changes
Parts:
- removed R41: 27k, 2024l2:res0603, symbol Device:R
- removed R42: 10k, 2024l2:res0603, symbol Device:R
- D1, D2: value B340 -> SS54
Connections:
- net BATT LVL: no longer names the net of U3.23 (23/A9)
- no-connect marks 41 -> 42
Changed lines of the file:
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@@
   (junction (at 226.695 57.785) (diameter 0) (color 0 0 0 0)
   )
-  (junction (at 110.6317 128.0367) (diameter 0) (color 0 0 0 0)
-  )
   (junction (at 226.822 92.329) (diameter 0) (color 0 0 0 0)
   )
@@
   (no_connect (at 80.01 209.55))
   (no_connect (at 116.2285 180.1169))
+  (no_connect (at 80.01 184.15))
   (no_connect (at 142.24 186.69))
   (no_connect (at 187.96 176.53))
@@
     (stroke (width 0) (type default))
   )
-  (wire (pts (xy 80.01 184.15) (xy 92.6113 184.15))
-    (stroke (width 0) (type default))
-  )
   (wire (pts (xy 226.822 81.407) (xy 226.822 82.169))
     (stroke (width 0) (type default))
@@
     (stroke (width 0) (type default))
   )
-  (wire (pts (xy 110.6317 128.0367) (xy 123.233 128.0367))
-    (stroke (width 0) (type default))
-  )
   (wire (pts (xy 106.68 76.2) (xy 106.68 77.47))
     (stroke (width 0) (type default))
@@
     (effects (font (size 1.27 1.27)) (justify left bottom))
   )
-  (label "BATT LVL" (at 113.9626 128.0367 0) (fields_autoplaced)
-    (effects (font (size 1.27 1.27)) (justify left bottom))
-  )
   (label "M1 INA" (at 167.259 33.528 0) (fields_autoplaced)
     (effects (font (size 1.27 1.27)) (justify left bottom))
@@
     (effects (font (size 1.27 1.27)) (justify left bottom))
   )
-  (label "BATT LVL" (at 83.3409 184.15 0) (fields_autoplaced)
-    (effects (font (size 1.27 1.27)) (justify left bottom))
-  )
   (label "L3 TX" (at 90.17 138.43 180) (fields_autoplaced)
     (effects (font (size 1.27 1.27)) (justify right bottom))
@@
     )
   )
-  (symbol (lib_id "Device:R") (at 110.6317 124.2267 0) (unit 1)
-    (in_bom yes) (on_board yes) (dnp no)
-    (property "Reference" "R41" (at 112.5367 125.6237 90)
-      (effects (font (size 1.27 1.27)) (justify left))
-    )
-    (property "Value" "27k" (at 110.6384 126.0148 90)
-      (effects (font (size 1.27 1.27)) (justify left))
-    )
-    (property "Footprint" "2024l2:res0603" (at 108.8537 124.2267 90)
-      (effects (font (size 1.27 1.27)) hide)
-    )
-    (property "Datasheet" "~" (at 110.6317 124.2267 0)
-      (effects (font (size 1.27 1.27)) hide)
-    )
-    (pin "1")
-    (pin "2")
-    (instances
-      (project "2024l2 (VNH5019)"
-        (path "/36f2ccec-186b-4304-87fe-6495d5655b87"
-          (reference "R41") (unit 1)
-        )
-      )
-    )
-  )
   (symbol (lib_id "Device:R") (at 288.036 84.201 90) (unit 1)
     (in_bom yes) (on_board yes) (dnp no)
@@
     )
   )
-  (symbol (lib_id "power:GND") (at 110.6317 135.6567 0) (unit 1)
-    (in_bom yes) (on_board yes) (dnp no) (fields_autoplaced)
-    (property "Reference" "#PWR047" (at 110.6317 142.0067 0)
-      (effects (font (size 1.27 1.27)) hide)
-    )
-    (property "Value" "GND" (at 110.6317 141.2279 0)
-      (effects (font (size 1.27 1.27)))
-    )
-    (property "Footprint" "" (at 110.6317 135.6567 0)
-      (effects (font (size 1.27 1.27)) hide)
-    )
-    (property "Datasheet" "" (at 110.6317 135.6567 0)
-      (effects (font (size 1.27 1.27)) hide)
-    )
-    (pin "1")
-    (instances
-      (project "2024l2 (VNH5019)"
-        (path "/36f2ccec-186b-4304-87fe-6495d5655b87"
-          (reference "#PWR047") (unit 1)
-        )
-      )
-    )
-  )
   (symbol (lib_id "power:GND") (at 278.2205 210.0175 0) (unit 1)
     (in_bom yes) (on_board yes) (dnp no) (fields_autoplaced)
@@
   (symbol (lib_id "Diode:B340") (at 77.47 26.67 270) (unit 1)
     (in_bom yes) (on_board yes) (dnp no) (fields_autoplaced)
-    (property "Reference" "D1" (at 80.01 25.0825 90)
+    (property "Reference" "D1" (at 80.01 25.7175 90)
       (effects (font (size 1.27 1.27)) (justify left))
     )
-    (property "Value" "B340" (at 80.01 27.6225 90)
+    (property "Value" "SS54" (at 80.01 28.2575 90)
       (effects (font (size 1.27 1.27)) (justify left))
     )
@@
     )
   )
-  (symbol (lib_id "Device:R") (at 110.6317 131.8467 0) (unit 1)
-    (in_bom yes) (on_board yes) (dnp no)
-    (property "Reference" "R42" (at 112.5367 133.2437 90)
-      (effects (font (size 1.27 1.27)) (justify left))
-    )
-    (property "Value" "10k" (at 110.6384 133.6348 90)
-      (effects (font (size 1.27 1.27)) (justify left))
-    )
-    (property "Footprint" "2024l2:res0603" (at 108.8537 131.8467 90)
-      (effects (font (size 1.27 1.27)) hide)
-    )
-    (property "Datasheet" "~" (at 110.6317 131.8467 0)
-      (effects (font (size 1.27 1.27)) hide)
-    )
-    (pin "1")
-    (pin "2")
-    (instances
-      (project "2024l2 (VNH5019)"
-        (path "/36f2ccec-186b-4304-87fe-6495d5655b87"
-          (reference "R42") (unit 1)
-        )
-      )
-    )
-  )
   (symbol (lib_id "Mechanical:MountingHole_Pad") (at 165.1 194.31 0) (unit 1)
     (in_bom no) (on_board yes) (dnp no) (fields_autoplaced)
@@
   (symbol (lib_id "Diode:B340") (at 77.47 72.39 270) (unit 1)
     (in_bom yes) (on_board yes) (dnp no) (fields_autoplaced)
-    (property "Reference" "D2" (at 80.01 70.8025 90)
+    (property "Reference" "D2" (at 80.01 71.4375 90)
       (effects (font (size 1.27 1.27)) (justify left))
     )
-    (property "Value" "B340" (at 80.01 73.3425 90)
+    (property "Value" "SS54" (at 80.01 73.9775 90)
       (effects (font (size 1.27 1.27)) (justify left))
     )
@@
         )
       )
-    )
-  )
-  (symbol (lib_id "power:+12V") (at 110.6317 120.4167 0) (unit 1)
-    (in_bom yes) (on_board yes) (dnp no) (fields_autoplaced)
-    (property "Reference" "#PWR046" (at 110.6317 124.2267 0)
-      (effects (font (size 1.27 1.27)) hide)
-    )
-    (property "Value" "+12V" (at 110.6317 116.84 0)
-      (effects (font (size 1.27 1.27)))
-    )
-    (property "Footprint" "" (at 110.6317 120.4167 0)
-      (effects (font (size 1.27 1.27)) hide)
-    )
-    (property "Datasheet" "" (at 110.6317 120.4167 0)
-      (effects (font (size 1.27 1.27)) hide)
-    )
-    (pin "1")
-    (instances
-      (project "2024l2 (VNH5019)"
-        (path "/36f2ccec-186b-4304-87fe-6495d5655b87"
-          (reference "#PWR046") (unit 1)
-        )
-      )

Commit message: L2 edits
Parts:
- removed J11, J12, J13, J14: Conn_01x02, 2024l2:AMASS_XT30-F, symbol Connector_Generic:Conn_01x02
- added C21, C22: 220u, Capacitor_SMD:CP_Elec_10x10.5, symbol Device:C_Polarized
- D1, D2: footprint 2024l2:B340 -> 2024l2:SMA (DO-214AC)
Connections:
- net +48V: now also C21.1, C22.1
- net GND: now also C21.2, C22.2
- no-connect marks 42 -> 34
