File: 2025l1/2025l1.kicad_pcb (KiCad board)
At the start: 2 copper layers, 152 parts, among them IC1 LM2587S-ADJ, IC2 VNH5019ATR-E, IC3 VNH5019ATR-E, IC4 VNH5019ATR-E, IC5 VNH5019ATR-E, J1 LED, J10 Conn_01x01, J11 Conn_01x01, J12 Conn_01x01, J13 Conn_01x01, J14 Conn_01x01, J15 Conn_01x01, J16 Conn_01x01, J17 Conn_01x01, J2 Conn_01x01, J3 Conn_01x01, J5 Conn_01x02, J6 XT30, J7 LDR, J9 Conn_01x04, Q1 STP75NF75, Q2 IRLML6344TRPBF, Q3 AON6354, Q4 AON6354, Q5 AON6354, Q6 AON6354, SW1 SW_SPST, SW2 SW_SPDT, U1 CD74HC4067SM, U2 CD74HC4067SM, U3 TPS5430DDA, U4 TPS5430DDA

Commit message: 75% L1
Parts:
- removed C12: 220uF, Capacitor_SMD:CP_Elec_10x10.5
- removed C6: 100u, Capacitor_SMD:CP_Elec_8x6.5
- removed D33, D34: LED, 2025:led0603
- removed IC1: LM2587S-ADJ, 2025:TO170P1435X465-6N
- removed IC2, IC3, IC4, IC5: VNH5019ATR-E, 2025:VNH5019A-E
- removed J1: LED, Connector_PinSocket_2.54mm:PinSocket_1x02_P2.54mm_Vertical
- removed J10, J11, J12, J13, J14, J15, J16, J17: Conn_01x01, 2025:18 AWG
- removed J2, J3: Conn_01x01, 2025:14 AWG
- removed J6: XT30, 2025:AMASS_XT30-F
- removed J7: LDR, Connector_PinSocket_2.54mm:PinSocket_1x02_P2.54mm_Vertical
- removed J9: Conn_01x04, Connector_JST:JST_XH_B4B-XH-A_1x04_P2.50mm_Vertical
- removed L1: 68uH, 2025:1040 One Piece Inductor
- removed Q1: STP75NF75, 2025:TO-220-3_Vertical
- removed Q2: IRLML6344TRPBF, 2025:SOT95P237X112-3N
- removed Q3, Q4, Q5, Q6: AON6354, 2025:8-DFN (5x6)
- removed R30, R32, R43, R50, R51, R66, R67: 10K, 2025:res0603
- removed R33, R34: C146233, 2025:ALS-PT19 (Top Side)
- removed R35: 2k94, 2025:res0603
- removed R36: 57K, 2025:res0603
- removed R37: 1K5, 2025:res0603
- removed R42: 10k, 2025:res0603
- removed R44, R46, R54, R55, R56, R57, R58, R59, R60, R61, R62, R63, R70, R71, R72, R73, R74, R75, R76, R77, R78, R79: 1K, 2025:res0603
- removed R45: 20k, 2025:res0603
- removed R47: 20R, 2025:res0603
- removed R48, R49, R52, R53, R64, R65, R68, R69: 3K3, 2025:res0603
- removed SW1: SW_SPST, Connector_JST:JST_XH_B2B-XH-A_1x02_P2.50mm_Vertical
- removed SW2: SW_SPDT, 2025:SS12D00G3
- added C10: 220u, 2025:EIA-7343-D, F.Cu at (39.5, 99.9)
- added C11: 220u, 2025:EIA-7343-D, F.Cu at (185.7, 100.7)
- added C13: 0u1, 2025:cap0603, F.Cu at (48.8, 92.2)
- added C14: 0u1, 2025:cap0603, F.Cu at (187.8, 94.9)
- added C4: 10u, 2025:cap0603, F.Cu at (48.3, 108.2)
- added C5: 10u, 2025:cap0603, F.Cu at (195.7, 108.6)
- added C8: 10n, 2025:cap0603, F.Cu at (37.7, 105.9)
- added C9: 10n, 2025:cap0603, F.Cu at (185.1, 106.5)
- added D1: LED, 2025:led0603, B.Cu at (115.3, 160.0)
- added D2: LED, 2025:led0603, B.Cu at (127.3, 158.7)
- added D3: LED, 2025:led0603, B.Cu at (138.7, 155.0)
- D10, D11, D12, D13, D14, D15, D16, D17, D18, D19, D20, D21, D22, D23, D24, D25, D26, D27, D28, D29, D30, D5, D6, D7, D8, D9, R1, R10, R11, R12, R13, R14, R15, R16, R17, R18, R19, R2, R20, R21, R22, R23, R24, R25, R26, R27, R28, R29, R3, R31, R4, R5, R7, R9, U1, U2: moved to B.Cu
- D31, D32: value LED -> SS54; footprint 2025:led0603 -> 2025:SMA (DO-214AC)
- D4: value 1N5401 -> LED; footprint Diode_THT:D_DO-201AD_P15.24mm_Horizontal -> 2025:led0603; moved to B.Cu
- R6, R8: value 3K24 -> C146233; footprint 2025:res0603 -> 2025:ALS-PT19 (Top Side); moved to B.Cu
- moved L3 388.5 mm to (192.3, 101.4), turned to 180 degrees
- moved R40 360.0 mm to (185.1, 108.5)
- moved R41 360.0 mm to (185.1, 110.5), turned to 180 degrees
- moved U4 359.3 mm to (190.8, 108.5)
- moved R1 334.1 mm to (172.8, 102.5), turned to 180 degrees
- moved R2 331.5 mm to (171.5, 90.6), turned to -168 degrees
- moved R3 327.1 mm to (167.8, 79.2), turned to -156 degrees
- moved R4 321.0 mm to (161.8, 68.8), turned to -144 degrees
- moved R31 319.2 mm to (171.5, 114.5), turned to 168 degrees
- moved R29 318.2 mm to (167.8, 125.9), turned to 156 degrees
- moved R28 315.1 mm to (161.8, 136.3), turned to 144 degrees
- moved R5 313.4 mm to (153.8, 59.8), turned to -132 degrees
- moved R27 308.8 mm to (153.8, 145.2), turned to 132 degrees
- moved R6 304.4 mm to (144.1, 52.8), turned to -120 degrees
- moved D32 301.9 mm to (192.9, 95.5), turned to 180 degrees
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Connections:
- D31 pad 1: GND -> Net-(D31-K)
- D31 pad 2: +3V3 -> GND
- D32 pad 1: GND -> Net-(D32-K)
- D32 pad 2: +3V3 -> GND
- D4 pad 1: +48V -> GND
- D4 pad 2: Net-(D4-A) -> +3V3
- L2 pad 1: Net-(D1-K) -> Net-(D31-K)
- L2 pad 2: Net-(C10-Pad1) -> +3V3
- L3 pad 1: Net-(D2-K) -> Net-(D32-K)
- L3 pad 2: Net-(C11-Pad1) -> +5V
- R1 pad 2: Net-(U1-I0) -> Net-(U2-I0)
- R10 pad 2: Net-(U2-I3) -> Net-(U2-I9)
- R11 pad 2: Net-(U1-I4) -> Net-(U2-I10)
- R12 pad 2: Net-(U2-I4) -> Net-(U2-I11)
- R13 pad 2: Net-(U1-I5) -> Net-(U2-I12)
- R14 pad 2: Net-(U2-I5) -> Net-(U2-I13)
- R15 pad 2: Net-(U1-I6) -> Net-(U2-I14)
- R16 pad 2: Net-(U2-I6) -> Net-(U1-I0)
- R17 pad 2: Net-(U1-I7) -> Net-(U1-I1)
- R18 pad 2: Net-(U2-I7) -> Net-(U1-I2)
- R19 pad 2: Net-(U1-I8) -> Net-(U1-I3)
- R2 pad 2: Net-(U2-I0) -> Net-(U2-I1)
- R20 pad 2: Net-(U2-I8) -> Net-(U1-I4)
- R21 pad 2: Net-(U1-I9) -> Net-(U1-I5)
- R22 pad 2: Net-(U2-I9) -> Net-(U1-I6)
- R23 pad 2: Net-(U1-I10) -> Net-(U1-I7)
- R24 pad 2: Net-(U2-I10) -> Net-(U1-I8)
- R25 pad 2: Net-(U1-I11) -> Net-(U1-I9)
- R26 pad 2: Net-(U2-I11) -> Net-(U1-I10)
- R27 pad 2: Net-(U1-I12) -> Net-(U1-I11)
- R28 pad 2: Net-(U2-I12) -> Net-(U1-I12)
- R3 pad 2: Net-(U1-I1) -> Net-(U2-I2)
- R31 pad 2: Net-(U2-I13) -> Net-(U1-I14)
- R38 pad 1: Net-(C10-Pad1) -> +3V3
- R4 pad 2: Net-(U2-I1) -> Net-(U2-I3)
- R40 pad 1: Net-(C11-Pad1) -> +5V
- R5 pad 2: Net-(U1-I2) -> Net-(U2-I4)
- R6 pad 1: GND -> +3V3
- R6 pad 2: /LED Ring/mux/M2 -> Net-(U2-I5)
- R7 pad 2: Net-(U2-I2) -> Net-(U2-I6)
- R8 pad 1: GND -> +3V3
- R8 pad 2: /LED Ring/mux/M1 -> Net-(U2-I7)
- R9 pad 2: Net-(U1-I3) -> Net-(U2-I8)
- U3 pad 8: Net-(D1-K) -> Net-(D31-K)
- U4 pad 8: Net-(D2-K) -> Net-(D32-K)
Routing:
- net Net-(U1-I0): track 0.00 -> 62.9 mm
- net Net-(U2-I0): track 0.00 -> 57.5 mm
- net Net-(U1-I1): track 0.00 -> 57.1 mm
- net Net-(U1-I14): track 0.00 -> 57.0 mm
- net Net-(U2-I11): track 0.00 -> 55.4 mm
- net Net-(U2-I4): track 0.00 -> 55.4 mm
- net Net-(U2-I13): track 0.00 -> 52.7 mm
- net Net-(U2-I2): track 0.00 -> 52.6 mm
- net Net-(U2-I14): track 0.00 -> 52.0 mm
- net Net-(U2-I1): track 0.00 -> 51.8 mm
- net Net-(U2-I12): track 0.00 -> 50.8 mm
- net Net-(U2-I3): track 0.00 -> 50.6 mm
- net Net-(U1-I2): track 0.00 -> 49.0 mm
- net Net-(U1-I13): track 0.00 -> 48.9 mm
- net Net-(U2-I6): track 0.00 -> 47.2 mm
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- added copper zone on F.Cu, net +12V
- added copper zone on F.Cu, net +5V
Other:
- board outline added: 176 x 170 mm
- board text added: "BOTTOM TEXT"
- board text added: "JLCJLCJLCJLC"
- board text added: "NOT CRINGE TEXT HERE"
- board text added: "hwa chong robotics"
