File: 2025l1/buckboost.kicad_sch (KiCad schematic)
At the start: 32 parts, among them IC1 LM2587S-ADJ, U3 TPS5430DDA, U4 TPS5430DDA

Commit message: 75% L1
Parts:
- removed F1, F2, F3: Fuse, symbol Device:Fuse
- C10, C11: footprint 2024l2:EIA-7343-D -> 2025:EIA-7343-D
- C13, C14, C15, C3, C4, C5, C7, C8, C9: footprint 2024l2:cap0603 -> 2025:cap0603
- D31: renamed from D1; footprint 2024l2:SMA (DO-214AC) -> 2025:SMA (DO-214AC)
- D32: renamed from D2; footprint 2024l2:SMA (DO-214AC) -> 2025:SMA (DO-214AC)
- D33: renamed from D3; footprint 2024l2:SMA (DO-214AC) -> 2025:SMA (DO-214AC)
- R39: value 5K9 -> 3K24
- R41: value 3K24 -> 5K9
Connections:
- net +3V3: now also C10.1, C13.1, L2.2, R38.1
- net +48V: now also C12.1, C15.1, D33.1 (K), R36.1
- net +5V: now also C11.1, C14.1, L3.2, R40.1
