File: 2025l1/caps.kicad_sch (KiCad schematic)
At the start: 7 parts, among them SW2 SW_SPDT

Commit message: 75% L1
Parts:
- C25, C26, C27, C28, C29: footprint 2024l1:CP_Radial_D16.0mm_P7.50mm -> 2025:CP_Radial_D16.0mm_P7.50mm
Changed lines of the file:
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@@
 			)
 		)
-		(property "Footprint" "2024l1:CP_Radial_D16.0mm_P7.50mm"
+		(property "Footprint" "2025:CP_Radial_D16.0mm_P7.50mm"
 			(at 185.6367 74.5195 0)
 			(effects
@@
 			)
 		)
-		(property "Footprint" "2024l1:CP_Radial_D16.0mm_P7.50mm"
+		(property "Footprint" "2025:CP_Radial_D16.0mm_P7.50mm"
 			(at 127.2167 74.5195 0)
 			(effects
@@
 			)
 		)
-		(property "Footprint" "2024l1:CP_Radial_D16.0mm_P7.50mm"
+		(property "Footprint" "2025:CP_Radial_D16.0mm_P7.50mm"
 			(at 139.9167 74.5195 0)
 			(effects
@@
 			)
 		)
-		(property "Footprint" "2024l1:CP_Radial_D16.0mm_P7.50mm"
+		(property "Footprint" "2025:CP_Radial_D16.0mm_P7.50mm"
 			(at 155.1567 74.5195 0)
 			(effects
@@
 			)
 		)
-		(property "Footprint" "2024l1:CP_Radial_D16.0mm_P7.50mm"
+		(property "Footprint" "2025:CP_Radial_D16.0mm_P7.50mm"
 			(at 170.3967 74.5195 0)
 			(effects
