File: 2025l1/conn.kicad_sch (KiCad schematic)
At the start: 8 parts, among them J1 LED, J2 Conn_01x01, J3 Conn_01x01, J5 Conn_01x02, J7 LDR, J8 Conn_01x04, J9 Conn_01x04

Commit message: 75% L1
Parts:
- J8: footprint (none) -> Connector_PinHeader_2.54mm:PinHeader_1x04_P2.54mm_Vertical
Changed lines of the file:
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@@
 			)
 		)
-		(property "Footprint" ""
+		(property "Footprint" "Connector_PinHeader_2.54mm:PinHeader_1x04_P2.54mm_Vertical"
 			(at 104.14 106.68 0)
 			(effects
