File: 2025l1/ledringmux.kicad_sch (KiCad schematic)
At the start: 38 parts, among them U1 CD74HC4067SM, U2 CD74HC4067SM

Commit message: 75% L1
Parts:
- removed R33, R34: C146233, 2025:ALS-PT19 (Top Side), symbol Device (Modified):ALS-PT19
- removed R6, R8: 3K24, 2025:res0603, symbol vincent:R
- added R33, R34: R, 2025:res0603, symbol Device:R
- added R6, R8: C146233, 2025:ALS-PT19 (Top Side), symbol Device (Modified):ALS-PT19
- C1, C2: footprint 2024l1:cap0603 -> 2025:cap0603
Connections:
- net +3V3: now also R6.1, R8.1
- net GND: now also R33.2, R34.2
- net M1: now also R34.1
- net M2: now also R33.1
- net at R5.2: now also U2.5 (I4); no longer U1.7 (I2)
- net at U1.22 (I9): now also R25.2; no longer R21.2
- net at U1.2 (I7): now also R23.2; no longer R17.2
- net at R1.2: now also U2.9 (I0); no longer U1.9 (I0)
- net at U2.17 (I14): now also R15.2
- net at R4.2: now also U2.6 (I3); no longer U2.8 (I1)
- net at U2.18 (I13): now also R14.2; no longer R31.2
- net at R28.2: now also U1.19 (I12); no longer U2.19 (I12)
- net at U2.2 (I7): now also R8.2; no longer R18.2
- net at R26.2: now also U1.21 (I10); no longer U2.20 (I11)
- net at U2.21 (I10): now also R11.2; no longer R24.2
- net at U2.22 (I9): now also R10.2; no longer R22.2
- net at R20.2: now also U1.5 (I4); no longer U2.23 (I8)
- net at U2.3 (I6): now also R7.2; no longer R16.2
- net at U2.4 (I5): now also R6.2; no longer R14.2
- net at R12.2: now also U2.20 (I11); no longer U2.5 (I4)
- net at U2.7 (I2): now also R3.2; no longer R7.2
- net at R2.2: now also U2.8 (I1); no longer U2.9 (I0)
- net at U1.3 (I6): now also R22.2; no longer R15.2
- net at R27.2: now also U1.20 (I11); no longer U1.19 (I12)
- net at R9.2: now also U2.23 (I8); no longer U1.6 (I3)
- net at U1.17 (I14): now also R31.2
- net at R13.2: now also U2.19 (I12); no longer U1.4 (I5)
- net at U1.8 (I1): now also R17.2; no longer R3.2
- net at R19.2: now also U1.6 (I3); no longer U1.23 (I8)
- new net: R18.2, U1.7 (I2)
- new net: R24.2, U1.23 (I8)
- new net: R16.2, U1.9 (I0)
- new net: R21.2, U1.4 (I5)
