File: 2025l1/leds.kicad_sch (KiCad schematic)
At the start: 30 parts

Commit message: 75% L1
Parts:
- renumbered D31 to D1, D32 to D2, D33 to D3, D34 to D4
Changed lines of the file:
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@@
 		(dnp no)
 		(fields_autoplaced yes)
-		(property "Reference" "D32"
+		(property "Reference" "D2"
 			(at 177.8 76.5174 90)
 			(effects
@@
 			(project "2025l1"
 				(path "/42f1a342-2581-49f6-a220-6ea8add89dfb/c64c4b1b-d73d-4041-97d2-d557e1412053/4b5b3d0c-e9d6-468d-9491-c6676e24121a"
-					(reference "D32")
+					(reference "D2")
 					(unit 1)
 				)
@@
 		(dnp no)
 		(fields_autoplaced yes)
-		(property "Reference" "D31"
+		(property "Reference" "D1"
 			(at 167.64 103.1874 90)
 			(effects
@@
 			(project "2025l1"
 				(path "/42f1a342-2581-49f6-a220-6ea8add89dfb/c64c4b1b-d73d-4041-97d2-d557e1412053/4b5b3d0c-e9d6-468d-9491-c6676e24121a"
-					(reference "D31")
+					(reference "D1")
 					(unit 1)
 				)
@@
 		(dnp no)
 		(fields_autoplaced yes)
-		(property "Reference" "D34"
+		(property "Reference" "D4"
 			(at 177.8 103.1874 90)
 			(effects
@@
 			(project "2025l1"
 				(path "/42f1a342-2581-49f6-a220-6ea8add89dfb/c64c4b1b-d73d-4041-97d2-d557e1412053/4b5b3d0c-e9d6-468d-9491-c6676e24121a"
-					(reference "D34")
+					(reference "D4")
 					(unit 1)
 				)
@@
 		(dnp no)
 		(fields_autoplaced yes)
-		(property "Reference" "D33"
+		(property "Reference" "D3"
 			(at 177.8 89.2174 90)
 			(effects
@@
 			(project "2025l1"
 				(path "/42f1a342-2581-49f6-a220-6ea8add89dfb/c64c4b1b-d73d-4041-97d2-d557e1412053/4b5b3d0c-e9d6-468d-9491-c6676e24121a"
-					(reference "D33")
-					(unit 1)
-				)
+					(reference "D3")
+					(unit 1)
+				)
