File: 2025l1/misc.kicad_sch (KiCad schematic)
At the start: 5 parts

Commit message: 75% L1
Parts:
- added H1, H10, H11, H12, H2, H3, H4, H5, H6, H7, H8, H9: MountingHole_Pad, MountingHole:MountingHole_3.2mm_M3_Pad_Via, symbol Mechanical:MountingHole_Pad
Connections:
- no-connect marks 0 -> 12
