File: 2025l1/motordriver.kicad_sch (KiCad schematic)
At the start: 58 parts, among them IC2 VNH5019ATR-E, IC3 VNH5019ATR-E, IC4 VNH5019ATR-E, IC5 VNH5019ATR-E, J10 Conn_01x01, J11 Conn_01x01, J12 Conn_01x01, J13 Conn_01x01, J14 Conn_01x01, J15 Conn_01x01, J16 Conn_01x01, J17 Conn_01x01, J4 Conn_01x12, Q3 AON6354, Q4 AON6354, Q5 AON6354, Q6 AON6354, SW1 SW_SPST

Commit message: 75% L1
Parts:
- C17, C18, C21, C22: footprint 2024l2:CP_Radial_D8.0mm_P3.50mm -> 2025:CP_Radial_D8.0mm_P3.50mm
- C19, C20, C23, C24: footprint 2024l2:cap0603 -> 2025:cap0603
Changed lines of the file:
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@@
 			)
 		)
-		(property "Footprint" "2024l2:cap0603"
+		(property "Footprint" "2025:cap0603"
 			(at 192.0748 76.2 0)
 			(effects
@@
 			)
 		)
-		(property "Footprint" "2024l2:cap0603"
+		(property "Footprint" "2025:cap0603"
 			(at 192.0748 135.89 0)
 			(effects
@@
 			)
 		)
-		(property "Footprint" "2024l2:cap0603"
+		(property "Footprint" "2025:cap0603"
 			(at 99.3648 74.93 0)
 			(effects
@@
 			)
 		)
-		(property "Footprint" "2024l2:cap0603"
+		(property "Footprint" "2025:cap0603"
 			(at 99.3648 134.62 0)
 			(effects
@@
 			)
 		)
-		(property "Footprint" "2024l2:CP_Radial_D8.0mm_P3.50mm"
+		(property "Footprint" "2025:CP_Radial_D8.0mm_P3.50mm"
 			(at 88.5952 134.62 0)
 			(effects
@@
 			)
 		)
-		(property "Footprint" "2024l2:CP_Radial_D8.0mm_P3.50mm"
+		(property "Footprint" "2025:CP_Radial_D8.0mm_P3.50mm"
 			(at 181.3052 135.89 0)
 			(effects
@@
 			)
 		)
-		(property "Footprint" "2024l2:CP_Radial_D8.0mm_P3.50mm"
+		(property "Footprint" "2025:CP_Radial_D8.0mm_P3.50mm"
 			(at 181.3052 76.2 0)
 			(effects
@@
 			)
 		)
-		(property "Footprint" "2024l2:CP_Radial_D8.0mm_P3.50mm"
+		(property "Footprint" "2025:CP_Radial_D8.0mm_P3.50mm"
 			(at 88.5952 74.93 0)
 			(effects
