File: 2025l1/solenoid activation.kicad_sch (KiCad schematic)
At the start: 9 parts, among them J6 XT30, Q1 STP75NF75, Q2 IRLML6344TRPBF

Commit message: 75% L1
Parts:
- C16: footprint 2024l1:cap0603 -> 2025:cap0603
- renumbered D4 to D34
Changed lines of the file:
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@@
 			)
 		)
-		(property "Footprint" "2024l1:cap0603"
+		(property "Footprint" "2025:cap0603"
 			(at 103.8352 107.95 0)
 			(effects
@@
 		(on_board yes)
 		(dnp no)
-		(property "Reference" "D4"
+		(property "Reference" "D34"
 			(at 77.47 80.01 90)
 			(effects
@@
 			(project "2025l1"
 				(path "/42f1a342-2581-49f6-a220-6ea8add89dfb/2141b66e-45d0-43fd-aaef-c9fd4e16da7c/5e82c284-ab28-4c6b-8caa-f59246f3779e"
-					(reference "D4")
+					(reference "D34")
 					(unit 1)
 				)
